Commit message: Solved the issue of knuckle link not appearing in v1

File: softhands_description/urdf/v1.0/sh_v1.xacro (robot description, xacro)
@@ -88,6 +88,6 @@
 			# Thumb finger
 			<xacro:thumb_v1 type="thumb"
-		 		ns = "${type}_hand_v1"
-		 		sign = "1"
+				ns = "${type}_hand_v1"
+				sign = "1"
 				position="0.00566972 0.0296160 0.0553140"
 				orientation="0.0 -0.38397275793662144 1.5707963267948966">
@@ -160,9 +160,5 @@
 			</link>
 			# Thumb finger
-			<xacro:thumb_v1 type="thumb"
-		 		ns = "${type}_hand_v1"
-		 		sign = "-1"
-				position="0.005669722 -0.029616 0.055314"
-				orientation="0.0 -0.38397275793662144 -1.5707963267948966">
+			<xacro:thumb_v1 type="thumb" ns = "${type}_hand_v1" sign = "-1" position="0.005669722 -0.029616 0.055314" orientation="0.0 -0.38397275793662144 -1.5707963267948966">
 			</xacro:thumb_v1>
 			# Index finger

File: softhands_description/urdf/v1.0_simple/finger.xacro (robot description, xacro)
@@ -38,5 +38,5 @@
 -->
 <robot xmlns:xacro="http://www.ros.org/wiki/xacro">
-  <xacro:macro name="finger_v1" params="type ns sign position orientation">
+  <xacro:macro name="finger_v1_simple" params="type ns sign position orientation">
     <!-- KNUCKLE -->
     <joint name="${ns}_${type}_knuckle_joint" type="revolute">

File: softhands_description/urdf/v1.0_simple/sh_v1_simple.xacro (robot description, xacro)
@@ -86,13 +86,13 @@
 			</link>
 			# Thumb finger
-			<xacro:thumb_v1 type="thumb" ns="${type}_hand_v1s" sign="1" position="0.00566972 0.0296160 0.0553140" orientation="0.0 -0.38397275793662144 1.5707963267948966"></xacro:thumb_v1>
+			<xacro:thumb_v1_simple type="thumb" ns="${type}_hand_v1s" sign="1" position="0.00566972 0.0296160 0.0553140" orientation="0.0 -0.38397275793662144 1.5707963267948966"></xacro:thumb_v1_simple>
 			# Index finger
-			<xacro:finger_v1 type="index" ns="${type}_hand_v1s" sign="1" position="-0.0033 0.0195 0.0936994" orientation="1.5707963267948966 -1.4835299330931884 1.5707963267948966"></xacro:finger_v1>
+			<xacro:finger_v1_simple type="index" ns="${type}_hand_v1s" sign="1" position="-0.0033 0.0195 0.0936994" orientation="1.5707963267948966 -1.4835299330931884 1.5707963267948966"></xacro:finger_v1_simple>
 			# Middle finger
-			<xacro:finger_v1 type="middle" ns="${type}_hand_v1s" sign="1" position="-0.003300000 0.0 0.100699" orientation="3.141592 -1.5707963267948966 0.0"></xacro:finger_v1>
+			<xacro:finger_v1_simple type="middle" ns="${type}_hand_v1s" sign="1" position="-0.003300000 0.0 0.100699" orientation="3.141592 -1.5707963267948966 0.0"></xacro:finger_v1_simple>
 			# Ring finger
-			<xacro:finger_v1 type="ring" ns="${type}_hand_v1s" sign="1" position="-0.0033 -0.0195 0.0936994" orientation="-1.5707963267948966 -1.5184364298870514 -1.5707963267948966"></xacro:finger_v1>
+			<xacro:finger_v1_simple type="ring" ns="${type}_hand_v1s" sign="1" position="-0.0033 -0.0195 0.0936994" orientation="-1.5707963267948966 -1.5184364298870514 -1.5707963267948966"></xacro:finger_v1_simple>
 			# Little finger
-			<xacro:finger_v1 type="little" ns="${type}_hand_v1s" sign="1" position="-0.0033 -0.039 0.0836994" orientation="-1.5707963267948966 -1.4835299330931884 -1.5707963267948966"></xacro:finger_v1>
+			<xacro:finger_v1_simple type="little" ns="${type}_hand_v1s" sign="1" position="-0.0033 -0.039 0.0836994" orientation="-1.5707963267948966 -1.4835299330931884 -1.5707963267948966"></xacro:finger_v1_simple>
 		</xacro:if>
 		# LEFT HAND
@@ -134,13 +134,13 @@
 			</link>
 			# Thumb finger
-			<xacro:thumb_v1 type="thumb" ns="${type}_hand_v1s" sign="-1" position="0.005669722 -0.029616 0.055314" orientation="0.0 -0.38397275793662144 -1.5707963267948966"></xacro:thumb_v1>
+			<xacro:thumb_v1_simple type="thumb" ns="${type}_hand_v1s" sign="-1" position="0.005669722 -0.029616 0.055314" orientation="0.0 -0.38397275793662144 -1.5707963267948966"></xacro:thumb_v1_simple>
 			# Index finger
-			<xacro:finger_v1 type="index" ns="${type}_hand_v1s" sign="-1" position="-0.0033 -0.0195 0.0936994" orientation="-1.5707963267948966 -1.4835299330931884 -1.5707963267948966"></xacro:finger_v1>
+			<xacro:finger_v1_simple type="index" ns="${type}_hand_v1s" sign="-1" position="-0.0033 -0.0195 0.0936994" orientation="-1.5707963267948966 -1.4835299330931884 -1.5707963267948966"></xacro:finger_v1_simple>
 			# Middle finger
-			<xacro:finger_v1 type="middle" ns="${type}_hand_v1s" sign="-1" position="-0.0033 0.0 0.100699" orientation="3.1415 -1.5707963267948966 0.0"></xacro:finger_v1>
+			<xacro:finger_v1_simple type="middle" ns="${type}_hand_v1s" sign="-1" position="-0.0033 0.0 0.100699" orientation="3.1415 -1.5707963267948966 0.0"></xacro:finger_v1_simple>
 			# Ring finger
-			<xacro:finger_v1 type="ring" ns="${type}_hand_v1s" sign="-1" position="-0.0033 0.0195 0.0936994" orientation="1.5707963267948966 -1.5184364298870514 1.5707963267948966"></xacro:finger_v1>
+			<xacro:finger_v1_simple type="ring" ns="${type}_hand_v1s" sign="-1" position="-0.0033 0.0195 0.0936994" orientation="1.5707963267948966 -1.5184364298870514 1.5707963267948966"></xacro:finger_v1_simple>
 			# Little finger
-			<xacro:finger_v1 type="little" ns="${type}_hand_v1s" sign="-1" position="-0.0033 0.039 0.0836994" orientation="1.5707963267948966 -1.4835299330931884 1.5707963267948966"></xacro:finger_v1>
+			<xacro:finger_v1_simple type="little" ns="${type}_hand_v1s" sign="-1" position="-0.0033 0.039 0.0836994" orientation="1.5707963267948966 -1.4835299330931884 1.5707963267948966"></xacro:finger_v1_simple>
 		</xacro:if>
 		# Gazebo NEW custom synergy-plugin

File: softhands_description/urdf/v1.0_simple/thumb.xacro (robot description, xacro)
@@ -38,5 +38,5 @@
 -->
 <robot xmlns:xacro="http://www.ros.org/wiki/xacro">
-  <xacro:macro name="thumb_v1" params="type ns sign position orientation">
+  <xacro:macro name="thumb_v1_simple" params="type ns sign position orientation">
     <!-- KNUCKLE -->
     <joint name="${ns}_${type}_knuckle_joint" type="continuous">
