Commit message: added new folder structur and macro for the finger

File: softhands_description/urdf/xacro/header.xacro (robot description, xacro)
@@ -39,7 +39,10 @@
 <robot xmlns:xacro="http://www.ros.org/wiki/xacro" name="header">
   <!-- Include xacro macro -->
- 	<xacro:include filename="$(find softhands_description)/urdf/xacro/include/macro/v1.0_simple/sh_v1_simple.xacro"/>
-	<xacro:include filename="$(find softhands_description)/urdf/xacro/include/macro/v1.0_simple/finger.xacro" />
-	<xacro:include filename="$(find softhands_description)/urdf/xacro/include/macro/v1.0_simple/thumb.xacro" />
+	<xacro:include filename="$(find softhands_description)/urdf/xacro/include/macro/v1.0_simple/finger_v1_simple.xacro" />
+	<xacro:include filename="$(find softhands_description)/urdf/xacro/include/macro/v1.0_simple/thumb_v1_simple.xacro" />
 	<xacro:include filename="$(find softhands_description)/urdf/xacro/include/macro/v1.0_simple/palm.xacro" />
+	<xacro:include filename="$(find softhands_description)/urdf/xacro/include/macro/common/phalanges/knuckle.xacro" />
+	<xacro:include filename="$(find softhands_description)/urdf/xacro/include/macro/common/phalanges/thumb_knuckle.xacro" />
+	<xacro:include filename="$(find softhands_description)/urdf/xacro/include/macro/common/phalanges/fingertip.xacro" />
+	<xacro:include filename="$(find softhands_description)/urdf/xacro/include/macro/common/phalanges/phalanx.xacro" />
 </robot>

File: softhands_description/urdf/xacro/include/macro/v1.0_simple/palm.xacro (robot description, xacro)
@@ -82,4 +82,8 @@
 			</collision>
 		</link>
+    <gazebo reference="${type}_hand_v1s_palm_link">
+      <material>Gazebo/Grey</material>
+      <selfCollide>true</selfCollide>
+	  </gazebo>
 	</xacro:macro>
 </robot>

File: softhands_description/urdf/xacro/include/macro/v1.0_simple/thumb_v1_simple.xacro (robot description, xacro)
@@ -31,5 +31,5 @@
  * OF THIS SOFTWARE, EVEN IF ADVISED OF THE POSSIBILITY OF SUCH DAMAGE.
  *
- * \file      finger.xacro
+ * \file      thumb.xacro
  *
  * \author       _Centro di Ricerca "E.Piaggio"_
@@ -38,37 +38,17 @@
 -->
 <robot xmlns:xacro="http://www.ros.org/wiki/xacro">
-  <xacro:macro name="finger_v1" params="type ns sign position orientation">
+  <xacro:macro name="thumb_v1_simple" params="type ns sign position orientation">
     <!-- KNUCKLE -->
-    <joint name="${ns}_${type}_knuckle_joint" type="revolute">
-      <origin xyz="${position}" rpy="${orientation}"/>
-      <parent link="${ns}_palm_link"/>
-      <child link="${ns}_${type}_knuckle_link"/>
-      <limit effort="30" velocity="1.0" lower="-1.57" upper="1.57" />
-      <axis xyz="0 0 ${sign*1}" />
-      <dynamics damping="0.08" friction="0.0" />
-    </joint>
-    <link name="${ns}_${type}_knuckle_link">
-      <inertial>
-        <origin xyz="0.001285644 0 0.000425011"/>
-        <mass value="0.09"/>
-        <inertia ixx="0.001" ixy="0" ixz="0" iyy="0.001" iyz="0" izz="0.001"/>
-      </inertial>
-      <visual>
-        <geometry>
-          <mesh filename="package://softhands_description/meshes/softhands/v1.0/common/knuckle_m.stl"/>
-        </geometry>
-      </visual>
-      <collision>
-        <geometry>
-          <mesh filename="package://softhands_description/meshes/softhands/v1.0/common/knuckle_m.stl"/>
-        </geometry>
-      </collision>
-    </link>
+    <xacro:thumb_knuckle
+      ns="${ns}"
+      position="${position}"
+      type="${type}"
+      orientation="${orientation}">
+    </xacro:thumb_knuckle>
     <!-- PROXIMAL PHALANGE -->
-    <joint name="${ns}_${type}_proximal_joint" type="revolute">
-      <origin xyz="0.020 0 0" rpy="0 0 0" />
+    <joint name="${ns}_${type}_proximal_joint" type="continuous">
+      <origin xyz="0.033500000 ${sign*-0.003300000} 0.0" rpy="${sign*0.426627741408745} 0 0.0" />
       <parent link="${ns}_${type}_knuckle_link"/>
       <child link="${ns}_${type}_proximal_link"/>
-      <limit effort="30" velocity="1.0" lower="-1.57" upper="1.57" />
       <axis xyz="0 -1 0" />
       <dynamics damping="0.08" friction="0.0" />
@@ -91,35 +71,9 @@
       </collision>
     </link>
-    <!-- MIDDLE PHALANGE -->
-    <joint name="${ns}_${type}_middle_joint" type="revolute">
-      <origin xyz="0.020 0 0" rpy="0 0 0" />
+    <!-- DISTAL PHALANGE -->
+    <joint name="${ns}_${type}_distal_joint" type="continuous">
+      <origin xyz="0.020 0 0.0" rpy="0 0 0" />
       <parent link="${ns}_${type}_proximal_link"/>
-      <child link="${ns}_${type}_middle_link"/>
-      <limit effort="30" velocity="1.0" lower="-1.57" upper="1.57" />
-      <axis xyz="0 -1 0" />
-    </joint>
-    <link name="${ns}_${type}_middle_link">
-      <inertial>
-        <origin xyz="0.005074337 0 -0.000262953"/>
-        <mass value="0.05"/>
-        <inertia ixx="0.001" ixy="0" ixz="0" iyy="0.001" iyz="0" izz="0.001"/>
-      </inertial>
-      <visual>
-        <geometry>
-          <mesh filename="package://softhands_description/meshes/softhands/v1.0/common/phalanx_m.stl"/>
-        </geometry>
-      </visual>
-      <collision>
-        <geometry>
-          <mesh filename="package://softhands_description/meshes/softhands/v1.0/common/phalanx_m.stl"/>
-        </geometry>
-      </collision>
-    </link>
-    <!-- DISTAL PHALANGE -->
-    <joint name="${ns}_${type}_distal_joint" type="revolute">
-      <origin xyz="0.020 0 0" rpy="0 0 0" />
-      <parent link="${ns}_${type}_middle_link"/>
       <child link="${ns}_${type}_distal_link"/>
-      <limit effort="30" velocity="1.0" lower="-1.57" upper="1.57" />
       <axis xyz="0 -1 0" />
       <dynamics damping="0.08" friction="0.0" />
@@ -133,10 +87,10 @@
       <visual>
         <geometry>
-          <mesh filename="package://softhands_description/meshes/softhands/v1.0/common/fingertip_m.stl"/>
+          <mesh filename="package://softhands_description/meshes/softhands/v1.0/common/fingertip_m.stl" />
         </geometry>
       </visual>
       <collision>
         <geometry>
-          <mesh filename="package://softhands_description/meshes/softhands/v1.0/common/fingertip_m.stl"/>
+          <mesh filename="package://softhands_description/meshes/softhands/v1.0/common/fingertip_m.stl" />
         </geometry>
       </collision>

File: softhands_description/urdf/xacro/sh_v1_simple.xacro (robot description, xacro)
@@ -58,6 +58,6 @@
 		sign="$(arg sign)"
 		ns="$(arg type)_hand_v1s"
-		position="0.00566972 0.0296160 0.0553140"
-		orientation="0.0 -0.38397275793662144 1.5707963267948966">
+		position="0.00566972 ${$(arg sign)*0.0296160} 0.0553140"
+		orientation="0.0 -0.38397275793662144 ${$(arg sign)*1.5707963267948966}">
 	</xacro:thumb_v1_simple>
 	<!-- # Index finger -->
@@ -65,6 +65,6 @@
 		type="index"
 		ns="$(arg type)_hand_v1s"
-		position="-0.0033 0.0195 0.0936994"
-		orientation="1.5707963267948966 -1.4835299330931884 1.5707963267948966">
+		position="-0.0033 ${$(arg sign)*0.0195} 0.0936994"
+		orientation="${$(arg sign)*1.5707963267948966} -1.4835299330931884 ${$(arg sign)*1.5707963267948966}">
 	</xacro:finger_v1_simple>
 	<!-- # Middle finger -->
@@ -79,6 +79,6 @@
 		type="ring"
 		ns="$(arg type)_hand_v1s"
-		position="-0.0033 -0.0195 0.0936994"
-		orientation="-1.5707963267948966 -1.5184364298870514 -1.5707963267948966">
+		position="-0.0033 ${$(arg sign)*-0.0195} 0.0936994"
+		orientation="${$(arg sign)*-1.5707963267948966} -1.5184364298870514 ${$(arg sign)*-1.5707963267948966}">
 	</xacro:finger_v1_simple>
 	<!-- # Little finger -->
@@ -86,6 +86,6 @@
 		type="little"
 		ns="$(arg type)_hand_v1s"
-		position="-0.0033 -0.039 0.0836994"
-		orientation="-1.5707963267948966 -1.4835299330931884 -1.5707963267948966">
+		position="-0.0033 ${$(arg sign)*-0.039} 0.0836994"
+		orientation="${$(arg sign)*-1.5707963267948966} -1.4835299330931884 ${$(arg sign)*-1.5707963267948966}">
 	</xacro:finger_v1_simple>
 		<!-- # Gazebo NEW custom synergy-plugin -->

Commit message: added thumb's macro and found wrong orientation of the finger's phalanges

File: softhands_description/urdf/xacro/header.xacro (robot description, xacro)
@@ -42,7 +42,7 @@
 	<xacro:include filename="$(find softhands_description)/urdf/xacro/include/macro/v1.0_simple/thumb_v1_simple.xacro" />
 	<xacro:include filename="$(find softhands_description)/urdf/xacro/include/macro/v1.0_simple/palm.xacro" />
-	<xacro:include filename="$(find softhands_description)/urdf/xacro/include/macro/common/phalanges/knuckle.xacro" />
-	<xacro:include filename="$(find softhands_description)/urdf/xacro/include/macro/common/phalanges/thumb_knuckle.xacro" />
-	<xacro:include filename="$(find softhands_description)/urdf/xacro/include/macro/common/phalanges/fingertip.xacro" />
-	<xacro:include filename="$(find softhands_description)/urdf/xacro/include/macro/common/phalanges/phalanx.xacro" />
+	<xacro:include filename="$(find softhands_description)/urdf/xacro/include/macro/v1.0_simple/phalanges/knuckle.xacro" />
+	<xacro:include filename="$(find softhands_description)/urdf/xacro/include/macro/v1.0_simple/phalanges/thumb_knuckle.xacro" />
+	<xacro:include filename="$(find softhands_description)/urdf/xacro/include/macro/v1.0_simple/phalanges/fingertip.xacro" />
+	<xacro:include filename="$(find softhands_description)/urdf/xacro/include/macro/v1.0_simple/phalanges/phalanx.xacro" />
 </robot>

File: softhands_description/urdf/xacro/include/macro/v1.0_simple/phalanges/phalanx.xacro (robot description, xacro)
@@ -41,5 +41,5 @@
     <!-- PROXIMAL PHALANGE -->
     <joint name="${ns}_${type}_${name}_joint" type="revolute">
-      <origin xyz="${position}" rpy="0 0 0" />
+      <origin xyz="${position}" rpy="${orientation}" />
       <parent link="${ns}_${type}_${parent}_link"/>
       <child link="${ns}_${type}_${name}_link"/>

File: softhands_description/urdf/xacro/include/macro/v1.0_simple/phalanges/thumb_knuckle.xacro (robot description, xacro)
@@ -40,8 +40,9 @@
   <xacro:macro name="thumb_knuckle" params="type ns position orientation">
     <!-- KNUCKLE -->
-    <joint name="${ns}_${type}_knuckle_joint" type="continuous">
+    <joint name="${ns}_${type}_knuckle_joint" type="revolute">
       <origin xyz="${position}" rpy="${orientation}"/>
       <parent link="${ns}_palm_link"/>
       <child link="${ns}_${type}_knuckle_link"/>
+      <limit effort="30" velocity="1.0" lower="-1.57" upper="1.57" />
       <axis xyz="0 0 ${sign*-1}" />
       <dynamics damping="0.08" friction="0.0" />

File: softhands_description/urdf/xacro/include/macro/v1.0_simple/thumb_v1_simple.xacro (robot description, xacro)
@@ -47,53 +47,21 @@
     </xacro:thumb_knuckle>
     <!-- PROXIMAL PHALANGE -->
-    <joint name="${ns}_${type}_proximal_joint" type="continuous">
-      <origin xyz="0.033500000 ${sign*-0.003300000} 0.0" rpy="${sign*0.426627741408745} 0 0.0" />
-      <parent link="${ns}_${type}_knuckle_link"/>
-      <child link="${ns}_${type}_proximal_link"/>
-      <axis xyz="0 -1 0" />
-      <dynamics damping="0.08" friction="0.0" />
-    </joint>
-    <link name="${ns}_${type}_proximal_link">
-      <inertial>
-        <origin xyz="0.005074337 0 -0.000262953"/>
-        <mass value="0.05"/>
-        <inertia ixx="0.001" ixy="0" ixz="0" iyy="0.001" iyz="0" izz="0.001"/>
-      </inertial>
-      <visual>
-        <geometry>
-          <mesh filename="package://softhands_description/meshes/softhands/v1.0/common/phalanx_m.stl"/>
-        </geometry>
-      </visual>
-      <collision>
-        <geometry>
-          <mesh filename="package://softhands_description/meshes/softhands/v1.0/common/phalanx_m.stl"/>
-        </geometry>
-      </collision>
-    </link>
+    <xacro:phalanx
+      parent="knuckle"
+      name="proximal"
+      ns="${ns}"
+      position="0.033500000 ${sign*-0.003300000} 0.0"
+      type="${type}"
+      orientation="${sign*0.426627741408745} 0 0.0">
+    </xacro:phalanx>
     <!-- DISTAL PHALANGE -->
-    <joint name="${ns}_${type}_distal_joint" type="continuous">
-      <origin xyz="0.020 0 0.0" rpy="0 0 0" />
-      <parent link="${ns}_${type}_proximal_link"/>
-      <child link="${ns}_${type}_distal_link"/>
-      <axis xyz="0 -1 0" />
-      <dynamics damping="0.08" friction="0.0" />
-    </joint>
-    <link name="${ns}_${type}_distal_link">
-      <inertial>
-            <origin xyz="0.009849094 0 0.000820286"/>
-        <mass value="0.1"/>
-        <inertia ixx="0.001" ixy="0" ixz="0" iyy="0.001" iyz="0" izz="0.001"/>
-      </inertial>
-      <visual>
-        <geometry>
-          <mesh filename="package://softhands_description/meshes/softhands/v1.0/common/fingertip_m.stl" />
-        </geometry>
-      </visual>
-      <collision>
-        <geometry>
-          <mesh filename="package://softhands_description/meshes/softhands/v1.0/common/fingertip_m.stl" />
-        </geometry>
-      </collision>
-    </link>
+    <xacro:fingertip
+      parent="proximal"
+      name="distal"
+      ns="${ns}"
+      position="0.020 0 0"
+      type="${type}"
+      orientation="0 0 0">
+    </xacro:fingertip>
   </xacro:macro>
 </robot>
