Commit message: added stl of sh_v3

File: softhands_description/urdf/xacro/header.xacro (robot description, xacro)
@@ -39,10 +39,11 @@
 <robot xmlns:xacro="http://www.ros.org/wiki/xacro" name="header">
   <!-- Include xacro macro -->
-	<xacro:include filename="$(find softhands_description)/urdf/xacro/include/macro/v1.0_simple/finger_v1_simple.xacro" />
-	<xacro:include filename="$(find softhands_description)/urdf/xacro/include/macro/v1.0_simple/thumb_v1_simple.xacro" />
-	<xacro:include filename="$(find softhands_description)/urdf/xacro/include/macro/v1.0_simple/palm.xacro" />
-	<xacro:include filename="$(find softhands_description)/urdf/xacro/include/macro/v1.0_simple/phalanges/knuckle.xacro" />
-	<xacro:include filename="$(find softhands_description)/urdf/xacro/include/macro/v1.0_simple/phalanges/thumb_knuckle.xacro" />
-	<xacro:include filename="$(find softhands_description)/urdf/xacro/include/macro/v1.0_simple/phalanges/fingertip.xacro" />
-	<xacro:include filename="$(find softhands_description)/urdf/xacro/include/macro/v1.0_simple/phalanges/phalanx.xacro" />
+	<xacro:include filename="$(arg root_dir)/finger.xacro" />
+	<xacro:include filename="$(arg root_dir)/thumb.xacro" />
+	<xacro:include filename="$(arg root_dir)/base.xacro" />
+	<xacro:include filename="$(arg root_dir)/palm.xacro" />
+	<xacro:include filename="$(arg root_dir)/phalanges/knuckle.xacro" />
+	<xacro:include filename="$(arg root_dir)/phalanges/thumb_knuckle.xacro" />
+	<xacro:include filename="$(arg root_dir)/phalanges/fingertip.xacro" />
+	<xacro:include filename="$(arg root_dir)/phalanges/phalanx.xacro" />
 </robot>

File: softhands_description/urdf/xacro/include/macro/v3_simple/base.xacro (robot description, xacro)
@@ -31,5 +31,5 @@
  * OF THIS SOFTWARE, EVEN IF ADVISED OF THE POSSIBILITY OF SUCH DAMAGE.
  *
- * \file      test_SHs_v2.urdf.xacro
+ * \file      sh_v1_simple.xacro
  *
  * \author       _Centro di Ricerca "E.Piaggio"_
@@ -37,13 +37,35 @@
  *
 -->
-<robot name="softhand" xmlns:xacro="http://www.ros.org/wiki/xacro">
-  	<xacro:arg name="sh_version" default="v1_simple"/>
-  	<xacro:arg name="root_dir" default="$(find softhands_description)/urdf/xacro/include/macro/$(arg sh_version)"/>
-  	<xacro:arg name="parent" default="world"/>
-  	<xacro:arg name="type" default="left"/>
-  	<xacro:arg name="position" default="0 0 0"/>
-  	<xacro:arg name="orientation" default="0 0 0"/>
-  	<xacro:arg name="operation_mode" default="0"/>
-	<xacro:include filename="$(find softhands_description)/urdf/xacro/header.xacro"/>
-	<xacro:include filename="$(find softhands_description)/urdf/xacro/$(arg sh_version).xacro"/>
+<robot name="Palm_v1_simple" xmlns:xacro="http://www.ros.org/wiki/xacro">
+	<xacro:macro name="base" params="type sign parent position orientation operation_mode">
+		<link name="root_link"/>
+		<joint name="qbhand_base_fixed_joint" type="fixed">
+			<origin rpy="0 0 0" xyz="0 0 0"/>
+			<parent link="root_link"/>
+			<child link="qbhand_base_link"/>
+		</joint>
+		<link name="qbhand_base_link">
+			<inertial>
+			<mass value="0.45"/>
+			<origin rpy="0 0 0" xyz="0.0030 -0.0449 0.0135"/>
+			<inertia ixx="0.00045" ixy="0.0" ixz="0.0" iyy="0.0006" iyz="0.0" izz="0.00025"/>
+			</inertial>
+			<visual>
+			<origin rpy="0 0 0" xyz="0 0 0"/>
+			<geometry>
+				<mesh filename="package://softhands_description/meshes/softhands/v3.0/flange_iso_04.stl" scale="0.001 0.001 0.001"/>
+			</geometry>
+			<material name="qbhand/base"/>
+			</visual>
+			<collision>
+			<origin rpy="0 0 0" xyz="0 0 0"/>
+			<geometry>
+				<mesh filename="package://softhands_description/meshes/softhands/v3.0/flange_iso_04.stl" scale="0.001 0.001 0.001"/>
+			</geometry>
+			</collision>
+		</link>
+		<gazebo reference="qbhand_base_link">
+			<self_collide>1</self_collide>
+		</gazebo>
+	</xacro:macro>
 </robot>

File: softhands_description/urdf/xacro/include/macro/v3_simple/palm.xacro (robot description, xacro)
@@ -31,5 +31,5 @@
  * OF THIS SOFTWARE, EVEN IF ADVISED OF THE POSSIBILITY OF SUCH DAMAGE.
  *
- * \file      test_SHs_v2.urdf.xacro
+ * \file      sh_v1_simple.xacro
  *
  * \author       _Centro di Ricerca "E.Piaggio"_
@@ -37,13 +37,31 @@
  *
 -->
-<robot name="softhand" xmlns:xacro="http://www.ros.org/wiki/xacro">
-  	<xacro:arg name="sh_version" default="v1_simple"/>
-  	<xacro:arg name="root_dir" default="$(find softhands_description)/urdf/xacro/include/macro/$(arg sh_version)"/>
-  	<xacro:arg name="parent" default="world"/>
-  	<xacro:arg name="type" default="left"/>
-  	<xacro:arg name="position" default="0 0 0"/>
-  	<xacro:arg name="orientation" default="0 0 0"/>
-  	<xacro:arg name="operation_mode" default="0"/>
-	<xacro:include filename="$(find softhands_description)/urdf/xacro/header.xacro"/>
-	<xacro:include filename="$(find softhands_description)/urdf/xacro/$(arg sh_version).xacro"/>
+<robot name="Palm_v1_simple" xmlns:xacro="http://www.ros.org/wiki/xacro">
+	<xacro:macro name="palm" params="type sign parent position orientation operation_mode">
+	  <joint name="qbhand_palm_fixed_joint" type="fixed">
+    <origin rpy="1.57 0 0" xyz="-0.0045 0.0145 0.144"/>
+    <parent link="qbhand_base_link"/>
+    <child link="qbhand_palm_link"/>
+  </joint>
+  <link name="qbhand_palm_link">
+    <inertial>
+      <mass value="0.45"/>
+      <origin rpy="0 0 0" xyz="0.0030 -0.0449 0.0135"/>
+      <inertia ixx="0.00045" ixy="0.0" ixz="0.0" iyy="0.0006" iyz="0.0" izz="0.00025"/>
+    </inertial>
+    <visual>
+      <origin rpy="0 0 0" xyz="0 0 0"/>
+      <geometry>
+        <mesh filename="package://softhands_description/meshes/softhands/v3.0/palm_pinch_r.stl" scale="0.001 0.001 0.001"/>
+      </geometry>
+      <material name="qbhand/palm"/>
+    </visual>
+    <collision>
+      <origin rpy="0 0 0" xyz="0 0 0"/>
+      <geometry>
+        <mesh filename="package://softhands_description/meshes/softhands/v3.0/palm_pinch_r.stl" scale="0.001 0.001 0.001"/>
+      </geometry>
+    </collision>
+  </link>
+	</xacro:macro>
 </robot>

File: softhands_description/urdf/xacro/include/macro/v3_simple/phalanges/knuckle.xacro (robot description, xacro)
@@ -38,39 +38,35 @@
 -->
 <robot xmlns:xacro="http://www.ros.org/wiki/xacro">
-  <xacro:macro name="finger_v1_simple" params="type ns position orientation">
+  <xacro:macro name="knuckle" params="type ns position orientation">
     <!-- KNUCKLE -->
-    <xacro:knuckle
-      ns="${ns}"
-      position="${position}"
-      type="${type}"
-      orientation="${orientation}">
-    </xacro:knuckle>
-    <!-- PROXIMAL PHALANGE -->
-    <xacro:phalanx
-      parent="knuckle"
-      name="proximal"
-      ns="${ns}"
-      position="0.020 0 0"
-      type="${type}"
-      orientation="${orientation}">
-    </xacro:phalanx>
-    <!-- MIDDLE PHALANGE -->
-    <xacro:phalanx
-      parent="proximal"
-      name="middle"
-      ns="${ns}"
-      position="0.020 0 0"
-      type="${type}"
-      orientation="${orientation}">
-    </xacro:phalanx>
-    <!-- DISTAL PHALANGE -->
-    <xacro:fingertip
-      parent="middle"
-      name="distal"
-      ns="${ns}"
-      position="0.020 0 0"
-      type="${type}"
-      orientation="${orientation}">
-    </xacro:fingertip>
+    <joint name="${ns}_${type}_knuckle_joint" type="revolute">
+      <origin xyz="${position}" rpy="${orientation}"/>
+      <parent link="${ns}_palm_link"/>
+      <child link="${ns}_${type}_knuckle_link"/>
+      <limit effort="30" velocity="1.0" lower="-1.57" upper="1.57" />
+      <axis xyz="0 0 $(arg sign)" />
+      <dynamics damping="0.08" friction="0.0" />
+    </joint>
+    <link name="${ns}_${type}_knuckle_link">
+      <inertial>
+        <origin xyz="0.001285644 0 0.000425011"/>
+        <mass value="0.09"/>
+        <inertia ixx="0.001" ixy="0" ixz="0" iyy="0.001" iyz="0" izz="0.001"/>
+      </inertial>
+      <visual>
+        <geometry>
+          <mesh filename="package://softhands_description/meshes/softhands/v1.0/common/knuckle_m.stl"/>
+        </geometry>
+      </visual>
+      <collision>
+        <geometry>
+          <mesh filename="package://softhands_description/meshes/softhands/v1.0/common/knuckle_m.stl"/>
+        </geometry>
+      </collision>
+    </link>
+    <gazebo reference="${ns}_${type}_knuckle_link">
+      <material>Gazebo/Grey</material>
+      <selfCollide>true</selfCollide>
+	  </gazebo>
   </xacro:macro>
 </robot>

File: softhands_description/urdf/xacro/v3_simple.xacro (robot description, xacro)
@@ -45,4 +45,12 @@
 		<xacro:arg name="sign" default="-1"/>
     </xacro:if>
+	<xacro:base
+		type="$(arg type)"
+		sign="$(arg sign)"
+		parent = "$(arg parent)"
+		position ="$(arg position)"
+		orientation ="$(arg orientation)"
+		operation_mode = "$(arg operation_mode)">
+	</xacro:base>
 	<xacro:palm
 		type="$(arg type)"
@@ -53,47 +61,3 @@
 		operation_mode = "$(arg operation_mode)">
 	</xacro:palm>
-	<!-- # Thumb finger -->
-	<xacro:thumb_v1_simple
-		type="thumb"
-		sign="$(arg sign)"
-		ns="$(arg type)_hand_v1s"
-		position="0.00566972 ${$(arg sign)*0.0296160} 0.0553140"
-		orientation="0.0 -0.38397275793662144 ${$(arg sign)*1.5707963267948966}">
-	</xacro:thumb_v1_simple>
-	<!-- # Index finger -->
-	<xacro:finger_v1_simple
-		type="index"
-		ns="$(arg type)_hand_v1s"
-		position="-0.0033 ${$(arg sign)*0.0195} 0.0936994"
-		orientation="${$(arg sign)*1.5707963267948966} -1.4835299330931884 ${$(arg sign)*1.5707963267948966}">
-	</xacro:finger_v1_simple>
-	<!-- # Middle finger -->
-	<xacro:finger_v1_simple
-		type="middle"
-		ns="$(arg type)_hand_v1s"
-		position="-0.003300000 0.0 0.100699"
-		orientation="3.141592 -1.5707963267948966 0.0">
-	</xacro:finger_v1_simple>
-	<!-- # Ring finger -->
-	<xacro:finger_v1_simple
-		type="ring"
-		ns="$(arg type)_hand_v1s"
-		position="-0.0033 ${$(arg sign)*-0.0195} 0.0936994"
-		orientation="${$(arg sign)*-1.5707963267948966} -1.5184364298870514 ${$(arg sign)*-1.5707963267948966}">
-	</xacro:finger_v1_simple>
-	<!-- # Little finger -->
-	<xacro:finger_v1_simple
-		type="little"
-		ns="$(arg type)_hand_v1s"
-		position="-0.0033 ${$(arg sign)*-0.039} 0.0836994"
-		orientation="${$(arg sign)*-1.5707963267948966} -1.4835299330931884 ${$(arg sign)*-1.5707963267948966}">
-	</xacro:finger_v1_simple>
-		<!-- # Gazebo NEW custom synergy-plugin -->
-	<gazebo>
-		<plugin name="synergy_plugin" filename="libsofthand_plugin.so">
-			<namespace>$(arg type)_hand_v1s</namespace>
-			<operation_mode>$(arg operation_mode)</operation_mode>
-			<!-- TODO: Insert here the OPTIONAL tags available! -->
-		</plugin>
-	</gazebo>
 </robot>
