Commit message: first draft with full urdf

File: softhands_description/urdf/xacro/include/macro/v_wide/header.xacro (robot description, xacro)
@@ -38,7 +38,18 @@
 -->
 <robot xmlns:xacro="http://www.ros.org/wiki/xacro" name="header">
-  <!-- Include xacro macro -->
-	<xacro:include filename="$(arg root_dir)/modules/palm_central.xacro" />
-	<xacro:include filename="$(arg root_dir)/modules/palm_thumb.xacro" />
+  <!-- Include xacro macro  Palm-->
+	<xacro:include filename="$(arg root_dir)/modules/palm/palm_central.xacro" />
+	<xacro:include filename="$(arg root_dir)/modules/palm/palm_thumb.xacro" />
+  <xacro:include filename="$(arg root_dir)/modules/palm/palm_little.xacro" />
+  <!-- Include xacro macro Thumb -->
+  <xacro:include filename="$(arg root_dir)/modules/thumb.xacro" />
+  <xacro:include filename="$(arg root_dir)/modules/thumb/thumb_prox.xacro" />
+  <xacro:include filename="$(arg root_dir)/modules/thumb/thumb_mid.xacro" />
+  <xacro:include filename="$(arg root_dir)/modules/thumb/thumb_dist.xacro" />
+  <!-- Include xacro macro Finger -->
+  <xacro:include filename="$(arg root_dir)/modules/finger/phalanx_prox_sup.xacro" />
+  <xacro:include filename="$(arg root_dir)/modules/finger/phalanx.xacro" />
+  <xacro:include filename="$(arg root_dir)/modules/finger/phalanx_dist.xacro" />
+  <xacro:include filename="$(arg root_dir)/modules/finger.xacro" />
   <!-- Color definitions -->
   <xacro:include filename="$(arg root_dir)/color.xacro" />

File: softhands_description/urdf/xacro/include/macro/v_wide/modules/thumb/thumb_dist.xacro (robot description, xacro)
@@ -1,5 +1,6 @@
 <?xml version="1.0"?>
 <robot xmlns:xacro="http://www.ros.org/wiki/xacro">
-    <xacro:macro name="palm_thumb" params="name parent side *origin">
+    <xacro:macro name="thumb_dist" params="name parent side *origin">
+		<!-- Thumb middle  -->
 		<joint name="${side}_${name}_joint" type="revolute">
 			<parent link="${side}_${parent}_link"/>
@@ -15,5 +16,5 @@
 					<geometry>
 					<mesh
-						filename="package://softhands_description/meshes/softhands/wide/${side}/palm_thumb.stl"
+						filename="package://softhands_description/meshes/softhands/wide/${side}/phalanx_dist_thumb.stl"
 						scale="0.001 0.001 0.001" />
 					</geometry>
@@ -30,5 +31,5 @@
 					<geometry>
 					<mesh
-						filename="package://softhands_description/meshes/softhands/wide/${side}/palm_thumb.stl"
+						filename="package://softhands_description/meshes/softhands/wide/${side}/phalanx_dist_thumb.stl"
 						scale="0.001 0.001 0.001" />
 					</geometry>
@@ -36,9 +37,4 @@
 				</collision>
 		</link>
-		<!--
-		<gazebo reference="base_link">
-			<material>Gazebo/SkyBlue</material>
-			<selfCollide>true</selfCollide>
-		</gazebo> -->
     </xacro:macro>
 </robot>

File: softhands_description/urdf/xacro/include/macro/v_wide/modules/thumb/thumb_prox.xacro (robot description, xacro)
@@ -1,13 +1,13 @@
 <?xml version="1.0"?>
 <robot xmlns:xacro="http://www.ros.org/wiki/xacro">
-    <xacro:macro name="palm_central" params="name parent side *origin">
-		<!-- World -->
-		<link name="${parent}">
-		</link>
-		<!-- World to palm base -->
-		<joint name="${side}_${name}_joint" type="fixed">
-			<parent link="${parent}"/>
+    <xacro:macro name="thumb_prox" params="name parent side *origin">
+		<!-- Thumb Proximal  -->
+		<joint name="${side}_${name}_joint" type="revolute">
+			<parent link="${side}_${parent}_link"/>
 			<child link="${side}_${name}_link"/>
 			<xacro:insert_block name="origin"/>
+			<axis xyz="0 0 1" />
+      		<limit effort="30" velocity="1.0" lower="0" upper="1.57" />
+			<dynamics damping="0.08" friction="0.0" />
 		</joint>
 		<link name="${side}_${name}_link">
@@ -16,5 +16,5 @@
 					<geometry>
 					<mesh
-						filename="package://softhands_description/meshes/softhands/wide/${side}/palm_central.stl"
+						filename="package://softhands_description/meshes/softhands/wide/${side}/phalanx_pros_thumb.stl"
 						scale="0.001 0.001 0.001" />
 					</geometry>
@@ -31,5 +31,5 @@
 					<geometry>
 					<mesh
-						filename="package://softhands_description/meshes/softhands/wide/${side}/palm_central.stl"
+						filename="package://softhands_description/meshes/softhands/wide/${side}/phalanx_pros_thumb.stl"
 						scale="0.001 0.001 0.001" />
 					</geometry>
@@ -37,13 +37,13 @@
 				</collision>
 		</link>
-		<!-- palm base to mobile thumb -->
-		<joint name="${side}_${name}_to_mobile_thumb_joint" type="revolute">
+		<!-- thumb proximal to mobile thumb proximal   -->
+		<joint name="${side}_${name}_to_mobile_joint" type="revolute">
 			<axis xyz="0 0 1"/>
 			<limit effort="0.0" lower="0" upper="0"  velocity="0.0"/>
-			<origin xyz="39.6398e-3 32.5059e-3 0" rpy="1.5707963 0 1.9198617"/>
+			<origin xyz=" 31.2357e-3 23.0197e-3 0.167417e-3" rpy=" 0.1745395 0.0000165 0.7597087"/>
 			<parent link="${side}_${name}_link"/>
-			<child link="${side}_${name}_to_mobile_thumb_link"/>
+			<child link="${side}_${name}_to_mobile_link"/>
 		</joint>
-	    <link name="${side}_${name}_to_mobile_thumb_link">
+	    <link name="${side}_${name}_to_mobile_link">
 		   <inertial>
 			<origin xyz="0 0 0" rpy="0 0 0"/>
@@ -54,4 +54,9 @@
 		   </inertial>
 	    </link>
+		<!--
+		<gazebo reference="base_link">
+			<material>Gazebo/SkyBlue</material>
+			<selfCollide>true</selfCollide>
+		</gazebo> -->
     </xacro:macro>
 </robot>

File: softhands_description/urdf/xacro/v_wide.xacro (robot description, xacro)
@@ -53,3 +53,27 @@
 		<origin rpy="0 0 0 " xyz="12e-3 -0.0000414746e-3 0"/>
 	</xacro:palm_thumb>
+	<!-- # palm little -->
+	<xacro:palm_little name="palm_little" parent="palm_central_to_mobile_little" side="$(arg side)">
+		<origin rpy="0 0 0 " xyz="12e-3 -0.0000466576e-3 0"/>
+	</xacro:palm_little>
+	<!-- # thumb -->
+	<xacro:thumb name="thumb" parent="palm_thumb_support" side="$(arg side)">
+		<origin rpy="1.5707963 0.7598972 0" xyz="21.9577e-3 0 -2.8e-3"/>
+	</xacro:thumb>
+	<!-- # Index -->
+	<xacro:finger name="index" parent="palm_central" side="$(arg side)">
+		<origin xyz="5e-3 44.8953e-3 112.230e-3" rpy="1.5707963 -1.3962636 1.5707963"/>
+	</xacro:finger>
+	<!-- # Middle -->
+	<xacro:finger name="middle" parent="palm_central" side="$(arg side)">
+		<origin xyz="5e-3 12.5e-3 115e-3" rpy="0 -1.5707963 -3.1415927"/>
+	</xacro:finger>
+	<!-- # Ring -->
+	<xacro:finger name="ring" parent="palm_little" side="$(arg side)">
+	    <origin xyz=" 8.6355e-3 5e-3 44.4863e-3" rpy="-1.5707963 -1.3089971 0"/>
+	</xacro:finger>
+    <!-- # Little -->
+	<xacro:finger name="little" parent="palm_little" side="$(arg side)">
+		<origin xyz="39.2985e-3 5e-3 34.8419e-3" rpy="-1.5707963 -1.221731 0"/>
+	</xacro:finger>
 </robot>
