Commit message: added structure of v2

File: softhands_description/urdf/old/v2.0/thumb.xacro (robot description, xacro)
@@ -203,5 +203,5 @@
       <inertial>
         <origin xyz="0.005074337 0 0"/>
-        <mass value="0.05"/>
+        <mass value="0.05"/>Giancarlo Magalli
         <inertia ixx="0.001" ixy="0" ixz="0" iyy="0.001" iyz="0" izz="0.001"/>
       </inertial>

File: softhands_description/urdf/softhand.urdf.xacro (robot description, xacro)
@@ -38,9 +38,10 @@
 -->
 <robot name="softhand" xmlns:xacro="http://www.ros.org/wiki/xacro">
-  	<xacro:arg name="sh_version" default="v1_simple"/>
+  	<xacro:arg name="sh_version" default="v2"/>
   	<xacro:arg name="root_dir" default="$(find softhands_description)/urdf/xacro/include/macro/$(arg sh_version)"/>
   	<xacro:arg name="parent" default="world"/>
-  	<xacro:arg name="type" default="left"/>
-  	<xacro:arg name="position" default="0 0 0"/>
+  	<xacro:arg name="side" default="right"/>
+  	<xacro:arg name="ns" default="$(arg side)_hand_$(arg sh_version)"/>
+  	<xacro:arg name="position" default="0 0 0.01"/>
   	<xacro:arg name="orientation" default="0 0 0"/>
   	<xacro:arg name="operation_mode" default="0"/>

File: softhands_description/urdf/xacro/include/macro/v2/base.xacro (robot description, xacro)
@@ -37,31 +37,36 @@
  *
 -->
-<robot name="Palm_v1_simple" xmlns:xacro="http://www.ros.org/wiki/xacro">
-	<xacro:macro name="palm" params="type sign parent position orientation operation_mode">
-	  <joint name="qbhand_palm_fixed_joint" type="fixed">
-    <origin rpy="1.57 0 0" xyz="-0.0045 0.0145 0.144"/>
-    <parent link="qbhand_base_link"/>
-    <child link="qbhand_palm_link"/>
-  </joint>
-  <link name="qbhand_palm_link">
-    <inertial>
-      <mass value="0.45"/>
-      <origin rpy="0 0 0" xyz="0.0030 -0.0449 0.0135"/>
-      <inertia ixx="0.00045" ixy="0.0" ixz="0.0" iyy="0.0006" iyz="0.0" izz="0.00025"/>
-    </inertial>
-    <visual>
-      <origin rpy="0 0 0" xyz="0 0 0"/>
-      <geometry>
-        <mesh filename="package://softhands_description/meshes/softhands/v3.0/palm_pinch_r.stl" scale="0.001 0.001 0.001"/>
-      </geometry>
-      <material name="qbhand/palm"/>
-    </visual>
-    <collision>
-      <origin rpy="0 0 0" xyz="0 0 0"/>
-      <geometry>
-        <mesh filename="package://softhands_description/meshes/softhands/v3.0/palm_pinch_r.stl" scale="0.001 0.001 0.001"/>
-      </geometry>
-    </collision>
-  </link>
+<robot name="base_v3" xmlns:xacro="http://www.ros.org/wiki/xacro">
+	<xacro:macro name="base" params="sign ns parent position orientation operation_mode">
+		<link name="${parent}"/>
+		<joint name="${ns}_base_joint" type="fixed">
+			<origin rpy="${orientation}" xyz="${position}"/>
+			<parent link="${parent}" />
+			<child link="${ns}_palm_base_link" />
+		</joint>
+		<link name="${ns}_palm_base_link">
+			<inertial>
+				<mass value="0.45"/>
+				<origin rpy="0 0 0" xyz="0.0030 -0.0449 0.0135"/>
+				<inertia ixx="0.00045" ixy="0.0" ixz="0.0" iyy="0.0006" iyz="0.0" izz="0.00025"/>
+			</inertial>
+			<visual>
+				<origin rpy="0 0 0" xyz="0 0 0"/>
+				<geometry>
+					<mesh filename="package://softhands_description/meshes/softhands/v3.0/flange_iso_04.stl" scale="0.001 0.001 0.001"/>
+				</geometry>
+				<material name="qbhand/base"/>
+			</visual>
+			<collision>
+			<origin rpy="0 0 0" xyz="0 0 0"/>
+			<geometry>
+				<mesh filename="package://softhands_description/meshes/softhands/v3.0/flange_iso_04.stl" scale="0.001 0.001 0.001"/>
+			</geometry>
+			</collision>
+		</link>
+		<gazebo reference="${ns}_palm_base_link">
+    	  	<material>Gazebo/Grey</material>
+			<selfCollide>true</selfCollide>
+	  	</gazebo>
 	</xacro:macro>
 </robot>

File: softhands_description/urdf/xacro/include/macro/v2/finger.xacro (robot description, xacro)
@@ -38,35 +38,39 @@
 -->
 <robot xmlns:xacro="http://www.ros.org/wiki/xacro">
-  <xacro:macro name="phalanx" params="type ns parent name position orientation">
+  <xacro:macro name="finger_v3_simple" params="type ns position orientation">
+    <!-- KNUCKLE -->
+    <xacro:knuckle
+      ns="${ns}"
+      position="${position}"
+      type="${type}"
+      orientation="${orientation}">
+    </xacro:knuckle>
     <!-- PROXIMAL PHALANGE -->
-    <joint name="${ns}_${type}_${name}_joint" type="revolute">
-      <origin xyz="${position}" rpy="${orientation}" />
-      <parent link="${ns}_${type}_${parent}_link"/>
-      <child link="${ns}_${type}_${name}_link"/>
-      <limit effort="30" velocity="1.0" lower="-1.57" upper="1.57" />
-      <axis xyz="0 -1 0" />
-      <dynamics damping="0.08" friction="0.0" />
-    </joint>
-    <link name="${ns}_${type}_${name}_link">
-      <inertial>
-        <origin xyz="0.005074337 0 -0.000262953"/>
-        <mass value="0.05"/>
-        <inertia ixx="0.001" ixy="0" ixz="0" iyy="0.001" iyz="0" izz="0.001"/>
-      </inertial>
-      <visual>
-        <geometry>
-          <mesh filename="package://softhands_description/meshes/softhands/v1.0/common/phalanx_m.stl"/>
-        </geometry>
-      </visual>
-      <collision>
-        <geometry>
-          <mesh filename="package://softhands_description/meshes/softhands/v1.0/common/phalanx_m.stl"/>
-        </geometry>
-      </collision>
-    </link>
-    <gazebo reference="${ns}_${type}_${name}_link">
-      <material>Gazebo/Grey</material>
-      <selfCollide>true</selfCollide>
-	  </gazebo>
+    <xacro:phalanx
+      parent="knuckle"
+      name="proximal"
+      ns="${ns}"
+      position="0.020 0 0"
+      type="${type}"
+      orientation="0 0 0">
+    </xacro:phalanx>
+    <!-- MIDDLE PHALANGE -->
+    <xacro:phalanx
+      parent="proximal"
+      name="middle"
+      ns="${ns}"
+      position="0.020 0 0"
+      type="${type}"
+      orientation="0 0 0">
+    </xacro:phalanx>
+    <!-- DISTAL PHALANGE -->
+    <xacro:fingertip
+      parent="middle"
+      name="distal"
+      ns="${ns}"
+      position="0.020 0 0"
+      type="${type}"
+      orientation="0 0 0">
+    </xacro:fingertip>
   </xacro:macro>
 </robot>

File: softhands_description/urdf/xacro/include/macro/v2/palm.xacro (robot description, xacro)
@@ -37,27 +37,50 @@
  *
 -->
-<robot name="sh_v1_simple" xmlns:xacro="http://www.ros.org/wiki/xacro">
-	<xacro:property name="side" value="$(arg type)"/>
-    <xacro:if value="${side == 'right'}">
-		<xacro:arg name="sign" default="1"/>
-	</xacro:if>
-    <xacro:if value="${side == 'left'}">
-		<xacro:arg name="sign" default="-1"/>
-    </xacro:if>
-	<xacro:base
-		type="$(arg type)"
-		sign="$(arg sign)"
-		parent = "$(arg parent)"
-		position ="$(arg position)"
-		orientation ="$(arg orientation)"
-		operation_mode = "$(arg operation_mode)">
-	</xacro:base>
-	<xacro:palm
-		type="$(arg type)"
-		sign="$(arg sign)"
-		parent = "$(arg parent)"
-		position ="$(arg position)"
-		orientation ="$(arg orientation)"
-		operation_mode = "$(arg operation_mode)">
-	</xacro:palm>
+<robot name="palm_v3" xmlns:xacro="http://www.ros.org/wiki/xacro">
+	<xacro:macro name="palm" params="sign ns parent position orientation operation_mode">
+	  	<joint name="${ns}_palm_joint" type="fixed">
+			<origin rpy="${orientation}" xyz="${position}"/>
+			<parent link="${ns}_palm_base_link" />
+			<child link="${ns}_palm_link" />
+		</joint>
+		<link name="${ns}_palm_link">
+			<inertial>
+			<mass value="0.45"/>
+			<origin rpy="0 0 0" xyz="0.0030 -0.0449 0.0135"/>
+			<inertia ixx="0.00045" ixy="0.0" ixz="0.0" iyy="0.0006" iyz="0.0" izz="0.00025"/>
+			</inertial>
+			<visual>
+			<origin rpy="0 0 0" xyz="0 0 0"/>
+			<geometry>
+				<mesh filename="package://softhands_description/meshes/softhands/v3.0/palm_pinch_r.stl" scale="0.001 0.001 0.001"/>
+			</geometry>
+			<material name="qbhand/palm"/>
+			</visual>
+			<collision>
+			<origin rpy="0 0 0" xyz="0 0 0"/>
+			<geometry>
+				<mesh filename="package://softhands_description/meshes/softhands/v3.0/palm_pinch_r.stl" scale="0.001 0.001 0.001"/>
+			</geometry>
+			</collision>
+		</link>
+		<joint name="${ns}_synergy_joint" type="revolute">
+			<origin rpy="0 0 0" xyz="0 0 0"/>
+			<parent link="${ns}_palm_link"/>
+			<child link="${ns}_synergy_tendon_virtual_link"/>
+			<axis xyz="0 0 1"/>
+			<dynamics damping="0.0" friction="0.0"/>
+			<limit effort="100" lower="0.0" upper="1.0" velocity="100"/>
+		</joint>
+		<link name="${ns}_synergy_tendon_virtual_link">
+			<inertial>
+			<origin rpy="0 0 0" xyz="0 0 0"/>
+			<mass value="1e-4"/>
+			<inertia ixx="1e-9" ixy="0.0" ixz="0.0" iyy="1e-9" iyz="0.0" izz="1e-9"/>
+			</inertial>
+		</link>
+	<gazebo reference="${ns}_palm_link">
+		<material>Gazebo/Grey</material>
+		<selfCollide>true</selfCollide>
+	</gazebo>
+	</xacro:macro>
 </robot>

File: softhands_description/urdf/xacro/include/macro/v2/phalanges/fingertip.xacro (robot description, xacro)
@@ -39,34 +39,54 @@
 <robot xmlns:xacro="http://www.ros.org/wiki/xacro">
   <xacro:macro name="fingertip" params="type ns parent name position orientation">
-    <!-- DISTAL PHALANGE -->
-    <joint name="${ns}_${type}_${name}_joint" type="revolute">
-      <origin xyz="${position}" rpy="0 0 0" />
+    <joint name="${ns}_${type}_${parent}_${name}_joint" type="revolute">
+      <origin rpy="${orientation}" xyz="${position}"/>
       <parent link="${ns}_${type}_${parent}_link"/>
-      <child link="${ns}_${type}_${name}_link"/>
+      <child link="${ns}_${type}_${parent}_${name}_virtual_link"/>
+      <axis xyz="0 0 -1"/>
+      <dynamics damping="0.0" friction="0.0"/>
       <limit effort="30" velocity="1.0" lower="-1.57" upper="1.57" />
-      <axis xyz="0 -1 0" />
-      <dynamics damping="0.08" friction="0.0" />
+      <mimic joint="${ns}_synergy_joint" multiplier="0.785"/>
     </joint>
-    <link name="${ns}_${type}_${name}_link">
-      <inertial>
-            <origin xyz="0.009849094 0 0.000820286"/>
-        <mass value="0.1"/>
-        <inertia ixx="0.001" ixy="0" ixz="0" iyy="0.001" iyz="0" izz="0.001"/>
-      </inertial>
-      <visual>
-        <geometry>
-          <mesh filename="package://softhands_description/meshes/softhands/v1.0/common/fingertip_m.stl"/>
-        </geometry>
-      </visual>
-      <collision>
-        <geometry>
-          <mesh filename="package://softhands_description/meshes/softhands/v1.0/common/fingertip_m.stl"/>
-        </geometry>
-      </collision>
-    </link>
-    <gazebo reference="${ns}_${type}_${name}_link">
-      <material>Gazebo/Grey</material>
-      <selfCollide>true</selfCollide>
-	  </gazebo>
+  <!-- <link name="${ns}_${parent}_${name}_virtual_link">
+    <inertial>
+      <origin rpy="0 0 0" xyz="0 0 0"/>
+      <mass value="1e-4"/>
+      <inertia ixx="1e-9" ixy="0.0" ixz="0.0" iyy="1e-9" iyz="0.0" izz="1e-9"/>
+    </inertial>
+  </link> -->
+<!--
+  <joint name="${ns}_${parent}_${name}_virtual_joint" type="revolute">
+    <origin rpy="0 0 0" xyz="0.013 0 0"/>
+    <parent link="${ns}_${parent}_${name}_virtual_link"/>
+    <child link="${ns}_${parent}_${name}_link"/>
+    <axis xyz="0 0 -1"/>
+    <dynamics damping="0.0" friction="0.0"/>
+    <limit effort="100" lower="0.0" upper="0.785" velocity="100"/>
+    <mimic joint="${ns}_${parent}_${name}_joint" multiplier="1.0"/>
+  </joint>
+  <link name="${ns}_${parent}_${name}_link">
+    <inertial>
+      <mass value="0.009"/>
+      <origin rpy="0 0 0" xyz="8.8025467e-03 -1.7219289e-03 0.0"/>
+      <inertia ixx="2.6586142e-07" ixy="1.2416847e-08" ixz="0.0" iyy="5.9935767e-07" iyz="0.0" izz="6.6781963e-07"/>
+    </inertial>
+    <visual>
+      <origin rpy="0 0 0" xyz="0 0 0"/>
+      <geometry>
+        <mesh filename="package://softhands_description/meshes/softhands/v3.0/ph_distal.stl" scale="0.001 0.001 0.001"/>
+      </geometry>
+      <material name="qbhand/distal"/>
+    </visual>
+    <collision>
+      <origin rpy="0 0 0" xyz="0 0 0"/>
+      <geometry>
+        <mesh filename="package://softhands_description/meshes/softhands/v3.0/ph_distal_collision.stl" scale="0.001 0.001 0.001"/>
+      </geometry>
+    </collision>
+  </link>
+  <gazebo reference="${ns}_${parent}_${name}_link">
+    <material>Gazebo/Grey</material>
+    <self_collide>false</self_collide>
+  </gazebo> -->
   </xacro:macro>
 </robot>

File: softhands_description/urdf/xacro/include/macro/v2/phalanges/thumb_knuckle.xacro (robot description, xacro)
@@ -31,5 +31,5 @@
  * OF THIS SOFTWARE, EVEN IF ADVISED OF THE POSSIBILITY OF SUCH DAMAGE.
  *
- * \file      thumb.xacro
+ * \file      finger.xacro
  *
  * \author       _Centro di Ricerca "E.Piaggio"_
@@ -38,30 +38,39 @@
 -->
 <robot xmlns:xacro="http://www.ros.org/wiki/xacro">
-  <xacro:macro name="thumb_v1_simple" params="type ns sign position orientation">
+  <xacro:macro name="thumb_knuckle" params="type ns position orientation">
     <!-- KNUCKLE -->
-    <xacro:thumb_knuckle
-      ns="${ns}"
-      position="${position}"
-      type="${type}"
-      orientation="${orientation}">
-    </xacro:thumb_knuckle>
-    <!-- PROXIMAL PHALANGE -->
-    <xacro:phalanx
-      parent="knuckle"
-      name="proximal"
-      ns="${ns}"
-      position="0.033500000 ${sign*-0.003300000} 0.0"
-      type="${type}"
-      orientation="${sign*0.426627741408745} 0 0.0">
-    </xacro:phalanx>
-    <!-- DISTAL PHALANGE -->
-    <xacro:fingertip
-      parent="proximal"
-      name="distal"
-      ns="${ns}"
-      position="0.020 0 0"
-      type="${type}"
-      orientation="0 0 0">
-    </xacro:fingertip>
+    <joint name="${ns}_${type}_knuckle_joint" type="revolute">
+      <origin xyz="${position}" rpy="${orientation}"/>
+      <parent link="${ns}_palm_link"/>
+      <child link="${ns}_${type}_knuckle_link"/>
+      <axis xyz="0 0 -1"/>
+      <dynamics damping="0.0" friction="0.0"/>
+      <limit effort="100" lower="0.0" upper="1.571" velocity="100"/>
+      <mimic joint="${ns}_synergy_joint" multiplier="2.542"/>
+    </joint>
+    <link name="${ns}_${type}_knuckle_link">
+      <inertial>
+        <mass value="0.01"/>
+        <origin rpy="0 0 0" xyz="1.3071561e-02 -2.7357764e-03 6.4347823e-04"/>
+        <inertia ixx="3.5865978e-07" ixy="2.0944224e-07" ixz="-6.8657569e-08" iyy="1.3885564e-06" iyz="3.2170608e-08" izz="1.3571203e-06"/>
+      </inertial>
+      <visual>
+        <origin rpy="0 0 0" xyz="0 0 0"/>
+        <geometry>
+          <mesh filename="package://softhands_description/meshes/softhands/v3.0/ph_thumb_r.stl" scale="0.001 0.001 0.001"/>
+        </geometry>
+        <material name="qbhand/knuckle"/>
+      </visual>
+      <collision>
+        <origin rpy="0 0 0" xyz="0 0 0"/>
+        <geometry>
+          <mesh filename="package://softhands_description/meshes/softhands/v3.0/ph_thumb_r_collision.stl" scale="0.001 0.001 0.001"/>
+        </geometry>
+      </collision>
+    </link>
+    <gazebo reference="${ns}_${type}_knuckle_link">
+      <material>Gazebo/Grey</material>
+      <selfCollide>false</selfCollide>
+	  </gazebo>
   </xacro:macro>
 </robot>

File: softhands_description/urdf/xacro/include/macro/v2/thumb.xacro (robot description, xacro)
@@ -31,5 +31,5 @@
  * OF THIS SOFTWARE, EVEN IF ADVISED OF THE POSSIBILITY OF SUCH DAMAGE.
  *
- * \file      finger.xacro
+ * \file      thumb.xacro
  *
  * \author       _Centro di Ricerca "E.Piaggio"_
@@ -38,39 +38,31 @@
 -->
 <robot xmlns:xacro="http://www.ros.org/wiki/xacro">
-  <xacro:macro name="finger_v1_simple" params="type ns position orientation">
+  <xacro:macro name="thumb" params="type ns sign position orientation">
     <!-- KNUCKLE -->
-    <xacro:knuckle
+    <xacro:thumb_knuckle
       ns="${ns}"
       position="${position}"
       type="${type}"
       orientation="${orientation}">
-    </xacro:knuckle>
+    </xacro:thumb_knuckle>
     <!-- PROXIMAL PHALANGE -->
     <xacro:phalanx
+      type="${type}"
       parent="knuckle"
       name="proximal"
       ns="${ns}"
-      position="0.020 0 0"
-      type="${type}"
-      orientation="0 0 0">
-    </xacro:phalanx>
-    <!-- MIDDLE PHALANGE -->
-    <xacro:phalanx
-      parent="proximal"
-      name="middle"
-      ns="${ns}"
-      position="0.020 0 0"
-      type="${type}"
-      orientation="0 0 0">
+      position="0.0255 -0.0038 -0.00012"
+      orientation="-1.1415 0.0 0.0">
     </xacro:phalanx>
     <!-- DISTAL PHALANGE -->
-    <xacro:fingertip
-      parent="middle"
+    <!-- <xacro:fingertip
+      type="${type}"
+      parent="proximal"
       name="distal"
       ns="${ns}"
-      position="0.020 0 0"
-      type="${type}"
+      position="0.009 0 0"
       orientation="0 0 0">
     </xacro:fingertip>
+    -->
   </xacro:macro>
 </robot>

File: softhands_description/urdf/xacro/v2.xacro (robot description, xacro)
@@ -37,35 +37,43 @@
  *
 -->
-<robot name="Palm_v1_simple" xmlns:xacro="http://www.ros.org/wiki/xacro">
-	<xacro:macro name="base" params="type sign parent position orientation operation_mode">
-		<link name="root_link"/>
-		<joint name="qbhand_base_fixed_joint" type="fixed">
-			<origin rpy="0 0 0" xyz="0 0 0"/>
-			<parent link="root_link"/>
-			<child link="qbhand_base_link"/>
-		</joint>
-		<link name="qbhand_base_link">
-			<inertial>
-			<mass value="0.45"/>
-			<origin rpy="0 0 0" xyz="0.0030 -0.0449 0.0135"/>
-			<inertia ixx="0.00045" ixy="0.0" ixz="0.0" iyy="0.0006" iyz="0.0" izz="0.00025"/>
-			</inertial>
-			<visual>
-			<origin rpy="0 0 0" xyz="0 0 0"/>
-			<geometry>
-				<mesh filename="package://softhands_description/meshes/softhands/v3.0/flange_iso_04.stl" scale="0.001 0.001 0.001"/>
-			</geometry>
-			<material name="qbhand/base"/>
-			</visual>
-			<collision>
-			<origin rpy="0 0 0" xyz="0 0 0"/>
-			<geometry>
-				<mesh filename="package://softhands_description/meshes/softhands/v3.0/flange_iso_04.stl" scale="0.001 0.001 0.001"/>
-			</geometry>
-			</collision>
-		</link>
-		<gazebo reference="qbhand_base_link">
-			<self_collide>1</self_collide>
-		</gazebo>
-	</xacro:macro>
+<robot name="v3" xmlns:xacro="http://www.ros.org/wiki/xacro">
+	<xacro:property name="side_" value="$(arg side)"/>
+    <xacro:if value="${side_ == 'right'}">
+		<xacro:arg name="sign" default="1"/>
+	</xacro:if>
+    <xacro:if value="${side_ == 'left'}">
+		<xacro:arg name="sign" default="-1"/>
+    </xacro:if>
+	<!-- type: right/left -->
+	<!-- parent: root_link/world -->
+	<xacro:base
+		sign="$(arg sign)"
+		ns="$(arg ns)"
+		parent = "$(arg parent)"
+		position ="$(arg position)"
+		orientation ="$(arg orientation)"
+		operation_mode = "$(arg operation_mode)">
+	</xacro:base>
+	<xacro:palm
+		sign="$(arg sign)"
+		ns="$(arg ns)"
+		parent = "$(arg parent)"
+		position ="-0.0045 0.0145 0.144"
+		orientation ="1.57 0 0"
+		operation_mode = "$(arg operation_mode)">
+	</xacro:palm>
+	<!-- # Thumb finger -->
+	<xacro:thumb
+		type="thumb"
+		sign="$(arg sign)"
+		ns="$(arg ns)"
+		position="-0.044 -0.0465 -0.002"
+		orientation="-1.57 3.14 0.0">
+	</xacro:thumb>
+	<!-- <gazebo>
+		<plugin name="synergy_plugin" filename="libsofthand_plugin.so">
+			<namespace>$(arg type)_hand_v3s</namespace>
+			<operation_mode>$(arg operation_mode)</operation_mode>
+		</plugin>
+	</gazebo> -->
 </robot>
