Commit message: update v_wide softhand

File: softhands_description/urdf/old/v2.0/thumb.xacro (robot description, xacro)
@@ -55,16 +55,16 @@
       </inertial>
       <visual>
-	<geometry>
-	  <mesh filename="package://softhands_description/meshes/softhands/v2.0/right/qbh_prox_thumb_ng.stl" scale="0.001 0.001 0.001"/>
-	</geometry>
-	<material name="qbmove/default"/>
-	<origin xyz="0 0 0" rpy="0 0 0"/>
-      </visual>
-      <collision>
-	<geometry>
-	  <mesh filename="package://softhands_description/meshes/softhands/v2.0/right/qbh_prox_thumb_ng_collision.stl" scale="0.001 0.001 0.001"/>
-	</geometry>
-	<origin xyz="0 0 0" rpy="0 0 0"/>
-      </collision>
+        <geometry>
+          <mesh filename="package://softhands_description/meshes/softhands/v2.0/right/qbh_prox_thumb_ng.stl" scale="0.001 0.001 0.001"/>
+        </geometry>
+        <material name="qbmove/default"/>
+        <origin xyz="0 0 0" rpy="0 0 0"/>
+            </visual>
+            <collision>
+        <geometry>
+          <mesh filename="package://softhands_description/meshes/softhands/v2.0/right/qbh_prox_thumb_ng_collision.stl" scale="0.001 0.001 0.001"/>
+        </geometry>
+        <origin xyz="0 0 0" rpy="0 0 0"/>
+            </collision>
     </link>
     <gazebo reference="${ns}_${type}_knuckle_link">
@@ -130,16 +130,16 @@
       </inertial>
       <visual>
-	<geometry>
-	  <mesh filename="package://softhands_description/meshes/softhands/v2.0/right/phalanx_std_ng.stl" scale="0.001 0.001 0.001"/>
-	</geometry>
-	<material name="qbmove/default"/>
-	<origin xyz="0 0 0" rpy="0 0 0"/>
-      </visual>
-      <collision>
-        <geometry>
-          <mesh filename="package://softhands_description/meshes/softhands/v2.0/right/phalanx_std_ng_collision.stl" scale="0.001 0.001 0.001"/>
-        </geometry>
-        <origin xyz="0 0 0" rpy="0 0 0"/>
-      </collision>
+      <geometry>
+        <mesh filename="package://softhands_description/meshes/softhands/v2.0/right/phalanx_std_ng.stl" scale="0.001 0.001 0.001"/>
+      </geometry>
+      <material name="qbmove/default"/>
+      <origin xyz="0 0 0" rpy="0 0 0"/>
+          </visual>
+          <collision>
+            <geometry>
+              <mesh filename="package://softhands_description/meshes/softhands/v2.0/right/phalanx_std_ng_collision.stl" scale="0.001 0.001 0.001"/>
+            </geometry>
+            <origin xyz="0 0 0" rpy="0 0 0"/>
+          </collision>
     </link>
     <gazebo reference="${ns}_${type}_proximal_link">

File: softhands_description/urdf/xacro/include/macro/v2/header.xacro (robot description, xacro)
@@ -31,5 +31,5 @@
  * OF THIS SOFTWARE, EVEN IF ADVISED OF THE POSSIBILITY OF SUCH DAMAGE.
  *
- * \file      test_SHs_v2.urdf.xacro
+ *
  *
  * \author       _Centro di Ricerca "E.Piaggio"_
@@ -37,14 +37,13 @@
  *
 -->
-<robot name="softhand" xmlns:xacro="http://www.ros.org/wiki/xacro">
-  	<xacro:arg name="sh_version" default="v2"/>
-  	<xacro:arg name="root_dir" default="$(find softhands_description)/urdf/xacro/include/macro/$(arg sh_version)"/>
-  	<xacro:arg name="parent" default="world"/>
-  	<xacro:arg name="side" default="right"/>
-  	<xacro:arg name="ns" default="$(arg side)_hand_$(arg sh_version)"/>
-  	<xacro:arg name="position" default="0 0 0.01"/>
-  	<xacro:arg name="orientation" default="0 0 0"/>
-  	<xacro:arg name="operation_mode" default="0"/>
-	<xacro:include filename="$(find softhands_description)/urdf/xacro/header.xacro"/>
-	<xacro:include filename="$(find softhands_description)/urdf/xacro/$(arg sh_version).xacro"/>
+<robot xmlns:xacro="http://www.ros.org/wiki/xacro" name="header">
+  <!-- Include xacro macro -->
+	<xacro:include filename="$(arg root_dir)/finger.xacro" />
+	<xacro:include filename="$(arg root_dir)/thumb.xacro" />
+	<xacro:include filename="$(arg root_dir)/base.xacro" />
+	<xacro:include filename="$(arg root_dir)/palm.xacro" />
+	<xacro:include filename="$(arg root_dir)/phalanges/knuckle.xacro" />
+	<xacro:include filename="$(arg root_dir)/phalanges/thumb_knuckle.xacro" />
+	<xacro:include filename="$(arg root_dir)/phalanges/fingertip.xacro" />
+	<xacro:include filename="$(arg root_dir)/phalanges/phalanx.xacro" />
 </robot>

File: softhands_description/urdf/xacro/include/macro/v_wide/color.xacro (robot description, xacro)
@@ -22,3 +22,9 @@
     <color rgba="0.50 0.50 0.50 1.0" />
   </material>
+  <material name="grey">
+    <color rgba="0.3 0.3 0.3 1.0" />
+  </material>
+    <material name="white">
+    <color rgba="0.9 0.9 0.9 1.0" />
+  </material>
 </robot>
