Commit message: small update

File: softhands_description/urdf/old/v2.0/thumb.xacro (robot description, xacro)
@@ -81,4 +81,5 @@
       </surface>
     </gazebo>
+    <!-- Proximal -->
     <joint name="${ns}_${type}_proximal_joint" type="revolute">
       <origin xyz="0.017 -0.00343074 0.00392231" rpy="1.6580634 -0.15 0"/> <!-- added offset on orientation -->
@@ -156,4 +157,5 @@
       </surface>
     </gazebo>
+    <!-- Distal -->
     <joint name="${ns}_${type}_distal_joint" type="revolute">
       <origin xyz="0.009 0 0" rpy="0 0 0.15"/> <!-- added offset on orientation -->
@@ -166,57 +168,57 @@
     <link name="${ns}_${type}_distal_link_fake">
      <inertial>
-	<origin xyz="0 0 0" rpy="0 0 0"/>
-	<mass value="0.001"/>
-	<inertia ixx="0.0001"  ixy="0"  	    ixz="0"
-				iyy="0.0001" 	    iyz="0"
-						    izz="0.0001" />
-      </inertial>
-      <visual>
-        <geometry>
-          <box size="0.001 0.001 0.001"/>
-        </geometry>
-        <origin xyz="0 0 0" rpy="0 0 0"/>
-      </visual>
-    </link>
-    <gazebo reference="${ns}_${type}_distal_link_fake">
-      <material>Gazebo/Grey</material>
-      <kp value="1e4" />
-      <kd value="1e2" />
-      <surface>
-       <friction>
-        <ode>
-         <mu>0.133</mu>
-         <mu2>0.133</mu2>
-        </ode>
-       </friction>
-      </surface>
-    </gazebo>
-    <joint name="${ns}_${type}_distal_virtual_joint" type="revolute">
-      <origin xyz="0.013 0 0" rpy="0 0 0.15"/> <!-- added offset on orientation -->
-      <parent link="${ns}_${type}_distal_link_fake"/>
-      <child link="${ns}_${type}_distal_link"/>
-      <limit effort="30" velocity="1.0" lower="-0.785398" upper="0.785398" />
-      <dynamics damping="0.05" friction="0.0" />
-      <axis xyz="0 0 1" />
-    </joint>
-    <link name="${ns}_${type}_distal_link">
-      <inertial>
-        <origin xyz="0.005074337 0 0"/>
-        <mass value="0.05"/>Giancarlo Magalli
-        <inertia ixx="0.001" ixy="0" ixz="0" iyy="0.001" iyz="0" izz="0.001"/>
-      </inertial>
-      <visual>
-	<geometry>
-	  <mesh filename="package://softhands_description/meshes/softhands/v2.0/right/qb_distal_ng.stl" scale="0.001 0.001 0.001"/>
-	</geometry>
-	<material name="qbmove/default"/>
-	<origin xyz="0 0 0" rpy="0 0 0"/>
-      </visual>
-      <collision>
-        <geometry>
-          <mesh filename="package://softhands_description/meshes/softhands/v2.0/right/qb_distal_ng_collision.stl" scale="0.001 0.001 0.001"/>
-        </geometry>
-        <origin xyz="0 0 0" rpy="0 0 0"/>
-      </collision>
+      <origin xyz="0 0 0" rpy="0 0 0"/>
+      <mass value="0.001"/>
+      <inertia ixx="0.0001"  ixy="0"  	    ixz="0"
+            iyy="0.0001" 	    iyz="0"
+                    izz="0.0001" />
+          </inertial>
+          <visual>
+            <geometry>
+              <box size="0.001 0.001 0.001"/>
+            </geometry>
+            <origin xyz="0 0 0" rpy="0 0 0"/>
+          </visual>
+        </link>
+        <gazebo reference="${ns}_${type}_distal_link_fake">
+          <material>Gazebo/Grey</material>
+          <kp value="1e4" />
+          <kd value="1e2" />
+          <surface>
+          <friction>
+            <ode>
+            <mu>0.133</mu>
+            <mu2>0.133</mu2>
+            </ode>
+          </friction>
+          </surface>
+        </gazebo>
+        <joint name="${ns}_${type}_distal_virtual_joint" type="revolute">
+          <origin xyz="0.013 0 0" rpy="0 0 0.15"/> <!-- added offset on orientation -->
+          <parent link="${ns}_${type}_distal_link_fake"/>
+          <child link="${ns}_${type}_distal_link"/>
+          <limit effort="30" velocity="1.0" lower="-0.785398" upper="0.785398" />
+          <dynamics damping="0.05" friction="0.0" />
+          <axis xyz="0 0 1" />
+        </joint>
+        <link name="${ns}_${type}_distal_link">
+          <inertial>
+            <origin xyz="0.005074337 0 0"/>
+            <mass value="0.05"/>Giancarlo Magalli
+            <inertia ixx="0.001" ixy="0" ixz="0" iyy="0.001" iyz="0" izz="0.001"/>
+          </inertial>
+          <visual>
+      <geometry>
+        <mesh filename="package://softhands_description/meshes/softhands/v2.0/right/qb_distal_ng.stl" scale="0.001 0.001 0.001"/>
+      </geometry>
+      <material name="qbmove/default"/>
+      <origin xyz="0 0 0" rpy="0 0 0"/>
+          </visual>
+          <collision>
+            <geometry>
+              <mesh filename="package://softhands_description/meshes/softhands/v2.0/right/qb_distal_ng_collision.stl" scale="0.001 0.001 0.001"/>
+            </geometry>
+            <origin xyz="0 0 0" rpy="0 0 0"/>
+          </collision>
     </link>
     <gazebo reference="${ns}_${type}_distal_link">

File: softhands_description/urdf/softhands.urdf.xacro (robot description, xacro)
@@ -38,6 +38,7 @@
 -->
 <robot name="softhand" xmlns:xacro="http://www.ros.org/wiki/xacro">
-  	<xacro:arg name="sh_version" default="v_wide"/>
+  	<xacro:arg name="sh_version" default="v2.0_qb"/>
   	<xacro:arg name="root_dir" default="$(find softhands_description)/urdf/xacro/include/macro/$(arg sh_version)"/>
+  	<xacro:arg name="meshes_dir" default="package://softhands_description/meshes/softhands/$(arg sh_version)"/>
   	<xacro:arg name="root_link" default="world"/>
   	<xacro:arg name="side" default="right"/>

File: softhands_description/urdf/xacro/include/macro/v1.0_wide/modules/finger.xacro (robot description, xacro)
@@ -13,5 +13,5 @@
       <xacro:phalanx name="${name}_phalanx_mid" parent="${name}_phalanx_prox_virtual" side="$(arg side)">
         <origin rpy="0 0 0" xyz="9e-3 0 0"/>
-      </xacro:phalanx >
+      </xacro:phalanx>
       <!-- Distal -->
       <xacro:phalanx_dist name="${name}_phalanx_dist" parent="${name}_phalanx_mid_virtual" side="$(arg side)">

File: softhands_description/urdf/xacro/include/macro/v1.0_wide/modules/finger/phalanx.xacro (robot description, xacro)
@@ -1,13 +1,10 @@
 <?xml version="1.0"?>
 <robot xmlns:xacro="http://www.ros.org/wiki/xacro">
-    <xacro:macro name="thumb_mid" params="name parent side *origin">
-		<!-- Thumb middle  -->
-		<joint name="${side}_${name}_joint" type="revolute">
-			<parent link="${side}_${parent}_link"/>
+    <xacro:macro name="phalanx" params="name parent side *origin">
+		<!-- Proximal phalanx -->
+		<joint name="${side}_${parent}_${name}_joint" type="fixed">
+			<xacro:insert_block name="origin"/>
+            <parent link="${side}_${parent}_link"/>
 			<child link="${side}_${name}_link"/>
-			<xacro:insert_block name="origin"/>
-			<axis xyz="0 0 1" />
-      		<limit effort="30" velocity="1.0" lower="0" upper="1.57" />
-			<dynamics damping="0.08" friction="0.0" />
 		</joint>
 		<link name="${side}_${name}_link">
@@ -16,5 +13,5 @@
 					<geometry>
 					<mesh
-						filename="package://softhands_description/meshes/softhands/wide/${side}/phalanx_medium_thumb.stl"
+						filename="package://softhands_description/meshes/softhands/wide/${side}/phalanx.stl"
 						scale="0.001 0.001 0.001" />
 					</geometry>
@@ -31,5 +28,5 @@
 					<geometry>
 					<mesh
-						filename="package://softhands_description/meshes/softhands/wide/${side}/phalanx_medium_thumb.stl"
+						filename="package://softhands_description/meshes/softhands/wide/${side}/phalanx.stl"
 						scale="0.001 0.001 0.001" />
 					</geometry>
@@ -37,19 +34,19 @@
 				</collision>
 		</link>
-		<!-- thumb middle to mobile thumb middle   -->
-		<joint name="${side}_${name}_to_mobile_joint" type="revolute">
+		<!-- Finger prox/mid virtual  -->
+		<joint name="${side}_${parent}_${name}_virtual_joint" type="revolute">
 			<axis xyz="0 0 1"/>
 			<limit effort="0.0" lower="0" upper="0"  velocity="0.0"/>
 			<origin xyz="41e-3 0 0" rpy="0 0 0"/>
 			<parent link="${side}_${name}_link"/>
-			<child link="${side}_${name}_to_mobile_link"/>
+			<child link="${side}_${name}_virtual_link"/>
 		</joint>
-	    <link name="${side}_${name}_to_mobile_link">
+		<link name="${side}_${name}_virtual_link">
 		   <inertial>
-			<origin xyz="0 0 0" rpy="0 0 0"/>
-			<mass value="1e-6"/>
-			<inertia ixx="1e-6"  ixy="0"  	  	ixz="0"
-								 iyy="1e-6" 	iyz="0"
-												izz="1e-6" />
+				<origin xyz="0 0 0" rpy="0 0 0"/>
+				<mass value="1e-6"/>
+				<inertia ixx="1e-6"  ixy="0"  	  	ixz="0"
+									iyy="1e-6" 	iyz="0"
+													izz="1e-6" />
 		   </inertial>
 	    </link>

File: softhands_description/urdf/xacro/include/macro/v1.0_wide/modules/finger/phalanx_prox_sup.xacro (robot description, xacro)
@@ -34,5 +34,5 @@
 				</collision>
 		</link>
-		<!-- Finger support to mobile  -->
+		<!-- Finger support Virtual  -->
 		<joint name="${side}_${name}_virtual_joint" type="revolute">
 			<axis xyz="0 0 1"/>

File: softhands_description/urdf/xacro/include/macro/v1.0_wide/modules/palm/palm_central.xacro (robot description, xacro)
@@ -37,13 +37,13 @@
 				</collision>
 		</link>
-		<!-- palm base to mobile thumb -->
-		<joint name="${side}_${name}_to_mobile_thumb_joint" type="revolute">
+		<!-- palm base virtual -->
+		<joint name="${side}_${name}_thumb_virtual_joint" type="revolute">
 			<axis xyz="0 0 1"/>
 			<limit effort="0.0" lower="0" upper="0"  velocity="0.0"/>
 			<origin xyz=" -0.0000000021 32.5059e-3 39.6398e-3" rpy="0 0.3490656 1.5707963"/>
 			<parent link="${side}_${name}_link"/>
-			<child link="${side}_${name}_to_mobile_thumb_link"/>
+			<child link="${side}_${name}_thumb_virtual_link"/>
 		</joint>
-	    <link name="${side}_${name}_to_mobile_thumb_link">
+	    <link name="${side}_${name}_thumb_virtual_link">
 		   <inertial>
 			<origin xyz="0 0 0" rpy="0 0 0"/>
@@ -54,13 +54,13 @@
 		   </inertial>
 	    </link>
-		<!-- palm base to mobile little -->
-		<joint name="${side}_${name}_to_mobile_little_joint" type="revolute">
+		<!-- palm base virtual -->
+		<joint name="${side}_${name}_little_virtual_joint" type="revolute">
 			<axis xyz="0 0 1"/>
 			<limit effort="0.0" lower="0" upper="0"  velocity="0.0"/>
 			<origin xyz=" -0.0000000091 -10.6603e-3 66.1817e-3" rpy="0 -0.1745327 -1.5707963"/>
 			<parent link="${side}_${name}_link"/>
-			<child link="${side}_${name}_to_mobile_little_link"/>
+			<child link="${side}_${name}_little_virtual_link"/>
 		</joint>
-		<link name="${side}_${name}_to_mobile_little_link">
+		<link name="${side}_${name}_little_virtual_link">
 		   <inertial>
 				<origin xyz="0 0 0" rpy="0 0 0"/>

File: softhands_description/urdf/xacro/include/macro/v1.0_wide/modules/thumb.xacro (robot description, xacro)
@@ -7,9 +7,9 @@
       </xacro:thumb_prox>
       <!-- Middle -->
-      <xacro:thumb_mid name="thumb_mid" parent="thumb_prox_to_mobile" side="$(arg side)">
+      <xacro:thumb_mid name="thumb_mid" parent="thumb_prox_virtual" side="$(arg side)">
         <origin rpy="0 0 0" xyz="9e-3 0 0"/>
       </xacro:thumb_mid>
       <!-- Distal -->
-      <xacro:thumb_dist name="thumb_dist" parent="thumb_mid_to_mobile" side="$(arg side)">
+      <xacro:thumb_dist name="thumb_dist" parent="thumb_mid_virtual" side="$(arg side)">
         <origin rpy="0 0.0101229 0" xyz="8.99947e-3 0 -0.0973875e-3"/>
       </xacro:thumb_dist>

File: softhands_description/urdf/xacro/include/macro/v1.0_wide/modules/thumb/thumb_mid.xacro (robot description, xacro)
@@ -1,6 +1,6 @@
 <?xml version="1.0"?>
 <robot xmlns:xacro="http://www.ros.org/wiki/xacro">
-    <xacro:macro name="thumb_prox" params="name parent side *origin">
-		<!-- Thumb Proximal  -->
+    <xacro:macro name="thumb_mid" params="name parent side *origin">
+		<!-- Thumb middle  -->
 		<joint name="${side}_${name}_joint" type="revolute">
 			<parent link="${side}_${parent}_link"/>
@@ -16,5 +16,5 @@
 					<geometry>
 					<mesh
-						filename="package://softhands_description/meshes/softhands/wide/${side}/phalanx_pros_thumb.stl"
+						filename="package://softhands_description/meshes/softhands/wide/${side}/phalanx_medium_thumb.stl"
 						scale="0.001 0.001 0.001" />
 					</geometry>
@@ -31,5 +31,5 @@
 					<geometry>
 					<mesh
-						filename="package://softhands_description/meshes/softhands/wide/${side}/phalanx_pros_thumb.stl"
+						filename="package://softhands_description/meshes/softhands/wide/${side}/phalanx_medium_thumb.stl"
 						scale="0.001 0.001 0.001" />
 					</geometry>
@@ -37,13 +37,13 @@
 				</collision>
 		</link>
-		<!-- thumb proximal to mobile thumb proximal   -->
-		<joint name="${side}_${name}_to_mobile_joint" type="revolute">
+		<!-- thumb middle virtual thumb middle   -->
+		<joint name="${side}_${name}_virtual_joint" type="revolute">
 			<axis xyz="0 0 1"/>
 			<limit effort="0.0" lower="0" upper="0"  velocity="0.0"/>
-			<origin xyz=" 31.2357e-3 23.0197e-3 0.167417e-3" rpy=" 0.1745395 0.0000165 0.7597087"/>
+			<origin xyz="41e-3 0 0" rpy="0 0 0"/>
 			<parent link="${side}_${name}_link"/>
-			<child link="${side}_${name}_to_mobile_link"/>
+			<child link="${side}_${name}_virtual_link"/>
 		</joint>
-	    <link name="${side}_${name}_to_mobile_link">
+	    <link name="${side}_${name}_virtual_link">
 		   <inertial>
 			<origin xyz="0 0 0" rpy="0 0 0"/>
@@ -54,9 +54,4 @@
 		   </inertial>
 	    </link>
-		<!--
-		<gazebo reference="base_link">
-			<material>Gazebo/SkyBlue</material>
-			<selfCollide>true</selfCollide>
-		</gazebo> -->
     </xacro:macro>
 </robot>

File: softhands_description/urdf/xacro/include/macro/v2.0_qb/header.xacro (robot description, xacro)
@@ -31,5 +31,5 @@
  * OF THIS SOFTWARE, EVEN IF ADVISED OF THE POSSIBILITY OF SUCH DAMAGE.
  *
- * \file      sh_v1_simple.xacro
+ *
  *
  * \author       _Centro di Ricerca "E.Piaggio"_
@@ -37,50 +37,17 @@
  *
 -->
-<robot name="palm_v3" xmlns:xacro="http://www.ros.org/wiki/xacro">
-	<xacro:macro name="palm" params="sign ns parent position orientation operation_mode">
-	  	<joint name="${ns}_palm_joint" type="fixed">
-			<origin rpy="${orientation}" xyz="${position}"/>
-			<parent link="${ns}_palm_base_link" />
-			<child link="${ns}_palm_link" />
-		</joint>
-		<link name="${ns}_palm_link">
-			<inertial>
-			<mass value="0.45"/>
-			<origin rpy="0 0 0" xyz="0.0030 -0.0449 0.0135"/>
-			<inertia ixx="0.00045" ixy="0.0" ixz="0.0" iyy="0.0006" iyz="0.0" izz="0.00025"/>
-			</inertial>
-			<visual>
-			<origin rpy="0 0 0" xyz="0 0 0"/>
-			<geometry>
-				<mesh filename="package://softhands_description/meshes/softhands/v3.0/palm_pinch_r.stl" scale="0.001 0.001 0.001"/>
-			</geometry>
-			<material name="qbhand/palm"/>
-			</visual>
-			<collision>
-			<origin rpy="0 0 0" xyz="0 0 0"/>
-			<geometry>
-				<mesh filename="package://softhands_description/meshes/softhands/v3.0/palm_pinch_r.stl" scale="0.001 0.001 0.001"/>
-			</geometry>
-			</collision>
-		</link>
-		<joint name="${ns}_synergy_joint" type="revolute">
-			<origin rpy="0 0 0" xyz="0 0 0"/>
-			<parent link="${ns}_palm_link"/>
-			<child link="${ns}_synergy_tendon_virtual_link"/>
-			<axis xyz="0 0 1"/>
-			<dynamics damping="0.0" friction="0.0"/>
-			<limit effort="100" lower="0.0" upper="1.0" velocity="100"/>
-		</joint>
-		<link name="${ns}_synergy_tendon_virtual_link">
-			<inertial>
-			<origin rpy="0 0 0" xyz="0 0 0"/>
-			<mass value="1e-4"/>
-			<inertia ixx="1e-9" ixy="0.0" ixz="0.0" iyy="1e-9" iyz="0.0" izz="1e-9"/>
-			</inertial>
-		</link>
-	<gazebo reference="${ns}_palm_link">
-		<material>Gazebo/Grey</material>
-		<selfCollide>true</selfCollide>
-	</gazebo>
-	</xacro:macro>
+<robot xmlns:xacro="http://www.ros.org/wiki/xacro" name="header">
+  <!-- Include xacro macro  Palm-->
+	<xacro:include filename="$(arg root_dir)/modules/palm/palm.xacro" />
+	<xacro:include filename="$(arg root_dir)/modules/iso.xacro" />
+  <!-- Include xacro macro Thumb -->
+  <xacro:include filename="$(arg root_dir)/modules/thumb.xacro" />
+  <xacro:include filename="$(arg root_dir)/modules/thumb/thumb_prox.xacro" />
+  <!-- Include xacro macro Finger -->
+  <xacro:include filename="$(arg root_dir)/modules/finger/phalanx_prox.xacro" />
+  <xacro:include filename="$(arg root_dir)/modules/finger/phalanx.xacro" />
+  <xacro:include filename="$(arg root_dir)/modules/finger/phalanx_dist.xacro" />
+  <xacro:include filename="$(arg root_dir)/modules/finger.xacro" />
+  <!-- Color definitions -->
+  <xacro:include filename="$(arg root_dir)/color.xacro" />
 </robot>

File: softhands_description/urdf/xacro/include/macro/v2.0_qb/modules/finger/phalanx.xacro (robot description, xacro)
@@ -38,5 +38,5 @@
 -->
 <robot xmlns:xacro="http://www.ros.org/wiki/xacro">
-  <xacro:macro name="fingertip" params="type ns parent name position orientation">
+  <xacro:macro name="phalanx" params="type ns parent name position orientation">
     <joint name="${ns}_${type}_${parent}_${name}_joint" type="revolute">
       <origin rpy="${orientation}" xyz="${position}"/>
@@ -48,45 +48,44 @@
       <mimic joint="${ns}_synergy_joint" multiplier="0.785"/>
     </joint>
-  <!-- <link name="${ns}_${parent}_${name}_virtual_link">
-    <inertial>
-      <origin rpy="0 0 0" xyz="0 0 0"/>
-      <mass value="1e-4"/>
-      <inertia ixx="1e-9" ixy="0.0" ixz="0.0" iyy="1e-9" iyz="0.0" izz="1e-9"/>
-    </inertial>
-  </link> -->
-<!--
-  <joint name="${ns}_${parent}_${name}_virtual_joint" type="revolute">
-    <origin rpy="0 0 0" xyz="0.013 0 0"/>
-    <parent link="${ns}_${parent}_${name}_virtual_link"/>
-    <child link="${ns}_${parent}_${name}_link"/>
-    <axis xyz="0 0 -1"/>
-    <dynamics damping="0.0" friction="0.0"/>
-    <limit effort="100" lower="0.0" upper="0.785" velocity="100"/>
-    <mimic joint="${ns}_${parent}_${name}_joint" multiplier="1.0"/>
-  </joint>
-  <link name="${ns}_${parent}_${name}_link">
-    <inertial>
-      <mass value="0.009"/>
-      <origin rpy="0 0 0" xyz="8.8025467e-03 -1.7219289e-03 0.0"/>
-      <inertia ixx="2.6586142e-07" ixy="1.2416847e-08" ixz="0.0" iyy="5.9935767e-07" iyz="0.0" izz="6.6781963e-07"/>
-    </inertial>
-    <visual>
-      <origin rpy="0 0 0" xyz="0 0 0"/>
-      <geometry>
-        <mesh filename="package://softhands_description/meshes/softhands/v3.0/ph_distal.stl" scale="0.001 0.001 0.001"/>
-      </geometry>
-      <material name="qbhand/distal"/>
-    </visual>
-    <collision>
-      <origin rpy="0 0 0" xyz="0 0 0"/>
-      <geometry>
-        <mesh filename="package://softhands_description/meshes/softhands/v3.0/ph_distal_collision.stl" scale="0.001 0.001 0.001"/>
-      </geometry>
-    </collision>
-  </link>
-  <gazebo reference="${ns}_${parent}_${name}_link">
-    <material>Gazebo/Grey</material>
-    <self_collide>false</self_collide>
-  </gazebo> -->
+    <link name="${ns}_${type}_${parent}_${name}_virtual_link">
+      <inertial>
+        <origin rpy="0 0 0" xyz="0 0 0"/>
+        <mass value="1e-4"/>
+        <inertia ixx="1e-9" ixy="0.0" ixz="0.0" iyy="1e-9" iyz="0.0" izz="1e-9"/>
+      </inertial>
+    </link>
+    <!-- Virtual -->
+    <joint name="${ns}_${type}_${parent}_${name}_virtual_joint" type="revolute">
+      <origin rpy="0 0 0" xyz="0.013 0 0"/>
+      <parent link="${ns}_${type}_${parent}_${name}_virtual_link"/>
+      <child link="${ns}_${type}_${name}_link"/>
+      <axis xyz="0 0 -1"/>
+      <dynamics damping="0.0" friction="0.0"/>
+      <limit effort="30" velocity="1.0" lower="-1.57" upper="1.57" />
+      <mimic joint="${ns}_${type}_${parent}_${name}_joint" multiplier="1.0"/>
+    </joint>
+    <link name="${ns}_${type}_${name}_link">
+      <inertial>
+        <mass value="0.0063"/>
+        <origin rpy="0 0 0" xyz="4.7601567e-03 -1.3786947e-03 0.0"/>
+        <inertia ixx="1.8024201e-07" ixy="5.756798e-09" ixz="0.0" iyy="2.3516266e-07" iyz="0.0" izz="2.691504e-07"/>
+      </inertial>
+      <visual>
+        <origin rpy="0 0 0" xyz="0 0 0"/>
+        <geometry>
+          <mesh filename="package://softhands_description/meshes/softhands/v2.0_qb/ph_short.stl" scale="0.001 0.001 0.001"/>
+        </geometry>
+      </visual>
+      <collision>
+        <origin rpy="0 0 0" xyz="0 0 0"/>
+        <geometry>
+          <mesh filename="package://softhands_description/meshes/softhands/v2.0_qb/ph_short_collision.stl" scale="0.001 0.001 0.001"/>
+        </geometry>
+      </collision>
+    </link>
+    <gazebo reference="${ns}_${type}_${name}_link">
+      <material>Gazebo/Grey</material>
+      <self_collide>false</self_collide>
+    </gazebo>
   </xacro:macro>
 </robot>
