Commit message: small update

File: softhands_description/urdf/xacro/include/macro/v2.0_qb/modules/finger/phalanx_dist.xacro (robot description, xacro)
@@ -38,15 +38,15 @@
 -->
 <robot xmlns:xacro="http://www.ros.org/wiki/xacro">
-  <xacro:macro name="phalanx" params="type ns parent name position orientation">
-  <joint name="${ns}_${type}_${parent}_${name}_joint" type="revolute">
-    <origin rpy="${orientation}" xyz="${position}"/>
-    <parent link="${ns}_${type}_${parent}_link"/>
-    <child link="${ns}_${type}_${parent}_${name}_virtual_link"/>
-    <axis xyz="0 0 -1"/>
-    <dynamics damping="0.0" friction="0.0"/>
-    <limit effort="30" velocity="1.0" lower="-1.57" upper="1.57" />
-    <mimic joint="${ns}_synergy_joint" multiplier="0.785"/>
-  </joint>
-  <link name="${ns}_${type}_${parent}_${name}_virtual_link">
+  <xacro:macro name="fingertip" params="type ns parent name position orientation">
+    <joint name="${ns}_${type}_${parent}_${name}_joint" type="revolute">
+      <origin rpy="${orientation}" xyz="${position}"/>
+      <parent link="${ns}_${type}_${parent}_link"/>
+      <child link="${ns}_${type}_${parent}_${name}_virtual_link"/>
+      <axis xyz="0 0 -1"/>
+      <dynamics damping="0.0" friction="0.0"/>
+      <limit effort="30" velocity="1.0" lower="-1.57" upper="1.57" />
+      <mimic joint="${ns}_synergy_joint" multiplier="0.785"/>
+    </joint>
+  <!-- <link name="${ns}_${parent}_${name}_virtual_link">
     <inertial>
       <origin rpy="0 0 0" xyz="0 0 0"/>
@@ -54,37 +54,39 @@
       <inertia ixx="1e-9" ixy="0.0" ixz="0.0" iyy="1e-9" iyz="0.0" izz="1e-9"/>
     </inertial>
-  </link>
-  <joint name="${ns}_${type}_${parent}_${name}_virtual_joint" type="revolute">
+  </link> -->
+<!--
+  <joint name="${ns}_${parent}_${name}_virtual_joint" type="revolute">
     <origin rpy="0 0 0" xyz="0.013 0 0"/>
-    <parent link="${ns}_${type}_${parent}_${name}_virtual_link"/>
-    <child link="${ns}_${type}_${name}_link"/>
+    <parent link="${ns}_${parent}_${name}_virtual_link"/>
+    <child link="${ns}_${parent}_${name}_link"/>
     <axis xyz="0 0 -1"/>
     <dynamics damping="0.0" friction="0.0"/>
-    <limit effort="30" velocity="1.0" lower="-1.57" upper="1.57" />
-    <mimic joint="${ns}_${type}_${parent}_${name}_joint" multiplier="1.0"/>
+    <limit effort="100" lower="0.0" upper="0.785" velocity="100"/>
+    <mimic joint="${ns}_${parent}_${name}_joint" multiplier="1.0"/>
   </joint>
-  <link name="${ns}_${type}_${name}_link">
+  <link name="${ns}_${parent}_${name}_link">
     <inertial>
-      <mass value="0.0063"/>
-      <origin rpy="0 0 0" xyz="4.7601567e-03 -1.3786947e-03 0.0"/>
-      <inertia ixx="1.8024201e-07" ixy="5.756798e-09" ixz="0.0" iyy="2.3516266e-07" iyz="0.0" izz="2.691504e-07"/>
+      <mass value="0.009"/>
+      <origin rpy="0 0 0" xyz="8.8025467e-03 -1.7219289e-03 0.0"/>
+      <inertia ixx="2.6586142e-07" ixy="1.2416847e-08" ixz="0.0" iyy="5.9935767e-07" iyz="0.0" izz="6.6781963e-07"/>
     </inertial>
     <visual>
       <origin rpy="0 0 0" xyz="0 0 0"/>
       <geometry>
-        <mesh filename="package://softhands_description/meshes/softhands/v3.0/ph_short.stl" scale="0.001 0.001 0.001"/>
+        <mesh filename="package://softhands_description/meshes/softhands/v2.0_qb/ph_distal.stl" scale="0.001 0.001 0.001"/>
       </geometry>
+      <material name="qbhand/distal"/>
     </visual>
     <collision>
       <origin rpy="0 0 0" xyz="0 0 0"/>
       <geometry>
-        <mesh filename="package://softhands_description/meshes/softhands/v3.0/ph_short_collision.stl" scale="0.001 0.001 0.001"/>
+        <mesh filename="package://softhands_description/meshes/softhands/v2.0_qb/ph_distal_collision.stl" scale="0.001 0.001 0.001"/>
       </geometry>
     </collision>
   </link>
-  <gazebo reference="${ns}_${type}_${name}_link">
+  <gazebo reference="${ns}_${parent}_${name}_link">
     <material>Gazebo/Grey</material>
     <self_collide>false</self_collide>
-  </gazebo>
+  </gazebo> -->
   </xacro:macro>
 </robot>

File: softhands_description/urdf/xacro/include/macro/v2.0_qb/modules/iso.xacro (robot description, xacro)
@@ -31,5 +31,5 @@
  * OF THIS SOFTWARE, EVEN IF ADVISED OF THE POSSIBILITY OF SUCH DAMAGE.
  *
- *
+ * \file      sh_v1_simple.xacro
  *
  * \author       _Centro di Ricerca "E.Piaggio"_
@@ -37,13 +37,39 @@
  *
 -->
-<robot xmlns:xacro="http://www.ros.org/wiki/xacro" name="header">
-  <!-- Include xacro macro -->
-	<xacro:include filename="$(arg root_dir)/finger.xacro" />
-	<xacro:include filename="$(arg root_dir)/thumb.xacro" />
-	<xacro:include filename="$(arg root_dir)/base.xacro" />
-	<xacro:include filename="$(arg root_dir)/palm.xacro" />
-	<xacro:include filename="$(arg root_dir)/phalanges/knuckle.xacro" />
-	<xacro:include filename="$(arg root_dir)/phalanges/thumb_knuckle.xacro" />
-	<xacro:include filename="$(arg root_dir)/phalanges/fingertip.xacro" />
-	<xacro:include filename="$(arg root_dir)/phalanges/phalanx.xacro" />
+<robot name="iso_v2" xmlns:xacro="http://www.ros.org/wiki/xacro">
+	<xacro:macro name="iso" params="ns name parent *origin side">
+		<!-- World -->
+		<link name="${parent}">
+		</link>
+		<!-- World to palm base -->
+		<joint name="${ns}_${name}_joint" type="fixed">
+			<parent link="${parent}"/>
+			<child link="${ns}_${name}_link"/>
+			<xacro:insert_block name="origin"/>
+		</joint>
+		<link name="${ns}_${name}_link">
+			<inertial>
+				<mass value="0.45"/>
+				<origin rpy="0 0 0" xyz="0.0030 -0.0449 0.0135"/>
+				<inertia ixx="0.00045" ixy="0.0" ixz="0.0" iyy="0.0006" iyz="0.0" izz="0.00025"/>
+			</inertial>
+			<visual>
+				<origin rpy="0 0 0" xyz="0 0 0"/>
+				<geometry>
+					<mesh filename="$(arg meshes_dir)/flange_iso_04.stl" scale="0.001 0.001 0.001"/>
+				</geometry>
+				<material name="qbhand/base"/>
+			</visual>
+			<collision>
+			<origin rpy="0 0 0" xyz="0 0 0"/>
+			<geometry>
+				<mesh filename="$(arg meshes_dir)/flange_iso_04.stl" scale="0.001 0.001 0.001"/>
+			</geometry>
+			</collision>
+		</link>
+		<gazebo reference="${ns}_${name}_link">
+    	  	<material>Gazebo/Grey</material>
+			<selfCollide>true</selfCollide>
+	  	</gazebo>
+	</xacro:macro>
 </robot>

File: softhands_description/urdf/xacro/include/macro/v2.0_qb/modules/palm/palm.xacro (robot description, xacro)
@@ -37,43 +37,35 @@
  *
 -->
-<robot name="v3" xmlns:xacro="http://www.ros.org/wiki/xacro">
-	<xacro:property name="side_" value="$(arg side)"/>
-    <xacro:if value="${side_ == 'right'}">
-		<xacro:arg name="sign" default="1"/>
-	</xacro:if>
-    <xacro:if value="${side_ == 'left'}">
-		<xacro:arg name="sign" default="-1"/>
-    </xacro:if>
-	<!-- type: right/left -->
-	<!-- parent: root_link/world -->
-	<xacro:base
-		sign="$(arg sign)"
-		ns="$(arg ns)"
-		parent = "$(arg parent)"
-		position ="$(arg position)"
-		orientation ="$(arg orientation)"
-		operation_mode = "$(arg operation_mode)">
-	</xacro:base>
-	<xacro:palm
-		sign="$(arg sign)"
-		ns="$(arg ns)"
-		parent = "$(arg parent)"
-		position ="-0.0045 0.0145 0.144"
-		orientation ="1.57 0 0"
-		operation_mode = "$(arg operation_mode)">
-	</xacro:palm>
-	<!-- # Thumb finger -->
-	<xacro:thumb
-		type="thumb"
-		sign="$(arg sign)"
-		ns="$(arg ns)"
-		position="-0.044 -0.0465 -0.002"
-		orientation="-1.57 3.14 0.0">
-	</xacro:thumb>
-	<!-- <gazebo>
-		<plugin name="synergy_plugin" filename="libsofthand_plugin.so">
-			<namespace>$(arg type)_hand_v3s</namespace>
-			<operation_mode>$(arg operation_mode)</operation_mode>
-		</plugin>
-	</gazebo> -->
+<robot name="palm_v2" xmlns:xacro="http://www.ros.org/wiki/xacro">
+	<xacro:macro name="palm" params="ns name parent *origin side">
+	  	<joint name="${ns}_palm_joint" type="fixed">
+			<xacro:insert_block name="origin"/>
+			<parent link="${ns}_${parent}_link" />
+			<child link="${ns}_palm_link" />
+		</joint>
+		<link name="${ns}_palm_link">
+			<inertial>
+			<mass value="0.45"/>
+			<origin rpy="0 0 0" xyz="0.0030 -0.0449 0.0135"/>
+			<inertia ixx="0.00045" ixy="0.0" ixz="0.0" iyy="0.0006" iyz="0.0" izz="0.00025"/>
+			</inertial>
+			<visual>
+			<origin rpy="0 0 0" xyz="0 0 0"/>
+			<geometry>
+				<mesh filename="$(arg meshes_dir)/palm_pinch_r.stl" scale="0.001 0.001 0.001"/>
+			</geometry>
+			<material name="qbhand/palm"/>
+			</visual>
+			<collision>
+			<origin rpy="0 0 0" xyz="0 0 0"/>
+			<geometry>
+				<mesh filename="$(arg meshes_dir)/palm_pinch_r.stl" scale="0.001 0.001 0.001"/>
+			</geometry>
+			</collision>
+		</link>
+	<gazebo reference="${ns}_palm_link">
+		<material>Gazebo/Grey</material>
+		<selfCollide>true</selfCollide>
+	</gazebo>
+	</xacro:macro>
 </robot>

File: softhands_description/urdf/xacro/include/macro/v2.0_qb/modules/thumb.xacro (robot description, xacro)
@@ -31,5 +31,5 @@
  * OF THIS SOFTWARE, EVEN IF ADVISED OF THE POSSIBILITY OF SUCH DAMAGE.
  *
- * \file      finger.xacro
+ * \file      thumb.xacro
  *
  * \author       _Centro di Ricerca "E.Piaggio"_
@@ -38,39 +38,23 @@
 -->
 <robot xmlns:xacro="http://www.ros.org/wiki/xacro">
-  <xacro:macro name="thumb_knuckle" params="type ns position orientation">
-    <!-- KNUCKLE -->
-    <joint name="${ns}_${type}_knuckle_joint" type="revolute">
-      <origin xyz="${position}" rpy="${orientation}"/>
-      <parent link="${ns}_palm_link"/>
-      <child link="${ns}_${type}_knuckle_link"/>
-      <axis xyz="0 0 -1"/>
-      <dynamics damping="0.0" friction="0.0"/>
-      <limit effort="100" lower="0.0" upper="1.571" velocity="100"/>
-      <mimic joint="${ns}_synergy_joint" multiplier="2.542"/>
-    </joint>
-    <link name="${ns}_${type}_knuckle_link">
-      <inertial>
-        <mass value="0.01"/>
-        <origin rpy="0 0 0" xyz="1.3071561e-02 -2.7357764e-03 6.4347823e-04"/>
-        <inertia ixx="3.5865978e-07" ixy="2.0944224e-07" ixz="-6.8657569e-08" iyy="1.3885564e-06" iyz="3.2170608e-08" izz="1.3571203e-06"/>
-      </inertial>
-      <visual>
-        <origin rpy="0 0 0" xyz="0 0 0"/>
-        <geometry>
-          <mesh filename="package://softhands_description/meshes/softhands/v3.0/ph_thumb_r.stl" scale="0.001 0.001 0.001"/>
-        </geometry>
-        <material name="qbhand/knuckle"/>
-      </visual>
-      <collision>
-        <origin rpy="0 0 0" xyz="0 0 0"/>
-        <geometry>
-          <mesh filename="package://softhands_description/meshes/softhands/v3.0/ph_thumb_r_collision.stl" scale="0.001 0.001 0.001"/>
-        </geometry>
-      </collision>
-    </link>
-    <gazebo reference="${ns}_${type}_knuckle_link">
-      <material>Gazebo/Grey</material>
-      <selfCollide>false</selfCollide>
-	  </gazebo>
+  <xacro:macro name="thumb" params="ns name parent *origin side">
+    <!-- Proximal -->
+    <xacro:thumb_prox name="thumb_prox" parent="${parent}" ns="$(arg ns)" side="$(arg side)">
+      <origin rpy="-1.57 3.14 0.0" xyz="-0.044 -0.0465 -0.002"/>
+    </xacro:thumb_prox>
+    <!-- Middle  -->
+    <!-- <xacro:phalanx name="thumb_mid" parent="${parent}" ns="$(arg ns)" side="$(arg side)">
+      <origin rpy="-1.57 3.14 0.0" xyz="-0.044 -0.0465 -0.002"/>
+    </xacro:phalanx> -->
+    <!-- DISTAL PHALANGE -->
+    <!-- <xacro:fingertip
+      type="${type}"
+      parent="proximal"
+      name="distal"
+      ns="${ns}"
+      position="0.009 0 0"
+      orientation="0 0 0">
+    </xacro:fingertip>
+    -->
   </xacro:macro>
 </robot>

File: softhands_description/urdf/xacro/v1.0_simple.xacro (robot description, xacro)
@@ -37,5 +37,5 @@
  *
 -->
-<robot name="v1_simple" xmlns:xacro="http://www.ros.org/wiki/xacro">
+<robot name="v1.0_simple" xmlns:xacro="http://www.ros.org/wiki/xacro">
 	<xacro:property name="side" value="$(arg type)"/>
     <xacro:if value="${side == 'right'}">

File: softhands_description/urdf/xacro/v2.0_qb.xacro (robot description, xacro)
@@ -37,43 +37,16 @@
  *
 -->
-<robot name="sh_wide" xmlns:xacro="http://www.ros.org/wiki/xacro">
-	<!-- <xacro:property name="side_" value="$(arg side)"/>
-    <xacro:if value="${side_ == 'right'}">
-		<xacro:arg name="sign" default="1"/>
-	</xacro:if>
-    <xacro:if value="${side_ == 'left'}">
-		<xacro:arg name="sign" default="-1"/>
-    </xacro:if> -->
-	<!-- # palm central -->
-	<xacro:palm_central name="palm_central" parent="$(arg root_link)" side="$(arg side)">
+<robot name="v2.0_qb" xmlns:xacro="http://www.ros.org/wiki/xacro">
+	<!-- # iso -->
+	<xacro:iso name="iso" parent="$(arg root_link)" ns="$(arg ns)" side="$(arg side)">
 		<origin rpy="$(arg orientation)" xyz="$(arg position)"/>
-	</xacro:palm_central>
-	<!-- # palm thumb -->
-	<xacro:palm_thumb name="palm_thumb" parent="palm_central_to_mobile_thumb" side="$(arg side)">
-		<origin rpy="0 0 0 " xyz="12e-3 -0.0000414746e-3 0"/>
-	</xacro:palm_thumb>
-	<!-- # palm little -->
-	<xacro:palm_little name="palm_little" parent="palm_central_to_mobile_little" side="$(arg side)">
-		<origin rpy="0 0 0 " xyz="12e-3 -0.0000466576e-3 0"/>
-	</xacro:palm_little>
+	</xacro:iso>
+	<!-- # palm  -->
+	<xacro:palm name="palm" parent="iso" ns="$(arg ns)" side="$(arg side)">
+		<origin rpy="1.57 0 0" xyz="-0.0045 0.0145 0.144"/>
+	</xacro:palm>
 	<!-- # thumb -->
-	<xacro:thumb name="thumb" parent="palm_thumb_support" side="$(arg side)">
-		<origin rpy="1.5707963 0.7598972 0" xyz="21.9577e-3 0 -2.8e-3"/>
+	<xacro:thumb name="thumb" parent="palm" ns="$(arg ns)" side="$(arg side)">
+		<origin rpy="-1.57 3.14 0.0" xyz="-0.044 -0.0465 -0.002"/>
 	</xacro:thumb>
-	<!-- # Index -->
-	<xacro:finger name="index" parent="palm_central" side="$(arg side)">
-		<origin xyz="5e-3 44.8953e-3 112.230e-3" rpy="1.5707963 -1.3962636 1.5707963"/>
-	</xacro:finger>
-	<!-- # Middle -->
-	<xacro:finger name="middle" parent="palm_central" side="$(arg side)">
-		<origin xyz="5e-3 12.5e-3 115e-3" rpy="0 -1.5707963 -3.1415927"/>
-	</xacro:finger>
-	<!-- # Ring -->
-	<xacro:finger name="ring" parent="palm_little" side="$(arg side)">
-	    <origin xyz=" 8.6355e-3 5e-3 44.4863e-3" rpy="-1.5707963 -1.3089971 0"/>
-	</xacro:finger>
-    <!-- # Little -->
-	<xacro:finger name="little" parent="palm_little" side="$(arg side)">
-		<origin xyz="39.2985e-3 5e-3 34.8419e-3" rpy="-1.5707963 -1.221731 0"/>
-	</xacro:finger>
 </robot>
