Commit message: added collision meshes for wide hand

File: softhands_description/urdf/xacro/include/macro/v1_wide/modules/finger/phalanx.xacro (robot description, xacro)
@@ -45,5 +45,5 @@
 					<geometry>
 					<mesh
-						filename="$(arg meshes_dir)/phalanx.stl"
+						filename="$(arg meshes_dir)/phalanx_collision.stl"
 						scale="0.001 0.001 0.001" />
 					</geometry>
@@ -53,15 +53,5 @@
 		<gazebo reference="${ns}_${name}_link">
 			<material>Gazebo/Gray</material>
-			<selfCollide>$(arg selfCollide)</selfCollide>
-			<kp value="1e4" />
-			<kd value="1e2" />
-			<surface>
-			<friction>
-				<ode>
-				<mu>0.133</mu>
-				<mu2>0.133</mu2>
-				</ode>
-			</friction>
-			</surface>
+			<selfCollide>false</selfCollide>
 		</gazebo>
     </xacro:macro>

File: softhands_description/urdf/xacro/include/macro/v1_wide/modules/finger/phalanx_dist.xacro (robot description, xacro)
@@ -53,15 +53,5 @@
 		<gazebo reference="${ns}_${name}_link">
 			<material>Gazebo/Gray</material>
-			<selfCollide>$(arg selfCollide)</selfCollide>
-			<kp value="1e4" />
-			<kd value="1e2" />
-			<surface>
-			<friction>
-				<ode>
-				<mu>0.133</mu>
-				<mu2>0.133</mu2>
-				</ode>
-			</friction>
-			</surface>
+			<selfCollide>true</selfCollide>
 		</gazebo>
     </xacro:macro>

File: softhands_description/urdf/xacro/include/macro/v1_wide/modules/finger/phalanx_knuckle.xacro (robot description, xacro)
@@ -28,5 +28,5 @@
 					<geometry>
 					<mesh
-						filename="$(arg meshes_dir)/phalanx_pros_sup.stl"
+						filename="$(arg meshes_dir)/phalanx_pros_sup_collision.stl"
 						scale="0.001 0.001 0.001" />
 					</geometry>
@@ -34,18 +34,8 @@
 				</collision>
 		</link>
-	<gazebo reference="${ns}_${name}_link">
+		<gazebo reference="${ns}_${name}_link">
+			<selfCollide>false</selfCollide>
 			<material>Gazebo/White</material>
-			<selfCollide>$(arg selfCollide)</selfCollide>
-			<kp value="1e4" />
-			<kd value="1e2" />
-			<surface>
-			<friction>
-				<ode>
-				<mu>0.133</mu>
-				<mu2>0.133</mu2>
-				</ode>
-			</friction>
-			</surface>
-	</gazebo>
+		</gazebo>
     </xacro:macro>
 </robot>

File: softhands_description/urdf/xacro/include/macro/v1_wide/modules/palm/palm_central.xacro (robot description, xacro)
@@ -31,5 +31,5 @@
 					<geometry>
 					<mesh
-						filename="$(arg meshes_dir)/palm_central.stl"
+						filename="$(arg meshes_dir)/palm_central_collision.stl"
 						scale="0.001 0.001 0.001" />
 					</geometry>
@@ -41,5 +41,5 @@
 			<axis xyz="0 0 -1"/>
 			<limit effort="30" velocity="10" lower="0" upper="1.57" />
-			<dynamics damping="0.0" friction="0.0" />
+			<dynamics damping="$(arg virtual_damping)" friction="$(arg virtual_friction)"/>
 			<origin xyz=" -0.0000000021 32.5059e-3 39.6398e-3" rpy="0 0.3490656 1.5707963"/>
 			<parent link="${ns}_${name}_link"/>
@@ -58,5 +58,5 @@
 		<joint name="${ns}_${name}_little_joint" type="revolute">
 			<axis xyz="0 0 1"/>
-			<dynamics damping="0.0" friction="0.0"/>
+			<dynamics damping="$(arg virtual_damping)" friction="$(arg virtual_friction)"/>
 			<limit effort="100" lower="0.0" upper="0.4" velocity="100"/>
 			<origin xyz=" -0.0000000091 -10.6603e-3 66.1817e-3" rpy="0 -0.1745327 -1.5707963"/>
@@ -76,14 +76,4 @@
 			<selfCollide>false</selfCollide>
 			<material>Gazebo/Grey</material>
-			<kp value="1e4" />
-			<kd value="1e2" />
-			<surface>
-			<friction>
-				<ode>
-				<mu>0.133</mu>
-				<mu2>0.133</mu2>
-				</ode>
-			</friction>
-			</surface>
 		</gazebo>
     </xacro:macro>

File: softhands_description/urdf/xacro/include/macro/v1_wide/modules/palm/palm_little.xacro (robot description, xacro)
@@ -8,5 +8,5 @@
 			<axis xyz="0 0 1" />
       		<limit effort="30" velocity="1.0" lower="0" upper="0.3" />
-			<dynamics damping="0.0" friction="0.0" />
+			<dynamics damping="$(arg virtual_damping)" friction="$(arg virtual_friction)"/>
 		</joint>
 		<link name="${ns}_${name}_link">
@@ -30,5 +30,5 @@
 					<geometry>
 					<mesh
-						filename="$(arg meshes_dir)/palm_little.stl"
+						filename="$(arg meshes_dir)/palm_little_collision.stl"
 						scale="0.001 0.001 0.001" />
 					</geometry>
@@ -37,16 +37,6 @@
 		</link>
 		<gazebo reference="${ns}_${name}_link">
+			<selfCollide>false</selfCollide>
 			<material>Gazebo/Grey</material>
-			<selfCollide>false</selfCollide>
-			<kp value="1e4" />
-			<kd value="1e2" />
-			<surface>
-			<friction>
-				<ode>
-				<mu>0.133</mu>
-				<mu2>0.133</mu2>
-				</ode>
-			</friction>
-			</surface>
 		</gazebo>
     </xacro:macro>

File: softhands_description/urdf/xacro/include/macro/v1_wide/modules/palm/palm_thumb.xacro (robot description, xacro)
@@ -8,5 +8,5 @@
 			<axis xyz="0 0 -1" />
       		<limit effort="30" velocity="1.0" lower="0" upper="1.57" />
-			<dynamics damping="0.0" friction="0.0" />
+			<dynamics damping="$(arg virtual_damping)" friction="$(arg virtual_friction)"/>
 		</joint>
 		<link name="${ns}_${name}_link">
@@ -30,5 +30,5 @@
 					<geometry>
 					<mesh
-						filename="$(arg meshes_dir)/palm_thumb.stl"
+						filename="$(arg meshes_dir)/palm_thumb_collision.stl"
 						scale="0.001 0.001 0.001" />
 					</geometry>
@@ -62,5 +62,5 @@
 					<geometry>
 					<mesh
-						filename="$(arg meshes_dir)/thumb_support.stl"
+						filename="$(arg meshes_dir)/thumb_support_collision.stl"
 						scale="0.001 0.001 0.001" />
 					</geometry>
@@ -69,30 +69,10 @@
 		</link>
 		<gazebo reference="${ns}_${name}_link">
+			<selfCollide>false</selfCollide>
 			<material>Gazebo/Grey</material>
-			<selfCollide>false</selfCollide>
-			<kp value="1e4" />
-			<kd value="1e2" />
-			<surface>
-			<friction>
-				<ode>
-				<mu>0.133</mu>
-				<mu2>0.133</mu2>
-				</ode>
-			</friction>
-			</surface>
 		</gazebo>
 		<gazebo reference="${ns}_${name}_support_link">
-				<material>Gazebo/White</material>
-				<selfCollide>false</selfCollide>
-				<kp value="1e4" />
-				<kd value="1e2" />
-				<surface>
-				<friction>
-					<ode>
-					<mu>0.133</mu>
-					<mu2>0.133</mu2>
-					</ode>
-				</friction>
-				</surface>
+			<selfCollide>false</selfCollide>
+			<material>Gazebo/White</material>
 		</gazebo>
     </xacro:macro>

File: softhands_description/urdf/xacro/include/macro/v1_wide/modules/thumb/thumb_distal.xacro (robot description, xacro)
@@ -45,5 +45,5 @@
 					<geometry>
 					<mesh
-						filename="$(arg meshes_dir)/phalanx_dist_thumb.stl"
+						filename="$(arg meshes_dir)/phalanx_dist_thumb_collision.stl"
 						scale="0.001 0.001 0.001" />
 					</geometry>
@@ -53,15 +53,5 @@
 		<gazebo reference="${ns}_${name}_link">
 			<material>Gazebo/Grey</material>
-			<selfCollide>$(arg selfCollide)</selfCollide>
-			<kp value="1e4" />
-			<kd value="1e2" />
-			<surface>
-			<friction>
-				<ode>
-				<mu>0.133</mu>
-				<mu2>0.133</mu2>
-				</ode>
-			</friction>
-			</surface>
+			<selfCollide>true</selfCollide>
 		</gazebo>
     </xacro:macro>

File: softhands_description/urdf/xacro/include/macro/v1_wide/modules/thumb/thumb_knuckle.xacro (robot description, xacro)
@@ -29,5 +29,5 @@
 					<geometry>
 					<mesh
-						filename="$(arg meshes_dir)/phalanx_pros_thumb.stl"
+						filename="$(arg meshes_dir)/phalanx_pros_thumb_collision.stl"
 						scale="0.001 0.001 0.001" />
 					</geometry>
@@ -37,15 +37,5 @@
 		<gazebo reference="${ns}_${name}_link">
 			<material>Gazebo/Grey</material>
-			<selfCollide>$(arg selfCollide)</selfCollide>
-			<kp value="1e4" />
-			<kd value="1e2" />
-			<surface>
-			<friction>
-				<ode>
-				<mu>0.133</mu>
-				<mu2>0.133</mu2>
-				</ode>
-			</friction>
-			</surface>
+			<selfCollide>true</selfCollide>
 		</gazebo>
     </xacro:macro>

File: softhands_description/urdf/xacro/include/macro/v1_wide/modules/thumb/thumb_proximal.xacro (robot description, xacro)
@@ -45,5 +45,5 @@
 					<geometry>
 					<mesh
-						filename="$(arg meshes_dir)/phalanx_medium_thumb.stl"
+						filename="$(arg meshes_dir)/phalanx_medium_thumb_collision.stl"
 						scale="0.001 0.001 0.001" />
 					</geometry>
@@ -53,15 +53,5 @@
 		<gazebo reference="${ns}_${name}_link">
 			<material>Gazebo/Grey</material>
-			<selfCollide>$(arg selfCollide)</selfCollide>
-			<kp value="1e4" />
-			<kd value="1e2" />
-			<surface>
-			<friction>
-				<ode>
-				<mu>0.133</mu>
-				<mu2>0.133</mu2>
-				</ode>
-			</friction>
-			</surface>
+			<selfCollide>true</selfCollide>
 		</gazebo>
     </xacro:macro>
