Commit message: need to tune damping and friction for both the hands

File: softhands_description/urdf/xacro/include/macro/v1_2_research/modules/finger/phalanx_knuckle.xacro (robot description, xacro)
@@ -31,5 +31,5 @@
  * OF THIS SOFTWARE, EVEN IF ADVISED OF THE POSSIBILITY OF SUCH DAMAGE.
  *
- * \file      sh_v1_simple.xacro
+ * \file      finger.xacro
  *
  * \author       _Centro di Ricerca "E.Piaggio"_
@@ -37,36 +37,51 @@
  *
 -->
-<robot name="v1_wide" xmlns:xacro="http://www.ros.org/wiki/xacro">
-	<!-- # palm central -->
-	<xacro:palm_central name="palm_central" parent="$(arg root_link)" side="$(arg side)" ns="$(arg ns)">
-		<origin rpy="$(arg orientation)" xyz="$(arg position)"/>
-	</xacro:palm_central>
-	<!-- # palm thumb -->
-	<xacro:palm_thumb name="palm_thumb" parent="palm_central_thumb_virtual" side="$(arg side)" ns="$(arg ns)">
-		<origin rpy="0 0 0 " xyz="12e-3 -0.0000414746e-3 0"/>
-	</xacro:palm_thumb>
-	<!-- # palm little -->
-	<xacro:palm_little name="palm_little" parent="palm_central_little_virtual" side="$(arg side)" ns="$(arg ns)">
-		<origin rpy="0 0 0 " xyz="12e-3 -0.0000466576e-3 0"/>
-	</xacro:palm_little>
-	<!-- # thumb -->
-	<xacro:thumb name="thumb" parent="palm_thumb_support" side="$(arg side)" ns="$(arg ns)">
-		<origin rpy="-1.5707963 0 0" xyz="21.9577e-3 0 -2.8e-3"/>
-	</xacro:thumb>
-	<!-- # Index -->
-	<xacro:finger name="index" parent="palm_central" side="$(arg side)" ns="$(arg ns)">
-		<origin  rpy="-3.1415927  -1.396264 1.5707963" xyz="5e-3 44.8953e-3 112.230e-3"/>
-	</xacro:finger>
-	<!-- # Middle -->
-	<xacro:finger name="middle" parent="palm_central" side="$(arg side)" ns="$(arg ns)">
-		<origin  rpy="0 -1.5707963 -1.5707963" xyz="5e-3 12.5e-3 115e-3"/>
-	</xacro:finger>
-	<!-- # Ring -->
-	<xacro:finger name="ring" parent="palm_little" side="$(arg side)" ns="$(arg ns)">
-	    <origin rpy="0 -1.3089971 0" xyz=" 8.6355e-3 5e-3 44.4863e-3" />
-	</xacro:finger>
-    <!-- # Little -->
-	<xacro:finger name="little" parent="palm_little" side="$(arg side)" ns="$(arg ns)">
-		<origin rpy="0 -1.221731 0" xyz="39.2985e-3 5e-3 34.8419e-3" />
-	</xacro:finger>
+<robot xmlns:xacro="http://www.ros.org/wiki/xacro">
+  <xacro:macro name="phalanx_knuckle" params="ns name parent *origin side">
+    <!-- Proximal JOINT -->
+    <joint name="${ns}_${name}_joint" type="revolute">
+      <xacro:insert_block name="origin"/>
+      <parent link="${ns}_${parent}_link"/>
+      <child link="${ns}_${name}_link"/>
+      <axis xyz="0 0 -1"/>
+      <limit effort="30" velocity="1.0" lower="-0.524" upper="0.524" />
+      <dynamics damping="$(arg damping)" friction="$(arg friction)"/>
+    </joint>
+    <!-- LINK -->
+    <link name="${ns}_${name}_link">
+      <inertial>
+        <mass value="0.0095"/>
+        <origin rpy="0 0 0" xyz="4.2753603e-04  0.0 -1.4321738e-03"/>
+        <inertia ixx="6.4337303e-07" ixy="0.0" ixz="-3.9373913e-08" iyy="1.1253771e-06" iyz="0.0" izz="7.2336948e-07"/>
+      </inertial>
+      <visual>
+        <origin rpy="0 0 0" xyz="0 0 0"/>
+        <geometry>
+          <mesh filename="$(arg meshes_dir)/ph_knuckle.stl" scale="0.001 0.001 0.001"/>
+        </geometry>
+        <material name="qbhand/palm"/>
+      </visual>
+      <collision>
+        <origin rpy="0 0 0" xyz="0 0 0"/>
+        <geometry>
+          <mesh filename="$(arg meshes_dir)/ph_knuckle.stl" scale="0.001 0.001 0.001"/>
+        </geometry>
+      </collision>
+    </link>
+        <!-- GAZEBO REF -->
+    <gazebo reference="${ns}_${name}_link">
+      <material>Gazebo/Grey</material>
+      <!-- <selfCollide>false</selfCollide> -->
+      <kp value="1e4" />
+      <kd value="1e2" />
+      <surface>
+       <friction>
+        <ode>
+         <mu>0.133</mu>
+         <mu2>0.133</mu2>
+        </ode>
+       </friction>
+      </surface>
+    </gazebo>
+  </xacro:macro>
 </robot>

File: softhands_description/urdf/xacro/include/macro/v1_2_research/modules/palm/palm.xacro (robot description, xacro)
@@ -31,5 +31,5 @@
  * OF THIS SOFTWARE, EVEN IF ADVISED OF THE POSSIBILITY OF SUCH DAMAGE.
  *
- * \file      test_SHs_v2.urdf.xacro
+ * \file      sh_v1_simple.xacro
  *
  * \author       _Centro di Ricerca "E.Piaggio"_
@@ -37,26 +37,35 @@
  *
 -->
-<robot name="softhand" xmlns:xacro="http://www.ros.org/wiki/xacro">
-  	<!-- <xacro:arg name="sh_version" default="v1_2_research"/> -->
-  	<xacro:arg name="sh_version" default="v1_wide"/>
-  	<xacro:arg name="root_dir" default="$(find softhands_description)/urdf/xacro/include/macro/$(arg sh_version)"/>
-  	<xacro:arg name="root_link" default="world"/>
-  	<xacro:arg name="side" default="right"/>
-  	<xacro:arg name="meshes_dir" default="package://softhands_description/meshes/$(arg sh_version)/$(arg side)"/>
-  	<xacro:arg name="ns" default="$(arg side)_hand_$(arg sh_version)"/>
-  	<xacro:arg name="position" default="0 0 0.01"/>
-  	<xacro:arg name="roll" default="0"/>
-  	<xacro:arg name="pitch" default="0"/>
-  	<xacro:arg name="yaw" default="0"/>
-  	<xacro:arg name="orientation" default="$(arg roll) $(arg pitch) $(arg yaw)"/>
-  	<xacro:arg name="operation_mode" default="0"/>
-	<xacro:include filename="$(arg root_dir)/header.xacro"/>
-  	<xacro:arg name="high_friction" default="0.7"/>
-  	<xacro:arg name="friction" default="1e-3"/>
-  	<xacro:arg name="damping" default="1e-4"/>
-  	<xacro:arg name="virtual_friction" default="0.0"/>
-  	<xacro:arg name="virtual_damping" default="0.0"/>
-	<xacro:include filename="$(find softhands_description)/urdf/xacro/$(arg sh_version).xacro"/>
-	<!-- Include plugin -->
-	<xacro:include filename="$(find softhands_description)/urdf/xacro/include/macro/$(arg sh_version)/plugin.xacro"/>
+<robot name="palm_v2" xmlns:xacro="http://www.ros.org/wiki/xacro">
+	<xacro:macro name="palm" params="ns name parent *origin side">
+	  	<joint name="${ns}_palm_joint" type="fixed">
+			<xacro:insert_block name="origin"/>
+			<parent link="${ns}_${parent}_link" />
+			<child link="${ns}_palm_link" />
+		</joint>
+		<link name="${ns}_palm_link">
+			<inertial>
+				<mass value="0.45"/>
+				<origin rpy="0 0 0" xyz="0.0030 -0.0449 0.0135"/>
+				<inertia ixx="0.00045" ixy="0.0" ixz="0.0" iyy="0.0006" iyz="0.0" izz="0.00025"/>
+			</inertial>
+			<visual>
+			<origin rpy="0 0 0" xyz="0 0 0"/>
+			<geometry>
+				<mesh filename="$(arg meshes_dir)/palm_pinch.stl" scale="0.001 0.001 0.001"/>
+			</geometry>
+			<material name="qbhand/palm"/>
+			</visual>
+			<collision>
+			<origin rpy="0 0 0" xyz="0 0 0"/>
+			<geometry>
+				<mesh filename="$(arg meshes_dir)/palm_pinch.stl" scale="0.001 0.001 0.001"/>
+			</geometry>
+			</collision>
+		</link>
+		<gazebo reference="${ns}_palm_link">
+			<material>Gazebo/Grey</material>
+			<selfCollide>true</selfCollide>
+		</gazebo>
+	</xacro:macro>
 </robot>

File: softhands_description/urdf/xacro/include/macro/v1_2_research/modules/thumb/thumb_knuckle.xacro (robot description, xacro)
@@ -31,5 +31,5 @@
  * OF THIS SOFTWARE, EVEN IF ADVISED OF THE POSSIBILITY OF SUCH DAMAGE.
  *
- * \file      sh_v1_simple.xacro
+ * \file      finger.xacro
  *
  * \author       _Centro di Ricerca "E.Piaggio"_
@@ -37,36 +37,51 @@
  *
 -->
-<robot name="v1_wide" xmlns:xacro="http://www.ros.org/wiki/xacro">
-	<!-- # palm central -->
-	<xacro:palm_central name="palm_central" parent="$(arg root_link)" side="$(arg side)" ns="$(arg ns)">
-		<origin rpy="$(arg orientation)" xyz="$(arg position)"/>
-	</xacro:palm_central>
-	<!-- # palm thumb -->
-	<xacro:palm_thumb name="palm_thumb" parent="palm_central_thumb_virtual" side="$(arg side)" ns="$(arg ns)">
-		<origin rpy="0 0 0 " xyz="12e-3 -0.0000414746e-3 0"/>
-	</xacro:palm_thumb>
-	<!-- # palm little -->
-	<xacro:palm_little name="palm_little" parent="palm_central_little_virtual" side="$(arg side)" ns="$(arg ns)">
-		<origin rpy="0 0 0 " xyz="12e-3 -0.0000466576e-3 0"/>
-	</xacro:palm_little>
-	<!-- # thumb -->
-	<xacro:thumb name="thumb" parent="palm_thumb_support" side="$(arg side)" ns="$(arg ns)">
-		<origin rpy="-1.5707963 0 0" xyz="21.9577e-3 0 -2.8e-3"/>
-	</xacro:thumb>
-	<!-- # Index -->
-	<xacro:finger name="index" parent="palm_central" side="$(arg side)" ns="$(arg ns)">
-		<origin  rpy="-3.1415927  -1.396264 1.5707963" xyz="5e-3 44.8953e-3 112.230e-3"/>
-	</xacro:finger>
-	<!-- # Middle -->
-	<xacro:finger name="middle" parent="palm_central" side="$(arg side)" ns="$(arg ns)">
-		<origin  rpy="0 -1.5707963 -1.5707963" xyz="5e-3 12.5e-3 115e-3"/>
-	</xacro:finger>
-	<!-- # Ring -->
-	<xacro:finger name="ring" parent="palm_little" side="$(arg side)" ns="$(arg ns)">
-	    <origin rpy="0 -1.3089971 0" xyz=" 8.6355e-3 5e-3 44.4863e-3" />
-	</xacro:finger>
-    <!-- # Little -->
-	<xacro:finger name="little" parent="palm_little" side="$(arg side)" ns="$(arg ns)">
-		<origin rpy="0 -1.221731 0" xyz="39.2985e-3 5e-3 34.8419e-3" />
-	</xacro:finger>
+<robot xmlns:xacro="http://www.ros.org/wiki/xacro">
+  <xacro:macro name="thumb_knuckle" params="ns name parent *origin side">
+    <!-- Proximal JOINT -->
+    <joint name="${ns}_${name}_joint" type="revolute">
+      <xacro:insert_block name="origin"/>
+      <parent link="${ns}_${parent}_link"/>
+      <child link="${ns}_${name}_link"/>
+      <axis xyz="0 0 -1"/>
+      <limit effort="30" velocity="1.0" lower="0" upper="1.57" />
+      <dynamics damping="0.08" friction="$(arg friction)" />
+    </joint>
+    <!-- LINK -->
+    <link name="${ns}_${name}_link">
+      <inertial>
+        <mass value="0.01"/>
+        <origin rpy="0 0 0" xyz="1.3071561e-02 -2.7357764e-03 6.4347823e-04"/>
+        <inertia ixx="3.5865978e-07" ixy="2.0944224e-07" ixz="-6.8657569e-08" iyy="1.3885564e-06" iyz="3.2170608e-08" izz="1.3571203e-06"/>
+      </inertial>
+      <visual>
+        <origin rpy="0 0 0" xyz="0 0 0"/>
+        <geometry>
+          <mesh filename="$(arg meshes_dir)/ph_thumb.stl" scale="0.001 0.001 0.001"/>
+        </geometry>
+        <material name="qbhand/knuckle"/>
+      </visual>
+      <collision>
+        <origin rpy="0 0 0" xyz="0 0 0"/>
+        <geometry>
+          <mesh filename="$(arg meshes_dir)/ph_thumb.stl" scale="0.001 0.001 0.001"/>
+        </geometry>
+      </collision>
+    </link>
+    <!-- GAZEBO REF -->
+    <gazebo reference="${ns}_${name}_link">
+      <material>Gazebo/Grey</material>
+      <selfCollide>false</selfCollide>
+      <kp value="1e4" />
+      <kd value="1e2" />
+      <surface>
+       <friction>
+        <ode>
+         <mu>0.133</mu>
+         <mu2>0.133</mu2>
+        </ode>
+       </friction>
+      </surface>
+    </gazebo>
+  </xacro:macro>
 </robot>

File: softhands_description/urdf/xacro/include/macro/v1_2_research/plugin.xacro (robot description, xacro)
@@ -87,11 +87,3 @@
 		</plugin>
 	</gazebo>
-	  <!-- # Gazebo NEW custom synergy-plugin
-	  <gazebo>
-	          <plugin name="synergy_plugin" filename="libsofthand_plugin.so">
-	                      <namespace>$(arg ns)</namespace>
-	                      <operation_mode>0</operation_mode>
-	                      <spring_k>5</spring_k>
-	          </plugin>
-	  </gazebo> -->
 </robot>

File: softhands_description/urdf/xacro/include/macro/v1_wide/modules/finger/phalanx.xacro (robot description, xacro)
@@ -12,7 +12,7 @@
 		<link name="${ns}_${name}_virtual_link">
 		   <inertial>
-				<origin xyz="0 0 0" rpy="0 0 0"/>
-				<mass value="1e-3"/>
-				<inertia ixx="1e-6" ixy="0.0" ixz="0.0" iyy="1e-6" iyz="0.0" izz="1e-6"/>
+				<origin rpy="0 0 0" xyz="0 0 0"/>
+				<mass value="0.001"/>
+				<inertia ixx="0.0001" ixy="0" ixz="0" iyy="0.0001" iyz="0" izz="0.0001" />
 		   </inertial>
 	    </link>
@@ -50,6 +50,16 @@
 		</link>
 		<gazebo reference="${ns}_${name}_link">
-			<material>Gazebo/Grey</material>
+			<material>Gazebo/Gray</material>
 			<selfCollide>false</selfCollide>
+			<kp value="1e4" />
+			<kd value="1e2" />
+			<surface>
+			<friction>
+				<ode>
+				<mu>0.133</mu>
+				<mu2>0.133</mu2>
+				</ode>
+			</friction>
+			</surface>
 		</gazebo>
     </xacro:macro>

File: softhands_description/urdf/xacro/include/macro/v1_wide/modules/finger/phalanx_dist.xacro (robot description, xacro)
@@ -12,11 +12,11 @@
 		<link name="${ns}_${name}_virtual_link">
 		   <inertial>
-				<origin xyz="0 0 0" rpy="0 0 0"/>
-				<mass value="1e-3"/>
-				<inertia ixx="1e-6" ixy="0.0" ixz="0.0" iyy="1e-6" iyz="0.0" izz="1e-6"/>
+				<origin rpy="0 0 0" xyz="0 0 0"/>
+				<mass value="0.001"/>
+				<inertia ixx="0.0001" ixy="0" ixz="0" iyy="0.0001" iyz="0" izz="0.0001" />
 		   </inertial>
 	    </link>
 		<!-- Proximal phalanx -->
-		<joint name="${ns}_${parent}_${name}_joint" type="revolute">
+		<joint name="${ns}_${name}_joint" type="revolute">
 			<axis xyz="0 0 1"/>
 			<limit effort="30" velocity="1.0" lower="0" upper="0.785398" />
@@ -49,8 +49,18 @@
 				</collision>
 		</link>
-	<gazebo reference="${ns}_${name}_link">
-		<material>Gazebo/Grey</material>
-		<selfCollide>false</selfCollide>
-	</gazebo>
+		<gazebo reference="${ns}_${name}_link">
+			<material>Gazebo/Gray</material>
+			<selfCollide>false</selfCollide>
+			<kp value="1e4" />
+			<kd value="1e2" />
+			<surface>
+			<friction>
+				<ode>
+				<mu>0.133</mu>
+				<mu2>0.133</mu2>
+				</ode>
+			</friction>
+			</surface>
+		</gazebo>
     </xacro:macro>
 </robot>

File: softhands_description/urdf/xacro/include/macro/v1_wide/modules/finger/phalanx_knuckle.xacro (robot description, xacro)
@@ -5,5 +5,5 @@
 		<joint name="${ns}_${name}_joint" type="revolute">
 			<axis xyz="0 1 0"/>
-			<limit effort="30" velocity="1.0" lower="0" upper="0.0" />
+			<limit effort="30" velocity="1.0" lower="0.0" upper="0.0" />
 			<xacro:insert_block name="origin"/>
             <parent link="${ns}_${parent}_link"/>
@@ -35,6 +35,16 @@
 		</link>
 	<gazebo reference="${ns}_${name}_link">
-		<material>Gazebo/White</material>
-		<selfCollide>false</selfCollide>
+			<material>Gazebo/White</material>
+			<selfCollide>false</selfCollide>
+			<kp value="1e4" />
+			<kd value="1e2" />
+			<surface>
+			<friction>
+				<ode>
+				<mu>0.133</mu>
+				<mu2>0.133</mu2>
+				</ode>
+			</friction>
+			</surface>
 	</gazebo>
     </xacro:macro>

File: softhands_description/urdf/xacro/include/macro/v1_wide/modules/palm/palm_central.xacro (robot description, xacro)
@@ -38,5 +38,5 @@
 		</link>
 		<!-- palm base to Thumb -->
-		<joint name="${ns}_${name}_thumb_virtual_joint" type="fixed">
+		<joint name="${ns}_${name}_thumb_virtual_joint" type="revolute">
 			<axis xyz="0 0 -1"/>
 			<limit effort="30" velocity="10" lower="0" upper="1.57" />
@@ -48,14 +48,16 @@
 	    <link name="${ns}_${name}_thumb_virtual_link">
 		   <inertial>
-			<origin xyz="0 0 0" rpy="0 0 0"/>
-			<mass value="1e-3"/>
-			<inertia ixx="1e-6" ixy="0.0" ixz="0.0" iyy="1e-6" iyz="0.0" izz="1e-6"/>
+				<origin rpy="0 0 0" xyz="0 0 0"/>
+				<mass value="0.001"/>
+				<inertia  ixx="0.0001"      ixy="0"  	    ixz="0"
+						iyy="0.0001" 	    iyz="0"
+							izz="0.0001" />
 		   </inertial>
 	    </link>
 		<!-- palm base to Litte virtual -->
-		<joint name="${ns}_${name}_little_virtual_joint" type="fixed">
+		<joint name="${ns}_${name}_little_virtual_joint" type="revolute">
 			<axis xyz="0 0 1"/>
 			<dynamics damping="0.0" friction="0.0"/>
-			<limit effort="100" lower="0.0" upper="0.5" velocity="100"/>
+			<limit effort="100" lower="0.0" upper="0.4" velocity="100"/>
 			<origin xyz=" -0.0000000091 -10.6603e-3 66.1817e-3" rpy="0 -0.1745327 -1.5707963"/>
 			<parent link="${ns}_${name}_link"/>
@@ -64,12 +66,24 @@
 		<link name="${ns}_${name}_little_virtual_link">
 		   <inertial>
-				<origin xyz="0 0 0" rpy="0 0 0"/>
-				<mass value="1e-3"/>
-				<inertia ixx="1e-6" ixy="0.0" ixz="0.0" iyy="1e-6" iyz="0.0" izz="1e-6"/>
+			<origin rpy="0 0 0" xyz="0 0 0"/>
+			<mass value="0.001"/>
+			<inertia  ixx="0.0001"      ixy="0"  	    ixz="0"
+					iyy="0.0001" 	    iyz="0"
+						izz="0.0001" />
 		   </inertial>
 	    </link>
 		<gazebo reference="${ns}_${name}_link">
-		<selfCollide>false</selfCollide>
+			<selfCollide>false</selfCollide>
 			<material>Gazebo/Grey</material>
+			<kp value="1e4" />
+			<kd value="1e2" />
+			<surface>
+			<friction>
+				<ode>
+				<mu>0.133</mu>
+				<mu2>0.133</mu2>
+				</ode>
+			</friction>
+			</surface>
 		</gazebo>
     </xacro:macro>

File: softhands_description/urdf/xacro/include/macro/v1_wide/modules/palm/palm_little.xacro (robot description, xacro)
@@ -2,5 +2,5 @@
 <robot xmlns:xacro="http://www.ros.org/wiki/xacro">
     <xacro:macro name="palm_little" params="name parent side *origin ns">
-		<joint name="${ns}_${name}_joint" type="fixed">
+		<joint name="${ns}_${name}_joint" type="revolute">
 			<parent link="${ns}_${parent}_link"/>
 			<child link="${ns}_${name}_link"/>
@@ -36,8 +36,18 @@
 				</collision>
 		</link>
-	<gazebo reference="${ns}_${name}_link">
-		<selfCollide>false</selfCollide>
-		<material>Gazebo/Grey</material>
-	</gazebo>
+		<gazebo reference="${ns}_${name}_link">
+			<material>Gazebo/Grey</material>
+			<selfCollide>false</selfCollide>
+			<kp value="1e4" />
+			<kd value="1e2" />
+			<surface>
+			<friction>
+				<ode>
+				<mu>0.133</mu>
+				<mu2>0.133</mu2>
+				</ode>
+			</friction>
+			</surface>
+		</gazebo>
     </xacro:macro>
 </robot>

File: softhands_description/urdf/xacro/include/macro/v1_wide/modules/palm/palm_thumb.xacro (robot description, xacro)
@@ -2,5 +2,5 @@
 <robot xmlns:xacro="http://www.ros.org/wiki/xacro">
     <xacro:macro name="palm_thumb" params="name parent side *origin ns">
-		<joint name="${ns}_${name}_joint" type="fixed">
+		<joint name="${ns}_${name}_joint" type="revolute">
 			<parent link="${ns}_${parent}_link"/>
 			<child link="${ns}_${name}_link"/>
@@ -36,44 +36,64 @@
 				</collision>
 		</link>
-	<!-- Palm thumb to thumb support -->
-	<joint name="${ns}_${name}_support_joint" type="fixed">
-		<parent link="${ns}_${name}_link"/>
-		<child link="${ns}_${name}_support_link"/>
-		<origin xyz=" 24.2343e-3 -5.0e-3 9.13010e-3" rpy="-1.5707963 -1.0471972 0"/>
-	</joint>
-	<link name="${ns}_${name}_support_link">
-			<visual>
-			<material name="grey" />
-				<geometry>
-				<mesh
-					filename="$(arg meshes_dir)/thumb_support.stl"
-					scale="0.001 0.001 0.001" />
-				</geometry>
-			<origin xyz="0 0 0" rpy="0 0 0" />
-			</visual>
-			<inertial>
-			<origin xyz="1.1097412e-02 -4.2327979e-05 -4.7109856e-04" rpy="0 0 0" />
-			<mass value="1.6408860e-02" />
-				<inertia ixx="1.8835019e-06" ixy="-4.9293913e-09" ixz="-2.5700318e-08"
-										iyy="1.2828797e-06"  iyz="-4.0065947e-09"
-															izz="2.2986135e-06" />
-				</inertial>
-			<collision>
-				<geometry>
-				<mesh
-					filename="$(arg meshes_dir)/thumb_support.stl"
-					scale="0.001 0.001 0.001" />
-				</geometry>
-			<origin xyz="0 0 0" rpy="0 0 0" />
-			</collision>
-	</link>
-	<gazebo reference="${ns}_${name}_link">
-		<material>Gazebo/Grey</material>
-    	<selfCollide>false</selfCollide>
-	</gazebo>
-	<gazebo reference="${ns}_${name}_support_link">
-		<material>Gazebo/White</material>
-		<selfCollide>false</selfCollide>
-	</gazebo>
+		<!-- Palm thumb to thumb support -->
+		<joint name="${ns}_${name}_support_joint" type="fixed">
+			<parent link="${ns}_${name}_link"/>
+			<child link="${ns}_${name}_support_link"/>
+			<origin xyz=" 24.2343e-3 -5.0e-3 9.13010e-3" rpy="-1.5707963 -1.0471972 0"/>
+		</joint>
+		<link name="${ns}_${name}_support_link">
+				<visual>
+				<material name="grey" />
+					<geometry>
+					<mesh
+						filename="$(arg meshes_dir)/thumb_support.stl"
+						scale="0.001 0.001 0.001" />
+					</geometry>
+				<origin xyz="0 0 0" rpy="0 0 0" />
+				</visual>
+				<inertial>
+				<origin xyz="1.1097412e-02 -4.2327979e-05 -4.7109856e-04" rpy="0 0 0" />
+				<mass value="1.6408860e-02" />
+					<inertia ixx="1.8835019e-06" ixy="-4.9293913e-09" ixz="-2.5700318e-08"
+											iyy="1.2828797e-06"  iyz="-4.0065947e-09"
+																izz="2.2986135e-06" />
+					</inertial>
+				<collision>
+					<geometry>
+					<mesh
+						filename="$(arg meshes_dir)/thumb_support.stl"
+						scale="0.001 0.001 0.001" />
+					</geometry>
+				<origin xyz="0 0 0" rpy="0 0 0" />
+				</collision>
+		</link>
+		<gazebo reference="${ns}_${name}_link">
+			<material>Gazebo/Grey</material>
+			<selfCollide>false</selfCollide>
+			<kp value="1e4" />
+			<kd value="1e2" />
+			<surface>
+			<friction>
+				<ode>
+				<mu>0.133</mu>
+				<mu2>0.133</mu2>
+				</ode>
+			</friction>
+			</surface>
+		</gazebo>
+		<gazebo reference="${ns}_${name}_support_link">
+				<material>Gazebo/White</material>
+				<selfCollide>false</selfCollide>
+				<kp value="1e4" />
+				<kd value="1e2" />
+				<surface>
+				<friction>
+					<ode>
+					<mu>0.133</mu>
+					<mu2>0.133</mu2>
+					</ode>
+				</friction>
+				</surface>
+		</gazebo>
     </xacro:macro>
 </robot>

File: softhands_description/urdf/xacro/include/macro/v1_wide/modules/thumb/thumb_distal.xacro (robot description, xacro)
@@ -12,22 +12,9 @@
 	    <link name="${ns}_${name}_virtual_link">
 		   <inertial>
-			<origin xyz="0 0 0" rpy="0 0 0"/>
-			<mass value="1e-3"/>
-			<inertia ixx="1e-6" ixy="0.0" ixz="0.0" iyy="1e-6" iyz="0.0" izz="1e-6"/>
+				<origin rpy="0 0 0" xyz="0 0 0"/>
+				<mass value="0.001"/>
+				<inertia ixx="0.0001" ixy="0" ixz="0" iyy="0.0001" iyz="0" izz="0.0001" />
 		   </inertial>
 	    </link>
-		<gazebo reference="${ns}_${name}_virtual_link">
-			<material>Gazebo/Grey</material>
-			<kp value="1e4" />
-			<kd value="1e2" />
-			<surface>
-			<friction>
-				<ode>
-				<mu>0.133</mu>
-				<mu2>0.133</mu2>
-				</ode>
-			</friction>
-			</surface>
-		</gazebo>
 		<!-- Thumb middle  -->
 		<joint name="${ns}_${name}_joint" type="revolute">
@@ -65,4 +52,5 @@
 		<gazebo reference="${ns}_${name}_link">
 			<material>Gazebo/Grey</material>
+			<selfCollide>false</selfCollide>
 			<kp value="1e4" />
 			<kd value="1e2" />

File: softhands_description/urdf/xacro/include/macro/v1_wide/modules/thumb/thumb_knuckle.xacro (robot description, xacro)
@@ -37,4 +37,5 @@
 		<gazebo reference="${ns}_${name}_link">
 			<material>Gazebo/Grey</material>
+			<selfCollide>false</selfCollide>
 			<kp value="1e4" />
 			<kd value="1e2" />
