Commit message: need to tune damping and friction for both the hands

File: softhands_description/urdf/xacro/include/macro/v1_wide/modules/thumb/thumb_proximal.xacro (robot description, xacro)
@@ -12,22 +12,9 @@
 	    <link name="${ns}_${name}_virtual_link">
 		   <inertial>
-			<origin xyz="0 0 0" rpy="0 0 0"/>
-			<mass value="1e-3"/>
-			<inertia ixx="1e-6" ixy="0.0" ixz="0.0" iyy="1e-6" iyz="0.0" izz="1e-6"/>
+				<origin rpy="0 0 0" xyz="0 0 0"/>
+				<mass value="0.001"/>
+				<inertia ixx="0.0001" ixy="0" ixz="0" iyy="0.0001" iyz="0" izz="0.0001" />
 		   </inertial>
 	    </link>
-		<gazebo reference="${ns}_${name}_virtual_link">
-			<material>Gazebo/Grey</material>
-			<kp value="1e4" />
-			<kd value="1e2" />
-			<surface>
-			<friction>
-				<ode>
-				<mu>0.133</mu>
-				<mu2>0.133</mu2>
-				</ode>
-			</friction>
-			</surface>
-		</gazebo>
 		<!-- Thumb Proximal joint  -->
 		<joint name="${ns}_${name}_virtual_joint" type="revolute">
@@ -65,4 +52,5 @@
 		<gazebo reference="${ns}_${name}_link">
 			<material>Gazebo/Grey</material>
+			<selfCollide>false</selfCollide>
 			<kp value="1e4" />
 			<kd value="1e2" />

File: softhands_description/urdf/xacro/v1_2_research.xacro (robot description, xacro)
@@ -37,36 +37,32 @@
  *
 -->
-<robot name="v1_wide" xmlns:xacro="http://www.ros.org/wiki/xacro">
-	<!-- # palm central -->
-	<xacro:palm_central name="palm_central" parent="$(arg root_link)" side="$(arg side)" ns="$(arg ns)">
+<robot name="right_hand_v2" xmlns:xacro="http://www.ros.org/wiki/xacro">
+	<!-- # iso -->
+	<xacro:iso name="iso" parent="$(arg root_link)" ns="$(arg ns)" side="$(arg side)">
 		<origin rpy="$(arg orientation)" xyz="$(arg position)"/>
-	</xacro:palm_central>
-	<!-- # palm thumb -->
-	<xacro:palm_thumb name="palm_thumb" parent="palm_central_thumb_virtual" side="$(arg side)" ns="$(arg ns)">
-		<origin rpy="0 0 0 " xyz="12e-3 -0.0000414746e-3 0"/>
-	</xacro:palm_thumb>
-	<!-- # palm little -->
-	<xacro:palm_little name="palm_little" parent="palm_central_little_virtual" side="$(arg side)" ns="$(arg ns)">
-		<origin rpy="0 0 0 " xyz="12e-3 -0.0000466576e-3 0"/>
-	</xacro:palm_little>
+	</xacro:iso>
+	<!-- # palm  -->
+	<xacro:palm name="palm" parent="iso" ns="$(arg ns)" side="$(arg side)">
+		<origin rpy="1.57 0 0" xyz="-0.0045 0.0145 0.144"/>
+	</xacro:palm>
 	<!-- # thumb -->
-	<xacro:thumb name="thumb" parent="palm_thumb_support" side="$(arg side)" ns="$(arg ns)">
-		<origin rpy="-1.5707963 0 0" xyz="21.9577e-3 0 -2.8e-3"/>
+	<xacro:thumb name="thumb" parent="palm" ns="$(arg ns)" side="$(arg side)">
+		<origin rpy="-1.57 3.14 0.0" xyz="-0.044 -0.0465 -0.002"/>
 	</xacro:thumb>
 	<!-- # Index -->
-	<xacro:finger name="index" parent="palm_central" side="$(arg side)" ns="$(arg ns)">
-		<origin  rpy="-3.1415927  -1.396264 1.5707963" xyz="5e-3 44.8953e-3 112.230e-3"/>
+	<xacro:finger name="index" parent="palm" ns="$(arg ns)" side="$(arg side)">
+		<origin rpy="0 0 1.57" xyz="-0.02 -0.007 0.014"/>
 	</xacro:finger>
 	<!-- # Middle -->
-	<xacro:finger name="middle" parent="palm_central" side="$(arg side)" ns="$(arg ns)">
-		<origin  rpy="0 -1.5707963 -1.5707963" xyz="5e-3 12.5e-3 115e-3"/>
+	<xacro:finger name="middle" parent="palm" ns="$(arg ns)" side="$(arg side)">
+		<origin rpy="0 0 1.57" xyz="0 0 0.014"/>
 	</xacro:finger>
 	<!-- # Ring -->
-	<xacro:finger name="ring" parent="palm_little" side="$(arg side)" ns="$(arg ns)">
-	    <origin rpy="0 -1.3089971 0" xyz=" 8.6355e-3 5e-3 44.4863e-3" />
+	<xacro:finger name="ring" parent="palm" ns="$(arg ns)" side="$(arg side)">
+		<origin rpy="0 0 1.57" xyz="0.02 -0.007 0.014"/>
 	</xacro:finger>
-    <!-- # Little -->
-	<xacro:finger name="little" parent="palm_little" side="$(arg side)" ns="$(arg ns)">
-		<origin rpy="0 -1.221731 0" xyz="39.2985e-3 5e-3 34.8419e-3" />
+	<!-- # Little -->
+	<xacro:finger name="little" parent="palm" ns="$(arg ns)" side="$(arg side)">
+		<origin rpy="0 0 1.57" xyz="0.04 -0.012 0.014"/>
 	</xacro:finger>
 </robot>

Commit message: modified some parameters

File: softhands_description/urdf/xacro/include/macro/v1_2_research/modules/finger/phalanx_knuckle.xacro (robot description, xacro)
@@ -46,5 +46,5 @@
       <axis xyz="0 0 -1"/>
       <limit effort="30" velocity="1.0" lower="-0.524" upper="0.524" />
-       <dynamics damping="0.08" friction="0"/>
+       <dynamics damping="0.08" friction="$(arg friction)"/>
     </joint>
     <!-- LINK -->

File: softhands_description/urdf/xacro/include/macro/v1_2_research/modules/iso.xacro (robot description, xacro)
@@ -67,5 +67,5 @@
 		<gazebo reference="${ns}_${name}_link">
     	  	<material>Gazebo/Grey</material>
-			<selfCollide>true</selfCollide>
+			<selfCollide>$(arg selfCollide)</selfCollide>
 	  	</gazebo>
 	</xacro:macro>

File: softhands_description/urdf/xacro/include/macro/v1_2_research/modules/palm/palm.xacro (robot description, xacro)
@@ -41,5 +41,5 @@
 	  	<joint name="${ns}_palm_joint" type="fixed">
 			<xacro:insert_block name="origin"/>
-			<parent link="${parent}" />
+			<parent link="${ns}_${parent}_link" />
 			<child link="${ns}_palm_link" />
 		</joint>
@@ -66,5 +66,5 @@
 		<gazebo reference="${ns}_palm_link">
 			<material>Gazebo/Grey</material>
-			<selfCollide>true</selfCollide>
+			<selfCollide>$(arg selfCollide)</selfCollide>
 		</gazebo>
 	</xacro:macro>

File: softhands_description/urdf/xacro/include/macro/v1_2_research/modules/thumb/thumb_knuckle.xacro (robot description, xacro)
@@ -46,5 +46,5 @@
       <axis xyz="0 0 -1"/>
       <limit effort="30" velocity="1.0" lower="0" upper="1.57" />
-      <dynamics damping="0.0" friction="0.0" />
+      <dynamics damping="0.08" friction="0.0" />
     </joint>
     <!-- LINK -->
@@ -72,5 +72,5 @@
     <gazebo reference="${ns}_${name}_link">
       <material>Gazebo/Grey</material>
-      <selfCollide>$(arg selfCollide)</selfCollide>
+      <selfCollide>false</selfCollide>
     </gazebo>
   </xacro:macro>

File: softhands_description/urdf/xacro/include/macro/v1_wide/modules/finger/phalanx.xacro (robot description, xacro)
@@ -53,5 +53,5 @@
 		<gazebo reference="${ns}_${name}_link">
 			<material>Gazebo/Gray</material>
-			<selfCollide>false</selfCollide>
+			<selfCollide>$(arg selfCollide)</selfCollide>
 		</gazebo>
     </xacro:macro>

File: softhands_description/urdf/xacro/include/macro/v1_wide/modules/finger/phalanx_dist.xacro (robot description, xacro)
@@ -53,5 +53,5 @@
 		<gazebo reference="${ns}_${name}_link">
 			<material>Gazebo/Gray</material>
-			<selfCollide>true</selfCollide>
+			<selfCollide>$(arg selfCollide)</selfCollide>
 		</gazebo>
     </xacro:macro>

File: softhands_description/urdf/xacro/include/macro/v1_wide/modules/finger/phalanx_knuckle.xacro (robot description, xacro)
@@ -35,5 +35,5 @@
 		</link>
 		<gazebo reference="${ns}_${name}_link">
-			<selfCollide>false</selfCollide>
+			<selfCollide>$(arg selfCollide)</selfCollide>
 			<material>Gazebo/White</material>
 		</gazebo>

File: softhands_description/urdf/xacro/include/macro/v1_wide/modules/palm/palm_central.xacro (robot description, xacro)
@@ -74,5 +74,5 @@
 	    </link>
 		<gazebo reference="${ns}_${name}_link">
-			<selfCollide>false</selfCollide>
+			<selfCollide>$(arg selfCollide)</selfCollide>
 			<material>Gazebo/Grey</material>
 		</gazebo>

File: softhands_description/urdf/xacro/include/macro/v1_wide/modules/palm/palm_little.xacro (robot description, xacro)
@@ -37,5 +37,5 @@
 		</link>
 		<gazebo reference="${ns}_${name}_link">
-			<selfCollide>false</selfCollide>
+			<selfCollide>$(arg selfCollide)</selfCollide>
 			<material>Gazebo/Grey</material>
 		</gazebo>

File: softhands_description/urdf/xacro/include/macro/v1_wide/modules/palm/palm_thumb.xacro (robot description, xacro)
@@ -69,9 +69,9 @@
 		</link>
 		<gazebo reference="${ns}_${name}_link">
-			<selfCollide>false</selfCollide>
+			<selfCollide>$(arg selfCollide)</selfCollide>
 			<material>Gazebo/Grey</material>
 		</gazebo>
 		<gazebo reference="${ns}_${name}_support_link">
-			<selfCollide>false</selfCollide>
+			<selfCollide>$(arg selfCollide)</selfCollide>
 			<material>Gazebo/White</material>
 		</gazebo>

File: softhands_description/urdf/xacro/include/macro/v1_wide/modules/thumb/thumb_distal.xacro (robot description, xacro)
@@ -53,5 +53,5 @@
 		<gazebo reference="${ns}_${name}_link">
 			<material>Gazebo/Grey</material>
-			<selfCollide>true</selfCollide>
+			<selfCollide>$(arg selfCollide)</selfCollide>
 		</gazebo>
     </xacro:macro>

File: softhands_description/urdf/xacro/include/macro/v1_wide/modules/thumb/thumb_knuckle.xacro (robot description, xacro)
@@ -37,5 +37,5 @@
 		<gazebo reference="${ns}_${name}_link">
 			<material>Gazebo/Grey</material>
-			<selfCollide>true</selfCollide>
+			<selfCollide>$(arg selfCollide)</selfCollide>
 		</gazebo>
     </xacro:macro>

File: softhands_description/urdf/xacro/include/macro/v1_wide/modules/thumb/thumb_proximal.xacro (robot description, xacro)
@@ -53,5 +53,5 @@
 		<gazebo reference="${ns}_${name}_link">
 			<material>Gazebo/Grey</material>
-			<selfCollide>true</selfCollide>
+			<selfCollide>$(arg selfCollide)</selfCollide>
 		</gazebo>
     </xacro:macro>

File: softhands_description/urdf/xacro/v1_2_research.xacro (robot description, xacro)
@@ -42,10 +42,11 @@
 	</link>
 	<!-- # iso -->
-	<!-- <xacro:iso name="iso" parent="$(arg root_link)" ns="$(arg ns)" side="$(arg side)">
+	<xacro:iso name="iso" parent="$(arg root_link)" ns="$(arg ns)" side="$(arg side)">
 		<origin rpy="$(arg orientation)" xyz="$(arg position)"/>
-	</xacro:iso> -->
+	</xacro:iso>
 	<!-- # palm  -->
-	<xacro:palm name="palm" parent="$(arg root_link)" ns="$(arg ns)" side="$(arg side)">
+	<xacro:palm name="palm" parent="iso" ns="$(arg ns)" side="$(arg side)">
 		<origin rpy="1.57 0 0" xyz="-0.0045 0.0145 0.144"/>
+		<!-- <origin rpy="0 0 0" xyz="-0.0045 0.0145 0.144"/> -->
 	</xacro:palm>
 	<!-- # thumb -->
