Commit message: changed rotation of the  grasp link v1_2_research

File: softhands_description/urdf/xacro/include/macro/v1_2_research/modules/iso.xacro (robot description, xacro)
@@ -71,5 +71,5 @@
 		<!-- Fake joint and link for grasping -->
 	  	<joint name="${ns}_grasp_joint" type="fixed">
-			<origin rpy="0 0 0" xyz="0.03 0.06 0.10"/>
+			<origin rpy="0 0 1.57" xyz="0.03 0.06 0.10"/>
 			<parent link="${ns}_${name}_link" />
 			<child link="${ns}_grasp_link" />

Commit message: added xacro:if for left and right grasp_link

File: softhands_description/urdf/xacro/include/macro/v1_2_research/modules/iso.xacro (robot description, xacro)
@@ -70,5 +70,7 @@
 	  	</gazebo>
 		<!-- Fake joint and link for grasping -->
-	  	<joint name="${ns}_grasp_joint" type="fixed">
+		<!-- QUIRINO: added xacro:if for left and right grasp_link-->
+	  	<xacro:if value="${ns == 'right_hand_v1_2_research'}">
+		<joint name="${ns}_grasp_joint" type="fixed">
 			<origin rpy="0 0 1.57" xyz="-0.06 0.03 0.16"/>
 			<parent link="${ns}_${name}_link" />
@@ -76,4 +78,13 @@
 		</joint>
 		<link name="${ns}_grasp_link"/>
+		</xacro:if>
+		<xacro:if value="${ns == 'left_hand_v1_2_research'}">
+		<joint name="${ns}_grasp_joint" type="fixed">
+			<origin rpy="0 0 1.57" xyz="0.06 0.03 0.16"/>
+			<parent link="${ns}_${name}_link" />
+			<child link="${ns}_grasp_link" />
+		</joint>
+		<link name="${ns}_grasp_link"/>
+		</xacro:if>
 	</xacro:macro>
 </robot>

File: softhands_description/urdf/xacro/include/macro/v1_wide/modules/palm/palm_central.xacro (robot description, xacro)
@@ -34,10 +34,23 @@
 		</link>
 		<!-- Fake joint and link for grasping -->
-	  	<joint name="${ns}_grasp_joint" type="fixed">
-			<origin rpy="0 0 0" xyz="0.03 -0.09 0.10"/>
+		<!-- QUIRINO: added xacro:if for left and right grasp_link-->
+	  	<xacro:if value="${ns == 'right_hand_v1_wide'}">
+		<joint name="${ns}_grasp_joint" type="fixed">
+			<!-- QUIRINO: modified grasp_link for wide_hand-->
+			<origin rpy="0 0 0" xyz="0.03 0.10 0.15"/>
 			<parent link="${ns}_${name}_link" />
 			<child link="${ns}_grasp_link" />
 		</joint>
 		<link name="${ns}_grasp_link"/>
+		</xacro:if>
+		<xacro:if value="${ns == 'left_hand_v1_wide'}">
+		<joint name="${ns}_grasp_joint" type="fixed">
+			<!-- QUIRINO: modified grasp_link for wide_hand-->
+			<origin rpy="0 0 0" xyz="0.03 -0.10 0.15"/>
+			<parent link="${ns}_${name}_link" />
+			<child link="${ns}_grasp_link" />
+		</joint>
+		<link name="${ns}_grasp_link"/>
+		</xacro:if>
 		<!-- palm base to Thumb -->
 		<joint name="${ns}_${name}_thumb_joint" type="${joint_type}">
