Commit message: reduced xacro file, added spring with joints and a real inertia on the virtual link

File: softhands_description/urdf/softhands.xacro (robot description, xacro)
@@ -33,33 +33,28 @@
  * \file      test_SHs_v2.urdf.xacro
  *
- * \author       _Centro di Ricerca "E.Piaggio"_
- * \author       _Istituto Italiano di Tecnologia, Soft Robotics for Human Cooperation and Rehabilitation Lab_
+ * \author       Centro di Ricerca "E.Piaggio"
+ * \author       Istituto Italiano di Tecnologia, Soft Robotics for Human Cooperation and Rehabilitation Lab
  *
 -->
 <robot name="softhand" xmlns:xacro="http://www.ros.org/wiki/xacro">
-  	<xacro:arg name="sh_version" default="v1_2_research"/>
-  	<!-- <xacro:arg name="sh_version" default="v1_wide"/> -->
-  	<xacro:arg name="root_dir" default="$(find softhands_description)/urdf/xacro/include/macro/$(arg sh_version)"/>
-  	<xacro:arg name="root_link" default="world"/>
-  	<xacro:arg name="side" default="left"/>
-  	<xacro:arg name="meshes_dir" default="package://softhands_description/meshes/$(arg sh_version)/$(arg side)"/>
-  	<xacro:arg name="ns" default="$(arg side)_hand_$(arg sh_version)"/>
-  	<xacro:arg name="x" default="0"/>
-  	<xacro:arg name="y" default="0"/>
-  	<xacro:arg name="z" default="0"/>
-  	<xacro:arg name="position" default="$(arg x) $(arg y) $(arg z)"/>
-  	<xacro:arg name="roll" default="0"/>
-  	<xacro:arg name="pitch" default="0"/>
-  	<xacro:arg name="yaw" default="0"/>
-  	<xacro:arg name="orientation" default="$(arg roll) $(arg pitch) $(arg yaw)"/>
-  	<xacro:arg name="operation_mode" default="0"/>
-  	<xacro:arg name="selfCollide" default="0"/>
-	<xacro:include filename="$(arg root_dir)/header.xacro"/>
-  	<xacro:arg name="friction" default="0.0"/>
-  	<xacro:arg name="virtual_friction" default="0.0"/>
-  	<xacro:arg name="virtual_damping" default="3e-2"/>
-  	<xacro:arg name="damping" default="3e-2"/>
-	<xacro:include filename="$(find softhands_description)/urdf/xacro/$(arg sh_version).xacro"/>
-	<!-- Include plugin -->
-	<xacro:include filename="$(find softhands_description)/urdf/xacro/include/macro/$(arg sh_version)/plugin.xacro"/>
+	<xacro:macro name="softhands" params="side parent position orientation fixed_hands:='false'">
+		<xacro:arg name="sh_version" default="v1_2_research"/>
+		<!-- <xacro:arg name="sh_version" default="v1_wide"/> -->
+		<xacro:arg name="root_dir" default="$(find softhands_description)/urdf/xacro/include/macro/$(arg sh_version)"/>
+		<xacro:arg name="root_link" default="${parent}"/>
+		<xacro:arg name="side" default="left"/>
+		<xacro:arg name="meshes_dir" default="package://softhands_description/meshes/$(arg sh_version)/$(arg side)"/>
+		<xacro:arg name="ns" default="$(arg side)hand$(arg sh_version)"/>
+		<xacro:arg name="position" default="${position}"/>
+		<xacro:arg name="orientation" default="${orientation}"/>
+		<xacro:arg name="operation_mode" default="0"/>
+		<xacro:arg name="selfCollide" default="0"/>
+		<xacro:arg name="friction" default="0"/>
+		<xacro:arg name="virtual_friction" default="0"/>
+		<xacro:arg name="virtual_damping" default="0.0"/>
+		<xacro:arg name="damping" default="0.0"/>
+		<xacro:include filename="$(find softhands_description)/urdf/xacro/$(arg sh_version).xacro"/>
+		<!-- Include plugin -->
+		<!-- <xacro:include filename="$(find softhands_description)/urdf/xacro/include/macro/$(arg sh_version)/plugin.xacro"/> -->
+	</xacro:macro>
 </robot>

File: softhands_description/urdf/xacro/include/macro/v1_2_research/header.xacro (robot description, xacro)
@@ -43,12 +43,10 @@
   <!-- Include xacro macro Thumb -->
   <xacro:include filename="$(arg root_dir)/modules/thumb.xacro" />
-  <xacro:include filename="$(arg root_dir)/modules/thumb/thumb_knuckle.xacro" />
-  <xacro:include filename="$(arg root_dir)/modules/thumb/thumb_short.xacro" />
   <!-- Include xacro macro Finger -->
-  <xacro:include filename="$(arg root_dir)/modules/finger/phalanx_short.xacro" />
-  <xacro:include filename="$(arg root_dir)/modules/finger/phalanx_knuckle.xacro" />
-  <xacro:include filename="$(arg root_dir)/modules/finger/phalanx.xacro" />
-  <xacro:include filename="$(arg root_dir)/modules/finger/phalanx_distal.xacro" />
   <xacro:include filename="$(arg root_dir)/modules/finger.xacro" />
+  <!-- Phalanges -->
+  <xacro:include filename="$(arg root_dir)/modules/phalanges/phalanx_generic.xacro" />
+  <xacro:include filename="$(arg root_dir)/modules/phalanges/phalanx_knuckle.xacro" />
+  <xacro:include filename="$(arg root_dir)/modules/phalanges/thumb_knuckle.xacro" />
   <!-- Color definitions -->
   <xacro:include filename="$(arg root_dir)/color.xacro" />

File: softhands_description/urdf/xacro/include/macro/v1_2_research/modules/finger.xacro (robot description, xacro)
@@ -44,15 +44,24 @@
     </xacro:phalanx_knuckle>
     <!-- Proximal -->
-    <xacro:phalanx name="${name}_proximal" parent="${name}_knuckle" side="$(arg side)" ns="$(arg ns)">
-      <origin rpy="1.57 0 0" xyz="0.009 0 0"/>
-    </xacro:phalanx>
+    <xacro:phalanx_generic name="${name}_proximal" parent="${name}_knuckle" ns="$(arg ns)" mass="0.009" mesh="ph_medium">
+      <virtual_origin>  <origin rpy="1.57 0 0" xyz="0.009 0 0"/>                      </virtual_origin>
+      <real_origin>     <origin rpy="0.0 0 0" xyz="0.013 0 0"/>                       </real_origin>
+      <inertia_origin>  <origin rpy="0 0 0" xyz="8.7707437e-03 -1.7863138e-03 0.0"/>  </inertia_origin>
+      <inertia ixx="2.2722068e-07" ixy="1.1586053e-08" ixz="0.0" iyy="5.5947233e-07" iyz="0.0" izz="5.9562195e-07"/>
+    </xacro:phalanx_generic>
     <!-- Middle -->
-    <xacro:phalanx_short name="${name}_middle" parent="${name}_proximal" side="$(arg side)" ns="$(arg ns)">
-      <origin rpy="0.0 0.0 0.0" xyz="0.013 0 0 "/>
-    </xacro:phalanx_short>
+    <xacro:phalanx_generic name="${name}_middle" parent="${name}_proximal" ns="$(arg ns)" mass="0.0063" mesh="ph_short">
+      <virtual_origin>  <origin rpy="0.0 0.0 0.0" xyz="0.013 0 0 "/>                  </virtual_origin>
+      <real_origin>     <origin rpy="0 0 0" xyz="0.017 0 0"/>                         </real_origin>
+      <inertia_origin>  <origin rpy="0 0 0" xyz="4.7601567e-03 -1.3786947e-03 0.0"/>  </inertia_origin>
+      <inertia ixx="1.8024201e-07" ixy="5.756798e-09" ixz="0.0" iyy="2.3516266e-07" iyz="0.0" izz="2.691504e-07"/>
+    </xacro:phalanx_generic>
     <!-- Distal -->
-    <xacro:phalanx_distal name="${name}_distal" parent="${name}_middle" side="$(arg side)" ns="$(arg ns)">
-      <origin rpy="0 0 0" xyz="0.009 0 0"/>
-    </xacro:phalanx_distal>
+    <xacro:phalanx_generic name="${name}_distal" parent="${name}_middle" ns="$(arg ns)" mass="0.009" mesh="ph_distal">
+      <virtual_origin>  <origin rpy="0 0 0" xyz="0.009 0 0"/>                        </virtual_origin>
+      <real_origin>     <origin rpy="0 0 0" xyz="0.013 0 0"/>                         </real_origin>
+      <inertia_origin>  <origin rpy="0 0 0" xyz="8.8025467e-03 -1.7219289e-03 0.0"/>  </inertia_origin>
+      <inertia ixx="2.6586142e-07" ixy="1.2416847e-08" ixz="0.0" iyy="5.9935767e-07" iyz="0.0" izz="6.6781963e-07"/>
+    </xacro:phalanx_generic>
   </xacro:macro>
 </robot>

File: softhands_description/urdf/xacro/include/macro/v1_2_research/modules/iso.xacro (robot description, xacro)
@@ -47,11 +47,7 @@
 		<link name="${ns}_${name}_link">
 			<inertial>
+				<mass value="0.205"/>
 				<origin rpy="0 0 0" xyz="0.0 7.8738498e-04 1.5878899e-02"/>
-				<!-- Original value -->
-				<!--<mass value="0.205"/>
-				<inertia ixx="0.00012506929" ixy="0.0" ixz="0.0" iyy="0.0001338779" iyz="0.0" izz="0.00019218394"/> -->
-				<!-- Old value -->
-				<mass value="0.205"/>
-				<inertia ixx="0.001" ixy="0" ixz="0" iyy="0.001" iyz="0" izz="0.001"/>
+				<inertia ixx="0.00012506929" ixy="0.0" ixz="0.0" iyy="0.0001338779" iyz="0.0" izz="0.00019218394"/>
 			</inertial>
 			<visual>

File: softhands_description/urdf/xacro/include/macro/v1_2_research/modules/palm/palm.xacro (robot description, xacro)
@@ -48,9 +48,9 @@
 				<origin rpy="0 0 0" xyz="0.0030 -0.0449 ${sign*0.0135}"/>
 				<!-- Original value -->
-				<!-- <mass value="0.45"/>
-				<inertia ixx="0.00045" ixy="0.0" ixz="0.0" iyy="0.00025" iyz="0.0" izz="0.0006"/> -->
+				<mass value="0.45"/>
+				<inertia ixx="0.00045" ixy="0.0" ixz="0.0" iyy="0.00025" iyz="0.0" izz="0.0006"/>
 				<!-- Old value -->
-				<mass value="2.28"/>
-				<inertia ixx="0.001" ixy="0" ixz="0" iyy="0.001" iyz="0" izz="0.001"/>
+				<!-- <mass value="2.28"/>
+				<inertia ixx="0.001" ixy="0" ixz="0" iyy="0.001" iyz="0" izz="0.001"/>  -->
 			</inertial>
 			<visual>
@@ -71,14 +71,4 @@
 			<material>Gazebo/Grey</material>
 			<selfCollide>$(arg selfCollide)</selfCollide>
-			<kp value="1e4" />
-			<kd value="1e2" />
-			<surface>
-			<friction>
-				<ode>
-				<mu>0.133</mu>
-				<mu2>0.133</mu2>
-				</ode>
-			</friction>
-			</surface>
 		</gazebo>
 	</xacro:macro>

File: softhands_description/urdf/xacro/include/macro/v1_2_research/modules/phalanges/phalanx_generic.xacro (robot description, xacro)
@@ -38,29 +38,48 @@
 -->
 <robot xmlns:xacro="http://www.ros.org/wiki/xacro">
-  <xacro:macro name="phalanx_knuckle" params="ns name parent *origin side">
-    <!-- Proximal JOINT -->
+  <xacro:macro name="phalanx_generic" params="name parent ns mass mesh **virtual_origin **real_origin **inertia_origin *inertia">
+    <!-- Inner VIRTUAL JOINT -->
+		<joint name="${ns}_${name}_virtual_joint" type="revolute">
+      <axis xyz="0 0 -1"/>
+      <xacro:insert_block name="virtual_origin"/>
+			<parent link="${ns}_${parent}_link"/>
+			<child link="${ns}_${name}_virtual_link"/>
+      <limit effort="30" velocity="10.0" lower="0.0" upper="0.785398" />
+      <dynamics damping="$(arg virtual_damping)" friction="$(arg virtual_friction)" />
+		</joint>
+    <!-- VIRTUAL LINK -->
+    <link name="${ns}_${name}_virtual_link">
+      <inertial>
+        <origin rpy="0 0 0" xyz="0 0 0"/>
+        <mass value="${mass}"/>
+        <xacro:insert_block name="inertia"/>
+      </inertial>
+      <visual>
+        <geometry>
+          <box size="0.001 0.001 0.001"/>
+        </geometry>
+        <origin xyz="0 0 0" rpy="0 0 0"/>
+      </visual>
+    </link>
+    <!-- Outer JOINT -->
     <joint name="${ns}_${name}_joint" type="revolute">
-      <xacro:insert_block name="origin"/>
-      <parent link="${ns}_${parent}_link"/>
+      <axis xyz="0 0 -1"/>
+      <xacro:insert_block name="real_origin"/>
+      <parent link="${ns}_${name}_virtual_link"/>
       <child link="${ns}_${name}_link"/>
-      <axis xyz="0 0 -1"/>
-      <limit effort="30" velocity="1.0" lower="-0.524" upper="0.524" />
-       <dynamics damping="$(arg damping)" friction="$(arg friction)"/>
+      <limit effort="30" velocity="10.0" lower="0.0" upper="0.785398" />
+      <dynamics damping="$(arg damping)" friction="$(arg friction)"/>
     </joint>
     <!-- LINK -->
     <link name="${ns}_${name}_link">
-      <inertial>
-        <origin rpy="0 0 0" xyz="4.2753603e-04  0.0 -1.4321738e-03"/>
-        <!-- Original value -->
-        <!-- <mass value="0.0095"/>
-        <inertia ixx="6.4337303e-07" ixy="0.0" ixz="-3.9373913e-08" iyy="1.1253771e-06" iyz="0.0" izz="7.2336948e-07"/> -->
-        <!-- Old value -->
-        <mass value="0.005"/>
-        <inertia ixx="0.001" ixy="0" ixz="0" iyy="0.001" iyz="0" izz="0.001"/>
-      </inertial>
+        <inertial>
+          <mass value="${mass}"/>
+          <xacro:insert_block name="inertia"/>
+          <xacro:insert_block name="inertia_origin"/>
+        </inertial>
       <visual>
         <origin rpy="0 0 0" xyz="0 0 0"/>
         <geometry>
-          <mesh filename="$(arg meshes_dir)/ph_knuckle.stl" scale="0.001 0.001 0.001"/>
+          <mesh filename="$(arg meshes_dir)/${mesh}.stl" scale="0.001 0.001 0.001"/>
         </geometry>
         <material name="qbhand/palm"/>
@@ -69,23 +88,25 @@
         <origin rpy="0 0 0" xyz="0 0 0"/>
         <geometry>
-          <mesh filename="$(arg meshes_dir)/ph_knuckle.stl" scale="0.001 0.001 0.001"/>
+          <mesh filename="$(arg meshes_dir)/${mesh}.stl" scale="0.001 0.001 0.001"/>
         </geometry>
       </collision>
     </link>
-        <!-- GAZEBO REF -->
+    <!-- GAZEBO REF -->
     <gazebo reference="${ns}_${name}_link">
       <material>Gazebo/Grey</material>
       <selfCollide>$(arg selfCollide)</selfCollide>
-            <kp value="1e4" />
-      <kd value="1e2" />
-      <surface>
-       <friction>
-        <ode>
-         <mu>0.133</mu>
-         <mu2>0.133</mu2>
-        </ode>
-       </friction>
-      </surface>
-    </gazebo>
+	  </gazebo>
+        <!-- GAZEBO REF -->
+    <gazebo reference="${ns}_${name}_joint">
+      <implicitSpringDamper>true</implicitSpringDamper>
+			<springStiffness>0.4</springStiffness>
+			<springReference>0</springReference>
+	  </gazebo>
+        <!-- GAZEBO REF -->
+    <gazebo reference="${ns}_${name}_virtual_joint">
+      <implicitSpringDamper>true</implicitSpringDamper>
+			<springStiffness>0.4</springStiffness>
+			<springReference>0</springReference>
+	  </gazebo>
   </xacro:macro>
 </robot>

File: softhands_description/urdf/xacro/include/macro/v1_2_research/modules/phalanges/phalanx_knuckle.xacro (robot description, xacro)
@@ -38,54 +38,29 @@
 -->
 <robot xmlns:xacro="http://www.ros.org/wiki/xacro">
-  <xacro:macro name="phalanx_short" params="ns name parent *origin side">
-    <!-- VIRTUAL JOINT -->
-		<joint name="${ns}_${name}_joint" type="revolute">
-      <axis xyz="0 0 -1"/>
+  <xacro:macro name="phalanx_knuckle" params="ns name parent *origin side">
+    <!-- Proximal JOINT -->
+    <joint name="${ns}_${name}_joint" type="revolute">
       <xacro:insert_block name="origin"/>
-			<parent link="${ns}_${parent}_link"/>
-			<child link="${ns}_${name}_virtual_link"/>
-      <limit effort="30" velocity="10" lower="0.0" upper="0.785"/>
-      <dynamics damping="$(arg virtual_damping)" friction="$(arg virtual_friction)"/>
-		</joint>
-    <!-- VIRTUAL LINK -->
-    <link name="${ns}_${name}_virtual_link">
-      <inertial>
-      <origin rpy="0 0 0" xyz="0 0 0"/>
-        <mass value="0.001"/>
-        <inertia  ixx="0.0001"      ixy="0"  	    ixz="0"
-                  iyy="0.0001" 	    iyz="0"
-        		      izz="0.0001" />
-      </inertial>
-	      <visual>
-        <geometry>
-          <cylinder length="0.005" radius="0.004"/>
-        </geometry>
-        <origin xyz="0 0 0" rpy="0 0 0"/>
-      </visual>
-    </link>
-    <!-- Proximal JOINT -->
-    <joint name="${ns}_${name}_virtual_joint" type="revolute">
-      <origin rpy="0 0 0" xyz="0.017 0 0"/>
-      <parent link="${ns}_${name}_virtual_link"/>
+      <parent link="${ns}_${parent}_link"/>
       <child link="${ns}_${name}_link"/>
       <axis xyz="0 0 -1"/>
-      <limit effort="30" velocity="1.0" lower="0.0" upper="0.785"/>
-      <dynamics damping="$(arg damping)" friction="$(arg friction)"/>
+      <limit effort="30" velocity="10.0" lower="-0.524" upper="0.524" />
+      <dynamics damping="$(arg damping)" friction="$(arg friction)" />
     </joint>
     <!-- LINK -->
     <link name="${ns}_${name}_link">
       <inertial>
-        <origin rpy="0 0 0" xyz="4.7601567e-03 -1.3786947e-03 0.0"/>
+        <origin rpy="0 0 0" xyz="4.2753603e-04  0.0 -1.4321738e-03"/>
         <!-- Original value -->
-        <!-- <mass value="0.0063"/>
-        <inertia ixx="1.8024201e-07" ixy="5.756798e-09" ixz="0.0" iyy="2.3516266e-07" iyz="0.0" izz="2.691504e-07"/> -->
+        <mass value="0.0095"/>
+        <inertia ixx="6.4337303e-07" ixy="0.0" ixz="-3.9373913e-08" iyy="1.1253771e-06" iyz="0.0" izz="7.2336948e-07"/>
         <!-- Old value -->
-        <mass value="0.005"/>
-        <inertia ixx="0.001" ixy="0" ixz="0" iyy="0.001" iyz="0" izz="0.001"/>
+        <!-- <mass value="0.005"/>
+        <inertia ixx="0.001" ixy="0" ixz="0" iyy="0.001" iyz="0" izz="0.001"/>  -->
       </inertial>
       <visual>
         <origin rpy="0 0 0" xyz="0 0 0"/>
         <geometry>
-          <mesh filename="$(arg meshes_dir)/ph_short.stl" scale="0.001 0.001 0.001"/>
+          <mesh filename="$(arg meshes_dir)/ph_knuckle.stl" scale="0.001 0.001 0.001"/>
         </geometry>
         <material name="qbhand/palm"/>
@@ -94,5 +69,5 @@
         <origin rpy="0 0 0" xyz="0 0 0"/>
         <geometry>
-          <mesh filename="$(arg meshes_dir)/ph_short.stl" scale="0.001 0.001 0.001"/>
+          <mesh filename="$(arg meshes_dir)/ph_knuckle.stl" scale="0.001 0.001 0.001"/>
         </geometry>
       </collision>
@@ -102,15 +77,11 @@
       <material>Gazebo/Grey</material>
       <selfCollide>$(arg selfCollide)</selfCollide>
-      <kp value="1e4" />
-      <kd value="1e2" />
-      <surface>
-       <friction>
-        <ode>
-         <mu>0.133</mu>
-         <mu2>0.133</mu2>
-        </ode>
-       </friction>
-      </surface>
     </gazebo>
+            <!-- GAZEBO REF -->
+    <gazebo reference="${ns}_${name}_joint">
+      <implicitSpringDamper>true</implicitSpringDamper>
+			<springStiffness>0.4</springStiffness>
+			<springReference>0</springReference>
+	  </gazebo>
   </xacro:macro>
 </robot>

File: softhands_description/urdf/xacro/include/macro/v1_2_research/modules/phalanges/thumb_knuckle.xacro (robot description, xacro)
@@ -38,61 +38,36 @@
 -->
 <robot xmlns:xacro="http://www.ros.org/wiki/xacro">
-  <xacro:macro name="phalanx_distal" params="ns name parent *origin side">
-    <!-- VIRTUAL JOINT -->
-		<joint name="${ns}_${name}_virtual_joint" type="revolute">
-      <axis xyz="0 0 -1"/>
-      <xacro:insert_block name="origin"/>
-			<parent link="${ns}_${parent}_link"/>
-			<child link="${ns}_${name}_virtual_link"/>
-      <limit effort="30" velocity="10" lower="0" upper="0.785398" />
-      <dynamics damping="$(arg virtual_damping)" friction="$(arg virtual_friction)"/>
-		</joint>
-    <!-- VIRTUAL LINK -->
-    <link name="${ns}_${name}_virtual_link">
-      <inertial>
-      <origin xyz="0 0 0" rpy="0 0 0"/>
-        <mass value="0.001"/>
-        <inertia  ixx="0.0001"      ixy="0"  	    ixz="0"
-                  iyy="0.0001" 	    iyz="0"
-        		      izz="0.0001" />
-      </inertial>
-      <visual>
-        <geometry>
-          <box size="0.001 0.001 0.001"/>
-        </geometry>
-        <origin xyz="0 0 0" rpy="0 0 0"/>
-      </visual>
-    </link>
+  <xacro:macro name="thumb_knuckle" params="ns name parent *origin side">
     <!-- Proximal JOINT -->
     <joint name="${ns}_${name}_joint" type="revolute">
-			<origin rpy="0 0 0" xyz="0.013 0 0"/>
-      <parent link="${ns}_${name}_virtual_link"/>
+      <xacro:insert_block name="origin"/>
+      <parent link="${ns}_${parent}_link"/>
       <child link="${ns}_${name}_link"/>
-      <axis xyz="0 0 -1"/>
-      <limit effort="30" velocity="1.0" lower="0" upper="0.785398" />
-       <dynamics damping="$(arg damping)" friction="$(arg friction)"/>
+      <axis xyz="0 0 ${sign*-1}"/>
+      <limit effort="30" velocity="10.0" lower="0.0" upper="1.57" />
+      <dynamics damping="$(arg damping)" friction="$(arg friction)" />
     </joint>
     <!-- LINK -->
     <link name="${ns}_${name}_link">
-        <inertial>
-          <origin rpy="0 0 0" xyz="8.8025467e-03 -1.7219289e-03 0.0"/>
-          <!-- Original value -->
-          <!-- <mass value="0.009"/>
-          <inertia ixx="2.6586142e-07" ixy="1.2416847e-08" ixz="0.0" iyy="5.9935767e-07" iyz="0.0" izz="6.6781963e-07"/> -->
-          <!-- Old value -->
-          <mass value="0.005"/>
-          <inertia ixx="0.001" ixy="0" ixz="0" iyy="0.001" iyz="0" izz="0.001"/>
-        </inertial>
+      <inertial>
+        <origin rpy="0 0 0" xyz="1.3071561e-02 ${sign*-2.7346340e-03} 6.4090487e-04"/>
+        <!-- Original value -->
+        <mass value="0.01"/>
+        <inertia ixx="3.5865978e-07" ixy="${sign*2.0944224e-07}" ixz="-6.8657569e-08" iyy="1.3885564e-06" iyz="${sign*3.2170608e-08}" izz="1.3571203e-06"/>
+        <!-- Old value -->
+        <!-- <mass value="0.005"/>
+        <inertia ixx="0.001" ixy="0" ixz="0" iyy="0.001" iyz="0" izz="0.001"/>  -->
+      </inertial>
       <visual>
         <origin rpy="0 0 0" xyz="0 0 0"/>
         <geometry>
-          <mesh filename="$(arg meshes_dir)/ph_distal.stl" scale="0.001 0.001 0.001"/>
+          <mesh filename="$(arg meshes_dir)/ph_thumb.stl" scale="0.001 0.001 0.001"/>
         </geometry>
-        <material name="qbhand/palm"/>
+        <material name="qbhand/knuckle"/>
       </visual>
       <collision>
         <origin rpy="0 0 0" xyz="0 0 0"/>
         <geometry>
-          <mesh filename="$(arg meshes_dir)/ph_distal.stl" scale="0.001 0.001 0.001"/>
+          <mesh filename="$(arg meshes_dir)/ph_thumb.stl" scale="0.001 0.001 0.001"/>
         </geometry>
       </collision>
@@ -102,14 +77,10 @@
       <material>Gazebo/Grey</material>
       <selfCollide>$(arg selfCollide)</selfCollide>
-      <kp value="1e4" />
-      <kd value="1e2" />
-      <surface>
-       <friction>
-        <ode>
-         <mu>0.133</mu>
-         <mu2>0.133</mu2>
-        </ode>
-       </friction>
-      </surface>
+    </gazebo>
+        <!-- GAZEBO REF -->
+    <gazebo reference="${ns}_${name}_joint">
+      <implicitSpringDamper>true</implicitSpringDamper>
+			<springStiffness>0.4</springStiffness>
+			<springReference>0</springReference>
 	  </gazebo>
   </xacro:macro>
