Commit message: reduced xacro file, added spring with joints and a real inertia on the virtual link

File: softhands_description/urdf/xacro/include/macro/v1_2_research/modules/thumb.xacro (robot description, xacro)
@@ -44,16 +44,22 @@
     </xacro:thumb_knuckle>
     <!-- Proximal  -->
-    <xacro:thumb_short name="${name}_proximal" parent="${name}_knuckle" ns="$(arg ns)" side="$(arg side)">
+    <xacro:phalanx_generic name="${name}_proximal" parent="${name}_knuckle" ns="$(arg ns)" mass="0.0063" mesh="ph_short">
       <xacro:if value="${side == 'left'}">
-        <origin rpy="-2 0.0 0.0" xyz="0.0255 0.0038 -0.00012"/>
+         <virtual_origin> <origin rpy="-2 0.0 0.0" xyz="0.0255 0.0038 -0.00012"/></virtual_origin>
       </xacro:if>
       <xacro:if value="${side == 'right'}">
-        <origin rpy="-1.1415 0.0 0.0" xyz="0.0255 -0.0038 -0.00012"/>
+         <virtual_origin> <origin rpy="-1.1415 0.0 0.0" xyz="0.0255 -0.0038 -0.00012"/></virtual_origin>
       </xacro:if>
-    </xacro:thumb_short>
+      <real_origin>     <origin rpy="0 0 0" xyz="0.013 0 0"/>                         </real_origin>
+      <inertia_origin>  <origin rpy="0 0 0" xyz="4.7601567e-03 -1.3786947e-03 0.0"/>  </inertia_origin>
+      <inertia ixx="1.8024201e-07" ixy="5.756798e-09" ixz="0.0" iyy="2.3516266e-07" iyz="0.0" izz="2.691504e-07"/>
+    </xacro:phalanx_generic>
     <!-- Distal  -->
-    <xacro:phalanx_distal name="${name}_distal" parent="${name}_proximal" ns="$(arg ns)" side="$(arg side)">
-      <origin rpy="0 0 0" xyz="0.009 0 0"/>
-    </xacro:phalanx_distal>
+    <xacro:phalanx_generic name="${name}_distal" parent="${name}_proximal" ns="$(arg ns)" mass="0.009" mesh="ph_distal">
+      <virtual_origin>  <origin rpy="0 0 0" xyz="0.009 0 0"/>                        </virtual_origin>
+      <real_origin>     <origin rpy="0 0 0" xyz="0.013 0 0"/>                         </real_origin>
+      <inertia_origin>  <origin rpy="0 0 0" xyz="8.8025467e-03 -1.7219289e-03 0.0"/>  </inertia_origin>
+      <inertia ixx="2.6586142e-07" ixy="1.2416847e-08" ixz="0.0" iyy="5.9935767e-07" iyz="0.0" izz="6.6781963e-07"/>
+    </xacro:phalanx_generic>
   </xacro:macro>
 </robot>

File: softhands_description/urdf/xacro/include/macro/v1_wide/modules/finger/phalanx.xacro (robot description, xacro)
@@ -5,5 +5,5 @@
 		<joint name="${ns}_${name}_virtual_joint" type="revolute">
 			<axis xyz="0 0 1"/>
-			<limit effort="30" velocity="1.0" lower="0" upper="0.785398" />
+			<limit effort="30" velocity="0.0" lower="0" upper="0.785398" />
 			<xacro:insert_block name="origin"/>
 			<parent link="${ns}_${parent}_link"/>
@@ -21,5 +21,5 @@
 		<joint name="${ns}_${name}_joint" type="revolute">
 			<axis xyz="0 0 1"/>
-			<limit effort="30" velocity="1.0" lower="0" upper="0.785398" />
+			<limit effort="30" velocity="0.0" lower="0" upper="0.785398" />
 			<origin rpy="0 0 0" xyz="9e-3 0 0"/>
             <parent link="${ns}_${name}_virtual_link"/>

File: softhands_description/urdf/xacro/include/macro/v1_wide/modules/finger/phalanx_dist.xacro (robot description, xacro)
@@ -5,5 +5,5 @@
 		<joint name="${ns}_${name}_virtual_joint" type="revolute">
 			<axis xyz="0 0 1"/>
-			<limit effort="30" velocity="1.0" lower="0" upper="0.785398" />
+			<limit effort="30" velocity="0.0" lower="0" upper="0.785398" />
 			<xacro:insert_block name="origin"/>
 			<parent link="${ns}_${parent}_link"/>
@@ -21,5 +21,5 @@
 		<joint name="${ns}_${name}_joint" type="revolute">
 			<axis xyz="0 0 1"/>
-			<limit effort="30" velocity="1.0" lower="0" upper="0.785398" />
+			<limit effort="30" velocity="0.0" lower="0" upper="0.785398" />
 			<origin rpy="0 0 0" xyz="9e-3 0 0"/>
             <parent link="${ns}_${name}_virtual_link"/>

File: softhands_description/urdf/xacro/include/macro/v1_wide/modules/finger/phalanx_knuckle.xacro (robot description, xacro)
@@ -5,5 +5,5 @@
 		<joint name="${ns}_${name}_joint" type="revolute">
 			<axis xyz="0 1 0"/>
-			<limit effort="30" velocity="1.0" lower="0.0" upper="0.0" />
+			<limit effort="30" velocity="0.0" lower="0.0" upper="0.0" />
 			<xacro:insert_block name="origin"/>
             <parent link="${ns}_${parent}_link"/>

File: softhands_description/urdf/xacro/include/macro/v1_wide/modules/palm/palm_central.xacro (robot description, xacro)
@@ -40,5 +40,5 @@
 		<joint name="${ns}_${name}_thumb_joint" type="revolute">
 			<axis xyz="0 0 -1"/>
-			<limit effort="30" velocity="10" lower="0" upper="1.57" />
+			<limit effort="30" velocity="0.0" lower="0" upper="1.57" />
 			<dynamics damping="$(arg virtual_damping)" friction="$(arg virtual_friction)"/>
 			<origin xyz=" -0.0000000021 32.5059e-3 39.6398e-3" rpy="0 0.3490656 1.5707963"/>
@@ -59,5 +59,5 @@
 			<axis xyz="0 0 1"/>
 			<dynamics damping="$(arg virtual_damping)" friction="$(arg virtual_friction)"/>
-			<limit effort="100" lower="0.0" upper="0.4" velocity="100"/>
+			<limit effort="100" lower="0.0" upper="0.4" velocity="0.00"/>
 			<origin xyz=" -0.0000000091 -10.6603e-3 66.1817e-3" rpy="0 -0.1745327 -1.5707963"/>
 			<parent link="${ns}_${name}_link"/>

File: softhands_description/urdf/xacro/include/macro/v1_wide/modules/palm/palm_little.xacro (robot description, xacro)
@@ -7,5 +7,5 @@
 			<xacro:insert_block name="origin"/>
 			<axis xyz="0 0 1" />
-      		<limit effort="30" velocity="1.0" lower="0" upper="0.3" />
+      		<limit effort="30" velocity="0.0" lower="0" upper="0.3" />
 			<dynamics damping="$(arg virtual_damping)" friction="$(arg virtual_friction)"/>
 		</joint>

File: softhands_description/urdf/xacro/include/macro/v1_wide/modules/palm/palm_thumb.xacro (robot description, xacro)
@@ -7,5 +7,5 @@
 			<xacro:insert_block name="origin"/>
 			<axis xyz="0 0 -1" />
-      		<limit effort="30" velocity="1.0" lower="0" upper="1.57" />
+      		<limit effort="30" velocity="0.0" lower="0" upper="1.57" />
 			<dynamics damping="$(arg virtual_damping)" friction="$(arg virtual_friction)"/>
 		</joint>

File: softhands_description/urdf/xacro/include/macro/v1_wide/modules/thumb/thumb_distal.xacro (robot description, xacro)
@@ -8,5 +8,5 @@
 			<parent link="${ns}_${parent}_link"/>
 			<child link="${ns}_${name}_virtual_link"/>
-			<limit effort="30" velocity="10" lower="0" upper="0.785398" />
+			<limit effort="30" velocity="0.0" lower="0" upper="0.785398" />
 			<dynamics damping="$(arg virtual_damping)" friction="$(arg virtual_friction)"/>
 		</joint>
@@ -24,5 +24,5 @@
 			<origin rpy="0 0.0101229 0" xyz="8.99947e-3 0 -0.0973875e-3"/>
 			<axis xyz="0 0 1" />
-      		<limit effort="30" velocity="1.0" lower="0" upper="0.785398" />
+      		<limit effort="30" velocity="0.0" lower="0" upper="0.785398" />
 			<dynamics damping="$(arg damping)" friction="$(arg friction)"/>
 		</joint>

File: softhands_description/urdf/xacro/include/macro/v1_wide/modules/thumb/thumb_knuckle.xacro (robot description, xacro)
@@ -8,5 +8,5 @@
 			<xacro:insert_block name="origin"/>
 			<axis xyz="0 0 1" />
-      		<limit effort="30" velocity="1.0" lower="0" upper="1.57" />
+      		<limit effort="30" velocity="0.0" lower="0" upper="1.57" />
 			<dynamics damping="$(arg damping)" friction="$(arg friction)"/>
 		</joint>

File: softhands_description/urdf/xacro/include/macro/v1_wide/modules/thumb/thumb_proximal.xacro (robot description, xacro)
@@ -5,5 +5,5 @@
 		<joint name="${ns}_${name}_joint" type="revolute">
 			<axis xyz="0 0 1"/>
-			<limit effort="30" velocity="10" lower="0" upper="0.785398" />
+			<limit effort="30" velocity="0.0" lower="0" upper="0.785398" />
 			<xacro:insert_block name="origin"/>
 			<parent link="${ns}_${parent}_link"/>
@@ -24,5 +24,5 @@
 			<origin rpy="0 0 0"  xyz="9e-3 0 0 "/>
 			<axis xyz="0 0 1" />
-      		<limit effort="30" velocity="1.0" lower="0" upper="0.785398" />
+      		<limit effort="30" velocity="0.0" lower="0" upper="0.785398" />
 			<dynamics damping="$(arg damping)" friction="$(arg friction)"/>
 		</joint>

File: softhands_description/urdf/xacro/v1_2_research.xacro (robot description, xacro)
@@ -44,6 +44,6 @@
 	</xacro:if>
 	<!-- World -->
-	<link name="$(arg root_link)">
-	</link>
+	<!-- <link name="$(arg root_link)">
+	</link> -->
 	<!-- # iso -->
 	<xacro:iso name="iso" parent="$(arg root_link)" ns="$(arg ns)">

Commit message: update meshes

File: softhands_description/urdf/softhands.xacro (robot description, xacro)
@@ -73,5 +73,5 @@
 				side="left"
 				parent="world"
-				position="0 -0.2 0"
+				position="0 -0.2 0.02"
 				orientation="${orientation}"
 				fixed_hands="false">
@@ -80,5 +80,5 @@
 				side="right"
 				parent="world"
-				position="0 0.2 0"
+				position="0 0.2 0.02"
 				orientation="${orientation}"
 				fixed_hands="false">

File: softhands_description/urdf/xacro/include/macro/v1_wide/modules/finger/phalanx_dist.xacro (robot description, xacro)
@@ -45,5 +45,5 @@
 					<geometry>
 					<mesh
-						filename="package://softhands_description/meshes/v1_wide/${side}/phalanx_dist.stl"
+						filename="package://softhands_description/meshes/v1_wide/${side}/phalanx_dist_collision.stl"
 						scale="0.0009 0.0009 0.0009" />
 					</geometry>

File: softhands_description/urdf/xacro/include/macro/v1_wide/modules/finger/phalanx_knuckle.xacro (robot description, xacro)
@@ -28,5 +28,5 @@
 					<mesh
 						filename="package://softhands_description/meshes/v1_wide/${side}/phalanx_pros_sup_collision.stl"
-						scale="0.001 0.001 0.001" />
+						scale="0.0009 0.0009 0.0009" />
 					</geometry>
 				<origin xyz="0 0 0" rpy="0 0 0" />
@@ -34,5 +34,5 @@
 		</link>
 		<gazebo reference="${ns}_${name}_link">
-			<selfCollide>$(arg selfCollide)</selfCollide>
+			<selfCollide>0</selfCollide>
 			<material>Gazebo/White</material>
 		</gazebo>

File: softhands_description/urdf/xacro/include/macro/v1_wide/modules/palm/palm_central.xacro (robot description, xacro)
@@ -27,5 +27,5 @@
 				<mesh
 					filename="package://softhands_description/meshes/v1_wide/${side}/palm_central_collision.stl"
-					scale="0.001 0.001 0.001" />
+					scale="0.0009 0.0009 0.0009" />
 				</geometry>
 			<origin xyz="0 0 0" rpy="0 0 0" />
@@ -44,5 +44,5 @@
 		   <inertial>
 				<origin rpy="0 0 0" xyz="0 0 0"/>
-				<mass value="${mass}"/>
+				<mass value="0.001"/>
 				<xacro:insert_block name="inertia"/>
 		   </inertial>
@@ -60,10 +60,10 @@
 			<inertial>
 				<origin rpy="0 0 0" xyz="0 0 0"/>
-				<mass value="${mass}"/>
+				<mass value="0.001"/>
 				<xacro:insert_block name="inertia"/>
 			</inertial>
 	    </link>
 		<gazebo reference="${ns}_${name}_link">
-			<selfCollide>$(arg selfCollide)</selfCollide>
+			<selfCollide>0</selfCollide>
 			<material>Gazebo/Grey</material>
 		</gazebo>

File: softhands_description/urdf/xacro/include/macro/v1_wide/modules/palm/palm_little.xacro (robot description, xacro)
@@ -29,5 +29,5 @@
 					<mesh
 						filename="package://softhands_description/meshes/v1_wide/${side}/palm_little_collision.stl"
-						scale="0.001 0.001 0.001" />
+						scale="0.0009 0.0009 0.0009" />
 					</geometry>
 				<origin xyz="0 0 0" rpy="0 0 0" />
@@ -35,5 +35,5 @@
 		</link>
 		<gazebo reference="${ns}_${name}_link">
-			<selfCollide>$(arg selfCollide)</selfCollide>
+			<selfCollide>0</selfCollide>
 			<material>Gazebo/Grey</material>
 		</gazebo>

File: softhands_description/urdf/xacro/include/macro/v1_wide/modules/palm/palm_thumb.xacro (robot description, xacro)
@@ -59,5 +59,5 @@
 					<mesh
 						filename="package://softhands_description/meshes/v1_wide/${side}/thumb_support_collision.stl"
-						scale="0.001 0.001 0.001" />
+						scale="0.0009 0.0009 0.0009" />
 					</geometry>
 				<origin xyz="0 0 0" rpy="0 0 0" />
@@ -65,9 +65,9 @@
 		</link>
 		<gazebo reference="${ns}_${name}_link">
-			<selfCollide>$(arg selfCollide)</selfCollide>
+			<selfCollide>0</selfCollide>
 			<material>Gazebo/Grey</material>
 		</gazebo>
 		<gazebo reference="${ns}_${name}_support_link">
-			<selfCollide>$(arg selfCollide)</selfCollide>
+			<selfCollide>0</selfCollide>
 			<material>Gazebo/White</material>
 		</gazebo>

File: softhands_description/urdf/xacro/include/macro/v1_wide/modules/thumb/thumb_knuckle.xacro (robot description, xacro)
@@ -37,5 +37,5 @@
 		<gazebo reference="${ns}_${name}_link">
 			<material>Gazebo/Grey</material>
-			<selfCollide>$(arg selfCollide)</selfCollide>
+			<selfCollide>0</selfCollide>
 		</gazebo>
 				        <!-- GAZEBO REF -->

File: softhands_description/urdf/xacro/v1_wide.xacro (robot description, xacro)
@@ -43,5 +43,5 @@
 		<xacro:arg name="virtual_damping" 	default="3e-2"/>
 		<xacro:arg name="damping" 			default="3e-2"/>
-		<xacro:arg name="selfCollide" 		default="0"/>
+		<xacro:arg name="selfCollide" 		default="1"/>
 		<!-- <xacro:property name="side" value="${side}"/> -->
 		<xacro:property name="sign" default="1"/>
@@ -49,5 +49,5 @@
 			<xacro:property name="sign" value="-1"/>
 		</xacro:if>
-    	<!-- <xacro:softhand_mimic_plugin ns="${side}_hand_v1_wide" wide="true"/> -->
+    	<xacro:softhand_mimic_plugin ns="${side}_hand_v1_wide" wide="true"/>
 		<!-- # palm central -->
 		<xacro:palm_central name="palm_central" parent="${parent}" side="${side}" ns="${side}_hand_v1_wide"  mass="5.5962922e-1">

Commit message: fixed hands for spawining

File: softhands_description/urdf/softhands.xacro (robot description, xacro)
@@ -46,5 +46,5 @@
 		<xacro:include filename="$(find softhands_description)/urdf/xacro/include/macro/plugin.xacro"/>
 		<!-- If you are using only the hand -->
-		<link name="world"/>
+		<!-- <link name="world"/> -->
 		<!-- IF VERSION == 1_2_Research -->
 		<xacro:if value="${version == 'v1_2_research'}">
@@ -53,14 +53,14 @@
 			<xacro:v1_2_research
 				side="left"
-				parent="world"
-				position="0 -0.2 0.02"
-				orientation="0 0 -1.57"
+				parent="arm_1_7"
+				position="0 -0. 0.00"
+				orientation="0 0 ${orientation}"
 				fixed_hands="false">
 			</xacro:v1_2_research>
 			<xacro:v1_2_research
 				side="right"
-				parent="world"
-				position="0 0.2 0.02"
-				orientation="0 0 -1.57"
+				parent="arm_2_7"
+				position="0 0.0 0.00"
+				orientation="0 0 ${orientation}"
 				fixed_hands="false">
 			</xacro:v1_2_research>
@@ -72,14 +72,14 @@
 			<xacro:v1_wide
 				side="left"
-				parent="world"
-				position="0 -0.2 0.02"
-				orientation="${orientation}"
+				parent="arm_1_7"
+				position="0 -0.0 0.00"
+				orientation="0 0 ${orientation}"
 				fixed_hands="false">
 			</xacro:v1_wide>
 			<xacro:v1_wide
 				side="right"
-				parent="world"
-				position="0 0.2 0.02"
-				orientation="${orientation}"
+				parent="arm_2_7"
+				position="0 0.0 0.0"
+				orientation="0 0 ${orientation}"
 				fixed_hands="false">
 			</xacro:v1_wide>
