Commit message: added mixed hands and changed the grasp link

File: softhands_description/urdf/softhands.xacro (robot description, xacro)
@@ -51,6 +51,6 @@
 				parent="arm_1_7"
 				position="0 -0. 0.00"
-				orientation="0 0 ${orientation}"
-				fixed_hands="false">
+				orientation="0 0 0"
+				fixed_hands="${fixed_hands}">
 			</xacro:v1_2_research>
 			<xacro:v1_2_research
@@ -58,6 +58,6 @@
 				parent="arm_2_7"
 				position="0 0.0 0.00"
-				orientation="0 0 ${orientation}"
-				fixed_hands="false">
+				orientation="0 0 3.14"
+				fixed_hands="${fixed_hands}">
 			</xacro:v1_2_research>
 		</xacro:if>
@@ -70,5 +70,5 @@
 				parent="arm_1_7"
 				position="0 0 0.0"
-				orientation="0 0 ${-orientation}"
+				orientation="0 0 0"
 				fixed_hands="false">
 			</xacro:v1_wide>
@@ -77,8 +77,29 @@
 				parent="arm_2_7"
 				position="0 0 0.0"
-				orientation="0 0 ${orientation}"
+				orientation="0 0 3.14"
 				fixed_hands="false">
 			</xacro:v1_wide>
 		</xacro:if>
+				<!-- IF VERSION == 1_wide -->
+		<xacro:if value="${version == 'mixed_hands'}">
+			<xacro:include filename="$(find softhands_description)/urdf/xacro/include/macro/v1_wide/header.xacro"/>
+			<xacro:include filename="$(find softhands_description)/urdf/xacro/v1_wide.xacro"/>
+			<xacro:include filename="$(find softhands_description)/urdf/xacro/include/macro/v1_2_research/header.xacro"/>
+			<xacro:include filename="$(find softhands_description)/urdf/xacro/v1_2_research.xacro"/>
+			<xacro:v1_wide
+				side="left"
+				parent="arm_1_7"
+				position="0 0 0.0"
+				orientation="0 0 ${orientation}"
+				fixed_hands="${fixed_hands}">
+			</xacro:v1_wide>
+			<xacro:v1_2_research
+				side="right"
+				parent="arm_2_7"
+				position="0 0.0 0.00"
+				orientation="0 0 3.14"
+				fixed_hands="${fixed_hands}">
+			</xacro:v1_2_research>
+		</xacro:if>
 	</xacro:macro>
 </robot>

File: softhands_description/urdf/xacro/include/macro/v1_2_research/modules/iso.xacro (robot description, xacro)
@@ -71,5 +71,5 @@
 		<!-- Fake joint and link for grasping -->
 	  	<joint name="${ns}_grasp_joint" type="fixed">
-			<origin rpy="0 0 1.57" xyz="0.03 0.06 0.10"/>
+			<origin rpy="0 0 1.57" xyz="-0.06 0.03 0.16"/>
 			<parent link="${ns}_${name}_link" />
 			<child link="${ns}_grasp_link" />

File: softhands_description/urdf/xacro/include/macro/v1_2_research/modules/phalanges/phalanx_generic.xacro (robot description, xacro)
@@ -40,5 +40,5 @@
   <xacro:macro name="phalanx_generic" params="name parent ns mass mesh **virtual_origin **real_origin **inertia_origin *inertia">
     <!-- Inner VIRTUAL JOINT -->
-		<joint name="${ns}_${name}_virtual_joint" type="revolute">
+		<joint name="${ns}_${name}_virtual_joint" type="${joint_type}">
       <axis xyz="0 0 -1"/>
       <xacro:insert_block name="virtual_origin"/>
@@ -57,5 +57,5 @@
     </link>
     <!-- Outer JOINT -->
-    <joint name="${ns}_${name}_joint" type="revolute">
+    <joint name="${ns}_${name}_joint" type="${joint_type}">
       <axis xyz="0 0 -1"/>
       <xacro:insert_block name="real_origin"/>

File: softhands_description/urdf/xacro/include/macro/v1_2_research/modules/phalanges/phalanx_knuckle.xacro (robot description, xacro)
@@ -40,5 +40,5 @@
   <xacro:macro name="phalanx_knuckle" params="ns name parent *origin side">
     <!-- Proximal JOINT -->
-    <joint name="${ns}_${name}_joint" type="revolute">
+    <joint name="${ns}_${name}_joint" type="${joint_type}">
       <xacro:insert_block name="origin"/>
       <parent link="${ns}_${parent}_link"/>

File: softhands_description/urdf/xacro/include/macro/v1_2_research/modules/phalanges/thumb_knuckle.xacro (robot description, xacro)
@@ -40,5 +40,5 @@
   <xacro:macro name="thumb_knuckle" params="ns name parent *origin side">
     <!-- Proximal JOINT -->
-    <joint name="${ns}_${name}_joint" type="revolute">
+    <joint name="${ns}_${name}_joint" type="${joint_type}">
       <xacro:insert_block name="origin"/>
       <parent link="${ns}_${parent}_link"/>

File: softhands_description/urdf/xacro/include/macro/v1_wide/modules/finger.xacro (robot description, xacro)
@@ -1,11 +1,11 @@
 <?xml version="1.0"?>
 <robot xmlns:xacro="http://www.ros.org/wiki/xacro">
-    <xacro:macro name="finger" params="name parent side *origin ns">
+    <xacro:macro name="wide_finger" params="name parent side *origin ns">
       <!-- Proximal Support -->
-      <xacro:phalanx_knuckle name="${name}_knuckle" parent="${parent}" side="${side}" ns="${ns}">
+      <xacro:wide_phalanx_knuckle name="${name}_knuckle" parent="${parent}" side="${side}" ns="${ns}">
         <xacro:insert_block name="origin"/>
-      </xacro:phalanx_knuckle>
+      </xacro:wide_phalanx_knuckle>
       <!-- Proximal -->
-      <xacro:phalanx name="${name}_proximal" parent="${name}_knuckle" side="${side}" ns="${ns}" mass="2.4190505e-02">
+      <xacro:wide_phalanx name="${name}_proximal" parent="${name}_knuckle" side="${side}" ns="${ns}" mass="2.4190505e-02">
         <xacro:if value="${side == 'left'}">
           <origin rpy="-1.5707963 -1.5707963 0" xyz=" -6.5e-3 0 24e-3" />
@@ -16,17 +16,17 @@
         <inertia_origin> <origin rpy="0 0 0" xyz=" 2.0923634e-02  8.4162795e-04 -5.2131884e-05"/> </inertia_origin>
         <inertia ixx="1.9981795e-06" ixy="-6.0806048e-08" ixz="0.0" iyy="4.7810654e-06" iyz="0.0" izz="5.0961924e-06"/>
-      </xacro:phalanx >
+      </xacro:wide_phalanx >
       <!-- Middle -->
-      <xacro:phalanx name="${name}_middle" parent="${name}_proximal" side="${side}" ns="${ns}"  mass="2.4190505e-02">
+      <xacro:wide_phalanx name="${name}_middle" parent="${name}_proximal" side="${side}" ns="${ns}"  mass="2.4190505e-02">
         <origin rpy="0 0 0" xyz="41e-3 0 0" />
         <inertia_origin> <origin rpy="0 0 0" xyz=" 2.0923634e-02  8.4162795e-04 -5.2131884e-05"/> </inertia_origin>
         <inertia ixx="1.9981795e-06" ixy="-6.0806048e-08" ixz="0.0" iyy="4.7810654e-06" iyz="0.0" izz="5.0961924e-06"/>
-      </xacro:phalanx>
+      </xacro:wide_phalanx>
       <!-- Distal -->
-      <xacro:phalanx_dist name="${name}_distal" parent="${name}_middle" side="${side}" ns="${ns}" mass="1.2475845e-02">
+      <xacro:wide_phalanx_dist name="${name}_distal" parent="${name}_middle" side="${side}" ns="${ns}" mass="1.2475845e-02">
         <origin xyz="41e-3 0 0" rpy="0 0 0"/>
         <inertia_origin><origin rpy="0 0 0" xyz="1.2887396e-02 6.2001804e-05 -1.1041989e-03"/></inertia_origin>
         <inertia ixx="7.5548908e-07" ixy="0.0" ixz="0.0" iyy="1.2532982e-06" iyz="0.0" izz="1.3218760e-06"/>
-      </xacro:phalanx_dist>
+      </xacro:wide_phalanx_dist>
     </xacro:macro>
 </robot>

File: softhands_description/urdf/xacro/include/macro/v1_wide/modules/finger/phalanx.xacro (robot description, xacro)
@@ -1,7 +1,7 @@
 <?xml version="1.0"?>
 <robot xmlns:xacro="http://www.ros.org/wiki/xacro">
-    <xacro:macro name="phalanx" params="name parent ns *origin side mass **inertia_origin *inertia">
+    <xacro:macro name="wide_phalanx" params="name parent ns *origin side mass **inertia_origin *inertia">
 		<!-- Virtual joint from knuckle->proximal or proximal->middle   -->
-		<joint name="${ns}_${name}_virtual_joint" type="revolute">
+		<joint name="${ns}_${name}_virtual_joint" type="${joint_type}">
 			<axis xyz="0 0 1"/>
 			<limit effort="30" velocity="0.0" lower="0" upper="0.785398" />
@@ -19,5 +19,5 @@
 	    </link>
 		<!-- Proximal phalanx -->
-		<joint name="${ns}_${name}_joint" type="revolute">
+		<joint name="${ns}_${name}_joint" type="${joint_type}">
 			<axis xyz="0 0 1"/>
 			<limit effort="30" velocity="0.0" lower="0" upper="0.785398" />

File: softhands_description/urdf/xacro/include/macro/v1_wide/modules/finger/phalanx_dist.xacro (robot description, xacro)
@@ -1,7 +1,7 @@
 <?xml version="1.0"?>
 <robot xmlns:xacro="http://www.ros.org/wiki/xacro">
-    <xacro:macro name="phalanx_dist" params="name parent side *origin ns mass **inertia_origin *inertia">
+    <xacro:macro name="wide_phalanx_dist" params="name parent side *origin ns mass **inertia_origin *inertia">
 		<!-- Virtual joint from middle->distal   -->
-		<joint name="${ns}_${name}_virtual_joint" type="revolute">
+		<joint name="${ns}_${name}_virtual_joint" type="${joint_type}">
 			<axis xyz="0 0 1"/>
 			<limit effort="30" velocity="0.0" lower="0" upper="0.785398" />
@@ -19,5 +19,5 @@
 	    </link>
 		<!-- Proximal phalanx -->
-		<joint name="${ns}_${name}_joint" type="revolute">
+		<joint name="${ns}_${name}_joint" type="${joint_type}">
 			<axis xyz="0 0 1"/>
 			<limit effort="30" velocity="0.0" lower="0" upper="0.785398" />

File: softhands_description/urdf/xacro/include/macro/v1_wide/modules/finger/phalanx_knuckle.xacro (robot description, xacro)
@@ -1,7 +1,7 @@
 <?xml version="1.0"?>
 <robot xmlns:xacro="http://www.ros.org/wiki/xacro">
-    <xacro:macro name="phalanx_knuckle" params="name parent side *origin ns">
+    <xacro:macro name="wide_phalanx_knuckle" params="name parent side *origin ns">
 		<!-- Support -->
-		<joint name="${ns}_${name}_joint" type="revolute">
+		<joint name="${ns}_${name}_joint" type="${joint_type}">
 			<axis xyz="0 1 0"/>
 			<limit effort="30" velocity="0.0" lower="0.0" upper="0.01" />

File: softhands_description/urdf/xacro/include/macro/v1_wide/modules/palm/palm_central.xacro (robot description, xacro)
@@ -35,5 +35,5 @@
 		<!-- Fake joint and link for grasping -->
 	  	<joint name="${ns}_grasp_joint" type="fixed">
-			<origin rpy="0 0 0" xyz="0.03 -0.06 0.10"/>
+			<origin rpy="0 0 0" xyz="0.03 -0.09 0.10"/>
 			<parent link="${ns}_${name}_link" />
 			<child link="${ns}_grasp_link" />
@@ -41,5 +41,5 @@
 		<link name="${ns}_grasp_link"/>
 		<!-- palm base to Thumb -->
-		<joint name="${ns}_${name}_thumb_joint" type="revolute">
+		<joint name="${ns}_${name}_thumb_joint" type="${joint_type}">
 			<axis xyz="0 0 ${sign*-1}"/>
 			<limit effort="30" velocity="0.0" lower="0" upper="0.17" />
@@ -57,5 +57,5 @@
 	    </link>
 		<!-- palm base to Litte virtual -->
-		<joint name="${ns}_${name}_little_joint" type="revolute">
+		<joint name="${ns}_${name}_little_joint" type="${joint_type}">
 			<axis xyz="0 0 1"/>
 			<dynamics damping="$(arg virtual_damping)" friction="$(arg virtual_friction)"/>

File: softhands_description/urdf/xacro/include/macro/v1_wide/modules/palm/palm_little.xacro (robot description, xacro)
@@ -2,5 +2,5 @@
 <robot xmlns:xacro="http://www.ros.org/wiki/xacro">
     <xacro:macro name="palm_little" params="name parent side ns mass *origin **inertia_origin *inertia ">
-		<joint name="${ns}_${parent}_virtual_joint" type="revolute">
+		<joint name="${ns}_${parent}_virtual_joint" type="${joint_type}">
 			<parent link="${ns}_${parent}_link"/>
 			<child link="${ns}_${name}_link"/>

File: softhands_description/urdf/xacro/include/macro/v1_wide/modules/palm/palm_thumb.xacro (robot description, xacro)
@@ -2,5 +2,5 @@
 <robot xmlns:xacro="http://www.ros.org/wiki/xacro">
     <xacro:macro name="palm_thumb" params="name parent side ns mass  **inertia_origin *inertia **palm_thumb_origin **thumb_support_origin">
-		<joint name="${ns}_${parent}_virtual_joint" type="revolute">
+		<joint name="${ns}_${parent}_virtual_joint" type="${joint_type}">
 			<parent link="${ns}_${parent}_link"/>
 			<child link="${ns}_${name}_link"/>

File: softhands_description/urdf/xacro/include/macro/v1_wide/modules/thumb.xacro (robot description, xacro)
@@ -1,21 +1,21 @@
 <?xml version="1.0"?>
 <robot xmlns:xacro="http://www.ros.org/wiki/xacro">
-    <xacro:macro name="thumb" params="name parent side *origin ns">
+    <xacro:macro name="wide_thumb" params="name parent side *origin ns">
       <!-- Proximal -->
-      <xacro:thumb_knuckle name="${name}_knuckle" parent="${parent}" side="${side}"  ns="${ns}">
+      <xacro:wide_thumb_knuckle name="${name}_knuckle" parent="${parent}" side="${side}"  ns="${ns}">
         <xacro:insert_block name="origin"/>
-      </xacro:thumb_knuckle>
+      </xacro:wide_thumb_knuckle>
       <!-- Middle -->
-      <xacro:thumb_proximal name="${name}_proximal" parent="${name}_knuckle" side="${side}" ns="${ns}" mass="3.3679189e-02">
+      <xacro:wide_thumb_proximal name="${name}_proximal" parent="${name}_knuckle" side="${side}" ns="${ns}" mass="3.3679189e-02">
         <origin rpy="${sign*-1.3962638} 0 0" xyz="38.5e-3 4.82952e-3 ${sign*-0.167417e-3}"/>
         <inertia_origin> <origin rpy="0 0 0" xyz="2.0950700e-02  1.1175133e-03 -3.7424390e-05"/> </inertia_origin>
         <inertia ixx="4.1328993e-06" ixy="-8.6599874e-08" ixz="0.0" iyy="7.4560101e-06" iyz="-1.0265429e-09" izz="6.6161853e-06"/>
-      </xacro:thumb_proximal>
+      </xacro:wide_thumb_proximal>
       <!-- Distal -->
-      <xacro:thumb_distal name="${name}_distal" parent="${name}_proximal" side="${side}" ns="${ns}" mass="2.3674554e-02">
+      <xacro:wide_thumb_distal name="${name}_distal" parent="${name}_proximal" side="${side}" ns="${ns}" mass="2.3674554e-02">
         <origin  rpy="0 0 0" xyz="41e-3 0 0"/>
         <inertia_origin> <origin rpy="0 0 0" xyz="1.6161362e-02  1.6241404e-03 -3.2684152e-05 "/> </inertia_origin>
         <inertia ixx="2.578454e-06" ixy="0.0" ixz="0.0" iyy="2.9887569e-06" iyz="0.0" izz="3.8277106e-06"/>
-      </xacro:thumb_distal>
+      </xacro:wide_thumb_distal>
     </xacro:macro>
 </robot>

File: softhands_description/urdf/xacro/include/macro/v1_wide/modules/thumb/thumb_distal.xacro (robot description, xacro)
@@ -1,7 +1,7 @@
 <?xml version="1.0"?>
 <robot xmlns:xacro="http://www.ros.org/wiki/xacro">
-    <xacro:macro name="thumb_distal" params="name parent side ns mass *origin **inertia_origin *inertia">
+    <xacro:macro name="wide_thumb_distal" params="name parent side ns mass *origin **inertia_origin *inertia">
 		<!-- Virtual joint from thumb proximal to thumb distal   -->
-		<joint name="${ns}_${name}_virtual_joint" type="revolute">
+		<joint name="${ns}_${name}_virtual_joint" type="${joint_type}">
 			<axis xyz="0 0 1"/>
 			<xacro:insert_block name="origin"/>
@@ -19,5 +19,5 @@
 	    </link>
 		<!-- Thumb middle  -->
-		<joint name="${ns}_${name}_joint" type="revolute">
+		<joint name="${ns}_${name}_joint" type="${joint_type}">
 			<parent link="${ns}_${name}_virtual_link"/>
 			<child link="${ns}_${name}_link"/>

File: softhands_description/urdf/xacro/include/macro/v1_wide/modules/thumb/thumb_knuckle.xacro (robot description, xacro)
@@ -1,7 +1,7 @@
 <?xml version="1.0"?>
 <robot xmlns:xacro="http://www.ros.org/wiki/xacro">
-    <xacro:macro name="thumb_knuckle" params="name parent side ns *origin">
+    <xacro:macro name="wide_thumb_knuckle" params="name parent side ns *origin">
 		<!-- Thumb Proximal  -->
-		<joint name="${ns}_${name}_joint" type="revolute">
+		<joint name="${ns}_${name}_joint" type="${joint_type}">
 			<parent link="${ns}_${parent}_link"/>
 			<child link="${ns}_${name}_link"/>

File: softhands_description/urdf/xacro/include/macro/v1_wide/modules/thumb/thumb_proximal.xacro (robot description, xacro)
@@ -1,7 +1,7 @@
 <?xml version="1.0"?>
 <robot xmlns:xacro="http://www.ros.org/wiki/xacro">
-    <xacro:macro name="thumb_proximal" params="name parent side ns mass *origin **inertia_origin *inertia">
+    <xacro:macro name="wide_thumb_proximal" params="name parent side ns mass *origin **inertia_origin *inertia">
 		<!-- Virtual joint from thumb knuckle to thumb proximal   -->
-		<joint name="${ns}_${name}_joint" type="revolute">
+		<joint name="${ns}_${name}_joint" type="${joint_type}">
 			<axis xyz="0 0 1"/>
 			<limit effort="30" velocity="0.0" lower="0" upper="0.785398" />
@@ -19,5 +19,5 @@
 	    </link>
 		<!-- Thumb Proximal joint  -->
-		<joint name="${ns}_${name}_virtual_joint" type="revolute">
+		<joint name="${ns}_${name}_virtual_joint" type="${joint_type}">
 			<parent link="${ns}_${name}_virtual_link"/>
 			<child link="${ns}_${name}_link"/>

File: softhands_description/urdf/xacro/v1_2_research.xacro (robot description, xacro)
@@ -44,4 +44,12 @@
 		<xacro:arg name="damping" 			default="3e-2"/>
 		<xacro:arg name="selfCollide" 		default="0"/>
+		<!-- <xacro:property name="fixed_hands" default="false"/> -->
+		<xacro:property name="joint_type" default="revolute"/>
+		<xacro:if value="${fixed_hands == True}">
+			<xacro:property name="joint_type" value="fixed"/>
+		</xacro:if>
+		<xacro:if value="${fixed_hands == False}">
+			<xacro:property name="joint_type" value="revolute"/>
+		</xacro:if>
 		<xacro:property name="sign" default="1"/>
 		<xacro:if value="${side == 'left'}">

File: softhands_description/urdf/xacro/v1_wide.xacro (robot description, xacro)
@@ -49,4 +49,11 @@
 			<xacro:property name="sign" value="-1"/>
 		</xacro:if>
+		<xacro:property name="joint_type" default="revolute"/>
+		<xacro:if value="${fixed_hands == True}">
+			<xacro:property name="joint_type" value="fixed"/>
+		</xacro:if>
+		<xacro:if value="${fixed_hands == False}">
+			<xacro:property name="joint_type" value="revolute"/>
+		</xacro:if>
     	<xacro:softhand_mimic_plugin ns="${side}_hand_v1_wide" wide="true"/>
 		<!-- # palm central -->
@@ -90,5 +97,5 @@
 		</xacro:palm_little>
 		<!-- # thumb -->
-		<xacro:thumb name="thumb" parent="palm_thumb_support" side="${side}" ns="${side}_hand_v1_wide">
+		<xacro:wide_thumb name="thumb" parent="palm_thumb_support" side="${side}" ns="${side}_hand_v1_wide">
 			<xacro:if value="${side == 'left'}">
 				<origin rpy="1.5707963 0 1.5707963" xyz="0 21.9577e-3 2.8e-3"/>
@@ -97,7 +104,7 @@
 				<origin rpy="-1.5707963 0 0" xyz="21.9577e-3 0 -2.8e-3"/>
 			</xacro:if>
-		</xacro:thumb>
+		</xacro:wide_thumb>
 		<!-- # Index -->
-		<xacro:finger name="index" parent="palm_central" side="${side}" ns="${side}_hand_v1_wide">
+		<xacro:wide_finger name="index" parent="palm_central" side="${side}" ns="${side}_hand_v1_wide">
 			<xacro:if value="${side == 'left'}">
 				<origin  rpy="0.1748327 0 0 " xyz="5e-3 -44.8953e-3 112.230e-3"/>
@@ -106,7 +113,7 @@
 				<origin  rpy="-3.1415927  -1.396264 1.5707963" xyz="5e-3 44.8953e-3 112.230e-3"/>
 			</xacro:if>
-		</xacro:finger>
+		</xacro:wide_finger>
 		<!-- # Middle -->
-		<xacro:finger name="middle" parent="palm_central" side="${side}" ns="${side}_hand_v1_wide">
+		<xacro:wide_finger name="middle" parent="palm_central" side="${side}" ns="${side}_hand_v1_wide">
 			<xacro:if value="${side == 'left'}">
 				<origin  rpy="0 0 0 " xyz="5e-3 -12.5e-3 115e-3"/>
@@ -115,7 +122,7 @@
 				<origin  rpy="0 -1.5707963 -1.5707963" xyz="5e-3 12.5e-3 115e-3"/>
 			</xacro:if>
-		</xacro:finger>
+		</xacro:wide_finger>
 		<!-- # Ring -->
-		<xacro:finger name="ring" parent="palm_little" side="${side}" ns="${side}_hand_v1_wide">
+		<xacro:wide_finger name="ring" parent="palm_little" side="${side}" ns="${side}_hand_v1_wide">
 			<xacro:if value="${side == 'left'}">
 				<origin rpy="2.8797933 0 1.5707963 " xyz=" 8.6355e-3 5e-3 -44.4863e-3" />
@@ -124,7 +131,7 @@
 				<origin rpy="0 -1.3089971 0" xyz=" 8.6355e-3 5e-3 44.4863e-3" />
 			</xacro:if>
-		</xacro:finger>
+		</xacro:wide_finger>
 		<!-- # Little -->
-		<xacro:finger name="little" parent="palm_little" side="${side}" ns="${side}_hand_v1_wide">
+		<xacro:wide_finger name="little" parent="palm_little" side="${side}" ns="${side}_hand_v1_wide">
 			<xacro:if value="${side == 'left'}">
 				<origin rpy="2.792527 0 1.5707963 " xyz="39.2985e-3 5e-3 -34.8419e-3" />
@@ -133,5 +140,5 @@
 				<origin rpy="0 -1.221731 0" xyz="39.2985e-3 5e-3 34.8419e-3" />
 			</xacro:if>
-		</xacro:finger>
+		</xacro:wide_finger>
 	</xacro:macro>
 </robot>

Commit message: updated hand orientations and grasp link

File: softhands_description/urdf/softhands.xacro (robot description, xacro)
@@ -91,5 +91,5 @@
 				parent="arm_1_7"
 				position="0 0 0.0"
-				orientation="0 0 ${orientation}"
+				orientation="0 0 ${orientation/2}"
 				fixed_hands="${fixed_hands}">
 			</xacro:v1_wide>
@@ -98,5 +98,5 @@
 				parent="arm_2_7"
 				position="0 0.0 0.00"
-				orientation="0 0 ${orientation/2}"
+				orientation="0 0 ${orientation}"
 				fixed_hands="${fixed_hands}">
 			</xacro:v1_2_research>

File: softhands_description/urdf/xacro/include/macro/v1_wide/modules/palm/palm_central.xacro (robot description, xacro)
@@ -38,5 +38,5 @@
 		<joint name="${ns}_grasp_joint" type="fixed">
 			<!-- QUIRINO: modified grasp_link for wide_hand-->
-			<origin rpy="0 0 0" xyz="0.03 0.10 0.15"/>
+			<origin rpy="0 0 1.57" xyz="0.03 0.10 0.15"/>
 			<parent link="${ns}_${name}_link" />
 			<child link="${ns}_grasp_link" />

Commit message: parameterised arguments for softhands

File: softhands_description/urdf/softhands.xacro (robot description, xacro)
@@ -38,5 +38,5 @@
 -->
 <robot name="softhands" xmlns:xacro="http://www.ros.org/wiki/xacro">
-	<xacro:macro name="softhands" params="version position orientation fixed_hands:='false'">
+	<xacro:macro name="softhands" params="version position orientation arm_1_parent arm_2_parent fixed_hands:='false'">
 		<xacro:include filename="$(find softhands_description)/urdf/xacro/include/macro/color.xacro" />
 		<xacro:include filename="$(find softhands_description)/urdf/xacro/include/macro/plugin.xacro"/>
@@ -49,6 +49,6 @@
 			<xacro:v1_2_research
 				side="left"
-				parent="arm_1_7"
-				position="0 -0. 0.00"
+				parent="${arm_1_parent}"
+				position="${position}"
 				orientation="0 0 ${orientation/2}"
 				fixed_hands="${fixed_hands}">
@@ -56,6 +56,6 @@
 			<xacro:v1_2_research
 				side="right"
-				parent="arm_2_7"
-				position="0 0.0 0.00"
+				parent="${arm_2_parent}"
+				position="${position}"
 				orientation="0 0 ${orientation/2}"
 				fixed_hands="${fixed_hands}">
@@ -68,6 +68,6 @@
 			<xacro:v1_wide
 				side="left"
-				parent="arm_1_7"
-				position="0 0 0.0"
+				parent="${arm_1_parent}"
+				position="${position}"
 				orientation="0 0 ${orientation}"
 				fixed_hands="${fixed_hands}">
@@ -75,6 +75,6 @@
 			<xacro:v1_wide
 				side="right"
-				parent="arm_2_7"
-				position="0 0 0.0"
+				parent="${arm_2_parent}"
+				position="${position}"
 				orientation="0 0 ${orientation}"
 				fixed_hands="${fixed_hands}">
@@ -89,14 +89,14 @@
 			<xacro:v1_wide
 				side="left"
-				parent="arm_1_7"
-				position="0 0 0.0"
-				orientation="0 0 ${orientation/2}"
+				parent="${arm_1_parent}"
+				position="${position}"
+				orientation="0 0 ${orientation}"
 				fixed_hands="${fixed_hands}">
 			</xacro:v1_wide>
 			<xacro:v1_2_research
 				side="right"
-				parent="arm_2_7"
-				position="0 0.0 0.00"
-				orientation="0 0 ${orientation}"
+				parent="${arm_2_parent}"
+				position="${position}"
+				orientation="0 0 ${orientation/2}"
 				fixed_hands="${fixed_hands}">
 			</xacro:v1_2_research>

File: softhands_description/urdf/xacro/include/macro/v1_wide/modules/palm/palm_thumb.xacro (robot description, xacro)
@@ -11,6 +11,6 @@
 		</joint>
 		<link name="${ns}_${name}_link">
-			<material name="grey" />
 			<visual>
+				<material name="grey" />
 				<geometry>
 				<mesh
@@ -41,6 +41,6 @@
 		</joint>
 		<link name="${ns}_${name}_support_link">
-				<material name="grey" />
 				<visual>
+					<material name="grey" />
 					<geometry>
 					<mesh
