Commit message: working on v1.2_research but its missing a damping between phalanges

File: softhands_description/urdf/softhands.urdf.xacro (robot description, xacro)
@@ -44,6 +44,6 @@
   	<xacro:arg name="side" default="right"/>
   	<xacro:arg name="meshes_dir" default="package://softhands_description/meshes/$(arg sh_version)/$(arg side)"/>
-  	<xacro:arg name="ns" default="$(arg side)_hand_$(arg sh_version)"/>
-  	<xacro:arg name="position" default="0 0 0.005"/>
+  	<xacro:arg name="ns" default="right_hand_v_wide"/>
+  	<xacro:arg name="position" default="0 0 0.01"/>
   	<xacro:arg name="orientation" default="0 0 0"/>
   	<xacro:arg name="operation_mode" default="0"/>
@@ -51,4 +51,4 @@
 	<xacro:include filename="$(find softhands_description)/urdf/xacro/$(arg sh_version).xacro"/>
 	<!-- Include plugin -->
-	<!-- <xacro:include filename="$(find softhands_description)/urdf/xacro/include/macro/$(arg sh_version)/plugin.xacro"/> -->
+	<xacro:include filename="$(find softhands_description)/urdf/xacro/include/macro/$(arg sh_version)/plugin.xacro"/>
 </robot>

File: softhands_description/urdf/xacro/include/macro/v1.2_research/modules/finger/phalanx.xacro (robot description, xacro)
@@ -40,11 +40,11 @@
   <xacro:macro name="phalanx" params="ns name parent *origin side">
     <!-- VIRTUAL JOINT -->
-		<joint name="${ns}_${name}_virtual_joint" type="fixed">
+		<joint name="${ns}_${name}_virtual_joint" type="revolute">
       <axis xyz="0 0 -1"/>
-      <dynamics damping="0.0" friction="0.0"/>
-      <limit effort="100" lower="0.0" upper="0.785" velocity="100"/>
 			<xacro:insert_block name="origin"/>
 			<parent link="${ns}_${parent}_link"/>
 			<child link="${ns}_${name}_virtual_link"/>
+      <dynamics damping="0.0" friction="0.0"/>
+      <limit effort="30" velocity="10" lower="0.0" upper="0.785"/>
 		</joint>
     <!-- VIRTUAL LINK -->
@@ -52,6 +52,8 @@
       <inertial>
         <origin rpy="0 0 0" xyz="0 0 0"/>
-        <mass value="1e-3"/>
-        <inertia ixx="1e-9" ixy="0.0" ixz="0.0" iyy="1e-9" iyz="0.0" izz="1e-9"/>
+        <mass value="0.001"/>
+        <inertia  ixx="0.0001"      ixy="0"  	    ixz="0"
+                  iyy="0.0001" 	    iyz="0"
+        		      izz="0.0001" />
       </inertial>
     </link>
@@ -63,5 +65,5 @@
       <axis xyz="0 0 -1"/>
       <dynamics damping="0.0" friction="0.0"/>
-      <limit effort="100" lower="0.0" upper="0.785" velocity="100"/>
+      <limit effort="30" velocity="1.0" lower="0.0" upper="0.785"/>
     </joint>
     <!-- LINK -->
@@ -87,8 +89,33 @@
     </link>
     <!-- GAZEBO REF -->
+    <gazebo reference="${ns}_${name}_virtual_link">
+      <material>Gazebo/Grey</material>
+      <selfCollide>false</selfCollide>
+      <kp value="1e4" />
+      <kd value="1e2" />
+      <surface>
+       <friction>
+        <ode>
+         <mu>0.133</mu>
+         <mu2>0.133</mu2>
+        </ode>
+       </friction>
+      </surface>
+    </gazebo>
+        <!-- GAZEBO REF -->
     <gazebo reference="${ns}_${name}_link">
       <material>Gazebo/Grey</material>
-      <selfCollide>true</selfCollide>
-	  </gazebo>
+      <selfCollide>false</selfCollide>
+      <kp value="1e4" />
+      <kd value="1e2" />
+      <surface>
+       <friction>
+        <ode>
+         <mu>0.133</mu>
+         <mu2>0.133</mu2>
+        </ode>
+       </friction>
+      </surface>
+    </gazebo>
   </xacro:macro>
 </robot>

File: softhands_description/urdf/xacro/include/macro/v1.2_research/modules/finger/phalanx_distal.xacro (robot description, xacro)
@@ -40,11 +40,11 @@
   <xacro:macro name="phalanx_distal" params="ns name parent *origin side">
     <!-- VIRTUAL JOINT -->
-		<joint name="${ns}_${name}_virtual_joint" type="fixed">
+		<joint name="${ns}_${name}_virtual_joint" type="revolute">
       <axis xyz="0 0 -1"/>
       <xacro:insert_block name="origin"/>
-      <dynamics damping="0.0" friction="0.0"/>
-      <limit effort="100" lower="0.0" upper="0.785" velocity="100"/>
 			<parent link="${ns}_${parent}_link"/>
 			<child link="${ns}_${name}_virtual_link"/>
+      <limit effort="30" velocity="10" lower="0" upper="0.785398" />
+      <dynamics damping="0.0" friction="0.0" />
 		</joint>
     <!-- VIRTUAL LINK -->
@@ -52,6 +52,8 @@
       <inertial>
         <origin rpy="0 0 0" xyz="0 0 0"/>
-        <mass value="1e-3"/>
-        <inertia ixx="1e-9" ixy="0.0" ixz="0.0" iyy="1e-9" iyz="0.0" izz="1e-9"/>
+        <mass value="0.001"/>
+        <inertia  ixx="0.0001"      ixy="0"  	    ixz="0"
+                  iyy="0.0001" 	    iyz="0"
+        		      izz="0.0001" />
       </inertial>
     </link>
@@ -62,6 +64,6 @@
       <child link="${ns}_${name}_link"/>
       <axis xyz="0 0 -1"/>
+      <limit effort="30" velocity="1.0" lower="0" upper="0.785398" />
       <dynamics damping="0.0" friction="0.0"/>
-      <limit effort="100" lower="0.0" upper="0.785" velocity="100"/>
     </joint>
     <!-- LINK -->
@@ -87,7 +89,32 @@
     </link>
     <!-- GAZEBO REF -->
+    <gazebo reference="${ns}_${name}_virtual_link">
+      <material>Gazebo/Grey</material>
+      <selfCollide>true</selfCollide>
+      <kp value="1e4" />
+      <kd value="1e2" />
+      <surface>
+       <friction>
+        <ode>
+         <mu>0.133</mu>
+         <mu2>0.133</mu2>
+        </ode>
+       </friction>
+      </surface>
+    </gazebo>
+    <!-- GAZEBO REF -->
     <gazebo reference="${ns}_${name}_link">
       <material>Gazebo/Grey</material>
       <selfCollide>true</selfCollide>
+      <kp value="1e4" />
+      <kd value="1e2" />
+      <surface>
+       <friction>
+        <ode>
+         <mu>0.133</mu>
+         <mu2>0.133</mu2>
+        </ode>
+       </friction>
+      </surface>
 	  </gazebo>
   </xacro:macro>

File: softhands_description/urdf/xacro/include/macro/v1.2_research/modules/finger/phalanx_knuckle.xacro (robot description, xacro)
@@ -46,5 +46,5 @@
       <axis xyz="0 0 -1"/>
       <dynamics damping="0.0" friction="0.0"/>
-      <limit effort="100" lower="-0.524" upper="0.524" velocity="100"/>
+      <limit effort="30" velocity="1.0" lower="-0.524" upper="0.524" />
     </joint>
     <!-- LINK -->
@@ -69,9 +69,19 @@
       </collision>
     </link>
-    <!-- GAZEBO REF -->
+        <!-- GAZEBO REF -->
     <gazebo reference="${ns}_${name}_link">
       <material>Gazebo/Grey</material>
       <selfCollide>true</selfCollide>
-	  </gazebo>
+      <kp value="1e4" />
+      <kd value="1e2" />
+      <surface>
+       <friction>
+        <ode>
+         <mu>0.133</mu>
+         <mu2>0.133</mu2>
+        </ode>
+       </friction>
+      </surface>
+    </gazebo>
   </xacro:macro>
 </robot>

File: softhands_description/urdf/xacro/include/macro/v1.2_research/modules/finger/phalanx_short.xacro (robot description, xacro)
@@ -40,11 +40,11 @@
   <xacro:macro name="phalanx_short" params="ns name parent *origin side">
     <!-- VIRTUAL JOINT -->
-		<joint name="${ns}_${name}_joint" type="fixed">
+		<joint name="${ns}_${name}_joint" type="revolute">
       <axis xyz="0 0 -1"/>
-      <dynamics damping="0.0" friction="0.0"/>
-      <limit effort="100" lower="0.0" upper="0.785" velocity="100"/>
       <xacro:insert_block name="origin"/>
 			<parent link="${ns}_${parent}_link"/>
 			<child link="${ns}_${name}_virtual_link"/>
+      <dynamics damping="0.0" friction="0.0"/>
+      <limit effort="30" velocity="10" lower="0.0" upper="0.785"/>
 		</joint>
     <!-- VIRTUAL LINK -->
@@ -52,6 +52,8 @@
       <inertial>
       <origin rpy="0 0 0" xyz="0 0 0"/>
-      <mass value="1e-3"/>
-      <inertia ixx="1e-9" ixy="0.0" ixz="0.0" iyy="1e-9" iyz="0.0" izz="1e-9"/>
+        <mass value="0.001"/>
+        <inertia  ixx="0.0001"      ixy="0"  	    ixz="0"
+                  iyy="0.0001" 	    iyz="0"
+        		      izz="0.0001" />
       </inertial>
     </link>
@@ -63,5 +65,5 @@
       <axis xyz="0 0 -1"/>
       <dynamics damping="0.0" friction="0.0"/>
-      <limit effort="100" lower="0.0" upper="0.785" velocity="100"/>
+      <limit effort="100" velocity="1.0" lower="0.0" upper="0.785"/>
     </joint>
     <!-- LINK -->
@@ -87,8 +89,33 @@
     </link>
     <!-- GAZEBO REF -->
+    <gazebo reference="${ns}_${name}_virtual_link">
+      <material>Gazebo/Grey</material>
+      <selfCollide>false</selfCollide>
+      <kp value="1e4" />
+      <kd value="1e2" />
+      <surface>
+       <friction>
+        <ode>
+         <mu>0.133</mu>
+         <mu2>0.133</mu2>
+        </ode>
+       </friction>
+      </surface>
+    </gazebo>
+        <!-- GAZEBO REF -->
     <gazebo reference="${ns}_${name}_link">
       <material>Gazebo/Grey</material>
-      <selfCollide>true</selfCollide>
-	  </gazebo>
+      <selfCollide>false</selfCollide>
+      <kp value="1e4" />
+      <kd value="1e2" />
+      <surface>
+       <friction>
+        <ode>
+         <mu>0.133</mu>
+         <mu2>0.133</mu2>
+        </ode>
+       </friction>
+      </surface>
+    </gazebo>
   </xacro:macro>
 </robot>

File: softhands_description/urdf/xacro/include/macro/v1.2_research/modules/thumb/thumb_knuckle.xacro (robot description, xacro)
@@ -45,6 +45,6 @@
       <child link="${ns}_${name}_link"/>
       <axis xyz="0 0 -1"/>
-      <dynamics damping="0.0" friction="0.0"/>
-      <limit effort="100" lower="0.0" upper="1.571" velocity="100"/>
+      <limit effort="30" velocity="1.0" lower="0" upper="1.57" />
+      <dynamics damping="0.08" friction="0.0" />
     </joint>
     <!-- LINK -->
@@ -73,5 +73,15 @@
       <material>Gazebo/Grey</material>
       <selfCollide>true</selfCollide>
-	  </gazebo>
+      <kp value="1e4" />
+      <kd value="1e2" />
+      <surface>
+       <friction>
+        <ode>
+         <mu>0.133</mu>
+         <mu2>0.133</mu2>
+        </ode>
+       </friction>
+      </surface>
+    </gazebo>
   </xacro:macro>
 </robot>

File: softhands_description/urdf/xacro/include/macro/v1.2_research/modules/thumb/thumb_short.xacro (robot description, xacro)
@@ -40,11 +40,11 @@
   <xacro:macro name="thumb_short" params="ns name parent *origin side">
     <!-- VIRTUAL JOINT -->
-		<joint name="${ns}_${name}_joint" type="fixed">
+		<joint name="${ns}_${name}_joint" type="revolute">
       <axis xyz="0 0 -1"/>
-      <dynamics damping="0.0" friction="0.0"/>
-      <limit effort="100" lower="0.0" upper="0.785" velocity="100"/>
       <xacro:insert_block name="origin"/>
 			<parent link="${ns}_${parent}_link"/>
 			<child link="${ns}_${name}_virtual_link"/>
+      <limit effort="30" velocity="10" lower="0" upper="0.785398" />
+      <dynamics damping="0.08" friction="0.0" />
 		</joint>
     <!-- VIRTUAL LINK -->
@@ -52,6 +52,8 @@
       <inertial>
       <origin rpy="0 0 0" xyz="0 0 0"/>
-      <mass value="1e-3"/>
-      <inertia ixx="1e-9" ixy="0.0" ixz="0.0" iyy="1e-9" iyz="0.0" izz="1e-9"/>
+        <mass value="0.001"/>
+        <inertia  ixx="0.0001"      ixy="0"  	    ixz="0"
+                  iyy="0.0001" 	    iyz="0"
+        		      izz="0.0001" />
       </inertial>
     </link>
@@ -62,6 +64,6 @@
       <child link="${ns}_${name}_link"/>
       <axis xyz="0 0 -1"/>
-      <dynamics damping="0.0" friction="0.0"/>
-      <limit effort="100" lower="0.0" upper="0.785" velocity="100"/>
+      <limit effort="30" velocity="1.0" lower="0.0" upper="0.785398" />
+      <dynamics damping="0.0" friction="0.0" />
     </joint>
     <!-- LINK -->
@@ -87,8 +89,33 @@
     </link>
     <!-- GAZEBO REF -->
+    <gazebo reference="${ns}_${name}_virtual_link">
+      <material>Gazebo/Grey</material>
+      <selfCollide>true</selfCollide>
+      <kp value="1e4" />
+      <kd value="1e2" />
+      <surface>
+       <friction>
+        <ode>
+         <mu>0.133</mu>
+         <mu2>0.133</mu2>
+        </ode>
+       </friction>
+      </surface>
+    </gazebo>
+        <!-- GAZEBO REF -->
     <gazebo reference="${ns}_${name}_link">
       <material>Gazebo/Grey</material>
       <selfCollide>true</selfCollide>
-	  </gazebo>
+      <kp value="1e4" />
+      <kd value="1e2" />
+      <surface>
+       <friction>
+        <ode>
+         <mu>0.133</mu>
+         <mu2>0.133</mu2>
+        </ode>
+       </friction>
+      </surface>
+    </gazebo>
   </xacro:macro>
 </robot>

File: softhands_description/urdf/xacro/include/macro/v1_wide/header.xacro (robot description, xacro)
@@ -38,4 +38,5 @@
 -->
 <robot xmlns:xacro="http://www.ros.org/wiki/xacro" name="header">
+  <xacro:include filename="$(arg root_dir)/modules/virtual_link.xacro" />
   <!-- Include xacro macro  Palm-->
 	<xacro:include filename="$(arg root_dir)/modules/palm/palm_central.xacro" />

File: softhands_description/urdf/xacro/include/macro/v1_wide/modules/finger.xacro (robot description, xacro)
@@ -7,14 +7,14 @@
       </xacro:phalanx_knuckle>
       <!-- Proximal -->
-      <xacro:phalanx name="${name}_prox" parent="${name}_knuckle" side="$(arg side)" ns="$(arg ns)">
-        <origin rpy="0 0 0" xyz="24e-3 0 -6.5e-3" />
+      <xacro:phalanx name="${name}_proximal" parent="${name}_knuckle" side="$(arg side)" ns="$(arg ns)">
+        <origin rpy="0 0 0" xyz="24e-3 -6.5e-3 0" />
       </xacro:phalanx >
       <!-- Middle -->
-      <xacro:phalanx name="${name}_mid" parent="${name}_prox" side="$(arg side)" ns="$(arg ns)">
+      <xacro:phalanx name="${name}_middle" parent="${name}_proximal" side="$(arg side)" ns="$(arg ns)">
         <origin rpy="0 0 0" xyz="41e-3 0 0" />
       </xacro:phalanx>
       <!-- Distal -->
-      <xacro:phalanx_dist name="${name}_dist" parent="${name}_mid" side="$(arg side)" ns="$(arg ns)">
-        <origin rpy="0 0 0" xyz="9e-3 0 0"/>
+      <xacro:phalanx_dist name="${name}_distal" parent="${name}_middle" side="$(arg side)" ns="$(arg ns)">
+        <origin xyz="41e-3 0 0" rpy="0 0 0"/>
       </xacro:phalanx_dist>
     </xacro:macro>

File: softhands_description/urdf/xacro/include/macro/v1_wide/modules/finger/phalanx.xacro (robot description, xacro)
@@ -3,7 +3,7 @@
     <xacro:macro name="phalanx" params="name parent ns *origin side">
 		<!-- Virtual joint from knuckle->proximal or proximal->middle   -->
-		<joint name="${ns}_${name}_virtual_joint" type="fixed">
-			<axis xyz="0 -1 0"/>
-			<limit effort="30" velocity="1.0" lower="-0.1" upper="0.1"/>
+		<joint name="${ns}_${name}_virtual_joint" type="revolute">
+			<axis xyz="0 0 1"/>
+			<limit effort="30" velocity="1.0" lower="0" upper="0.785398" />
 			<xacro:insert_block name="origin"/>
 			<parent link="${ns}_${parent}_link"/>
@@ -14,11 +14,11 @@
 				<origin xyz="0 0 0" rpy="0 0 0"/>
 				<mass value="1e-3"/>
-				<inertia ixx="1e-9" ixy="0.0" ixz="0.0" iyy="1e-9" iyz="0.0" izz="1e-9"/>
+				<inertia ixx="1e-6" ixy="0.0" ixz="0.0" iyy="1e-6" iyz="0.0" izz="1e-6"/>
 		   </inertial>
 	    </link>
 		<!-- Proximal phalanx -->
 		<joint name="${ns}_${name}_joint" type="revolute">
-			<axis xyz="0 -1 0"/>
-			<limit effort="30" velocity="1.0" lower="-0.785398" upper="0.785398" />
+			<axis xyz="0 0 1"/>
+			<limit effort="30" velocity="1.0" lower="0" upper="0.785398" />
 			<origin rpy="0 0 0" xyz="9e-3 0 0"/>
             <parent link="${ns}_${name}_virtual_link"/>
@@ -36,7 +36,7 @@
 				</visual>
 				<inertial>
-					<mass value="0.0082"/>
-					<origin rpy="0 0 0" xyz="8.7707437e-03 -1.7863138e-03 0.0"/>
-					<inertia ixx="2.2722068e-07" ixy="1.1586053e-08" ixz="0.0" iyy="5.5947233e-07" iyz="0.0" izz="5.9562195e-07"/>
+					<mass value="2.4190505e-02"/>
+					<origin rpy="0 0 0" xyz=" 2.0923634e-02  8.4162795e-04 -5.2131884e-05"/>
+					<inertia ixx="1.9981795e-06" ixy="-6.0806048e-08" ixz="0.0" iyy="4.7810654e-06" iyz="0.0" izz="5.0961924e-06"/>
 				</inertial>
 				<collision>
@@ -51,5 +51,5 @@
 		<gazebo reference="${ns}_${name}_link">
 			<material>Gazebo/Grey</material>
-			<selfCollide>true</selfCollide>
+			<selfCollide>false</selfCollide>
 		</gazebo>
     </xacro:macro>

File: softhands_description/urdf/xacro/include/macro/v1_wide/modules/finger/phalanx_dist.xacro (robot description, xacro)
@@ -3,8 +3,8 @@
     <xacro:macro name="phalanx_dist" params="name parent side *origin ns">
 		<!-- Virtual joint from middle->distal   -->
-		<joint name="${ns}_${name}_virtual_joint" type="fixed">
+		<joint name="${ns}_${name}_virtual_joint" type="revolute">
 			<axis xyz="0 0 1"/>
-			<limit effort="30" velocity="1.0" lower="-0.785398" upper="0.785398" />
-			<origin xyz="41e-3 0 0" rpy="0 0 0"/>
+			<limit effort="30" velocity="1.0" lower="0" upper="0.785398" />
+			<xacro:insert_block name="origin"/>
 			<parent link="${ns}_${parent}_link"/>
 			<child link="${ns}_${name}_virtual_link"/>
@@ -14,12 +14,12 @@
 				<origin xyz="0 0 0" rpy="0 0 0"/>
 				<mass value="1e-3"/>
-				<inertia ixx="1e-9" ixy="0.0" ixz="0.0" iyy="1e-9" iyz="0.0" izz="1e-9"/>
+				<inertia ixx="1e-6" ixy="0.0" ixz="0.0" iyy="1e-6" iyz="0.0" izz="1e-6"/>
 		   </inertial>
 	    </link>
 		<!-- Proximal phalanx -->
 		<joint name="${ns}_${parent}_${name}_joint" type="revolute">
-			<axis xyz="0 -1 0"/>
-			<limit effort="30" velocity="1.0" lower="-0.785398" upper="0.785398" />
-			<xacro:insert_block name="origin"/>
+			<axis xyz="0 0 1"/>
+			<limit effort="30" velocity="1.0" lower="0" upper="0.785398" />
+			<origin rpy="0 0 0" xyz="9e-3 0 0"/>
             <parent link="${ns}_${name}_virtual_link"/>
 			<child link="${ns}_${name}_link"/>
@@ -36,7 +36,7 @@
 				</visual>
 				<inertial>
-					<mass value="0.009"/>
-					<origin rpy="0 0 0" xyz="8.8025467e-03 -1.7219289e-03 0.0"/>
-					<inertia ixx="2.6586142e-07" ixy="1.2416847e-08" ixz="0.0" iyy="5.9935767e-07" iyz="0.0" izz="6.6781963e-07"/>
+					<mass value="1.2475845e-02"/>
+					<origin rpy="0 0 0" xyz="1.2887396e-02 6.2001804e-05 -1.1041989e-03"/>
+					<inertia ixx="7.5548908e-07" ixy="0.0" ixz="0.0" iyy="1.2532982e-06" iyz="0.0" izz="1.3218760e-06"/>
 				</inertial>
 				<collision>
@@ -51,5 +51,5 @@
 	<gazebo reference="${ns}_${name}_link">
 		<material>Gazebo/Grey</material>
-		<selfCollide>true</selfCollide>
+		<selfCollide>false</selfCollide>
 	</gazebo>
     </xacro:macro>

File: softhands_description/urdf/xacro/include/macro/v1_wide/modules/finger/phalanx_knuckle.xacro (robot description, xacro)
@@ -3,5 +3,7 @@
     <xacro:macro name="phalanx_knuckle" params="name parent side *origin ns">
 		<!-- Support -->
-		<joint name="${ns}_${name}_joint" type="fixed">
+		<joint name="${ns}_${name}_joint" type="revolute">
+			<axis xyz="0 1 0"/>
+			<limit effort="30" velocity="1.0" lower="0" upper="0.0" />
 			<xacro:insert_block name="origin"/>
             <parent link="${ns}_${parent}_link"/>
@@ -13,5 +15,5 @@
 					<geometry>
 					<mesh
-						filename="$(arg meshes_dir)/phalanx_prox_sup.stl"
+						filename="$(arg meshes_dir)/phalanx_pros_sup.stl"
 						scale="0.001 0.001 0.001" />
 					</geometry>
@@ -19,12 +21,12 @@
 				</visual>
 				<inertial>
-					<mass value="0.0095"/>
-					<origin rpy="0 0 0" xyz="4.2753603e-04  0.0 -1.4321738e-03"/>
-					<inertia ixx="6.4337303e-07" ixy="0.0" ixz="-3.9373913e-08" iyy="1.1253771e-06" iyz="0.0" izz="7.2336948e-07"/>
+					<mass value="7.4913242e-03"/>
+					<origin rpy="0 0 0" xyz="1.8035857e-02 -4.0351343e-03 -4.4165266e-05 "/>
+					<inertia ixx="5.3708642e-07" ixy="0.0" ixz="1.5304482e-07" iyy="6.1466440e-07" iyz="-4.4383298e-09" izz="5.5136271e-07"/>
 					</inertial>
 				<collision>
 					<geometry>
 					<mesh
-						filename="$(arg meshes_dir)/phalanx_prox_sup.stl"
+						filename="$(arg meshes_dir)/phalanx_pros_sup.stl"
 						scale="0.001 0.001 0.001" />
 					</geometry>
@@ -34,5 +36,5 @@
 	<gazebo reference="${ns}_${name}_link">
 		<material>Gazebo/White</material>
-		<selfCollide>true</selfCollide>
+		<selfCollide>false</selfCollide>
 	</gazebo>
     </xacro:macro>

File: softhands_description/urdf/xacro/include/macro/v1_wide/modules/palm/palm_central.xacro (robot description, xacro)
@@ -22,9 +22,9 @@
 				</visual>
 				<inertial>
-				<origin xyz="-9.4524165e-3 -3.2786419e-2 -1.9973598e-3" rpy="0 0 0" />
-				<mass value="1.2747079e-1" />
-					<inertia ixx=" 1.1656420e-4" ixy="-3.6262159e-5"  ixz="-2.3018113e-6"
-											iyy=" 5.3305451e-5"  iyz=" -5.5947664e-6"
-																izz=" 1.2416468e-4" />
+					<mass value="5.5962922e-1" />
+					<origin xyz="-7.3637766e-03 1.5857667e-02  6.7065321e-02" rpy="0 0 0" />
+					<inertia ixx="8.2936450e-04" ixy="-1.9292962e-06"  ixz="1.6410516e-05"
+											iyy="8.0447768e-04"  iyz="-1.3735281e-04"
+																izz="3.0664811e-04" />
 					</inertial>
 				<collision>
@@ -38,7 +38,8 @@
 		</link>
 		<!-- palm base to Thumb -->
-		<joint name="${ns}_${name}_thumb_virtual_joint" type="revolute">
+		<joint name="${ns}_${name}_thumb_virtual_joint" type="fixed">
 			<axis xyz="0 0 -1"/>
-			<limit effort="0.0" lower="0" upper="0"  velocity="0.0"/>
+			<limit effort="30" velocity="10" lower="0" upper="1.57" />
+			<dynamics damping="0.0" friction="0.0" />
 			<origin xyz=" -0.0000000021 32.5059e-3 39.6398e-3" rpy="0 0.3490656 1.5707963"/>
 			<parent link="${ns}_${name}_link"/>
@@ -49,13 +50,12 @@
 			<origin xyz="0 0 0" rpy="0 0 0"/>
 			<mass value="1e-3"/>
-			<inertia ixx="1e-6"  ixy="0"  	  	ixz="0"
-								 iyy="1e-6" 	iyz="0"
-												izz="1e-6" />
+			<inertia ixx="1e-6" ixy="0.0" ixz="0.0" iyy="1e-6" iyz="0.0" izz="1e-6"/>
 		   </inertial>
 	    </link>
 		<!-- palm base to Litte virtual -->
-		<joint name="${ns}_${name}_little_virtual_joint" type="revolute">
+		<joint name="${ns}_${name}_little_virtual_joint" type="fixed">
 			<axis xyz="0 0 1"/>
-			<limit effort="0.0" lower="0" upper="0"  velocity="0.0"/>
+			<dynamics damping="0.0" friction="0.0"/>
+			<limit effort="100" lower="0.0" upper="0.5" velocity="100"/>
 			<origin xyz=" -0.0000000091 -10.6603e-3 66.1817e-3" rpy="0 -0.1745327 -1.5707963"/>
 			<parent link="${ns}_${name}_link"/>
@@ -66,13 +66,11 @@
 				<origin xyz="0 0 0" rpy="0 0 0"/>
 				<mass value="1e-3"/>
-				<inertia ixx="1e-6"  ixy="0"  	  	ixz="0"
-									iyy="1e-6" 	iyz="0"
-													izz="1e-6" />
+				<inertia ixx="1e-6" ixy="0.0" ixz="0.0" iyy="1e-6" iyz="0.0" izz="1e-6"/>
 		   </inertial>
 	    </link>
-	<gazebo reference="${ns}_${name}_link">
-		<material>Gazebo/Grey</material>
-		<selfCollide>true</selfCollide>
-	</gazebo>
+		<gazebo reference="${ns}_${name}_link">
+		<selfCollide>false</selfCollide>
+			<material>Gazebo/Grey</material>
+		</gazebo>
     </xacro:macro>
 </robot>
