Commit message: working on v1.2_research but its missing a damping between phalanges

File: softhands_description/urdf/xacro/include/macro/v1_wide/modules/palm/palm_little.xacro (robot description, xacro)
@@ -2,11 +2,11 @@
 <robot xmlns:xacro="http://www.ros.org/wiki/xacro">
     <xacro:macro name="palm_little" params="name parent side *origin ns">
-		<joint name="${ns}_${name}_joint" type="revolute">
+		<joint name="${ns}_${name}_joint" type="fixed">
 			<parent link="${ns}_${parent}_link"/>
 			<child link="${ns}_${name}_link"/>
 			<xacro:insert_block name="origin"/>
 			<axis xyz="0 0 1" />
-      		<limit effort="30" velocity="1.0" lower="0" upper="1.57" />
-			<dynamics damping="0.08" friction="0.0" />
+      		<limit effort="30" velocity="1.0" lower="0" upper="0.3" />
+			<dynamics damping="0.0" friction="0.0" />
 		</joint>
 		<link name="${ns}_${name}_link">
@@ -21,9 +21,9 @@
 				</visual>
 				<inertial>
-				<origin xyz="-9.4524165e-3 -3.2786419e-2 -1.9973598e-3" rpy="0 0 0" />
-				<mass value="1.2747079e-1" />
-					<inertia ixx=" 1.1656420e-4" ixy="-3.6262159e-5"  ixz="-2.3018113e-6"
-											iyy=" 5.3305451e-5"  iyz=" -5.5947664e-6"
-																izz=" 1.2416468e-4" />
+				<origin xyz="1.9466642e-02  5.5041380e-03 -7.9253974e-04" rpy="0 0 0" />
+				<mass value="1.7998957e-1" />
+					<inertia ixx=" 2.4776164e-04" ixy="-2.2762031e-06"  ixz="-2.5699035e-05"
+											iyy="2.6460918e-04"  iyz=" 1.5348716e-05"
+																izz="5.9121350e-05" />
 					</inertial>
 				<collision>
@@ -37,6 +37,6 @@
 		</link>
 	<gazebo reference="${ns}_${name}_link">
+		<selfCollide>false</selfCollide>
 		<material>Gazebo/Grey</material>
-		<selfCollide>true</selfCollide>
 	</gazebo>
     </xacro:macro>

File: softhands_description/urdf/xacro/include/macro/v1_wide/modules/palm/palm_thumb.xacro (robot description, xacro)
@@ -2,5 +2,5 @@
 <robot xmlns:xacro="http://www.ros.org/wiki/xacro">
     <xacro:macro name="palm_thumb" params="name parent side *origin ns">
-		<joint name="${ns}_${name}_joint" type="revolute">
+		<joint name="${ns}_${name}_joint" type="fixed">
 			<parent link="${ns}_${parent}_link"/>
 			<child link="${ns}_${name}_link"/>
@@ -8,5 +8,5 @@
 			<axis xyz="0 0 -1" />
       		<limit effort="30" velocity="1.0" lower="0" upper="1.57" />
-			<dynamics damping="0.08" friction="0.0" />
+			<dynamics damping="0.0" friction="0.0" />
 		</joint>
 		<link name="${ns}_${name}_link">
@@ -21,9 +21,9 @@
 				</visual>
 				<inertial>
-				<origin xyz="-9.4524165e-3 -3.2786419e-2 -1.9973598e-3" rpy="0 0 0" />
-				<mass value="1.2747079e-1" />
-					<inertia ixx=" 1.1656420e-4" ixy="-3.6262159e-5"  ixz="-2.3018113e-6"
-											iyy=" 5.3305451e-5"  iyz=" -5.5947664e-6"
-																izz=" 1.2416468e-4" />
+				<origin xyz="1.3888149e-2 -7.0704771e-3  1.1337304e-3" rpy="0 0 0" />
+				<mass value="9.2767000e-02" />
+					<inertia ixx="5.2239281e-5" ixy="2.7341002e-6"  ixz="6.0525027e-6"
+											iyy="5.5447805e-5"  iyz="-4.6570702e-6"
+																izz="2.7144559e-5" />
 					</inertial>
 				<collision>
@@ -36,8 +36,4 @@
 				</collision>
 		</link>
-	<gazebo reference="${ns}_${name}_link">
-		<material>Gazebo/Grey</material>
-		<selfCollide>true</selfCollide>
-	</gazebo>
 	<!-- Palm thumb to thumb support -->
 	<joint name="${ns}_${name}_support_joint" type="fixed">
@@ -57,9 +53,9 @@
 			</visual>
 			<inertial>
-			<origin xyz="-9.4524165e-3 -3.2786419e-2 -1.9973598e-3" rpy="0 0 0" />
-			<mass value="1.2747079e-1" />
-				<inertia ixx=" 1.1656420e-4" ixy="-3.6262159e-5"  ixz="-2.3018113e-6"
-										iyy=" 5.3305451e-5"  iyz=" -5.5947664e-6"
-															izz=" 1.2416468e-4" />
+			<origin xyz="1.1097412e-02 -4.2327979e-05 -4.7109856e-04" rpy="0 0 0" />
+			<mass value="1.6408860e-02" />
+				<inertia ixx="1.8835019e-06" ixy="-4.9293913e-09" ixz="-2.5700318e-08"
+										iyy="1.2828797e-06"  iyz="-4.0065947e-09"
+															izz="2.2986135e-06" />
 				</inertial>
 			<collision>
@@ -72,7 +68,11 @@
 			</collision>
 	</link>
+	<gazebo reference="${ns}_${name}_link">
+		<material>Gazebo/Grey</material>
+    	<selfCollide>false</selfCollide>
+	</gazebo>
 	<gazebo reference="${ns}_${name}_support_link">
 		<material>Gazebo/White</material>
-		<selfCollide>true</selfCollide>
+		<selfCollide>false</selfCollide>
 	</gazebo>
     </xacro:macro>

File: softhands_description/urdf/xacro/include/macro/v1_wide/modules/thumb.xacro (robot description, xacro)
@@ -8,9 +8,9 @@
       <!-- Middle -->
       <xacro:thumb_proximal name="${name}_proximal" parent="${name}_knuckle" side="$(arg side)" ns="$(arg ns)">
-        <origin rpy="0 0 0" xyz="9e-3 0 0"/>
+        <origin rpy="-1.3962638 0 0" xyz="38.5e-3 4.82952e-3 -0.167417e-3"/>
       </xacro:thumb_proximal>
       <!-- Distal -->
       <xacro:thumb_distal name="${name}_distal" parent="${name}_proximal" side="$(arg side)" ns="$(arg ns)">
-        <origin rpy="0 0.0101229 0" xyz="8.99947e-3 0 -0.0973875e-3"/>
+        <origin  rpy="0 0 0" xyz="41e-3 0 0"/>
       </xacro:thumb_distal>
     </xacro:macro>

File: softhands_description/urdf/xacro/include/macro/v1_wide/modules/thumb/thumb_distal.xacro (robot description, xacro)
@@ -3,10 +3,10 @@
     <xacro:macro name="thumb_distal" params="name parent side ns *origin">
 		<!-- Virtual joint from thumb proximal to thumb distal   -->
-		<joint name="${ns}_${name}_virtual_joint" type="fixed">
-			<axis xyz="0 -1 0"/>
-			<limit effort="0.0" lower="0" upper="0"  velocity="0.0"/>
-			<origin xyz="41e-3 0 0" rpy="0 0 0"/>
+		<joint name="${ns}_${name}_virtual_joint" type="revolute">
+			<axis xyz="0 0 1"/>
+			<xacro:insert_block name="origin"/>
 			<parent link="${ns}_${parent}_link"/>
 			<child link="${ns}_${name}_virtual_link"/>
+			<limit effort="30" velocity="10" lower="0" upper="0.785398" />
 		</joint>
 	    <link name="${ns}_${name}_virtual_link">
@@ -14,10 +14,9 @@
 			<origin xyz="0 0 0" rpy="0 0 0"/>
 			<mass value="1e-3"/>
-			<inertia ixx="1e-9" ixy="0.0" ixz="0.0" iyy="1e-9" iyz="0.0" izz="1e-9"/>
+			<inertia ixx="1e-6" ixy="0.0" ixz="0.0" iyy="1e-6" iyz="0.0" izz="1e-6"/>
 		   </inertial>
 	    </link>
 		<gazebo reference="${ns}_${name}_virtual_link">
 			<material>Gazebo/Grey</material>
-			<selfCollide>true</selfCollide>
 			<kp value="1e4" />
 			<kd value="1e2" />
@@ -35,8 +34,8 @@
 			<parent link="${ns}_${name}_virtual_link"/>
 			<child link="${ns}_${name}_link"/>
-			<xacro:insert_block name="origin"/>
-			<axis xyz="0 -1 0" />
-      		<limit effort="30" velocity="1.0" lower="0" upper="1.57" />
-			<dynamics damping="0.08" friction="0.0" />
+			<origin rpy="0 0.0101229 0" xyz="8.99947e-3 0 -0.0973875e-3"/>
+			<axis xyz="0 0 1" />
+      		<limit effort="30" velocity="1.0" lower="0" upper="0.785398" />
+			<dynamics damping="0.0" friction="0.0" />
 		</joint>
 		<link name="${ns}_${name}_link">
@@ -51,7 +50,7 @@
 				</visual>
 				<inertial>
-					<mass value="0.009"/>
-					<origin rpy="0 0 0" xyz="8.8025467e-03 -1.7219289e-03 0.0"/>
-					<inertia ixx="2.6586142e-07" ixy="1.2416847e-08" ixz="0.0" iyy="5.9935767e-07" iyz="0.0" izz="6.6781963e-07"/>
+					<mass value="2.3674554e-02"/>
+					<origin rpy="0 0 0" xyz="1.6161362e-02  1.6241404e-03 -3.2684152e-05 "/>
+					<inertia ixx="2.578454e-06" ixy="0.0" ixz="0.0" iyy="2.9887569e-06" iyz="0.0" izz="3.8277106e-06"/>
 				</inertial>
 				<collision>
@@ -65,16 +64,15 @@
 		</link>
 		<gazebo reference="${ns}_${name}_link">
-		<material>Gazebo/Grey</material>
-		<selfCollide>true</selfCollide>
-		<kp value="1e4" />
-		<kd value="1e2" />
-		<surface>
-		<friction>
-			<ode>
-			<mu>0.133</mu>
-			<mu2>0.133</mu2>
-			</ode>
-		</friction>
-		</surface>
+			<material>Gazebo/Grey</material>
+			<kp value="1e4" />
+			<kd value="1e2" />
+			<surface>
+			<friction>
+				<ode>
+				<mu>0.133</mu>
+				<mu2>0.133</mu2>
+				</ode>
+			</friction>
+			</surface>
 		</gazebo>
     </xacro:macro>

File: softhands_description/urdf/xacro/include/macro/v1_wide/modules/thumb/thumb_knuckle.xacro (robot description, xacro)
@@ -9,5 +9,5 @@
 			<axis xyz="0 0 1" />
       		<limit effort="30" velocity="1.0" lower="0" upper="1.57" />
-			<dynamics damping="0.08" friction="0.0" />
+			<dynamics damping="0.0" friction="0.0" />
 		</joint>
 		<link name="${ns}_${name}_link">
@@ -22,7 +22,7 @@
 				</visual>
 				<inertial>
-					<mass value="0.01"/>
-					<origin rpy="0 0 0" xyz="1.3071561e-02 -2.7357764e-03 6.4347823e-04"/>
-					<inertia ixx="3.5865978e-07" ixy="2.0944224e-07" ixz="-6.8657569e-08" iyy="1.3885564e-06" iyz="3.2170608e-08" izz="1.3571203e-06"/>
+					<mass value="2.4657976e-02"/>
+					<origin rpy="0 0 0" xyz="2.2747515e-02  4.5872045e-03 -1.3868568e-03  "/>
+					<inertia ixx="2.6529131e-6" ixy="-2.6016685e-07" ixz="1.3433999e-07" iyy="4.4499492e-06" iyz="-7.5218787e-08" izz="5.0393400e-06"/>
 				</inertial>
 				<collision>
@@ -37,5 +37,4 @@
 		<gazebo reference="${ns}_${name}_link">
 			<material>Gazebo/Grey</material>
-			<selfCollide>true</selfCollide>
 			<kp value="1e4" />
 			<kd value="1e2" />

File: softhands_description/urdf/xacro/include/macro/v1_wide/modules/thumb/thumb_proximal.xacro (robot description, xacro)
@@ -3,8 +3,8 @@
     <xacro:macro name="thumb_proximal" params="name parent side ns *origin">
 		<!-- Virtual joint from thumb knuckle to thumb proximal   -->
-		<joint name="${ns}_${name}_joint" type="fixed">
+		<joint name="${ns}_${name}_joint" type="revolute">
 			<axis xyz="0 0 1"/>
-			<limit effort="0.0" lower="0" upper="0"  velocity="0.0"/>
-			<origin xyz=" 31.2357e-3 23.0197e-3 0.167417e-3" rpy=" 0.1745395 0.0000165 0.7597087"/>
+			<limit effort="30" velocity="10" lower="0" upper="0.785398" />
+			<xacro:insert_block name="origin"/>
 			<parent link="${ns}_${parent}_link"/>
 			<child link="${ns}_${name}_virtual_link"/>
@@ -14,10 +14,9 @@
 			<origin xyz="0 0 0" rpy="0 0 0"/>
 			<mass value="1e-3"/>
-			<inertia ixx="1e-9" ixy="0.0" ixz="0.0" iyy="1e-9" iyz="0.0" izz="1e-9"/>
+			<inertia ixx="1e-6" ixy="0.0" ixz="0.0" iyy="1e-6" iyz="0.0" izz="1e-6"/>
 		   </inertial>
 	    </link>
 		<gazebo reference="${ns}_${name}_virtual_link">
 			<material>Gazebo/Grey</material>
-			<selfCollide>true</selfCollide>
 			<kp value="1e4" />
 			<kd value="1e2" />
@@ -25,6 +24,6 @@
 			<friction>
 				<ode>
-					<mu>0.133</mu>
-					<mu2>0.133</mu2>
+				<mu>0.133</mu>
+				<mu2>0.133</mu2>
 				</ode>
 			</friction>
@@ -35,8 +34,8 @@
 			<parent link="${ns}_${name}_virtual_link"/>
 			<child link="${ns}_${name}_link"/>
-			<xacro:insert_block name="origin"/>
-			<axis xyz="0 -1 0" />
-      		<limit effort="30" velocity="1.0" lower="0" upper="1.57" />
-			<dynamics damping="0.08" friction="0.0" />
+			<origin rpy="0 0 0"  xyz="9e-3 0 0 "/>
+			<axis xyz="0 0 1" />
+      		<limit effort="30" velocity="1.0" lower="0" upper="0.785398" />
+			<dynamics damping="0.0" friction="0.0" />
 		</joint>
 		<link name="${ns}_${name}_link">
@@ -51,7 +50,7 @@
 				</visual>
 				<inertial>
-					<mass value="0.0063"/>
-					<origin rpy="0 0 0" xyz="4.7601567e-03 -1.3786947e-03 0.0"/>
-					<inertia ixx="1.8024201e-07" ixy="5.756798e-09" ixz="0.0" iyy="2.3516266e-07" iyz="0.0" izz="2.691504e-07"/>
+					<mass value="3.3679189e-02"/>
+					<origin rpy="0 0 0" xyz="2.0950700e-02  1.1175133e-03 -3.7424390e-05"/>
+					<inertia ixx="4.1328993e-06" ixy="-8.6599874e-08" ixz="0.0" iyy="7.4560101e-06" iyz="-1.0265429e-09" izz="6.6161853e-06"/>
 				</inertial>
 				<collision>
@@ -66,5 +65,4 @@
 		<gazebo reference="${ns}_${name}_link">
 			<material>Gazebo/Grey</material>
-			<selfCollide>true</selfCollide>
 			<kp value="1e4" />
 			<kd value="1e2" />

File: softhands_description/urdf/xacro/v1.2_research.xacro (robot description, xacro)
@@ -37,5 +37,5 @@
  *
 -->
-<robot name="v2.0_qb" xmlns:xacro="http://www.ros.org/wiki/xacro">
+<robot name="right_hand_v2" xmlns:xacro="http://www.ros.org/wiki/xacro">
 	<!-- # iso -->
 	<xacro:iso name="iso" parent="$(arg root_link)" ns="$(arg ns)" side="$(arg side)">
