Commit message: works on wide with parameter true-false on plugin xacro

File: softhands_description/urdf/softhands.urdf.xacro (robot description, xacro)
@@ -51,10 +51,10 @@
   	<xacro:arg name="orientation" default="$(arg roll) $(arg pitch) $(arg yaw)"/>
   	<xacro:arg name="operation_mode" default="0"/>
+  	<xacro:arg name="selfCollide" default="0"/>
 	<xacro:include filename="$(arg root_dir)/header.xacro"/>
-  	<xacro:arg name="high_friction" default="0.7"/>
-  	<xacro:arg name="friction" default="1e-3"/>
-  	<xacro:arg name="damping" default="1e-4"/>
-  	<xacro:arg name="virtual_friction" default="0.0"/>
+  	<xacro:arg name="friction" default="1e-2"/>
+  	<xacro:arg name="virtual_friction" default="1e-2"/>
   	<xacro:arg name="virtual_damping" default="0.0"/>
+  	<xacro:arg name="damping" default="0.0"/>
 	<xacro:include filename="$(find softhands_description)/urdf/xacro/$(arg sh_version).xacro"/>
 	<!-- Include plugin -->

File: softhands_description/urdf/xacro/include/macro/v1_2_research/modules/finger/phalanx.xacro (robot description, xacro)
@@ -46,5 +46,5 @@
 			<child link="${ns}_${name}_virtual_link"/>
       <limit effort="30" velocity="1.0" lower="0.0" upper="0.785"/>
-      <dynamics damping="$(arg virtual_damping)" friction="0.0"/>
+      <dynamics damping="$(arg virtual_damping)" friction="$(arg virtual_friction)"/>
 		</joint>
     <!-- VIRTUAL LINK -->
@@ -92,15 +92,5 @@
     <gazebo reference="${ns}_${name}_link">
       <material>Gazebo/Grey</material>
-      <selfCollide>false</selfCollide>
-      <kp value="1e4" />
-      <kd value="1e2" />
-      <surface>
-       <friction>
-        <ode>
-         <mu>0.133</mu>
-         <mu2>0.133</mu2>
-        </ode>
-       </friction>
-      </surface>
+      <selfCollide>$(arg selfCollide)</selfCollide>
     </gazebo>
   </xacro:macro>

File: softhands_description/urdf/xacro/include/macro/v1_2_research/modules/finger/phalanx_distal.xacro (robot description, xacro)
@@ -46,5 +46,5 @@
 			<child link="${ns}_${name}_virtual_link"/>
       <limit effort="30" velocity="10" lower="0" upper="0.785398" />
-       <dynamics damping="$(arg virtual_damping)" friction="0.0"/>
+      <dynamics damping="$(arg virtual_damping)" friction="$(arg virtual_friction)"/>
 		</joint>
     <!-- VIRTUAL LINK -->
@@ -92,14 +92,5 @@
     <gazebo reference="${ns}_${name}_link">
       <material>Gazebo/Grey</material>
-      <kp value="1e4" />
-      <kd value="1e2" />
-      <surface>
-       <friction>
-        <ode>
-         <mu>0.133</mu>
-         <mu2>0.133</mu2>
-        </ode>
-       </friction>
-      </surface>
+      <selfCollide>$(arg selfCollide)</selfCollide>
 	  </gazebo>
   </xacro:macro>

File: softhands_description/urdf/xacro/include/macro/v1_2_research/modules/finger/phalanx_knuckle.xacro (robot description, xacro)
@@ -46,5 +46,5 @@
       <axis xyz="0 0 -1"/>
       <limit effort="30" velocity="1.0" lower="-0.524" upper="0.524" />
-      <dynamics damping="$(arg damping)" friction="$(arg friction)"/>
+       <dynamics damping="0.08" friction="0"/>
     </joint>
     <!-- LINK -->
@@ -72,15 +72,5 @@
     <gazebo reference="${ns}_${name}_link">
       <material>Gazebo/Grey</material>
-      <!-- <selfCollide>false</selfCollide> -->
-      <kp value="1e4" />
-      <kd value="1e2" />
-      <surface>
-       <friction>
-        <ode>
-         <mu>0.133</mu>
-         <mu2>0.133</mu2>
-        </ode>
-       </friction>
-      </surface>
+      <selfCollide>$(arg selfCollide)</selfCollide>
     </gazebo>
   </xacro:macro>

File: softhands_description/urdf/xacro/include/macro/v1_2_research/modules/finger/phalanx_short.xacro (robot description, xacro)
@@ -46,5 +46,5 @@
 			<child link="${ns}_${name}_virtual_link"/>
       <limit effort="30" velocity="10" lower="0.0" upper="0.785"/>
-      <dynamics damping="$(arg virtual_damping)" friction="0.0"/>
+      <dynamics damping="$(arg virtual_damping)" friction="$(arg virtual_friction)"/>
 		</joint>
     <!-- VIRTUAL LINK -->
@@ -92,15 +92,5 @@
     <gazebo reference="${ns}_${name}_link">
       <material>Gazebo/Grey</material>
-      <!-- <selfCollide>false</selfCollide> -->
-      <kp value="1e4" />
-      <kd value="1e2" />
-      <surface>
-       <friction>
-        <ode>
-         <mu>0.133</mu>
-         <mu2>0.133</mu2>
-        </ode>
-       </friction>
-      </surface>
+      <selfCollide>$(arg selfCollide)</selfCollide>
     </gazebo>
   </xacro:macro>

File: softhands_description/urdf/xacro/include/macro/v1_2_research/modules/iso.xacro (robot description, xacro)
@@ -39,7 +39,4 @@
 <robot name="iso_v2" xmlns:xacro="http://www.ros.org/wiki/xacro">
 	<xacro:macro name="iso" params="ns name parent *origin side">
-		<!-- World -->
-		<link name="${parent}">
-		</link>
 		<!-- World to palm base -->
 		<joint name="${ns}_${name}_joint" type="fixed">

File: softhands_description/urdf/xacro/include/macro/v1_2_research/modules/palm/palm.xacro (robot description, xacro)
@@ -41,5 +41,5 @@
 	  	<joint name="${ns}_palm_joint" type="fixed">
 			<xacro:insert_block name="origin"/>
-			<parent link="${ns}_${parent}_link" />
+			<parent link="${parent}" />
 			<child link="${ns}_palm_link" />
 		</joint>
@@ -48,5 +48,5 @@
 				<mass value="0.45"/>
 				<origin rpy="0 0 0" xyz="0.0030 -0.0449 0.0135"/>
-				<inertia ixx="0.00045" ixy="0.0" ixz="0.0" iyy="0.0006" iyz="0.0" izz="0.00025"/>
+				<inertia ixx="0.00045" ixy="0.0" ixz="0.0" iyy="0.00025" iyz="0.0" izz="0.0006"/>
 			</inertial>
 			<visual>

File: softhands_description/urdf/xacro/include/macro/v1_2_research/modules/thumb/thumb_knuckle.xacro (robot description, xacro)
@@ -46,5 +46,5 @@
       <axis xyz="0 0 -1"/>
       <limit effort="30" velocity="1.0" lower="0" upper="1.57" />
-      <dynamics damping="0.08" friction="$(arg friction)" />
+      <dynamics damping="0.0" friction="0.0" />
     </joint>
     <!-- LINK -->
@@ -72,15 +72,5 @@
     <gazebo reference="${ns}_${name}_link">
       <material>Gazebo/Grey</material>
-      <selfCollide>false</selfCollide>
-      <kp value="1e4" />
-      <kd value="1e2" />
-      <surface>
-       <friction>
-        <ode>
-         <mu>0.133</mu>
-         <mu2>0.133</mu2>
-        </ode>
-       </friction>
-      </surface>
+      <selfCollide>$(arg selfCollide)</selfCollide>
     </gazebo>
   </xacro:macro>

File: softhands_description/urdf/xacro/include/macro/v1_2_research/modules/thumb/thumb_short.xacro (robot description, xacro)
@@ -46,5 +46,5 @@
 			<child link="${ns}_${name}_virtual_link"/>
       <limit effort="30" velocity="10" lower="0" upper="0.785398" />
-      <dynamics damping="0.05" friction="0.0" />
+      <dynamics damping="$(arg virtual_damping)" friction="$(arg virtual_friction)"/>
 		</joint>
     <!-- VIRTUAL LINK -->
@@ -65,5 +65,5 @@
       <axis xyz="0 0 -1"/>
       <limit effort="30" velocity="1.0" lower="0.0" upper="0.785398" />
-      <dynamics damping="0.0" friction="$(arg friction)" />
+      <dynamics damping="$(arg damping)" friction="$(arg friction)" />
     </joint>
     <!-- LINK -->
@@ -96,15 +96,5 @@
     <gazebo reference="${ns}_${name}_link">
       <material>Gazebo/Grey</material>
-      <selfCollide>false</selfCollide>
-      <kp value="1e4" />
-      <kd value="1e2" />
-      <surface>
-       <friction>
-        <ode>
-         <mu>0.133</mu>
-         <mu2>0.133</mu2>
-        </ode>
-       </friction>
-      </surface>
+      <selfCollide>$(arg selfCollide)</selfCollide>
     </gazebo>
   </xacro:macro>

File: softhands_description/urdf/xacro/include/macro/v1_2_research/plugin.xacro (robot description, xacro)
@@ -42,5 +42,4 @@
 			<namespace>$(arg ns)</namespace>
 			<operation_mode>$(arg operation_mode)</operation_mode>
-			<close_rate>0.001</close_rate>
 			<spring_k>0.5</spring_k>
 			<r_finger>0.0033</r_finger>

File: softhands_description/urdf/xacro/include/macro/v1_wide/modules/finger/phalanx.xacro (robot description, xacro)
@@ -9,4 +9,5 @@
 			<parent link="${ns}_${parent}_link"/>
 			<child link="${ns}_${name}_virtual_link"/>
+			<dynamics damping="$(arg virtual_damping)" friction="$(arg virtual_friction)"/>
 		</joint>
 		<link name="${ns}_${name}_virtual_link">
@@ -24,4 +25,5 @@
             <parent link="${ns}_${name}_virtual_link"/>
 			<child link="${ns}_${name}_link"/>
+			<dynamics damping="$(arg damping)" friction="$(arg friction)"/>
 		</joint>
 		<link name="${ns}_${name}_link">
@@ -51,5 +53,5 @@
 		<gazebo reference="${ns}_${name}_link">
 			<material>Gazebo/Gray</material>
-			<selfCollide>false</selfCollide>
+			<selfCollide>$(arg selfCollide)</selfCollide>
 			<kp value="1e4" />
 			<kd value="1e2" />

File: softhands_description/urdf/xacro/include/macro/v1_wide/modules/finger/phalanx_dist.xacro (robot description, xacro)
@@ -9,4 +9,5 @@
 			<parent link="${ns}_${parent}_link"/>
 			<child link="${ns}_${name}_virtual_link"/>
+			<dynamics damping="$(arg virtual_damping)" friction="$(arg virtual_friction)"/>
 		</joint>
 		<link name="${ns}_${name}_virtual_link">
@@ -24,4 +25,5 @@
             <parent link="${ns}_${name}_virtual_link"/>
 			<child link="${ns}_${name}_link"/>
+			<dynamics damping="$(arg damping)" friction="$(arg friction)"/>
 		</joint>
 		<link name="${ns}_${name}_link">
@@ -51,5 +53,5 @@
 		<gazebo reference="${ns}_${name}_link">
 			<material>Gazebo/Gray</material>
-			<selfCollide>false</selfCollide>
+			<selfCollide>$(arg selfCollide)</selfCollide>
 			<kp value="1e4" />
 			<kd value="1e2" />

File: softhands_description/urdf/xacro/include/macro/v1_wide/modules/finger/phalanx_knuckle.xacro (robot description, xacro)
@@ -36,5 +36,5 @@
 	<gazebo reference="${ns}_${name}_link">
 			<material>Gazebo/White</material>
-			<selfCollide>false</selfCollide>
+			<selfCollide>$(arg selfCollide)</selfCollide>
 			<kp value="1e4" />
 			<kd value="1e2" />

File: softhands_description/urdf/xacro/include/macro/v1_wide/modules/palm/palm_central.xacro (robot description, xacro)
@@ -38,5 +38,5 @@
 		</link>
 		<!-- palm base to Thumb -->
-		<joint name="${ns}_${name}_thumb_virtual_joint" type="revolute">
+		<joint name="${ns}_${name}_thumb_joint" type="revolute">
 			<axis xyz="0 0 -1"/>
 			<limit effort="30" velocity="10" lower="0" upper="1.57" />
@@ -44,7 +44,7 @@
 			<origin xyz=" -0.0000000021 32.5059e-3 39.6398e-3" rpy="0 0.3490656 1.5707963"/>
 			<parent link="${ns}_${name}_link"/>
-			<child link="${ns}_${name}_thumb_virtual_link"/>
+			<child link="${ns}_${name}_thumb_link"/>
 		</joint>
-	    <link name="${ns}_${name}_thumb_virtual_link">
+	    <link name="${ns}_${name}_thumb_link">
 		   <inertial>
 				<origin rpy="0 0 0" xyz="0 0 0"/>
@@ -56,5 +56,5 @@
 	    </link>
 		<!-- palm base to Litte virtual -->
-		<joint name="${ns}_${name}_little_virtual_joint" type="revolute">
+		<joint name="${ns}_${name}_little_joint" type="revolute">
 			<axis xyz="0 0 1"/>
 			<dynamics damping="0.0" friction="0.0"/>
@@ -62,7 +62,7 @@
 			<origin xyz=" -0.0000000091 -10.6603e-3 66.1817e-3" rpy="0 -0.1745327 -1.5707963"/>
 			<parent link="${ns}_${name}_link"/>
-			<child link="${ns}_${name}_little_virtual_link"/>
+			<child link="${ns}_${name}_little_link"/>
 		</joint>
-		<link name="${ns}_${name}_little_virtual_link">
+		<link name="${ns}_${name}_little_link">
 		   <inertial>
 			<origin rpy="0 0 0" xyz="0 0 0"/>

File: softhands_description/urdf/xacro/include/macro/v1_wide/modules/palm/palm_little.xacro (robot description, xacro)
@@ -2,5 +2,5 @@
 <robot xmlns:xacro="http://www.ros.org/wiki/xacro">
     <xacro:macro name="palm_little" params="name parent side *origin ns">
-		<joint name="${ns}_${name}_joint" type="revolute">
+		<joint name="${ns}_${parent}_virtual_joint" type="revolute">
 			<parent link="${ns}_${parent}_link"/>
 			<child link="${ns}_${name}_link"/>

File: softhands_description/urdf/xacro/include/macro/v1_wide/modules/palm/palm_thumb.xacro (robot description, xacro)
@@ -2,5 +2,5 @@
 <robot xmlns:xacro="http://www.ros.org/wiki/xacro">
     <xacro:macro name="palm_thumb" params="name parent side *origin ns">
-		<joint name="${ns}_${name}_joint" type="revolute">
+		<joint name="${ns}_${parent}_virtual_joint" type="revolute">
 			<parent link="${ns}_${parent}_link"/>
 			<child link="${ns}_${name}_link"/>

File: softhands_description/urdf/xacro/include/macro/v1_wide/modules/thumb/thumb_distal.xacro (robot description, xacro)
@@ -9,4 +9,5 @@
 			<child link="${ns}_${name}_virtual_link"/>
 			<limit effort="30" velocity="10" lower="0" upper="0.785398" />
+			<dynamics damping="$(arg virtual_damping)" friction="$(arg virtual_friction)"/>
 		</joint>
 	    <link name="${ns}_${name}_virtual_link">
@@ -24,5 +25,5 @@
 			<axis xyz="0 0 1" />
       		<limit effort="30" velocity="1.0" lower="0" upper="0.785398" />
-			<dynamics damping="0.0" friction="0.0" />
+			<dynamics damping="$(arg damping)" friction="$(arg friction)"/>
 		</joint>
 		<link name="${ns}_${name}_link">
@@ -52,5 +53,5 @@
 		<gazebo reference="${ns}_${name}_link">
 			<material>Gazebo/Grey</material>
-			<selfCollide>false</selfCollide>
+			<selfCollide>$(arg selfCollide)</selfCollide>
 			<kp value="1e4" />
 			<kd value="1e2" />

File: softhands_description/urdf/xacro/include/macro/v1_wide/modules/thumb/thumb_knuckle.xacro (robot description, xacro)
@@ -9,5 +9,5 @@
 			<axis xyz="0 0 1" />
       		<limit effort="30" velocity="1.0" lower="0" upper="1.57" />
-			<dynamics damping="0.0" friction="0.0" />
+			<dynamics damping="$(arg damping)" friction="$(arg friction)"/>
 		</joint>
 		<link name="${ns}_${name}_link">
@@ -37,5 +37,5 @@
 		<gazebo reference="${ns}_${name}_link">
 			<material>Gazebo/Grey</material>
-			<selfCollide>false</selfCollide>
+			<selfCollide>$(arg selfCollide)</selfCollide>
 			<kp value="1e4" />
 			<kd value="1e2" />

File: softhands_description/urdf/xacro/include/macro/v1_wide/modules/thumb/thumb_proximal.xacro (robot description, xacro)
@@ -9,4 +9,5 @@
 			<parent link="${ns}_${parent}_link"/>
 			<child link="${ns}_${name}_virtual_link"/>
+			<dynamics damping="$(arg virtual_damping)" friction="$(arg virtual_friction)"/>
 		</joint>
 	    <link name="${ns}_${name}_virtual_link">
@@ -24,5 +25,5 @@
 			<axis xyz="0 0 1" />
       		<limit effort="30" velocity="1.0" lower="0" upper="0.785398" />
-			<dynamics damping="0.0" friction="0.0" />
+			<dynamics damping="$(arg damping)" friction="$(arg friction)"/>
 		</joint>
 		<link name="${ns}_${name}_link">
@@ -52,5 +53,5 @@
 		<gazebo reference="${ns}_${name}_link">
 			<material>Gazebo/Grey</material>
-			<selfCollide>false</selfCollide>
+			<selfCollide>$(arg selfCollide)</selfCollide>
 			<kp value="1e4" />
 			<kd value="1e2" />

File: softhands_description/urdf/xacro/include/macro/v1_wide/plugin.xacro (robot description, xacro)
@@ -42,6 +42,6 @@
 			<namespace>$(arg ns)</namespace>
 			<operation_mode>$(arg operation_mode)</operation_mode>
-			<close_rate>0.001</close_rate>
 			<spring_k>0.5</spring_k>
+			<wide>true</wide>
 			<r_finger>0.0033</r_finger>
 			<R_pulley>0.0053</R_pulley>
@@ -85,4 +85,10 @@
 			<k_little_j3>0.5</k_little_j3>
 			<k_little_j4>0.5</k_little_j4>
+			<synS_palm_j1>0.1</synS_palm_j1>
+			<synS_palm_j2>1.57</synS_palm_j2>
+			<k_palm_j1>0.5</k_palm_j1>
+			<k_palm_j2>0.5</k_palm_j2>
+			<k_palm_j1_mimic>0.5</k_palm_j1_mimic>
+			<k_palm_j2_mimic>0.5</k_palm_j2_mimic>
 		</plugin>
 	</gazebo>
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