Commit message: added left hand

File: softhands_description/urdf/softhands.urdf.xacro (robot description, xacro)
@@ -38,12 +38,15 @@
 -->
 <robot name="softhand" xmlns:xacro="http://www.ros.org/wiki/xacro">
-  	<!-- <xacro:arg name="sh_version" default="v1_2_research"/> -->
-  	<xacro:arg name="sh_version" default="v1_wide"/>
+  	<xacro:arg name="sh_version" default="v1_2_research"/>
+  	<!-- <xacro:arg name="sh_version" default="v1_wide"/> -->
   	<xacro:arg name="root_dir" default="$(find softhands_description)/urdf/xacro/include/macro/$(arg sh_version)"/>
   	<xacro:arg name="root_link" default="world"/>
-  	<xacro:arg name="side" default="right"/>
+  	<xacro:arg name="side" default="left"/>
   	<xacro:arg name="meshes_dir" default="package://softhands_description/meshes/$(arg sh_version)/$(arg side)"/>
   	<xacro:arg name="ns" default="$(arg side)_hand_$(arg sh_version)"/>
-  	<xacro:arg name="position" default="0 0 0.01"/>
+  	<xacro:arg name="x" default="0"/>
+  	<xacro:arg name="y" default="0"/>
+  	<xacro:arg name="z" default="0"/>
+  	<xacro:arg name="position" default="$(arg x) $(arg y) $(arg z)"/>
   	<xacro:arg name="roll" default="0"/>
   	<xacro:arg name="pitch" default="0"/>
@@ -53,8 +56,8 @@
   	<xacro:arg name="selfCollide" default="0"/>
 	<xacro:include filename="$(arg root_dir)/header.xacro"/>
-  	<xacro:arg name="friction" default="1e-2"/>
-  	<xacro:arg name="virtual_friction" default="1e-2"/>
-  	<xacro:arg name="virtual_damping" default="0.0"/>
-  	<xacro:arg name="damping" default="0.0"/>
+  	<xacro:arg name="friction" default="0"/>
+  	<xacro:arg name="virtual_friction" default="0"/>
+  	<xacro:arg name="virtual_damping" default="0.05"/>
+  	<xacro:arg name="damping" default="0.05"/>
 	<xacro:include filename="$(find softhands_description)/urdf/xacro/$(arg sh_version).xacro"/>
 	<!-- Include plugin -->

File: softhands_description/urdf/xacro/include/macro/v1_2_research/modules/finger/phalanx.xacro (robot description, xacro)
@@ -57,4 +57,10 @@
         		      izz="0.0001" />
       </inertial>
+      <visual>
+        <geometry>
+          <cylinder length="0.005" radius="0.004"/>
+        </geometry>
+          <origin xyz="0 0 0" rpy="0 0 0"/>
+      </visual>
     </link>
     <!-- Proximal JOINT -->
@@ -70,8 +76,11 @@
     <link name="${ns}_${name}_link">
       <inertial>
-        <mass value="0.0082"/>
         <origin rpy="0 0 0" xyz="8.7707437e-03 -1.7863138e-03 0.0"/>
-        <inertia ixx="2.2722068e-07" ixy="1.1586053e-08" ixz="0.0" iyy="5.5947233e-07" iyz="0.0" izz="5.9562195e-07"/>
-        <!-- <inertia ixx="0.001" ixy="0" ixz="0" iyy="0.001" iyz="0" izz="0.001"/> -->
+        <!-- Original value -->
+        <!-- <mass value="0.0082"/>
+        <inertia ixx="2.2722068e-07" ixy="1.1586053e-08" ixz="0.0" iyy="5.5947233e-07" iyz="0.0" izz="5.9562195e-07"/> -->
+        <!-- Old value -->
+        <mass value="0.005"/>
+        <inertia ixx="0.001" ixy="0" ixz="0" iyy="0.001" iyz="0" izz="0.001"/>
       </inertial>
       <visual>
@@ -93,4 +102,14 @@
       <material>Gazebo/Grey</material>
       <selfCollide>$(arg selfCollide)</selfCollide>
+      <kp value="1e4" />
+      <kd value="1e2" />
+      <surface>
+       <friction>
+        <ode>
+         <mu>0.133</mu>
+         <mu2>0.133</mu2>
+        </ode>
+       </friction>
+      </surface>
     </gazebo>
   </xacro:macro>

File: softhands_description/urdf/xacro/include/macro/v1_2_research/modules/finger/phalanx_distal.xacro (robot description, xacro)
@@ -51,5 +51,5 @@
     <link name="${ns}_${name}_virtual_link">
       <inertial>
-        <origin rpy="0 0 0" xyz="0 0 0"/>
+      <origin xyz="0 0 0" rpy="0 0 0"/>
         <mass value="0.001"/>
         <inertia  ixx="0.0001"      ixy="0"  	    ixz="0"
@@ -57,4 +57,10 @@
         		      izz="0.0001" />
       </inertial>
+      <visual>
+        <geometry>
+          <box size="0.001 0.001 0.001"/>
+        </geometry>
+        <origin xyz="0 0 0" rpy="0 0 0"/>
+      </visual>
     </link>
     <!-- Proximal JOINT -->
@@ -70,8 +76,11 @@
     <link name="${ns}_${name}_link">
         <inertial>
-          <mass value="0.009"/>
           <origin rpy="0 0 0" xyz="8.8025467e-03 -1.7219289e-03 0.0"/>
-          <inertia ixx="2.6586142e-07" ixy="1.2416847e-08" ixz="0.0" iyy="5.9935767e-07" iyz="0.0" izz="6.6781963e-07"/>
-          <!-- <inertia ixx="0.001" ixy="0" ixz="0" iyy="0.001" iyz="0" izz="0.001"/> -->
+          <!-- Original value -->
+          <!-- <mass value="0.009"/>
+          <inertia ixx="2.6586142e-07" ixy="1.2416847e-08" ixz="0.0" iyy="5.9935767e-07" iyz="0.0" izz="6.6781963e-07"/> -->
+          <!-- Old value -->
+          <mass value="0.005"/>
+          <inertia ixx="0.001" ixy="0" ixz="0" iyy="0.001" iyz="0" izz="0.001"/>
         </inertial>
       <visual>
@@ -93,4 +102,14 @@
       <material>Gazebo/Grey</material>
       <selfCollide>$(arg selfCollide)</selfCollide>
+      <kp value="1e4" />
+      <kd value="1e2" />
+      <surface>
+       <friction>
+        <ode>
+         <mu>0.133</mu>
+         <mu2>0.133</mu2>
+        </ode>
+       </friction>
+      </surface>
 	  </gazebo>
   </xacro:macro>

File: softhands_description/urdf/xacro/include/macro/v1_2_research/modules/finger/phalanx_knuckle.xacro (robot description, xacro)
@@ -46,12 +46,16 @@
       <axis xyz="0 0 -1"/>
       <limit effort="30" velocity="1.0" lower="-0.524" upper="0.524" />
-       <dynamics damping="0.08" friction="$(arg friction)"/>
+       <dynamics damping="$(arg damping)" friction="$(arg friction)"/>
     </joint>
     <!-- LINK -->
     <link name="${ns}_${name}_link">
       <inertial>
-        <mass value="0.0095"/>
         <origin rpy="0 0 0" xyz="4.2753603e-04  0.0 -1.4321738e-03"/>
-        <inertia ixx="6.4337303e-07" ixy="0.0" ixz="-3.9373913e-08" iyy="1.1253771e-06" iyz="0.0" izz="7.2336948e-07"/>
+        <!-- Original value -->
+        <!-- <mass value="0.0095"/>
+        <inertia ixx="6.4337303e-07" ixy="0.0" ixz="-3.9373913e-08" iyy="1.1253771e-06" iyz="0.0" izz="7.2336948e-07"/> -->
+        <!-- Old value -->
+        <mass value="0.005"/>
+        <inertia ixx="0.001" ixy="0" ixz="0" iyy="0.001" iyz="0" izz="0.001"/>
       </inertial>
       <visual>
@@ -73,4 +77,14 @@
       <material>Gazebo/Grey</material>
       <selfCollide>$(arg selfCollide)</selfCollide>
+            <kp value="1e4" />
+      <kd value="1e2" />
+      <surface>
+       <friction>
+        <ode>
+         <mu>0.133</mu>
+         <mu2>0.133</mu2>
+        </ode>
+       </friction>
+      </surface>
     </gazebo>
   </xacro:macro>

File: softhands_description/urdf/xacro/include/macro/v1_2_research/modules/finger/phalanx_short.xacro (robot description, xacro)
@@ -57,4 +57,10 @@
         		      izz="0.0001" />
       </inertial>
+	      <visual>
+        <geometry>
+          <cylinder length="0.005" radius="0.004"/>
+        </geometry>
+        <origin xyz="0 0 0" rpy="0 0 0"/>
+      </visual>
     </link>
     <!-- Proximal JOINT -->
@@ -70,8 +76,11 @@
     <link name="${ns}_${name}_link">
       <inertial>
-        <mass value="0.0063"/>
         <origin rpy="0 0 0" xyz="4.7601567e-03 -1.3786947e-03 0.0"/>
-        <inertia ixx="1.8024201e-07" ixy="5.756798e-09" ixz="0.0" iyy="2.3516266e-07" iyz="0.0" izz="2.691504e-07"/>
-        <!-- <inertia ixx="0.001" ixy="0" ixz="0" iyy="0.001" iyz="0" izz="0.001"/> -->
+        <!-- Original value -->
+        <!-- <mass value="0.0063"/>
+        <inertia ixx="1.8024201e-07" ixy="5.756798e-09" ixz="0.0" iyy="2.3516266e-07" iyz="0.0" izz="2.691504e-07"/> -->
+        <!-- Old value -->
+        <mass value="0.005"/>
+        <inertia ixx="0.001" ixy="0" ixz="0" iyy="0.001" iyz="0" izz="0.001"/>
       </inertial>
       <visual>
@@ -93,4 +102,14 @@
       <material>Gazebo/Grey</material>
       <selfCollide>$(arg selfCollide)</selfCollide>
+      <kp value="1e4" />
+      <kd value="1e2" />
+      <surface>
+       <friction>
+        <ode>
+         <mu>0.133</mu>
+         <mu2>0.133</mu2>
+        </ode>
+       </friction>
+      </surface>
     </gazebo>
   </xacro:macro>

File: softhands_description/urdf/xacro/include/macro/v1_2_research/modules/iso.xacro (robot description, xacro)
@@ -38,5 +38,5 @@
 -->
 <robot name="iso_v2" xmlns:xacro="http://www.ros.org/wiki/xacro">
-	<xacro:macro name="iso" params="ns name parent *origin side">
+	<xacro:macro name="iso" params="ns name parent *origin">
 		<!-- World to palm base -->
 		<joint name="${ns}_${name}_joint" type="fixed">
@@ -47,7 +47,11 @@
 		<link name="${ns}_${name}_link">
 			<inertial>
+				<origin rpy="0 0 0" xyz="0.0 7.8738498e-04 1.5878899e-02"/>
+				<!-- Original value -->
+				<!--<mass value="0.205"/>
+				<inertia ixx="0.00012506929" ixy="0.0" ixz="0.0" iyy="0.0001338779" iyz="0.0" izz="0.00019218394"/> -->
+				<!-- Old value -->
 				<mass value="0.205"/>
-				<origin rpy="0 0 0" xyz="0.0030 -0.0449 0.0135"/>
-				<inertia ixx="0.00012506929" ixy="0.0" ixz="0.0" iyy="0.0001338779" iyz="0.0" izz="0.00019218394"/>
+				<inertia ixx="0.001" ixy="0" ixz="0" iyy="0.001" iyz="0" izz="0.001"/>
 			</inertial>
 			<visual>

File: softhands_description/urdf/xacro/include/macro/v1_2_research/modules/palm/palm.xacro (robot description, xacro)
@@ -38,5 +38,5 @@
 -->
 <robot name="palm_v2" xmlns:xacro="http://www.ros.org/wiki/xacro">
-	<xacro:macro name="palm" params="ns name parent *origin side">
+	<xacro:macro name="palm" params="ns name parent *origin">
 	  	<joint name="${ns}_palm_joint" type="fixed">
 			<xacro:insert_block name="origin"/>
@@ -46,7 +46,11 @@
 		<link name="${ns}_palm_link">
 			<inertial>
-				<mass value="0.45"/>
-				<origin rpy="0 0 0" xyz="0.0030 -0.0449 0.0135"/>
-				<inertia ixx="0.00045" ixy="0.0" ixz="0.0" iyy="0.00025" iyz="0.0" izz="0.0006"/>
+				<origin rpy="0 0 0" xyz="0.0030 -0.0449 ${sign*0.0135}"/>
+				<!-- Original value -->
+				<!-- <mass value="0.45"/>
+				<inertia ixx="0.00045" ixy="0.0" ixz="0.0" iyy="0.00025" iyz="0.0" izz="0.0006"/> -->
+				<!-- Old value -->
+				<mass value="2.28"/>
+				<inertia ixx="0.001" ixy="0" ixz="0" iyy="0.001" iyz="0" izz="0.001"/>
 			</inertial>
 			<visual>
@@ -67,4 +71,14 @@
 			<material>Gazebo/Grey</material>
 			<selfCollide>$(arg selfCollide)</selfCollide>
+			<kp value="1e4" />
+			<kd value="1e2" />
+			<surface>
+			<friction>
+				<ode>
+				<mu>0.133</mu>
+				<mu2>0.133</mu2>
+				</ode>
+			</friction>
+			</surface>
 		</gazebo>
 	</xacro:macro>

File: softhands_description/urdf/xacro/include/macro/v1_2_research/modules/thumb.xacro (robot description, xacro)
@@ -41,9 +41,14 @@
     <!-- Knuckle -->
     <xacro:thumb_knuckle name="${name}_knuckle" parent="${parent}" ns="$(arg ns)" side="$(arg side)">
-      <origin rpy="-1.57 3.14 0.0" xyz="-0.044 -0.0465 -0.002"/>
+      <origin rpy="-1.57 3.14 0.0" xyz="-0.044 -0.0465 ${sign*-0.002}"/>
     </xacro:thumb_knuckle>
     <!-- Proximal  -->
     <xacro:thumb_short name="${name}_proximal" parent="${name}_knuckle" ns="$(arg ns)" side="$(arg side)">
-      <origin rpy="-1.1415 0.0 0.0" xyz="0.0255 -0.0038 -0.00012"/>
+      <xacro:if value="${side == 'left'}">
+        <origin rpy="-2 0.0 0.0" xyz="0.0255 0.0038 -0.00012"/>
+      </xacro:if>
+      <xacro:if value="${side == 'right'}">
+        <origin rpy="-1.1415 0.0 0.0" xyz="0.0255 -0.0038 -0.00012"/>
+      </xacro:if>
     </xacro:thumb_short>
     <!-- Distal  -->

File: softhands_description/urdf/xacro/include/macro/v1_2_research/modules/thumb/thumb_knuckle.xacro (robot description, xacro)
@@ -44,14 +44,18 @@
       <parent link="${ns}_${parent}_link"/>
       <child link="${ns}_${name}_link"/>
-      <axis xyz="0 0 -1"/>
+      <axis xyz="0 0 ${sign*-1}"/>
       <limit effort="30" velocity="1.0" lower="0" upper="1.57" />
-      <dynamics damping="0.08" friction="0.0" />
+      <dynamics damping="$(arg damping)" friction="$(arg friction)" />
     </joint>
     <!-- LINK -->
     <link name="${ns}_${name}_link">
       <inertial>
-        <mass value="0.01"/>
-        <origin rpy="0 0 0" xyz="1.3071561e-02 -2.7357764e-03 6.4347823e-04"/>
-        <inertia ixx="3.5865978e-07" ixy="2.0944224e-07" ixz="-6.8657569e-08" iyy="1.3885564e-06" iyz="3.2170608e-08" izz="1.3571203e-06"/>
+        <origin rpy="0 0 0" xyz="1.3071561e-02 ${sign*-2.7346340e-03} 6.4090487e-04"/>
+        <!-- Original value -->
+        <!-- <mass value="0.01"/>
+        <inertia ixx="3.5865978e-07" ixy="${sign*2.0944224e-07}" ixz="-6.8657569e-08" iyy="1.3885564e-06" iyz="${sign*3.2170608e-08}" izz="1.3571203e-06"/> -->
+        <!-- Old value -->
+        <mass value="0.005"/>
+        <inertia ixx="0.001" ixy="0" ixz="0" iyy="0.001" iyz="0" izz="0.001"/>
       </inertial>
       <visual>
@@ -72,5 +76,15 @@
     <gazebo reference="${ns}_${name}_link">
       <material>Gazebo/Grey</material>
-      <selfCollide>false</selfCollide>
+      <selfCollide>$(arg selfCollide)</selfCollide>
+      <!-- <kp value="1e4" />
+      <kd value="1e2" />
+      <surface>
+       <friction>
+        <ode>
+         <mu>0.133</mu>
+         <mu2>0.133</mu2>
+        </ode>
+       </friction>
+      </surface> -->
     </gazebo>
   </xacro:macro>

File: softhands_description/urdf/xacro/include/macro/v1_2_research/modules/thumb/thumb_short.xacro (robot description, xacro)
@@ -51,5 +51,5 @@
     <link name="${ns}_${name}_virtual_link">
       <inertial>
-      <origin rpy="0 0 0" xyz="0 0 0"/>
+      <origin xyz="0 0 0" rpy="0 0 0"/>
         <mass value="0.001"/>
         <inertia  ixx="0.0001"      ixy="0"  	    ixz="0"
@@ -57,4 +57,10 @@
         		      izz="0.0001" />
       </inertial>
+      <visual>
+        <geometry>
+          <box size="0.001 0.001 0.001"/>
+        </geometry>
+        <origin xyz="0 0 0" rpy="0 0 0"/>
+      </visual>
     </link>
     <!-- Proximal JOINT -->
@@ -70,8 +76,11 @@
     <link name="${ns}_${name}_link">
       <inertial>
-        <mass value="0.0063"/>
         <origin rpy="0 0 0" xyz="4.7601567e-03 -1.3786947e-03 0.0"/>
-        <inertia ixx="1.8024201e-07" ixy="5.756798e-09" ixz="0.0" iyy="2.3516266e-07" iyz="0.0" izz="2.691504e-07"/>
-        <!-- <inertia ixx="0.001" ixy="0" ixz="0" iyy="0.001" iyz="0" izz="0.001"/> -->
+        <!-- Original value -->
+        <!-- <mass value="0.0032"/>
+        <inertia ixx="1.8024201e-07" ixy="5.756798e-09" ixz="0.0" iyy="2.3516266e-07" iyz="0.0" izz="2.691504e-07"/> -->
+        <!-- Old value -->
+        <mass value="0.005"/>
+        <inertia ixx="0.001" ixy="0" ixz="0" iyy="0.001" iyz="0" izz="0.001"/>
       </inertial>
       <visual>
@@ -89,12 +98,18 @@
       </collision>
     </link>
-    <!-- GAZEBO REF -->
-    <gazebo reference="${ns}_${name}_virtual_link">
-      <material>Gazebo/Grey</material>
-    </gazebo>
         <!-- GAZEBO REF -->
     <gazebo reference="${ns}_${name}_link">
       <material>Gazebo/Grey</material>
       <selfCollide>$(arg selfCollide)</selfCollide>
+      <kp value="1e4" />
+      <kd value="1e2" />
+      <surface>
+       <friction>
+        <ode>
+         <mu>0.133</mu>
+         <mu2>0.133</mu2>
+        </ode>
+       </friction>
+      </surface>
     </gazebo>
   </xacro:macro>

File: softhands_description/urdf/xacro/include/macro/v1_2_research/plugin.xacro (robot description, xacro)
@@ -42,5 +42,5 @@
 			<namespace>$(arg ns)</namespace>
 			<operation_mode>$(arg operation_mode)</operation_mode>
-			<spring_k>0.5</spring_k>
+			<spring_k>5</spring_k>
 			<r_finger>0.0033</r_finger>
 			<R_pulley>0.0053</R_pulley>

File: softhands_description/urdf/xacro/v1_2_research.xacro (robot description, xacro)
@@ -38,15 +38,24 @@
 -->
 <robot name="right_hand_v2" xmlns:xacro="http://www.ros.org/wiki/xacro">
+	<xacro:property name="side" value="$(arg side)"/>
+	<xacro:property name="sign" default="1"/>
+	<xacro:if value="${side == 'left'}">
+		<xacro:property name="sign" value="-1"/>
+	</xacro:if>
 	<!-- World -->
 	<link name="$(arg root_link)">
 	</link>
 	<!-- # iso -->
-	<xacro:iso name="iso" parent="$(arg root_link)" ns="$(arg ns)" side="$(arg side)">
+	<xacro:iso name="iso" parent="$(arg root_link)" ns="$(arg ns)">
 		<origin rpy="$(arg orientation)" xyz="$(arg position)"/>
 	</xacro:iso>
 	<!-- # palm  -->
-	<xacro:palm name="palm" parent="iso" ns="$(arg ns)" side="$(arg side)">
-		<origin rpy="1.57 0 0" xyz="-0.0045 0.0145 0.144"/>
-		<!-- <origin rpy="0 0 0" xyz="-0.0045 0.0145 0.144"/> -->
+	<xacro:palm name="palm" parent="iso" ns="$(arg ns)">
+		<xacro:if value="${side == 'left'}">
+			<origin rpy="1.57 0  3.14" xyz="0.0045 0.0145 0.144"/>
+		</xacro:if>
+		<xacro:if value="${side == 'right'}">
+			<origin rpy="1.57 0 0" xyz="-0.0045 0.0145 0.144"/>
+		</xacro:if>
 	</xacro:palm>
 	<!-- # thumb -->
@@ -56,17 +65,37 @@
 	<!-- # Index -->
 	<xacro:finger name="index" parent="palm" ns="$(arg ns)" side="$(arg side)">
-		<origin rpy="0 0 1.57" xyz="-0.02 -0.007 0.014"/>
+		<xacro:if value="${side == 'left'}">
+			<origin rpy="0 3.14 -1.57" xyz="-0.02 -0.007 -0.014"/>
+		</xacro:if>
+		<xacro:if value="${side == 'right'}">
+			<origin rpy="0 0 1.57" xyz="-0.02 -0.007 0.014"/>
+		</xacro:if>
 	</xacro:finger>
 	<!-- # Middle -->
 	<xacro:finger name="middle" parent="palm" ns="$(arg ns)" side="$(arg side)">
-		<origin rpy="0 0 1.57" xyz="0 0 0.014"/>
+		<xacro:if value="${side == 'left'}">
+			<origin rpy="0 3.14 -1.57" xyz="0 0 -0.014"/>
+		</xacro:if>
+		<xacro:if value="${side == 'right'}">
+			<origin rpy="0 0 1.57" xyz="0 0 0.014"/>
+		</xacro:if>
 	</xacro:finger>
 	<!-- # Ring -->
 	<xacro:finger name="ring" parent="palm" ns="$(arg ns)" side="$(arg side)">
-		<origin rpy="0 0 1.57" xyz="0.02 -0.007 0.014"/>
+		<xacro:if value="${side == 'left'}">
+			<origin rpy="0 3.14 -1.57" xyz="0.02 -0.007 -0.014"/>
+		</xacro:if>
+		<xacro:if value="${side == 'right'}">
+			<origin rpy="0 0 1.57" xyz="0.02 -0.007 0.014"/>
+		</xacro:if>
 	</xacro:finger>
 	<!-- # Little -->
 	<xacro:finger name="little" parent="palm" ns="$(arg ns)" side="$(arg side)">
-		<origin rpy="0 0 1.57" xyz="0.04 -0.012 0.014"/>
+		<xacro:if value="${side == 'left'}">
+			<origin rpy="0 3.14 -1.57" xyz="0.04 -0.012 -0.014"/>
+		</xacro:if>
+		<xacro:if value="${side == 'right'}">
+			<origin rpy="0 0 1.57" xyz="0.04 -0.012 0.014"/>
+		</xacro:if>
 	</xacro:finger>
 </robot>
