Commit message: added grasp link and test on repair robot

File: softhands_description/urdf/softhands.urdf.xacro (robot description, xacro)
@@ -43,5 +43,5 @@
         version="$(arg sh_version)"
         position="0 0 0"
-        orientation="0 0 0"
+        orientation="0.78"
         fixed_hands="false">
     </xacro:softhands>

File: softhands_description/urdf/softhands.xacro (robot description, xacro)
@@ -39,8 +39,4 @@
 <robot name="softhands" xmlns:xacro="http://www.ros.org/wiki/xacro">
 	<xacro:macro name="softhands" params="version position orientation fixed_hands:='false'">
-		<xacro:property name="mm" value="1000"/>
-		<xacro:property name="mm2_to_m2" value="0.001"/>
-		<xacro:property name="gr_to_Kg" value="0.001"/>
-		<xacro:property name="negligible_mass" value="${10*gr_to_Kg}" />
 		<xacro:include filename="$(find softhands_description)/urdf/xacro/include/macro/color.xacro" />
 		<xacro:include filename="$(find softhands_description)/urdf/xacro/include/macro/plugin.xacro"/>
@@ -73,6 +69,6 @@
 				side="left"
 				parent="arm_1_7"
-				position="0 -0.0 0.00"
-				orientation="0 0 ${orientation}"
+				position="0 0 0.0"
+				orientation="0 0 ${-orientation}"
 				fixed_hands="false">
 			</xacro:v1_wide>
@@ -80,5 +76,5 @@
 				side="right"
 				parent="arm_2_7"
-				position="0 0.0 0.0"
+				position="0 0 0.0"
 				orientation="0 0 ${orientation}"
 				fixed_hands="false">

File: softhands_description/urdf/xacro/include/macro/v1_2_research/modules/iso.xacro (robot description, xacro)
@@ -69,4 +69,11 @@
 			<selfCollide>0</selfCollide>
 	  	</gazebo>
+		<!-- Fake joint and link for grasping -->
+	  	<joint name="${ns}_grasp_joint" type="fixed">
+			<origin rpy="0 0 0" xyz="0.03 0.06 0.10"/>
+			<parent link="${ns}_${name}_link" />
+			<child link="${ns}_grasp_link" />
+		</joint>
+		<link name="${ns}_grasp_link"/>
 	</xacro:macro>
 </robot>

File: softhands_description/urdf/xacro/include/macro/v1_wide/header.xacro (robot description, xacro)
@@ -38,4 +38,5 @@
 -->
 <robot xmlns:xacro="http://www.ros.org/wiki/xacro" name="header">
+  <xacro:include filename="$(find softhands_description)/urdf/xacro/include/macro/v1_wide/modules/iso.xacro" />
   <!-- Include xacro macro  Palm-->
 	<xacro:include filename="$(find softhands_description)/urdf/xacro/include/macro/v1_wide/modules/palm/palm_central.xacro" />

File: softhands_description/urdf/xacro/include/macro/v1_wide/modules/finger/phalanx_knuckle.xacro (robot description, xacro)
@@ -5,5 +5,5 @@
 		<joint name="${ns}_${name}_joint" type="revolute">
 			<axis xyz="0 1 0"/>
-			<limit effort="30" velocity="0.0" lower="0.0" upper="0.0" />
+			<limit effort="30" velocity="0.0" lower="0.0" upper="0.01" />
 			<xacro:insert_block name="origin"/>
             <parent link="${ns}_${parent}_link"/>
@@ -12,4 +12,5 @@
 		<link name="${ns}_${name}_link">
 				<visual>
+				<material name="grey" />
 					<geometry>
 					<mesh

File: softhands_description/urdf/xacro/include/macro/v1_wide/modules/iso.xacro (robot description, xacro)
@@ -37,35 +37,36 @@
  *
 -->
-<robot name="palm_v2" xmlns:xacro="http://www.ros.org/wiki/xacro">
-	<xacro:macro name="palm" params="ns name parent *origin">
-	  	<joint name="${ns}_palm_joint" type="fixed">
+<robot name="iso_v2" xmlns:xacro="http://www.ros.org/wiki/xacro">
+	<xacro:macro name="iso" params="ns name parent *origin">
+		<!-- World to palm base -->
+		<joint name="${ns}_${name}_joint" type="fixed">
+			<parent link="${parent}"/>
+			<child link="${ns}_${name}_link"/>
 			<xacro:insert_block name="origin"/>
-			<parent link="${ns}_${parent}_link" />
-			<child link="${ns}_palm_link" />
 		</joint>
-		<link name="${ns}_palm_link">
+		<link name="${ns}_${name}_link">
 			<inertial>
-				<origin rpy="0 0 0" xyz="0.0030 -0.0449 ${sign*0.0135}"/>
-				<mass value="0.45"/>
-				<inertia ixx="0.00045" ixy="0.0" ixz="0.0" iyy="0.00025" iyz="0.0" izz="0.0006"/>
+				<mass value="0.205"/>
+				<origin rpy="0 0 0" xyz="0.0 7.8738498e-04 1.5878899e-02"/>
+				<inertia ixx="0.00012506929" ixy="0.0" ixz="0.0" iyy="0.0001338779" iyz="0.0" izz="0.00019218394"/>
 			</inertial>
 			<visual>
-			<origin rpy="0 0 0" xyz="0 0 0"/>
-			<geometry>
-				<mesh filename="package://softhands_description/meshes/v1_2_research/${side}/palm_pinch.stl" scale="0.001 0.001 0.001"/>
-			</geometry>
-			<material name="qbhand/palm"/>
+				<origin rpy="0 0 0" xyz="0 0 0"/>
+				<geometry>
+					<mesh filename="package://softhands_description/meshes/v1_wide/${side}/flange_iso_04.stl" scale="0.001 0.001 0.001"/>
+				</geometry>
+				<material name="qbhand/base"/>
 			</visual>
 			<collision>
 			<origin rpy="0 0 0" xyz="0 0 0"/>
 			<geometry>
-				<mesh filename="package://softhands_description/meshes/v1_2_research/${side}/palm_pinch.stl" scale="0.001 0.001 0.001"/>
+				<mesh filename="package://softhands_description/meshes/v1_wide/${side}/flange_iso_04.stl" scale="0.001 0.001 0.001"/>
 			</geometry>
 			</collision>
 		</link>
-		<gazebo reference="${ns}_palm_link">
-			<material>Gazebo/Grey</material>
+		<gazebo reference="${ns}_${name}_link">
+    	  	<material>Gazebo/Grey</material>
 			<selfCollide>0</selfCollide>
-		</gazebo>
+	  	</gazebo>
 	</xacro:macro>
 </robot>

File: softhands_description/urdf/xacro/include/macro/v1_wide/modules/palm/palm_central.xacro (robot description, xacro)
@@ -11,4 +11,5 @@
 		<link name="${ns}_${name}_link">
 			<visual>
+				<material name="grey" />
 				<geometry>
 				<mesh
@@ -19,5 +20,5 @@
 			</visual>
 			<inertial>
-				<mass value="${mass}" />
+				<mass value="${mass/3}" />
 				<xacro:insert_block name="inertia_origin"/>
 				<xacro:insert_block name="inertia"/>
@@ -32,8 +33,15 @@
 			</collision>
 		</link>
+		<!-- Fake joint and link for grasping -->
+	  	<joint name="${ns}_grasp_joint" type="fixed">
+			<origin rpy="0 0 0" xyz="0.03 -0.06 0.10"/>
+			<parent link="${ns}_${name}_link" />
+			<child link="${ns}_grasp_link" />
+		</joint>
+		<link name="${ns}_grasp_link"/>
 		<!-- palm base to Thumb -->
 		<joint name="${ns}_${name}_thumb_joint" type="revolute">
 			<axis xyz="0 0 ${sign*-1}"/>
-			<limit effort="30" velocity="0.0" lower="0" upper="0.3" />
+			<limit effort="30" velocity="0.0" lower="0" upper="0.17" />
 			<dynamics damping="$(arg virtual_damping)" friction="$(arg virtual_friction)"/>
 			<xacro:insert_block name="thumb_origin"/>
@@ -44,5 +52,5 @@
 		   <inertial>
 				<origin rpy="0 0 0" xyz="0 0 0"/>
-				<mass value="0.001"/>
+				<mass value="${mass/3}" />
 				<xacro:insert_block name="inertia"/>
 		   </inertial>
@@ -52,5 +60,5 @@
 			<axis xyz="0 0 1"/>
 			<dynamics damping="$(arg virtual_damping)" friction="$(arg virtual_friction)"/>
-			<limit effort="100" velocity="0.00" lower="0.0" upper="0.3" />
+			<limit effort="100" velocity="0.00" lower="0.0" upper="0.17" />
 			<xacro:insert_block name="little_origin"/>
 			<parent link="${ns}_${name}_link"/>
@@ -60,5 +68,5 @@
 			<inertial>
 				<origin rpy="0 0 0" xyz="0 0 0"/>
-				<mass value="0.001"/>
+				<mass value="${mass/3}" />
 				<xacro:insert_block name="inertia"/>
 			</inertial>

File: softhands_description/urdf/xacro/include/macro/v1_wide/modules/palm/palm_little.xacro (robot description, xacro)
@@ -7,5 +7,5 @@
 			<xacro:insert_block name="origin"/>
 			<axis xyz="0 0 1" />
-      		<limit effort="30" velocity="0.0" lower="0" upper="0.35" />
+      		<limit effort="30" velocity="0.0" lower="0" upper="0.17" />
 			<dynamics damping="$(arg damping)" friction="$(arg friction)"/>
 		</joint>

File: softhands_description/urdf/xacro/include/macro/v1_wide/modules/palm/palm_thumb.xacro (robot description, xacro)
@@ -7,8 +7,9 @@
 			<xacro:insert_block name="palm_thumb_origin"/>
 			<axis xyz="0 0 ${sign*-1}" />
-      		<limit effort="30" velocity="0.0" lower="0" upper="0.35" />
+      		<limit effort="30" velocity="0.0" lower="0" upper="0.17" />
 			 <dynamics damping="$(arg damping)" friction="$(arg friction)"/>
 		</joint>
 		<link name="${ns}_${name}_link">
+			<material name="grey" />
 			<visual>
 				<geometry>
@@ -40,4 +41,5 @@
 		</joint>
 		<link name="${ns}_${name}_support_link">
+				<material name="grey" />
 				<visual>
 					<geometry>
@@ -57,9 +59,9 @@
 				<collision>
 					<geometry>
-					<mesh
-						filename="package://softhands_description/meshes/v1_wide/${side}/thumb_support_collision.stl"
-						scale="0.0009 0.0009 0.0009" />
+						<mesh
+							filename="package://softhands_description/meshes/v1_wide/${side}/thumb_support_collision.stl"
+							scale="0.0009 0.0009 0.0009" />
 					</geometry>
-				<origin xyz="0 0 0" rpy="0 0 0" />
+					<origin xyz="0 0 0" rpy="0 0 0" />
 				</collision>
 		</link>
@@ -70,5 +72,5 @@
 		<gazebo reference="${ns}_${name}_support_link">
 			<selfCollide>0</selfCollide>
-			<material>Gazebo/White</material>
+			<material>Gazebo/Grey</material>
 		</gazebo>
     </xacro:macro>

Commit message: update structure sh3

File: softhands_description/urdf/softhands.urdf.xacro (robot description, xacro)
@@ -43,5 +43,5 @@
         version="$(arg sh_version)"
         position="0 0 0"
-        orientation="0 0 0"
+        orientation="1.57 0 0"
         fixed_hands="false">
     </xacro:softhands>

File: softhands_description/urdf/xacro/include/macro/v3/modules/finger.xacro (robot description, xacro)
@@ -38,33 +38,5 @@
 -->
 <robot xmlns:xacro="http://www.ros.org/wiki/xacro">
-  <xacro:macro name="finger" params="ns name parent *origin side ">
-    <!-- Proximal -->
-    <xacro:phalanx_knuckle name="${name}_knuckle" parent="${parent}" ns="${ns}" side="${side}" mesh="${index.mesh.knuckle_mesh}">
-     <xacro:insert_block name="origin"/>
-     <inertia_origin> <origin rpy="0 0 0" xyz="8.2672528e-03  -2.7479334e-03 6.3742013e-05"/>   </inertia_origin>
-     <mass value="2.9531895e-03"/>
-     <inertia ixx="4.9114511e-08" ixy="2.4336199e-08" ixz="1.1336750e-09" iyy="1.6520715e-07" iyz="0.0" izz="1.7172503e-07"/>
-    </xacro:phalanx_knuckle>
-    <!-- Proximal -->
-    <!-- <xacro:phalanx_generic name="${name}_proximal" parent="${name}_knuckle" ns="${ns}" mass="3.4433482e-03" mesh="${proximal_mesh}">
-      <virtual_origin>  <origin rpy="1.57 0 0" xyz="15e-03 -3.7e-03 0"/>                      </virtual_origin>
-      <real_origin>     <origin rpy="0.0 0 0" xyz="9e-03 0 0"/>                       </real_origin>
-      <inertia_origin>  <origin rpy="0 0 0" xyz="8.2958878e-03 1.4867666e-04 0.0"/>  </inertia_origin>
-      <inertia ixx="5.9259154e-08" ixy="4.7090997e-09" ixz="0.0" iyy="2.0151714e-07" iyz="0.0" izz="2.1338410e-07"/>
-    </xacro:phalanx_generic> -->
-    <!-- Middle -->
-    <!-- <xacro:phalanx_generic name="${name}_middle" parent="${name}_proximal" ns="${ns}" mass="0.0063" mesh="${middle_mesh}">
-      <virtual_origin>  <origin rpy="0.0 0.0 0.0" xyz="16e-03 0 0 "/>                  </virtual_origin>
-      <real_origin>     <origin rpy="0 0 0" xyz="16e-03 0 0"/>                         </real_origin>
-      <inertia_origin>  <origin rpy="0 0 0" xyz="4.7601567e-03 -1.3786947e-03 0.0"/>  </inertia_origin>
-      <inertia ixx="1.8024201e-07" ixy="5.756798e-09" ixz="0.0" iyy="2.3516266e-07" iyz="0.0" izz="2.691504e-07"/>
-    </xacro:phalanx_generic> -->
-    <!-- Distal -->
-    <!-- <xacro:phalanx_generic name="${name}_distal" parent="${name}_middle" ns="${ns}" mass="0.009" mesh="ph_distal">
-      <virtual_origin>  <origin rpy="0 0 0" xyz="0.009 0 0"/>                        </virtual_origin>
-      <real_origin>     <origin rpy="0 0 0" xyz="0.013 0 0"/>                         </real_origin>
-      <inertia_origin>  <origin rpy="0 0 0" xyz="8.8025467e-03 -1.7219289e-03 0.0"/>  </inertia_origin>
-      <inertia ixx="2.6586142e-07" ixy="1.2416847e-08" ixz="0.0" iyy="5.9935767e-07" iyz="0.0" izz="6.6781963e-07"/>
-    </xacro:phalanx_generic> -->
+  <xacro:macro name="finger" params="yaml_file:=^ ">
   </xacro:macro>
 </robot>

File: softhands_description/urdf/xacro/include/macro/v3/modules/phalanges/phalanx_generic.xacro (robot description, xacro)
@@ -38,16 +38,16 @@
 -->
 <robot xmlns:xacro="http://www.ros.org/wiki/xacro">
-  <xacro:macro name="phalanx_generic" params="name parent ns mass mesh **virtual_origin **real_origin **inertia_origin *inertia">
+  <xacro:macro name="phalanx_generic" params="yaml_file:=^ name type parent ns">
     <!-- Inner VIRTUAL JOINT -->
-		<joint name="${ns}_${name}_virtual_joint" type="revolute">
+		<joint name="${ns}_${name}_${type}_virtual_joint" type="revolute">
       <axis xyz="0 0 -1"/>
-      <xacro:insert_block name="virtual_origin"/>
+      <origin rpy="${yaml_file['finger']['${name}']['${type}']['virtual_origin']['orientation']}" xyz="${yaml_file['finger']['${name}']['${type}']['virtual_origin']['position']}"/>
 			<parent link="${ns}_${parent}_link"/>
-			<child link="${ns}_${name}_virtual_link"/>
+			<child link="${ns}_${name}_${type}_virtual_link"/>
       <limit effort="30" velocity="10.0" lower="0.0" upper="0.785398" />
       <dynamics damping="$(arg virtual_damping)" friction="$(arg virtual_friction)" />
 		</joint>
     <!-- VIRTUAL LINK -->
-    <link name="${ns}_${name}_virtual_link">
+    <link name="${ns}_${name}_${type}_virtual_link">
       <inertial>
         <origin rpy="0 0 0" xyz="0 0 0"/>
@@ -57,14 +57,14 @@
     </link>
     <!-- Outer JOINT -->
-    <joint name="${ns}_${name}_joint" type="revolute">
+    <joint name="${ns}_${name}_${type}_joint" type="revolute">
       <axis xyz="0 0 -1"/>
-      <xacro:insert_block name="real_origin"/>
-      <parent link="${ns}_${name}_virtual_link"/>
-      <child link="${ns}_${name}_link"/>
+      <origin rpy="${yaml_file['finger']['${name}']['${type}']['real_origin']['orientation']}" xyz="${yaml_file['finger']['${name}']['${type}']['real_origin']['position']}"/>
+      <parent link="${ns}_${name}_${type}_virtual_link"/>
+      <child link="${ns}_${name}_${type}_link"/>
       <limit effort="30" velocity="10.0" lower="0.0" upper="0.785398" />
       <dynamics damping="$(arg damping)" friction="$(arg friction)"/>
     </joint>
     <!-- LINK -->
-    <link name="${ns}_${name}_link">
+    <link name="${ns}_${name}_${type}_link">
         <inertial>
           <mass value="${mass}"/>
@@ -87,10 +87,10 @@
     </link>
     <!-- GAZEBO REF -->
-    <gazebo reference="${ns}_${name}_link">
+    <gazebo reference="${ns}_${name}_${type}_link">
       <material>Gazebo/Grey</material>
       <selfCollide>$(arg selfCollide)</selfCollide>
 	  </gazebo>
         <!-- GAZEBO REF -->
-    <gazebo reference="${ns}_${name}_joint">
+    <gazebo reference="${ns}_${name}_${type}_joint">
       <implicitSpringDamper>true</implicitSpringDamper>
 			<springStiffness>0.4</springStiffness>
@@ -98,5 +98,5 @@
 	  </gazebo>
         <!-- GAZEBO REF -->
-    <gazebo reference="${ns}_${name}_virtual_joint">
+    <gazebo reference="${ns}_${name}_${type}_virtual_joint">
       <implicitSpringDamper>true</implicitSpringDamper>
 			<springStiffness>0.4</springStiffness>

File: softhands_description/urdf/xacro/include/macro/v3/modules/phalanges/phalanx_knuckle.xacro (robot description, xacro)
@@ -38,5 +38,5 @@
 -->
 <robot xmlns:xacro="http://www.ros.org/wiki/xacro">
-  <xacro:macro name="phalanx_knuckle" params="ns name parent *origin side mesh">
+  <xacro:macro name="phalanx_knuckle" params="ns name mass parent *origin **inertia_origin side mesh">
     <!-- Proximal JOINT -->
     <joint name="${ns}_${name}_joint" type="revolute">
@@ -58,5 +58,5 @@
         <origin rpy="0 0 0" xyz="0 0 0"/>
         <geometry>
-          <mesh filename="package://softhands_description/meshes/v3/${side}/${index.mesh.knuckle_mesh}" scale="0.001 0.001 0.001"/>
+          <mesh filename="package://softhands_description/meshes/v3/${side}/${mesh}" scale="0.001 0.001 0.001"/>
         </geometry>
         <material name="qbhand/palm"/>
@@ -65,26 +65,5 @@
         <origin rpy="0 0 0" xyz="0 0 0"/>
         <geometry>
-          <mesh filename="package://softhands_description/meshes/v3/${side}/${index.mesh.knuckle_mesh}" scale="0.001 0.001 0.001"/>
-        </geometry>
-      </collision>
-    </link>
-    <!-- LINK -->
-    <link name="${ns}_${name}_link">
-      <inertial>
-        <origin rpy="0 0 0" xyz="8.2672528e-03  -2.7479334e-03 6.3742013e-05"/>
-        <mass value="2.9531895e-03"/>
-        <inertia ixx="4.9114511e-08" ixy="2.4336199e-08" ixz="1.1336750e-09" iyy="1.6520715e-07" iyz="0.0" izz="1.7172503e-07"/>
-      </inertial>
-      <visual>
-        <origin rpy="0 0 0" xyz="0 0 0"/>
-        <geometry>
-          <mesh filename="package://softhands_description/meshes/v3/${side}/ph_knuckle.stl" scale="0.001 0.001 0.001"/>
-        </geometry>
-        <material name="qbhand/palm"/>
-      </visual>
-      <collision>
-        <origin rpy="0 0 0" xyz="0 0 0"/>
-        <geometry>
-          <mesh filename="package://softhands_description/meshes/v3/${side}/ph_knuckle.stl" scale="0.001 0.001 0.001"/>
+          <mesh filename="package://softhands_description/meshes/v3/${side}/${mesh}" scale="0.001 0.001 0.001"/>
         </geometry>
       </collision>

File: softhands_description/urdf/xacro/include/macro/v3/modules/phalanges/thumb_knuckle.xacro (robot description, xacro)
@@ -38,8 +38,8 @@
 -->
 <robot xmlns:xacro="http://www.ros.org/wiki/xacro">
-  <xacro:macro name="thumb_knuckle" params="ns name parent *origin side">
+  <xacro:macro name="thumb_knuckle" params="yaml_file:=^ ns name parent side">
     <!-- Proximal JOINT -->
     <joint name="${ns}_${name}_joint" type="revolute">
-      <xacro:insert_block name="origin"/>
+      <origin rpy="${yaml_file['finger']['thumb']['knuckle']['orientation']}" xyz="${yaml_file['finger']['thumb']['knuckle']['position']}"/>
       <parent link="${ns}_${parent}_link"/>
       <child link="${ns}_${name}_link"/>

File: softhands_description/urdf/xacro/include/macro/v3/modules/thumb.xacro (robot description, xacro)
@@ -38,28 +38,14 @@
 -->
 <robot xmlns:xacro="http://www.ros.org/wiki/xacro">
-  <xacro:macro name="thumb" params="ns name parent *origin side">
+  <xacro:macro name="thumb" params="yaml_file:=^ ns name parent side">
     <!-- Knuckle -->
     <xacro:thumb_knuckle name="${name}_knuckle" parent="${parent}" ns="${ns}" side="${side}">
-      <origin rpy="1.5707963 0 2.5307278" xyz="-0.0315281 -0.0276566 ${sign*-0.0024}"/>
     </xacro:thumb_knuckle>
     <!-- Proximal  -->
-    <xacro:phalanx_generic name="${name}_proximal" parent="${name}_knuckle" ns="${ns}" mass="3.4433482e-03" mesh="ph_short">
-      <xacro:if value="${side == 'left'}">
-         <virtual_origin> <origin rpy="-2 0.0 0.0" xyz="0.0255 0.0038 -0.00012"/></virtual_origin>
-      </xacro:if>
-      <xacro:if value="${side == 'right'}">
-         <virtual_origin> <origin rpy="-1.5707963 0.0 0.0" xyz="16.5e-03 -4.2e-03 0"/></virtual_origin>
-      </xacro:if>
+    <xacro:phalanx_generic name="${name}" type="prossimal" parent="${name}_knuckle" ns="${ns}">
       <real_origin>     <origin rpy="0 0 0" xyz="9e-03 0 0"/>                         </real_origin>
       <inertia_origin>  <origin rpy="0 0 0" xyz="8.2958878e-03 1.4867666e-04 0"/>  </inertia_origin>
       <inertia ixx="5.9259154e-08" ixy="4.7090997e-09" ixz="0" iyy="2.0151714e-07" iyz="0.0" izz="2.1338410e-07"/>
     </xacro:phalanx_generic>
-    <!-- Distal  -->
-    <xacro:phalanx_generic name="${name}_distal" parent="${name}_proximal" ns="${ns}" mass="2.3548400e-03" mesh="ph_distal">
-      <virtual_origin>  <origin rpy="0 0 0" xyz="16e-03 0 0"/>                        </virtual_origin>
-      <real_origin>     <origin rpy="0 0 0" xyz="9e-03 0 0"/>                         </real_origin>
-      <inertia_origin>  <origin rpy="0 0 0" xyz="2.3098353e-03 4.4361817e-04 -4.4968362e-04"/>  </inertia_origin>
-      <inertia ixx="2.8240100e-08" ixy="8.9271493e-10" ixz="1.2771999e-10" iyy="6.1297195e-10" iyz="0.0" izz="5.7464142e-08"/>
-    </xacro:phalanx_generic>
   </xacro:macro>
 </robot>

File: softhands_description/urdf/xacro/v3.xacro (robot description, xacro)
@@ -50,5 +50,5 @@
     	<xacro:softhand_mimic_plugin ns="${side}_hand_v3" wide="false"/>
 		<!-- Softhand v3 needs a config file because the finger are different from each other -->
-		<xacro:property name="params" from_yaml="$(find softhands_description)/urdf/config/params_v3.yaml"/>
+		<xacro:property name="yaml_file" value="${xacro.load_yaml('$(find softhands_description)/urdf/config/params_v3.yaml')}"/>
 		<!-- <xacro:println value="${params}"/> -->
 		<!-- # palm  -->
@@ -57,43 +57,5 @@
 		</xacro:palm>
 		<!-- # thumb -->
-		<!-- <xacro:thumb name="thumb" parent="palm" ns="${side}_hand_v3" side="${side}">
-			<origin rpy="-1.57 3.14 0.0" xyz="-0.044 -0.0465 -0.002"/>
-		</xacro:thumb> -->
-		<!-- # Index -->
-		<!-- <xacro:finger name="index" parent="palm" ns="${side}_hand_v3" side="${side}" mesh="${index.mesh.knuckle_mesh}" >
-			<xacro:if value="${side == 'left'}">
-				<origin rpy="0 3.14 -1.57" xyz="-0.02 -0.007 -0.014"/>
-			</xacro:if>
-			<xacro:if value="${side == 'right'}">
-				<origin rpy="0 0 1.7453293" xyz="-0.02 0 6.02670e-03"/>
-			</xacro:if>
-		</xacro:finger> -->
-		<!-- # Middle -->
-		<!-- <xacro:finger name="middle" parent="palm" ns="${side}_hand_v3" side="${side}">
-			<xacro:if value="${side == 'left'}">
-				<origin rpy="0 3.14 -1.57" xyz="0 0 -0.014"/>
-			</xacro:if>
-			<xacro:if value="${side == 'right'}">
-				<origin rpy="0 0 1.57" xyz="0 0 0.014"/>
-			</xacro:if>
-		</xacro:finger> -->
-		<!-- # Ring -->
-		<!-- <xacro:finger name="ring" parent="palm" ns="${side}_hand_v3" side="${side}">
-			<xacro:if value="${side == 'left'}">
-				<origin rpy="0 3.14 -1.57" xyz="0.02 -0.007 -0.014"/>
-			</xacro:if>
-			<xacro:if value="${side == 'right'}">
-				<origin rpy="0 0 1.57" xyz="0.02 -0.007 0.014"/>
-			</xacro:if>
-		</xacro:finger> -->
-		<!-- # Little -->
-		<!-- <xacro:finger name="little" parent="palm" ns="${side}_hand_v3" side="${side}">
-			<xacro:if value="${side == 'left'}">
-				<origin rpy="0 3.14 -1.57" xyz="0.04 -0.012 -0.014"/>
-			</xacro:if>
-			<xacro:if value="${side == 'right'}">
-				<origin rpy="0 0 1.57" xyz="0.04 -0.012 0.014"/>
-			</xacro:if>
-		</xacro:finger> -->
+		<xacro:thumb name="thumb" parent="palm" ns="${side}_hand_v3" side="${side}"/>
 	</xacro:macro>
 </robot>
