Commit message: first commit sh3

File: softhands_description/urdf/xacro/include/macro/v3/modules/finger.xacro (robot description, xacro)
@@ -38,30 +38,33 @@
 -->
 <robot xmlns:xacro="http://www.ros.org/wiki/xacro">
-  <xacro:macro name="finger" params="ns name parent *origin side">
+  <xacro:macro name="finger" params="ns name parent *origin side ">
     <!-- Proximal -->
-    <xacro:phalanx_knuckle name="${name}_knuckle" parent="${parent}" ns="${ns}" side="${side}">
-      <xacro:insert_block name="origin"/>
+    <xacro:phalanx_knuckle name="${name}_knuckle" parent="${parent}" ns="${ns}" side="${side}" mesh="${index.mesh.knuckle_mesh}">
+     <xacro:insert_block name="origin"/>
+     <inertia_origin> <origin rpy="0 0 0" xyz="8.2672528e-03  -2.7479334e-03 6.3742013e-05"/>   </inertia_origin>
+     <mass value="2.9531895e-03"/>
+     <inertia ixx="4.9114511e-08" ixy="2.4336199e-08" ixz="1.1336750e-09" iyy="1.6520715e-07" iyz="0.0" izz="1.7172503e-07"/>
     </xacro:phalanx_knuckle>
     <!-- Proximal -->
-    <xacro:phalanx_generic name="${name}_proximal" parent="${name}_knuckle" ns="${ns}" mass="0.009" mesh="ph_medium">
-      <virtual_origin>  <origin rpy="1.57 0 0" xyz="0.009 0 0"/>                      </virtual_origin>
-      <real_origin>     <origin rpy="0.0 0 0" xyz="0.013 0 0"/>                       </real_origin>
-      <inertia_origin>  <origin rpy="0 0 0" xyz="8.7707437e-03 -1.7863138e-03 0.0"/>  </inertia_origin>
-      <inertia ixx="2.2722068e-07" ixy="1.1586053e-08" ixz="0.0" iyy="5.5947233e-07" iyz="0.0" izz="5.9562195e-07"/>
-    </xacro:phalanx_generic>
+    <!-- <xacro:phalanx_generic name="${name}_proximal" parent="${name}_knuckle" ns="${ns}" mass="3.4433482e-03" mesh="${proximal_mesh}">
+      <virtual_origin>  <origin rpy="1.57 0 0" xyz="15e-03 -3.7e-03 0"/>                      </virtual_origin>
+      <real_origin>     <origin rpy="0.0 0 0" xyz="9e-03 0 0"/>                       </real_origin>
+      <inertia_origin>  <origin rpy="0 0 0" xyz="8.2958878e-03 1.4867666e-04 0.0"/>  </inertia_origin>
+      <inertia ixx="5.9259154e-08" ixy="4.7090997e-09" ixz="0.0" iyy="2.0151714e-07" iyz="0.0" izz="2.1338410e-07"/>
+    </xacro:phalanx_generic> -->
     <!-- Middle -->
-    <xacro:phalanx_generic name="${name}_middle" parent="${name}_proximal" ns="${ns}" mass="0.0063" mesh="ph_short">
-      <virtual_origin>  <origin rpy="0.0 0.0 0.0" xyz="0.013 0 0 "/>                  </virtual_origin>
-      <real_origin>     <origin rpy="0 0 0" xyz="0.017 0 0"/>                         </real_origin>
+    <!-- <xacro:phalanx_generic name="${name}_middle" parent="${name}_proximal" ns="${ns}" mass="0.0063" mesh="${middle_mesh}">
+      <virtual_origin>  <origin rpy="0.0 0.0 0.0" xyz="16e-03 0 0 "/>                  </virtual_origin>
+      <real_origin>     <origin rpy="0 0 0" xyz="16e-03 0 0"/>                         </real_origin>
       <inertia_origin>  <origin rpy="0 0 0" xyz="4.7601567e-03 -1.3786947e-03 0.0"/>  </inertia_origin>
       <inertia ixx="1.8024201e-07" ixy="5.756798e-09" ixz="0.0" iyy="2.3516266e-07" iyz="0.0" izz="2.691504e-07"/>
-    </xacro:phalanx_generic>
+    </xacro:phalanx_generic> -->
     <!-- Distal -->
-    <xacro:phalanx_generic name="${name}_distal" parent="${name}_middle" ns="${ns}" mass="0.009" mesh="ph_distal">
+    <!-- <xacro:phalanx_generic name="${name}_distal" parent="${name}_middle" ns="${ns}" mass="0.009" mesh="ph_distal">
       <virtual_origin>  <origin rpy="0 0 0" xyz="0.009 0 0"/>                        </virtual_origin>
       <real_origin>     <origin rpy="0 0 0" xyz="0.013 0 0"/>                         </real_origin>
       <inertia_origin>  <origin rpy="0 0 0" xyz="8.8025467e-03 -1.7219289e-03 0.0"/>  </inertia_origin>
       <inertia ixx="2.6586142e-07" ixy="1.2416847e-08" ixz="0.0" iyy="5.9935767e-07" iyz="0.0" izz="6.6781963e-07"/>
-    </xacro:phalanx_generic>
+    </xacro:phalanx_generic> -->
   </xacro:macro>
 </robot>

File: softhands_description/urdf/xacro/include/macro/v3/modules/iso.xacro (robot description, xacro)
@@ -37,5 +37,5 @@
  *
 -->
-<robot name="iso_v2" xmlns:xacro="http://www.ros.org/wiki/xacro">
+<robot name="iso_v3" xmlns:xacro="http://www.ros.org/wiki/xacro">
 	<xacro:macro name="iso" params="ns name parent *origin">
 		<!-- World to palm base -->

File: softhands_description/urdf/xacro/include/macro/v3/modules/palm/palm.xacro (robot description, xacro)
@@ -37,5 +37,5 @@
  *
 -->
-<robot name="palm_v2" xmlns:xacro="http://www.ros.org/wiki/xacro">
+<robot name="palm_v3" xmlns:xacro="http://www.ros.org/wiki/xacro">
 	<xacro:macro name="palm" params="ns name parent *origin">
 	  	<joint name="${ns}_palm_joint" type="fixed">

File: softhands_description/urdf/xacro/include/macro/v3/modules/phalanges/phalanx_knuckle.xacro (robot description, xacro)
@@ -38,5 +38,5 @@
 -->
 <robot xmlns:xacro="http://www.ros.org/wiki/xacro">
-  <xacro:macro name="phalanx_knuckle" params="ns name parent *origin side">
+  <xacro:macro name="phalanx_knuckle" params="ns name parent *origin side mesh">
     <!-- Proximal JOINT -->
     <joint name="${ns}_${name}_joint" type="revolute">
@@ -50,8 +50,29 @@
     <!-- LINK -->
     <link name="${ns}_${name}_link">
+        <inertial>
+          <mass value="${mass}"/>
+          <xacro:insert_block name="inertia"/>
+          <xacro:insert_block name="inertia_origin"/>
+        </inertial>
+      <visual>
+        <origin rpy="0 0 0" xyz="0 0 0"/>
+        <geometry>
+          <mesh filename="package://softhands_description/meshes/v3/${side}/${index.mesh.knuckle_mesh}" scale="0.001 0.001 0.001"/>
+        </geometry>
+        <material name="qbhand/palm"/>
+      </visual>
+      <collision>
+        <origin rpy="0 0 0" xyz="0 0 0"/>
+        <geometry>
+          <mesh filename="package://softhands_description/meshes/v3/${side}/${index.mesh.knuckle_mesh}" scale="0.001 0.001 0.001"/>
+        </geometry>
+      </collision>
+    </link>
+    <!-- LINK -->
+    <link name="${ns}_${name}_link">
       <inertial>
-        <origin rpy="0 0 0" xyz="4.2753603e-04  0.0 -1.4321738e-03"/>
-        <mass value="0.0095"/>
-        <inertia ixx="6.4337303e-07" ixy="0.0" ixz="-3.9373913e-08" iyy="1.1253771e-06" iyz="0.0" izz="7.2336948e-07"/>
+        <origin rpy="0 0 0" xyz="8.2672528e-03  -2.7479334e-03 6.3742013e-05"/>
+        <mass value="2.9531895e-03"/>
+        <inertia ixx="4.9114511e-08" ixy="2.4336199e-08" ixz="1.1336750e-09" iyy="1.6520715e-07" iyz="0.0" izz="1.7172503e-07"/>
       </inertial>
       <visual>

File: softhands_description/urdf/xacro/include/macro/v3/modules/phalanges/thumb_knuckle.xacro (robot description, xacro)
@@ -51,7 +51,7 @@
     <link name="${ns}_${name}_link">
       <inertial>
-        <origin rpy="0 0 0" xyz="1.3071561e-02 ${sign*-2.7346340e-03} 6.4090487e-04"/>
-        <mass value="0.01"/>
-        <inertia ixx="3.5865978e-07" ixy="${sign*2.0944224e-07}" ixz="-6.8657569e-08" iyy="1.3885564e-06" iyz="${sign*3.2170608e-08}" izz="1.3571203e-06"/>
+        <origin rpy="0 0 0" xyz="1.6018749e-3 ${sign*1.9731832e-04} -1.8504085e-03"/>
+        <mass value="3.2037862e-03"/>
+        <inertia ixx="6.5745301e-08" ixy="${sign*-3.1362083e-10}" ixz="3.5152512e-08" iyy="2.2281085e-07" iyz="${sign*-5.2782785e-11}" izz="2.0956023e-07"/>
       </inertial>
       <visual>

File: softhands_description/urdf/xacro/include/macro/v3/modules/thumb.xacro (robot description, xacro)
@@ -41,24 +41,24 @@
     <!-- Knuckle -->
     <xacro:thumb_knuckle name="${name}_knuckle" parent="${parent}" ns="${ns}" side="${side}">
-      <origin rpy="-1.57 3.14 0.0" xyz="-0.044 -0.0465 ${sign*-0.002}"/>
+      <origin rpy="1.5707963 0 2.5307278" xyz="-0.0315281 -0.0276566 ${sign*-0.0024}"/>
     </xacro:thumb_knuckle>
     <!-- Proximal  -->
-    <xacro:phalanx_generic name="${name}_proximal" parent="${name}_knuckle" ns="${ns}" mass="0.0063" mesh="ph_short">
+    <xacro:phalanx_generic name="${name}_proximal" parent="${name}_knuckle" ns="${ns}" mass="3.4433482e-03" mesh="ph_short">
       <xacro:if value="${side == 'left'}">
          <virtual_origin> <origin rpy="-2 0.0 0.0" xyz="0.0255 0.0038 -0.00012"/></virtual_origin>
       </xacro:if>
       <xacro:if value="${side == 'right'}">
-         <virtual_origin> <origin rpy="-1.1415 0.0 0.0" xyz="0.0255 -0.0038 -0.00012"/></virtual_origin>
+         <virtual_origin> <origin rpy="-1.5707963 0.0 0.0" xyz="16.5e-03 -4.2e-03 0"/></virtual_origin>
       </xacro:if>
-      <real_origin>     <origin rpy="0 0 0" xyz="0.013 0 0"/>                         </real_origin>
-      <inertia_origin>  <origin rpy="0 0 0" xyz="4.7601567e-03 -1.3786947e-03 0.0"/>  </inertia_origin>
-      <inertia ixx="1.8024201e-07" ixy="5.756798e-09" ixz="0.0" iyy="2.3516266e-07" iyz="0.0" izz="2.691504e-07"/>
+      <real_origin>     <origin rpy="0 0 0" xyz="9e-03 0 0"/>                         </real_origin>
+      <inertia_origin>  <origin rpy="0 0 0" xyz="8.2958878e-03 1.4867666e-04 0"/>  </inertia_origin>
+      <inertia ixx="5.9259154e-08" ixy="4.7090997e-09" ixz="0" iyy="2.0151714e-07" iyz="0.0" izz="2.1338410e-07"/>
     </xacro:phalanx_generic>
     <!-- Distal  -->
-    <xacro:phalanx_generic name="${name}_distal" parent="${name}_proximal" ns="${ns}" mass="0.009" mesh="ph_distal">
-      <virtual_origin>  <origin rpy="0 0 0" xyz="0.009 0 0"/>                        </virtual_origin>
-      <real_origin>     <origin rpy="0 0 0" xyz="0.013 0 0"/>                         </real_origin>
-      <inertia_origin>  <origin rpy="0 0 0" xyz="8.8025467e-03 -1.7219289e-03 0.0"/>  </inertia_origin>
-      <inertia ixx="2.6586142e-07" ixy="1.2416847e-08" ixz="0.0" iyy="5.9935767e-07" iyz="0.0" izz="6.6781963e-07"/>
+    <xacro:phalanx_generic name="${name}_distal" parent="${name}_proximal" ns="${ns}" mass="2.3548400e-03" mesh="ph_distal">
+      <virtual_origin>  <origin rpy="0 0 0" xyz="16e-03 0 0"/>                        </virtual_origin>
+      <real_origin>     <origin rpy="0 0 0" xyz="9e-03 0 0"/>                         </real_origin>
+      <inertia_origin>  <origin rpy="0 0 0" xyz="2.3098353e-03 4.4361817e-04 -4.4968362e-04"/>  </inertia_origin>
+      <inertia ixx="2.8240100e-08" ixy="8.9271493e-10" ixz="1.2771999e-10" iyy="6.1297195e-10" iyz="0.0" izz="5.7464142e-08"/>
     </xacro:phalanx_generic>
   </xacro:macro>

File: softhands_description/urdf/xacro/v3.xacro (robot description, xacro)
@@ -49,4 +49,7 @@
 		</xacro:if>
     	<xacro:softhand_mimic_plugin ns="${side}_hand_v3" wide="false"/>
+		<!-- Softhand v3 needs a config file because the finger are different from each other -->
+		<xacro:property name="params" from_yaml="$(find softhands_description)/urdf/config/params_v3.yaml"/>
+		<!-- <xacro:println value="${params}"/> -->
 		<!-- # palm  -->
 		<xacro:palm name="palm" parent="${parent}" ns="${side}_hand_v3">
@@ -54,18 +57,18 @@
 		</xacro:palm>
 		<!-- # thumb -->
-		<xacro:thumb name="thumb" parent="palm" ns="${side}_hand_v3" side="${side}">
+		<!-- <xacro:thumb name="thumb" parent="palm" ns="${side}_hand_v3" side="${side}">
 			<origin rpy="-1.57 3.14 0.0" xyz="-0.044 -0.0465 -0.002"/>
-		</xacro:thumb>
+		</xacro:thumb> -->
 		<!-- # Index -->
-		<xacro:finger name="index" parent="palm" ns="${side}_hand_v3" side="${side}">
+		<!-- <xacro:finger name="index" parent="palm" ns="${side}_hand_v3" side="${side}" mesh="${index.mesh.knuckle_mesh}" >
 			<xacro:if value="${side == 'left'}">
 				<origin rpy="0 3.14 -1.57" xyz="-0.02 -0.007 -0.014"/>
 			</xacro:if>
 			<xacro:if value="${side == 'right'}">
-				<origin rpy="0 0 1.57" xyz="-0.02 -0.007 0.014"/>
+				<origin rpy="0 0 1.7453293" xyz="-0.02 0 6.02670e-03"/>
 			</xacro:if>
-		</xacro:finger>
+		</xacro:finger> -->
 		<!-- # Middle -->
-		<xacro:finger name="middle" parent="palm" ns="${side}_hand_v3" side="${side}">
+		<!-- <xacro:finger name="middle" parent="palm" ns="${side}_hand_v3" side="${side}">
 			<xacro:if value="${side == 'left'}">
 				<origin rpy="0 3.14 -1.57" xyz="0 0 -0.014"/>
@@ -74,7 +77,7 @@
 				<origin rpy="0 0 1.57" xyz="0 0 0.014"/>
 			</xacro:if>
-		</xacro:finger>
+		</xacro:finger> -->
 		<!-- # Ring -->
-		<xacro:finger name="ring" parent="palm" ns="${side}_hand_v3" side="${side}">
+		<!-- <xacro:finger name="ring" parent="palm" ns="${side}_hand_v3" side="${side}">
 			<xacro:if value="${side == 'left'}">
 				<origin rpy="0 3.14 -1.57" xyz="0.02 -0.007 -0.014"/>
@@ -83,7 +86,7 @@
 				<origin rpy="0 0 1.57" xyz="0.02 -0.007 0.014"/>
 			</xacro:if>
-		</xacro:finger>
+		</xacro:finger> -->
 		<!-- # Little -->
-		<xacro:finger name="little" parent="palm" ns="${side}_hand_v3" side="${side}">
+		<!-- <xacro:finger name="little" parent="palm" ns="${side}_hand_v3" side="${side}">
 			<xacro:if value="${side == 'left'}">
 				<origin rpy="0 3.14 -1.57" xyz="0.04 -0.012 -0.014"/>
@@ -92,5 +95,5 @@
 				<origin rpy="0 0 1.57" xyz="0.04 -0.012 0.014"/>
 			</xacro:if>
-		</xacro:finger>
+		</xacro:finger> -->
 	</xacro:macro>
 </robot>

Commit message: update sh3

File: softhands_description/urdf/xacro/include/macro/v3/modules/finger.xacro (robot description, xacro)
@@ -38,5 +38,8 @@
 -->
 <robot xmlns:xacro="http://www.ros.org/wiki/xacro">
-  <xacro:macro name="finger" params="yaml_file:=^ ">
+  <xacro:macro name="finger" params="yaml_file:=^ ns name parent side ">
+    <!-- Knuckle -->
+    <xacro:phalanx_knuckle name="${name}_knuckle" parent="${parent}" ns="${ns}" side="${side}">
+    </xacro:phalanx_knuckle>
   </xacro:macro>
 </robot>

File: softhands_description/urdf/xacro/include/macro/v3/modules/phalanges/phalanx_knuckle.xacro (robot description, xacro)
@@ -38,8 +38,8 @@
 -->
 <robot xmlns:xacro="http://www.ros.org/wiki/xacro">
-  <xacro:macro name="phalanx_knuckle" params="ns name mass parent *origin **inertia_origin side mesh">
+  <xacro:macro name="phalanx_knuckle" params="yaml_file:=^ ns name parent side">
     <!-- Proximal JOINT -->
     <joint name="${ns}_${name}_joint" type="revolute">
-      <xacro:insert_block name="origin"/>
+    <origin rpy="${yaml_file['finger']['index']['knuckle']['orientation']}" xyz="${yaml_file['finger']['index']['knuckle']['position']}"/>
       <parent link="${ns}_${parent}_link"/>
       <child link="${ns}_${name}_link"/>
@@ -51,12 +51,12 @@
     <link name="${ns}_${name}_link">
         <inertial>
-          <mass value="${mass}"/>
-          <xacro:insert_block name="inertia"/>
-          <xacro:insert_block name="inertia_origin"/>
+          <mass value="${yaml_file['finger']['index']['knuckle']['mass']}"/>
+          <inertia ixx="${yaml_file['finger']['index']['knuckle']['inertia']['ixx']}" ixy="${yaml_file['finger']['index']['knuckle']['inertia']['ixy']}" ixz="${yaml_file['finger']['index']['knuckle']['inertia']['ixz']}" iyy="${yaml_file['finger']['index']['knuckle']['inertia']['iyy']}" iyz="${yaml_file['finger']['index']['knuckle']['inertia']['iyz']}" izz="${yaml_file['finger']['index']['knuckle']['inertia']['izz']}"/>
+          <origin rpy="0 0 0" xyz="${yaml_file['finger']['index']['knuckle']['inertia_origin']['position']}"/>
         </inertial>
       <visual>
         <origin rpy="0 0 0" xyz="0 0 0"/>
         <geometry>
-          <mesh filename="package://softhands_description/meshes/v3/${side}/${mesh}" scale="0.001 0.001 0.001"/>
+          <mesh filename="package://softhands_description/meshes/v3/${side}/${yaml_file['finger']['index']['knuckle']['mesh']}" scale="0.001 0.001 0.001"/>
         </geometry>
         <material name="qbhand/palm"/>
@@ -65,5 +65,5 @@
         <origin rpy="0 0 0" xyz="0 0 0"/>
         <geometry>
-          <mesh filename="package://softhands_description/meshes/v3/${side}/${mesh}" scale="0.001 0.001 0.001"/>
+          <mesh filename="package://softhands_description/meshes/v3/${side}/${yaml_file['finger']['index']['knuckle']['mesh']}" scale="0.001 0.001 0.001"/>
         </geometry>
       </collision>

File: softhands_description/urdf/xacro/include/macro/v3/modules/phalanges/thumb_knuckle.xacro (robot description, xacro)
@@ -51,12 +51,12 @@
     <link name="${ns}_${name}_link">
       <inertial>
-        <origin rpy="0 0 0" xyz="1.6018749e-3 ${sign*1.9731832e-04} -1.8504085e-03"/>
-        <mass value="3.2037862e-03"/>
-        <inertia ixx="6.5745301e-08" ixy="${sign*-3.1362083e-10}" ixz="3.5152512e-08" iyy="2.2281085e-07" iyz="${sign*-5.2782785e-11}" izz="2.0956023e-07"/>
+        <origin rpy="0 0 0" xyz="${yaml_file['finger']['thumb']['knuckle']['inertia_origin']['position']}"/>
+        <mass value="${yaml_file['finger']['thumb']['knuckle']['mass']}"/>
+        <inertia ixx="${yaml_file['finger']['thumb']['knuckle']['inertia']['ixx']}" ixy="${yaml_file['finger']['thumb']['knuckle']['inertia']['ixy']}" ixz="${yaml_file['finger']['thumb']['knuckle']['inertia']['ixz']}" iyy="${yaml_file['finger']['thumb']['knuckle']['inertia']['iyy']}" iyz="${yaml_file['finger']['thumb']['knuckle']['inertia']['iyz']}" izz="${yaml_file['finger']['thumb']['knuckle']['inertia']['izz']}"/>
       </inertial>
       <visual>
         <origin rpy="0 0 0" xyz="0 0 0"/>
         <geometry>
-          <mesh filename="package://softhands_description/meshes/v3/${side}/ph_thumb.stl" scale="0.001 0.001 0.001"/>
+          <mesh filename="package://softhands_description/meshes/v3/${side}/${yaml_file['finger']['thumb']['knuckle']['mesh']}" scale="0.001 0.001 0.001"/>
         </geometry>
         <material name="qbhand/knuckle"/>
@@ -65,5 +65,5 @@
         <origin rpy="0 0 0" xyz="0 0 0"/>
         <geometry>
-          <mesh filename="package://softhands_description/meshes/v3/${side}/ph_thumb.stl" scale="0.001 0.001 0.001"/>
+          <mesh filename="package://softhands_description/meshes/v3/${side}/${yaml_file['finger']['thumb']['knuckle']['mesh']}" scale="0.001 0.001 0.001"/>
         </geometry>
       </collision>

File: softhands_description/urdf/xacro/include/macro/v3/modules/thumb.xacro (robot description, xacro)
@@ -43,9 +43,9 @@
     </xacro:thumb_knuckle>
     <!-- Proximal  -->
-    <xacro:phalanx_generic name="${name}" type="prossimal" parent="${name}_knuckle" ns="${ns}">
+    <!-- <xacro:phalanx_generic name="${name}" type="prossimal" parent="${name}_knuckle" ns="${ns}">
       <real_origin>     <origin rpy="0 0 0" xyz="9e-03 0 0"/>                         </real_origin>
       <inertia_origin>  <origin rpy="0 0 0" xyz="8.2958878e-03 1.4867666e-04 0"/>  </inertia_origin>
       <inertia ixx="5.9259154e-08" ixy="4.7090997e-09" ixz="0" iyy="2.0151714e-07" iyz="0.0" izz="2.1338410e-07"/>
-    </xacro:phalanx_generic>
+    </xacro:phalanx_generic> -->
   </xacro:macro>
 </robot>

File: softhands_description/urdf/xacro/v3.xacro (robot description, xacro)
@@ -50,5 +50,5 @@
     	<xacro:softhand_mimic_plugin ns="${side}_hand_v3" wide="false"/>
 		<!-- Softhand v3 needs a config file because the finger are different from each other -->
-		<xacro:property name="yaml_file" value="${xacro.load_yaml('$(find softhands_description)/urdf/config/params_v3.yaml')}"/>
+		<xacro:property name="yaml_file" value="${xacro.load_yaml('$(find softhands_description)/urdf/config/params_v3.yaml')[side]}"/>
 		<!-- <xacro:println value="${params}"/> -->
 		<!-- # palm  -->
@@ -58,4 +58,8 @@
 		<!-- # thumb -->
 		<xacro:thumb name="thumb" parent="palm" ns="${side}_hand_v3" side="${side}"/>
+		<!-- # index -->
+		<xacro:finger name="index" parent="palm" ns="${side}_hand_v3" side="${side}"/>
+		<!-- # middle -->
+		<!-- <xacro:finger name="middle" parent="palm" ns="${side}_hand_v3" side="${side}"/> -->
 	</xacro:macro>
 </robot>
