Commit message: update sh3

File: softhands_description/urdf/xacro/include/macro/v3/modules/finger.xacro (robot description, xacro)
@@ -40,5 +40,5 @@
   <xacro:macro name="finger" params="yaml_file:=^ ns name parent side ">
     <!-- Knuckle -->
-    <xacro:phalanx_knuckle name="${name}_knuckle" parent="${parent}" ns="${ns}" side="${side}">
+    <xacro:phalanx_knuckle name="${name}" type="knuckle" parent="${parent}" ns="${ns}" side="${side}">
     </xacro:phalanx_knuckle>
   </xacro:macro>

File: softhands_description/urdf/xacro/include/macro/v3/modules/phalanges/phalanx_generic.xacro (robot description, xacro)
@@ -38,9 +38,9 @@
 -->
 <robot xmlns:xacro="http://www.ros.org/wiki/xacro">
-  <xacro:macro name="phalanx_generic" params="yaml_file:=^ name type parent ns">
+  <xacro:macro name="phalanx_generic" params="yaml_file:=^ name type side parent ns">
     <!-- Inner VIRTUAL JOINT -->
 		<joint name="${ns}_${name}_${type}_virtual_joint" type="revolute">
       <axis xyz="0 0 -1"/>
-      <origin rpy="${yaml_file['finger']['${name}']['${type}']['virtual_origin']['orientation']}" xyz="${yaml_file['finger']['${name}']['${type}']['virtual_origin']['position']}"/>
+      <origin rpy="${yaml_file[side]['finger'][name][type]['virtual_origin']['orientation']}" xyz="${yaml_file[side]['finger'][name][type]['virtual_origin']['position']}"/>
 			<parent link="${ns}_${parent}_link"/>
 			<child link="${ns}_${name}_${type}_virtual_link"/>
@@ -59,5 +59,5 @@
     <joint name="${ns}_${name}_${type}_joint" type="revolute">
       <axis xyz="0 0 -1"/>
-      <origin rpy="${yaml_file['finger']['${name}']['${type}']['real_origin']['orientation']}" xyz="${yaml_file['finger']['${name}']['${type}']['real_origin']['position']}"/>
+      <origin rpy="${yaml_file[side]['finger'][name][type]['real_origin']['orientation']}" xyz="${yaml_file[side]['finger'][name][type]['real_origin']['position']}"/>
       <parent link="${ns}_${name}_${type}_virtual_link"/>
       <child link="${ns}_${name}_${type}_link"/>
@@ -68,12 +68,12 @@
     <link name="${ns}_${name}_${type}_link">
         <inertial>
-          <mass value="${mass}"/>
-          <xacro:insert_block name="inertia"/>
-          <xacro:insert_block name="inertia_origin"/>
+          <mass value="${yaml_file[side]['finger'][name][type]['mass']}"/>
+          <inertia ixx="${yaml_file[side]['finger'][name][type]['inertia']['ixx']}" ixy="${yaml_file[side]['finger'][name][type]['inertia']['ixy']}" ixz="${yaml_file[side]['finger'][name][type]['inertia']['ixz']}" iyy="${yaml_file[side]['finger'][name][type]['inertia']['iyy']}" iyz="${yaml_file[side]['finger'][name][type]['inertia']['iyz']}" izz="${yaml_file[side]['finger'][name][type]['inertia']['izz']}"/>
+          <origin rpy="0 0 0" xyz="${yaml_file[side]['finger'][name][type]['inertia_origin']['position']}"/>
         </inertial>
       <visual>
         <origin rpy="0 0 0" xyz="0 0 0"/>
         <geometry>
-          <mesh filename="package://softhands_description/meshes/v3/${side}/${mesh}.stl" scale="0.001 0.001 0.001"/>
+          <mesh filename="package://softhands_description/meshes/v3/${side}/${yaml_file[side]['finger'][name][type]['mesh']}" scale="0.001 0.001 0.001"/>
         </geometry>
         <material name="qbhand/palm"/>
@@ -82,5 +82,5 @@
         <origin rpy="0 0 0" xyz="0 0 0"/>
         <geometry>
-          <mesh filename="package://softhands_description/meshes/v3/${side}/${mesh}.stl" scale="0.001 0.001 0.001"/>
+           <mesh filename="package://softhands_description/meshes/v3/${side}/${yaml_file['finger'][name][type]['mesh']}" scale="0.001 0.001 0.001"/>
         </geometry>
       </collision>

File: softhands_description/urdf/xacro/include/macro/v3/modules/phalanges/phalanx_knuckle.xacro (robot description, xacro)
@@ -38,10 +38,10 @@
 -->
 <robot xmlns:xacro="http://www.ros.org/wiki/xacro">
-  <xacro:macro name="phalanx_knuckle" params="yaml_file:=^ ns name parent side">
+  <xacro:macro name="phalanx_knuckle" params="yaml_file:=^ ns name type parent side">
     <!-- Proximal JOINT -->
-    <joint name="${ns}_${name}_joint" type="revolute">
-    <origin rpy="${yaml_file['finger']['index']['knuckle']['orientation']}" xyz="${yaml_file['finger']['index']['knuckle']['position']}"/>
+    <joint name="${ns}_${name}_${type}_joint" type="revolute">
+    <origin rpy="${yaml_file[side]['finger'][name][type]['orientation']}" xyz="${yaml_file[side]['finger'][name][type]['position']}"/>
       <parent link="${ns}_${parent}_link"/>
-      <child link="${ns}_${name}_link"/>
+      <child link="${ns}_${name}_${type}_link"/>
       <axis xyz="0 0 -1"/>
       <limit effort="30" velocity="10.0" lower="-0.524" upper="0.524" />
@@ -49,14 +49,14 @@
     </joint>
     <!-- LINK -->
-    <link name="${ns}_${name}_link">
+    <link name="${ns}_${name}_${type}_link">
         <inertial>
-          <mass value="${yaml_file['finger']['index']['knuckle']['mass']}"/>
-          <inertia ixx="${yaml_file['finger']['index']['knuckle']['inertia']['ixx']}" ixy="${yaml_file['finger']['index']['knuckle']['inertia']['ixy']}" ixz="${yaml_file['finger']['index']['knuckle']['inertia']['ixz']}" iyy="${yaml_file['finger']['index']['knuckle']['inertia']['iyy']}" iyz="${yaml_file['finger']['index']['knuckle']['inertia']['iyz']}" izz="${yaml_file['finger']['index']['knuckle']['inertia']['izz']}"/>
-          <origin rpy="0 0 0" xyz="${yaml_file['finger']['index']['knuckle']['inertia_origin']['position']}"/>
+          <mass value="${yaml_file[side]['finger'][name][type]['mass']}"/>
+          <inertia ixx="${yaml_file[side]['finger'][name][type]['inertia']['ixx']}" ixy="${yaml_file[side]['finger'][name][type]['inertia']['ixy']}" ixz="${yaml_file[side]['finger'][name][type]['inertia']['ixz']}" iyy="${yaml_file[side]['finger'][name][type]['inertia']['iyy']}" iyz="${yaml_file[side]['finger'][name][type]['inertia']['iyz']}" izz="${yaml_file[side]['finger'][name][type]['inertia']['izz']}"/>
+          <origin rpy="0 0 0" xyz="${yaml_file[side]['finger'][name][type]['inertia_origin']['position']}"/>
         </inertial>
       <visual>
         <origin rpy="0 0 0" xyz="0 0 0"/>
         <geometry>
-          <mesh filename="package://softhands_description/meshes/v3/${side}/${yaml_file['finger']['index']['knuckle']['mesh']}" scale="0.001 0.001 0.001"/>
+          <mesh filename="package://softhands_description/meshes/v3/${side}/${yaml_file[side]['finger'][name][type]['mesh']}" scale="0.001 0.001 0.001"/>
         </geometry>
         <material name="qbhand/palm"/>
@@ -65,15 +65,15 @@
         <origin rpy="0 0 0" xyz="0 0 0"/>
         <geometry>
-          <mesh filename="package://softhands_description/meshes/v3/${side}/${yaml_file['finger']['index']['knuckle']['mesh']}" scale="0.001 0.001 0.001"/>
+          <mesh filename="package://softhands_description/meshes/v3/${side}/${yaml_file[side]['finger'][name][type]['mesh']}" scale="0.001 0.001 0.001"/>
         </geometry>
       </collision>
     </link>
         <!-- GAZEBO REF -->
-    <gazebo reference="${ns}_${name}_link">
+    <gazebo reference="${ns}_${name}_${type}_link">
       <material>Gazebo/Grey</material>
       <selfCollide>$(arg selfCollide)</selfCollide>
     </gazebo>
             <!-- GAZEBO REF -->
-    <gazebo reference="${ns}_${name}_joint">
+    <gazebo reference="${ns}_${name}_${type}_joint">
       <implicitSpringDamper>true</implicitSpringDamper>
 			<springStiffness>0.8</springStiffness>

File: softhands_description/urdf/xacro/include/macro/v3/modules/phalanges/thumb_knuckle.xacro (robot description, xacro)
@@ -38,10 +38,10 @@
 -->
 <robot xmlns:xacro="http://www.ros.org/wiki/xacro">
-  <xacro:macro name="thumb_knuckle" params="yaml_file:=^ ns name parent side">
+  <xacro:macro name="thumb_knuckle" params="yaml_file:=^ ns name type parent side">
     <!-- Proximal JOINT -->
-    <joint name="${ns}_${name}_joint" type="revolute">
-      <origin rpy="${yaml_file['finger']['thumb']['knuckle']['orientation']}" xyz="${yaml_file['finger']['thumb']['knuckle']['position']}"/>
+    <joint name="${ns}_${name}_${type}_joint" type="revolute">
+      <origin rpy="${yaml_file[side]['finger'][name][type]['orientation']}" xyz="${yaml_file[side]['finger'][name][type]['position']}"/>
       <parent link="${ns}_${parent}_link"/>
-      <child link="${ns}_${name}_link"/>
+      <child link="${ns}_${name}_${type}_link"/>
       <axis xyz="0 0 ${sign*-1}"/>
       <limit effort="30" velocity="10.0" lower="0.0" upper="1.57" />
@@ -49,14 +49,14 @@
     </joint>
     <!-- LINK -->
-    <link name="${ns}_${name}_link">
+    <link name="${ns}_${name}_${type}_link">
       <inertial>
-        <origin rpy="0 0 0" xyz="${yaml_file['finger']['thumb']['knuckle']['inertia_origin']['position']}"/>
-        <mass value="${yaml_file['finger']['thumb']['knuckle']['mass']}"/>
-        <inertia ixx="${yaml_file['finger']['thumb']['knuckle']['inertia']['ixx']}" ixy="${yaml_file['finger']['thumb']['knuckle']['inertia']['ixy']}" ixz="${yaml_file['finger']['thumb']['knuckle']['inertia']['ixz']}" iyy="${yaml_file['finger']['thumb']['knuckle']['inertia']['iyy']}" iyz="${yaml_file['finger']['thumb']['knuckle']['inertia']['iyz']}" izz="${yaml_file['finger']['thumb']['knuckle']['inertia']['izz']}"/>
+        <origin rpy="0 0 0" xyz="${yaml_file[side]['finger'][name][type]['inertia_origin']['position']}"/>
+        <mass value="${yaml_file[side]['finger'][name][type]['mass']}"/>
+        <inertia ixx="${yaml_file[side]['finger'][name][type]['inertia']['ixx']}" ixy="${yaml_file[side]['finger'][name][type]['inertia']['ixy']}" ixz="${yaml_file[side]['finger'][name][type]['inertia']['ixz']}" iyy="${yaml_file[side]['finger'][name][type]['inertia']['iyy']}" iyz="${yaml_file[side]['finger'][name][type]['inertia']['iyz']}" izz="${yaml_file[side]['finger'][name][type]['inertia']['izz']}"/>
       </inertial>
       <visual>
         <origin rpy="0 0 0" xyz="0 0 0"/>
         <geometry>
-          <mesh filename="package://softhands_description/meshes/v3/${side}/${yaml_file['finger']['thumb']['knuckle']['mesh']}" scale="0.001 0.001 0.001"/>
+          <mesh filename="package://softhands_description/meshes/v3/${side}/${yaml_file[side]['finger'][name][type]['mesh']}" scale="0.001 0.001 0.001"/>
         </geometry>
         <material name="qbhand/knuckle"/>
@@ -65,15 +65,15 @@
         <origin rpy="0 0 0" xyz="0 0 0"/>
         <geometry>
-          <mesh filename="package://softhands_description/meshes/v3/${side}/${yaml_file['finger']['thumb']['knuckle']['mesh']}" scale="0.001 0.001 0.001"/>
+          <mesh filename="package://softhands_description/meshes/v3/${side}/${yaml_file[side]['finger'][name][type]['mesh']}" scale="0.001 0.001 0.001"/>
         </geometry>
       </collision>
     </link>
     <!-- GAZEBO REF -->
-    <gazebo reference="${ns}_${name}_link">
+    <gazebo reference="${ns}_${name}_${type}_link">
       <material>Gazebo/Grey</material>
       <selfCollide>$(arg selfCollide)</selfCollide>
     </gazebo>
         <!-- GAZEBO REF -->
-    <gazebo reference="${ns}_${name}_joint">
+    <gazebo reference="${ns}_${name}_${type}_joint">
       <implicitSpringDamper>true</implicitSpringDamper>
 			<springStiffness>0.4</springStiffness>

File: softhands_description/urdf/xacro/include/macro/v3/modules/thumb.xacro (robot description, xacro)
@@ -40,12 +40,9 @@
   <xacro:macro name="thumb" params="yaml_file:=^ ns name parent side">
     <!-- Knuckle -->
-    <xacro:thumb_knuckle name="${name}_knuckle" parent="${parent}" ns="${ns}" side="${side}">
+    <xacro:thumb_knuckle name="${name}" type="knuckle" parent="${parent}" ns="${ns}" side="${side}">
     </xacro:thumb_knuckle>
     <!-- Proximal  -->
-    <!-- <xacro:phalanx_generic name="${name}" type="prossimal" parent="${name}_knuckle" ns="${ns}">
-      <real_origin>     <origin rpy="0 0 0" xyz="9e-03 0 0"/>                         </real_origin>
-      <inertia_origin>  <origin rpy="0 0 0" xyz="8.2958878e-03 1.4867666e-04 0"/>  </inertia_origin>
-      <inertia ixx="5.9259154e-08" ixy="4.7090997e-09" ixz="0" iyy="2.0151714e-07" iyz="0.0" izz="2.1338410e-07"/>
-    </xacro:phalanx_generic> -->
+    <xacro:phalanx_generic name="${name}" type="prossimal" parent="${name}_knuckle" ns="${ns}" side="${side}">
+    </xacro:phalanx_generic>
   </xacro:macro>
 </robot>

File: softhands_description/urdf/xacro/v3.xacro (robot description, xacro)
@@ -50,5 +50,5 @@
     	<xacro:softhand_mimic_plugin ns="${side}_hand_v3" wide="false"/>
 		<!-- Softhand v3 needs a config file because the finger are different from each other -->
-		<xacro:property name="yaml_file" value="${xacro.load_yaml('$(find softhands_description)/urdf/config/params_v3.yaml')[side]}"/>
+		<xacro:property name="yaml_file" value="${xacro.load_yaml('$(find softhands_description)/urdf/config/params_v3.yaml')}"/>
 		<!-- <xacro:println value="${params}"/> -->
 		<!-- # palm  -->
@@ -61,5 +61,9 @@
 		<xacro:finger name="index" parent="palm" ns="${side}_hand_v3" side="${side}"/>
 		<!-- # middle -->
-		<!-- <xacro:finger name="middle" parent="palm" ns="${side}_hand_v3" side="${side}"/> -->
+		<xacro:finger name="middle" parent="palm" ns="${side}_hand_v3" side="${side}"/>
+		<!-- # ring -->
+		<xacro:finger name="ring" parent="palm" ns="${side}_hand_v3" side="${side}"/>
+		<!-- # little -->
+		<xacro:finger name="little" parent="palm" ns="${side}_hand_v3" side="${side}"/>
 	</xacro:macro>
 </robot>

Commit message: update sh3

File: softhands_description/urdf/xacro/include/macro/v3/modules/finger.xacro (robot description, xacro)
@@ -42,4 +42,7 @@
     <xacro:phalanx_knuckle name="${name}" type="knuckle" parent="${parent}" ns="${ns}" side="${side}">
     </xacro:phalanx_knuckle>
+    <!-- Proximal -->
+    <xacro:phalanx_generic name="${name}" type="proximal" parent="${name}_knuckle" ns="${ns}" side="${side}">
+    </xacro:phalanx_generic>
   </xacro:macro>
 </robot>

File: softhands_description/urdf/xacro/include/macro/v3/modules/phalanges/phalanx_generic.xacro (robot description, xacro)
@@ -52,6 +52,6 @@
       <inertial>
         <origin rpy="0 0 0" xyz="0 0 0"/>
-        <mass value="${mass}"/>
-        <xacro:insert_block name="inertia"/>
+        <mass value="${yaml_file[side]['finger'][name][type]['mass']}"/>
+        <inertia ixx="${yaml_file[side]['finger'][name][type]['inertia']['ixx']}" ixy="${yaml_file[side]['finger'][name][type]['inertia']['ixy']}" ixz="${yaml_file[side]['finger'][name][type]['inertia']['ixz']}" iyy="${yaml_file[side]['finger'][name][type]['inertia']['iyy']}" iyz="${yaml_file[side]['finger'][name][type]['inertia']['iyz']}" izz="${yaml_file[side]['finger'][name][type]['inertia']['izz']}"/>
       </inertial>
     </link>
@@ -82,5 +82,5 @@
         <origin rpy="0 0 0" xyz="0 0 0"/>
         <geometry>
-           <mesh filename="package://softhands_description/meshes/v3/${side}/${yaml_file['finger'][name][type]['mesh']}" scale="0.001 0.001 0.001"/>
+           <mesh filename="package://softhands_description/meshes/v3/${side}/${yaml_file[side]['finger'][name][type]['mesh']}" scale="0.001 0.001 0.001"/>
         </geometry>
       </collision>

File: softhands_description/urdf/xacro/include/macro/v3/modules/thumb.xacro (robot description, xacro)
@@ -43,5 +43,8 @@
     </xacro:thumb_knuckle>
     <!-- Proximal  -->
-    <xacro:phalanx_generic name="${name}" type="prossimal" parent="${name}_knuckle" ns="${ns}" side="${side}">
+    <xacro:phalanx_generic name="${name}" type="proximal" parent="${name}_knuckle" ns="${ns}" side="${side}">
+    </xacro:phalanx_generic>
+    <!--> Distal -->
+    <xacro:phalanx_generic name="${name}" type="distal" parent="${name}_proximal" ns="${ns}" side="${side}">
     </xacro:phalanx_generic>
   </xacro:macro>

File: softhands_description/urdf/xacro/v3.xacro (robot description, xacro)
@@ -51,5 +51,4 @@
 		<!-- Softhand v3 needs a config file because the finger are different from each other -->
 		<xacro:property name="yaml_file" value="${xacro.load_yaml('$(find softhands_description)/urdf/config/params_v3.yaml')}"/>
-		<!-- <xacro:println value="${params}"/> -->
 		<!-- # palm  -->
 		<xacro:palm name="palm" parent="${parent}" ns="${side}_hand_v3">

Commit message: need still to find the value of  friction and damping, try to change the mesh of the palm (to much vertex>100)

File: softhands_description/urdf/xacro/include/macro/v3/modules/finger.xacro (robot description, xacro)
@@ -45,4 +45,10 @@
     <xacro:phalanx_generic name="${name}" type="proximal" parent="${name}_knuckle" ns="${ns}" side="${side}">
     </xacro:phalanx_generic>
+    <!-- Middle -->
+    <xacro:phalanx_generic name="${name}" type="middle" parent="${name}_proximal" ns="${ns}" side="${side}">
+    </xacro:phalanx_generic>
+    <!-- Distal -->
+    <xacro:phalanx_generic name="${name}" type="distal" parent="${name}_middle" ns="${ns}" side="${side}">
+    </xacro:phalanx_generic>
   </xacro:macro>
 </robot>

File: softhands_description/urdf/xacro/include/macro/v3/modules/palm/palm.xacro (robot description, xacro)
@@ -46,7 +46,7 @@
 		<link name="${ns}_palm_link">
 			<inertial>
-				<origin rpy="0 0 0" xyz="0.0030 -0.0449 ${sign*0.0135}"/>
-				<mass value="0.45"/>
-				<inertia ixx="0.00045" ixy="0.0" ixz="0.0" iyy="0.00025" iyz="0.0" izz="0.0006"/>
+				<origin rpy="0 0 0" xyz="0.005 -4.037e-2 ${sign*1.214e-2}"/>
+				<mass value="2.27e-1"/>
+				<inertia ixx="1.14e-4" ixy="4.47e-6" ixz="-3.04e-6" iyy="7e-5" iyz="2.87e-6" izz="1.608e-4"/>
 			</inertial>
 			<visual>
@@ -58,8 +58,8 @@
 			</visual>
 			<collision>
-			<origin rpy="0 0 0" xyz="0 0 0"/>
-			<geometry>
-				<mesh filename="package://softhands_description/meshes/v3/${side}/palm_pinch.stl" scale="0.001 0.001 0.001"/>
-			</geometry>
+				<origin rpy="0 0 0" xyz="0 0 0"/>
+				<geometry>
+					<mesh filename="package://softhands_description/meshes/v3/${side}/palm_pinch_collision.stl" scale="0.001 0.001 0.001"/>
+				</geometry>
 			</collision>
 		</link>

File: softhands_description/urdf/xacro/include/macro/v3/modules/phalanges/phalanx_generic.xacro (robot description, xacro)
@@ -82,5 +82,5 @@
         <origin rpy="0 0 0" xyz="0 0 0"/>
         <geometry>
-           <mesh filename="package://softhands_description/meshes/v3/${side}/${yaml_file[side]['finger'][name][type]['mesh']}" scale="0.001 0.001 0.001"/>
+           <mesh filename="package://softhands_description/meshes/v3/${side}/${yaml_file[side]['finger'][name][type]['mesh_collision']}" scale="0.001 0.001 0.001"/>
         </geometry>
       </collision>
@@ -89,5 +89,10 @@
     <gazebo reference="${ns}_${name}_${type}_link">
       <material>Gazebo/Grey</material>
-      <selfCollide>$(arg selfCollide)</selfCollide>
+      <selfCollide>0</selfCollide>
+	  </gazebo>
+    <!-- GAZEBO REF -->
+    <gazebo reference="${ns}_${name}_${type}_virtual_link">
+      <material>Gazebo/Grey</material>
+      <selfCollide>0</selfCollide>
 	  </gazebo>
         <!-- GAZEBO REF -->

File: softhands_description/urdf/xacro/include/macro/v3/modules/phalanges/phalanx_knuckle.xacro (robot description, xacro)
@@ -41,5 +41,5 @@
     <!-- Proximal JOINT -->
     <joint name="${ns}_${name}_${type}_joint" type="revolute">
-    <origin rpy="${yaml_file[side]['finger'][name][type]['orientation']}" xyz="${yaml_file[side]['finger'][name][type]['position']}"/>
+      <origin rpy="${yaml_file[side]['finger'][name][type]['orientation']}" xyz="${yaml_file[side]['finger'][name][type]['position']}"/>
       <parent link="${ns}_${parent}_link"/>
       <child link="${ns}_${name}_${type}_link"/>
@@ -65,5 +65,5 @@
         <origin rpy="0 0 0" xyz="0 0 0"/>
         <geometry>
-          <mesh filename="package://softhands_description/meshes/v3/${side}/${yaml_file[side]['finger'][name][type]['mesh']}" scale="0.001 0.001 0.001"/>
+          <mesh filename="package://softhands_description/meshes/v3/${side}/${yaml_file[side]['finger'][name][type]['mesh_collision']}" scale="0.001 0.001 0.001"/>
         </geometry>
       </collision>

File: softhands_description/urdf/xacro/include/macro/v3/modules/phalanges/thumb_knuckle.xacro (robot description, xacro)
@@ -65,5 +65,5 @@
         <origin rpy="0 0 0" xyz="0 0 0"/>
         <geometry>
-          <mesh filename="package://softhands_description/meshes/v3/${side}/${yaml_file[side]['finger'][name][type]['mesh']}" scale="0.001 0.001 0.001"/>
+          <mesh filename="package://softhands_description/meshes/v3/${side}/${yaml_file[side]['finger'][name][type]['mesh_collision']}" scale="0.001 0.001 0.001"/>
         </geometry>
       </collision>

File: softhands_description/urdf/xacro/v3.xacro (robot description, xacro)
@@ -39,8 +39,8 @@
 <robot name="v3" xmlns:xacro="http://www.ros.org/wiki/xacro">
 	<xacro:macro name="v3" params="side parent position orientation fixed_hands:=false">
-		<xacro:arg name="friction"			default="0.0"/>
-		<xacro:arg name="virtual_friction" 	default="0.0"/>
-		<xacro:arg name="virtual_damping" 	default="3e-2"/>
-		<xacro:arg name="damping" 			default="3e-2"/>
+		<xacro:arg name="friction"			default="0.25"/>
+		<xacro:arg name="damping" 			default="4e-2"/>
+		<xacro:arg name="virtual_friction" 	default="0.25"/>
+		<xacro:arg name="virtual_damping" 	default="4e-2"/>
 		<xacro:arg name="selfCollide" 		default="0"/>
 		<xacro:property name="sign" default="1"/>
